File: G2/Connectors.sch (KiCad schematic (older format))
At the start: 6 parts, among them J301 Conn_01x09, J302 Conn_01x09, J303 Conn_01x09, J304 Conn_01x09, J305 Conn_01x09, J306 Conn_01x09

Commit message: Most things connected to MCU
Parts:
- added R? (x2): 100, Resistors_SMD:R_0805, symbol R
Connections:
- net GND: now also J303.2 (Pin_2), J305.9 (Pin_9), J306.2 (Pin_2), J306.4 (Pin_4), J306.6 (Pin_6), J306.8 (Pin_8)
- net Sense7_DUT: now reaches J306.1 (Pin_1)
- net Sense6_DUT: now reaches J306.3 (Pin_3)
- net Sense5_DUT: now reaches J306.5 (Pin_5)
- net Sense4_DUT: now reaches J306.7 (Pin_7)
- net Sense3_DUT: now reaches J306.9 (Pin_9)
- net Sense8_DUT: now reaches J305.8 (Pin_8)
- net Sense1_DUT: now reaches J303.1 (Pin_1)
- net Sense2_DUT: now reaches J303.3 (Pin_3)
- net at J303.8 (Pin_8): now also R?.1
- net at J303.9 (Pin_9): now also R?.1
- net DO1_GND renamed DO1_GND_CTRL
- net DO2_GND renamed DO2_GND_CTRL
- net DO3_GND renamed DO3_GND_CTRL
- net DO4_GND renamed DO4_GND_CTRL
- net DO5_GND renamed DO5_GND_CTRL
- net DO6_GND renamed DO6_GND_CTRL
- net DO7_GND renamed DO7_GND_CTRL
- net DO8_GND renamed DO8_GND_CTRL
- new net Wiegand_D1: R?.2
- new net Wiegand_D2: R?.2
Changed lines of the file:
@@
 LIBS:valves
 LIBS:diode
+LIBS:analog_devices
+LIBS:ADS1115IDGST
+LIBS:spark_esp32thing
+LIBS:sensors
+LIBS:Worldsemi
 LIBS:G2-cache
 EELAYER 26 0
@@
 $Descr A4 11693 8268
 encoding utf-8
-Sheet 3 6
+Sheet 3 7
 Title ""
 Date ""
@@
 DO1_PWR
 Text GLabel 2250 2350 0    60   Input ~ 0
-DO1_GND
+DO1_GND_CTRL
 Text GLabel 2250 2550 0    60   Input ~ 0
-DO2_GND
+DO2_GND_CTRL
 Text GLabel 2250 2750 0    60   Input ~ 0
-DO3_GND
+DO3_GND_CTRL
 Text GLabel 2250 3000 0    60   Input ~ 0
-DO4_GND
+DO4_GND_CTRL
 Text GLabel 2250 3200 0    60   Input ~ 0
-DO5_GND
+DO5_GND_CTRL
 Text GLabel 2250 3400 0    60   Input ~ 0
-DO6_GND
+DO6_GND_CTRL
 Text GLabel 2250 3600 0    60   Input ~ 0
-DO7_GND
+DO7_GND_CTRL
 Text GLabel 2250 3800 0    60   Input ~ 0
-DO8_GND
+DO8_GND_CTRL
+Text GLabel 2250 3950 0    60   Input ~ 0
+Sense1_DUT
+Text GLabel 2250 4150 0    60   Input ~ 0
+Sense2_DUT
+Text GLabel 3950 4800 0    60   Input ~ 0
+Sense3_DUT
+Text GLabel 3950 4600 0    60   Input ~ 0
+Sense4_DUT
+Text GLabel 3950 4200 0    60   Input ~ 0
+Sense6_DUT
+Text GLabel 3950 4000 0    60   Input ~ 0
+Sense7_DUT
+Text GLabel 3950 3750 0    60   Input ~ 0
+Sense8_DUT
+$Comp
+L GND #PWR070
+U 1 1 59C7AA8D
+P 3950 3850
+F 0 "#PWR070" H 3950 3600 50  0001 C CNN
+F 1 "GND" V 3955 3722 50  0000 R CNN
+F 2 "" H 3950 3850 50  0001 C CNN
+F 3 "" H 3950 3850 50  0001 C CNN
+	1    3950 3850
+	0    1    1    0
+$EndComp
+$Comp
+L GND #PWR071
+U 1 1 59C7AAA4
+P 3950 4100
+F 0 "#PWR071" H 3950 3850 50  0001 C CNN
+F 1 "GND" V 3955 3972 50  0000 R CNN
+F 2 "" H 3950 4100 50  0001 C CNN
+F 3 "" H 3950 4100 50  0001 C CNN
+	1    3950 4100
+	0    1    1    0
+$EndComp
+Text GLabel 3950 4400 0    60   Input ~ 0
+Sense5_DUT
+$Comp
+L GND #PWR072
+U 1 1 59C7AB8A
+P 3950 4300
+F 0 "#PWR072" H 3950 4050 50  0001 C CNN
+F 1 "GND" V 3955 4172 50  0000 R CNN
+F 2 "" H 3950 4300 50  0001 C CNN
+F 3 "" H 3950 4300 50  0001 C CNN
+	1    3950 4300
+	0    1    1    0
+$EndComp
+$Comp
+L GND #PWR073
+U 1 1 59C7ABA1
+P 3950 4500
+F 0 "#PWR073" H 3950 4250 50  0001 C CNN
+F 1 "GND" V 3955 4372 50  0000 R CNN
+F 2 "" H 3950 4500 50  0001 C CNN
+F 3 "" H 3950 4500 50  0001 C CNN
+	1    3950 4500
+	0    1    1    0
+$EndComp
+$Comp
+L GND #PWR074
+U 1 1 59C7ABB8
+P 3950 4700
+F 0 "#PWR074" H 3950 4450 50  0001 C CNN
+F 1 "GND" V 3955 4572 50  0000 R CNN
+F 2 "" H 3950 4700 50  0001 C CNN
+F 3 "" H 3950 4700 50  0001 C CNN
+	1    3950 4700
+	0    1    1    0
+$EndComp
+$Comp
+L GND #PWR075
+U 1 1 59C7ABCF
+P 2250 4050
+F 0 "#PWR075" H 2250 3800 50  0001 C CNN
+F 1 "GND" V 2255 3922 50  0000 R CNN
+F 2 "" H 2250 4050 50  0001 C CNN
+F 3 "" H 2250 4050 50  0001 C CNN
+	1    2250 4050
+	0    1    1    0
+$EndComp
+Text GLabel 1500 4650 0    60   Input ~ 0
+Wiegand_D1
+Text GLabel 1500 4750 0    60   Input ~ 0
+Wiegand_D2
+$Comp
+L R R?
+U 1 1 59C908AC
+P 1850 4750
+F 0 "R?" V 1950 4750 50  0000 C CNN
+F 1 "100" V 1850 4750 50  0000 C CNN
+F 2 "Resistors_SMD:R_0805" V 1780 4750 50  0001 C CNN
+F 3 "" H 1850 4750 50  0001 C CNN
+	1    1850 4750
+	0    1    1    0
+$EndComp
+$Comp
+L R R?
+U 1 1 59C93072
+P 1850 4650
+F 0 "R?" V 1750 4650 50  0000 C CNN
+F 1 "100" V 1850 4650 50  0000 C CNN
+F 2 "Resistors_SMD:R_0805" V 1780 4650 50  0001 C CNN
+F 3 "" H 1850 4650 50  0001 C CNN
+	1    1850 4650
+	0    1    1    0
+$EndComp
+Wire Wire Line
+	1500 4650 1700 4650
+Wire Wire Line
+	1500 4750 1700 4750
+Wire Wire Line
+	2000 4750 2250 4750
+Wire Wire Line
+	2000 4650 2250 4650
 $EndSCHEMATC

Commit message: Begun layout.
Parts:
- removed J301, J302, J303, J304, J305, J306: Conn_01x09, LocalComponents:MOLEX_1x9_39544-3009, symbol Conn_01x09
- removed R? (x2): 100, Resistors_SMD:R_0805, symbol R
