File: G2/G2.sch (KiCad schematic (older format))
At the start: 0 parts

Commit message: Completed digital IO. Begun analog sensing.
Changed lines of the file:
@@
 $Descr A4 11693 8268
 encoding utf-8
-Sheet 1 2
+Sheet 1 6
 Title ""
 Date ""
@@
 F1 "Power.sch" 60
 $EndSheet
+$Sheet
+S 1850 2300 1350 400
+U 59C2C5E7
+F0 "Connectors" 60
+F1 "Connectors.sch" 60
+$EndSheet
+$Sheet
+S 3600 1550 1100 350
+U 59C2CAC5
+F0 "DigitalIO" 60
+F1 "DigitalIO.sch" 60
+$EndSheet
+$Sheet
+S 4050 3100 1250 400
+U 59C69055
+F0 "MCU" 60
+F1 "MCU.sch" 60
+$EndSheet
+$Sheet
+S 1850 3100 1350 400
+U 59C692ED
+F0 "Analog Sense" 60
+F1 "AnalogSense.sch" 60
+$EndSheet
 $EndSCHEMATC

Commit message: Most things connected to MCU
Changed lines of the file:
@@
 LIBS:valves
 LIBS:diode
+LIBS:analog_devices
+LIBS:ADS1115IDGST
+LIBS:spark_esp32thing
+LIBS:sensors
+LIBS:Worldsemi
 LIBS:G2-cache
 EELAYER 26 0
@@
 $Descr A4 11693 8268
 encoding utf-8
-Sheet 1 6
+Sheet 1 7
 Title ""
 Date ""
@@
 $EndSheet
 $Sheet
-S 3600 1550 1100 350
+S 3500 1500 1100 350
 U 59C2CAC5
 F0 "DigitalIO" 60
@@
 $EndSheet
 $Sheet
-S 4050 3100 1250 400
+S 3500 2300 1250 400
 U 59C69055
 F0 "MCU" 60
@@
 F1 "AnalogSense.sch" 60
 $EndSheet
+$Sheet
+S 1850 3800 1300 300
+U 59C9A55D
+F0 "Status" 60
+F1 "Status.sch" 60
+$EndSheet
 $EndSCHEMATC

Commit message: Begun layout.
Changed lines of the file:
@@
 LIBS:sensors
 LIBS:Worldsemi
+LIBS:LocalPower
 LIBS:G2-cache
 EELAYER 26 0
@@
 $Descr A4 11693 8268
 encoding utf-8
-Sheet 1 7
+Sheet 1 6
 Title ""
 Date ""
@@
 $EndSheet
 $Sheet
-S 1850 2300 1350 400
-U 59C2C5E7
-F0 "Connectors" 60
-F1 "Connectors.sch" 60
-$EndSheet
-$Sheet
 S 3500 1500 1100 350
 U 59C2CAC5
@@
 $EndSheet
 $Sheet
-S 1850 3100 1350 400
+S 1850 2300 1350 400
 U 59C692ED
 F0 "Analog Sense" 60
@@
 $EndSheet
 $Sheet
-S 1850 3800 1300 300
+S 1850 3000 1300 300
 U 59C9A55D
 F0 "Status" 60
