File: G2/G2.kicad_pcb (KiCad board)
At the start: 2 copper layers, 156.2 x 174.4 mm, 0 parts

Commit message: Placed Molex connectors.
Parts:
- added C201: 100n, Capacitors_SMD:C_0805, F.Cu at (49.4, 60.6)
- added C202: 100n, Capacitors_SMD:C_0805, F.Cu at (73.8, 39.1)
- added C203: 100n, Capacitors_SMD:C_0805, F.Cu at (68.6, 51.3)
- added C204: 100n, Capacitors_SMD:C_0805, F.Cu at (78.2, 39.1)
- added C205: 100u, Capacitors_THT:CP_Radial_D6.3mm_P2.50mm, F.Cu at (34.7, 57.4)
- added C206: 100u, Capacitors_THT:CP_Radial_D6.3mm_P2.50mm, F.Cu at (42.2, 57.4)
- added D201: D, Diodes_SMD:D_SOD-123F, F.Cu at (68.9, 45.6)
- added D202: D, Diodes_SMD:D_SOD-123F, F.Cu at (54.8, 54.8)
- added D203: 3.3V, Diodes_SMD:D_SOD-123, F.Cu at (69.0, 39.6)
- added D204: 5.1V, Diodes_SMD:D_SOD-123, F.Cu at (49.7, 54.9)
- added J201: Conn_01x09, LocalComponents:MOLEX_1x9_39544-3009, F.Cu at (16.9, 93.6)
- added J202: Conn_01x09, LocalComponents:MOLEX_1x9_39544-3009, F.Cu at (69.8, 93.6)
- added J203: Conn_01x09, LocalComponents:MOLEX_1x9_39544-3009, F.Cu at (122.5, 93.6)
- added J204: Conn_01x09, LocalComponents:MOLEX_1x9_39544-3009, F.Cu at (17.4, 18.6)
- added J205: Conn_01x09, LocalComponents:MOLEX_1x9_39544-3009, F.Cu at (69.8, 18.6)
- added J206: Conn_01x09, LocalComponents:MOLEX_1x9_39544-3009, F.Cu at (122.5, 18.6)
- added U201: LM1084-3.3, TO_SOT_Packages_SMD:TO-263-3_TabPin2, F.Cu at (39.9, 43.0)
- added U202: LM1084-5.0, TO_SOT_Packages_SMD:TO-263-3_TabPin2, F.Cu at (57.9, 44.2)
Other:
- board size 156.2 x 174.4 mm -> 156.2 x 191.3 mm
- board text added: "Mount component side towards DIN rail"

Commit message: Power supply in place.
Parts:
- moved C206 118.6 mm to (159.9, 72.0)
- moved D204 111.5 mm to (161.2, 59.0)
- moved D202 95.3 mm to (147.5, 76.8), turned to 270 degrees
- moved U202 94.4 mm to (150.0, 64.9), turned to 90 degrees
- moved C202 87.2 mm to (152.5, 76.6), turned to 270 degrees
- moved C204 86.4 mm to (160.9, 64.1)
- moved D201 59.5 mm to (18.2, 76.8), turned to 270 degrees
- moved D203 41.9 mm to (31.9, 59.0)
- moved C203 39.2 mm to (31.6, 64.1)
- moved C201 30.6 mm to (23.3, 76.6), turned to 270 degrees
- moved U201 29.0 mm to (20.7, 64.9)
- moved C205 15.2 mm to (30.6, 72.0)
- moved J206 0.72 mm to (123.0, 18.0)
- moved J205 0.72 mm to (70.2, 18.0)
- moved J204 0.59 mm to (17.4, 18.0)
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Connections:
- net Net-(C201-Pad1) renamed /BackPlane/3.3V-Feed
- net Net-(C202-Pad1) renamed /BackPlane/5V-Feed
- J201 pad 3: GND -> Net-(J201-Pad3)
- J201 pad 4: +3V3 -> Net-(J201-Pad4)
- J201 pad 5: GND -> Net-(J201-Pad5)
- J201 pad 6: +5V -> Net-(J201-Pad6)
Routing:
- net +12V: track 0.00 -> 196.1 mm
- net +3V3: track 0.00 -> 32.8 mm
- net +5V: track 0.00 -> 29.0 mm
- net GND: track 0.00 -> 20.1 mm, vias 0 -> 10
- net /BackPlane/5V-Feed: track 0.00 -> 9.98 mm
- net /BackPlane/3.3V-Feed: track 0.00 -> 9.98 mm
- added copper zone on B.Cu, net GND
- added copper zone on F.Cu, net GND
Other:
- net class 12V-Supply added: clearance 0.2, trace_width 1.7, via_dia 0.8, via_drill 0.4
- net class 3.3V-Rail added: clearance 0.2, trace_width 2, via_dia 0.8, via_drill 0.4
- net class 5.5V-Rail added: clearance 0.2, trace_width 2, via_dia 0.8, via_drill 0.4
- board text added: "+12V"
- board text added: "GND"

Commit message: Single card with V-Grooves
Routing:
- net GND: track 20.1 -> 0.00 mm, vias 10 -> 0
Other:
- board size 156.2 x 191.3 mm -> 156.2 x 176.3 mm
- board text added: "V-Groove"
Changed lines of the file:
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@@
     (thickness 1.6)
     (drawings 15)
-    (tracks 56)
+    (tracks 34)
     (zones 0)
     (modules 18)
@@
     )
   )
+  (gr_text V-Groove (at 167.74 197.89 90) (layer Dwgs.User)
+    (effects (font (size 1.5 1.5) (thickness 0.3)))
+  )
+  (gr_line (start 167.9 99.32) (end 167.9 192.37) (layer Dwgs.User) (width 0.15))
+  (gr_line (start 12.4 188.7) (end 168.6 188.7) (layer Edge.Cuts) (width 0.15))
+  (gr_text "Mount component side towards DIN rail" (at 35.17 156.47) (layer F.SilkS)
+    (effects (font (size 1.5 1.5) (thickness 0.3)))
+  )
+  (gr_line (start 9.99 146.7) (end 170.34 146.7) (layer Dwgs.User) (width 0.2))
+  (gr_text V-Groove (at 4.46 146.58) (layer Dwgs.User)
+    (effects (font (size 1.5 1.5) (thickness 0.3)))
+  )
+  (gr_text V-Groove (at 176.09 146.79) (layer Dwgs.User)
+    (effects (font (size 1.5 1.5) (thickness 0.3)))
+  )
+  (gr_text V-Groove (at 176.43 99.34) (layer Dwgs.User)
+    (effects (font (size 1.5 1.5) (thickness 0.3)))
+  )
+  (gr_text V-Groove (at 4.37 99.12) (layer Dwgs.User)
+    (effects (font (size 1.5 1.5) (thickness 0.3)))
+  )
+  (gr_line (start 9.99 99.31) (end 170.34 99.31) (layer Dwgs.User) (width 0.2))
   (gr_text GND (at 16.648 87.478) (layer F.SilkS)
     (effects (font (size 1.5 1.5) (thickness 0.3)))
@@
     (effects (font (size 1.5 1.5) (thickness 0.3)))
   )
-  (gr_text "Mount component side towards DIN rail" (at 35.17 158.31) (layer F.SilkS)
-    (effects (font (size 1.5 1.5) (thickness 0.3)))
-  )
-  (gr_line (start 12.41 101.13) (end 12.41 159.83) (layer Edge.Cuts) (width 0.15))
-  (gr_line (start 167.41 101.13) (end 167.41 159.83) (layer Edge.Cuts) (width 0.15))
-  (gr_line (start 12.41 159.83) (end 167.41 159.83) (layer Edge.Cuts) (width 0.15))
-  (gr_line (start 12.41 101.13) (end 167.41 101.13) (layer Edge.Cuts) (width 0.15))
-  (gr_line (start 167.397489 161.739817) (end 167.397489 203.739817) (layer Edge.Cuts) (width 0.15))
-  (gr_line (start 12.397489 161.739817) (end 12.397489 203.739817) (layer Edge.Cuts) (width 0.15))
-  (gr_line (start 12.397489 203.739817) (end 167.397489 203.739817) (layer Edge.Cuts) (width 0.15))
-  (gr_line (start 12.397489 161.739817) (end 167.397489 161.739817) (layer Edge.Cuts) (width 0.15))
-  (gr_line (start 168.6 12.4) (end 168.6 99.3) (layer Edge.Cuts) (width 0.15))
-  (gr_line (start 12.4 12.4) (end 12.4 99.3) (layer Edge.Cuts) (width 0.15))
-  (gr_line (start 12.4 99.3) (end 168.6 99.3) (layer Edge.Cuts) (width 0.15))
+  (gr_line (start 168.6 12.4) (end 168.6 188.7) (layer Edge.Cuts) (width 0.15))
+  (gr_line (start 12.4 12.4) (end 12.4 188.7) (layer Edge.Cuts) (width 0.15))
   (gr_line (start 12.4 12.4) (end 168.6 12.4) (layer Edge.Cuts) (width 0.15))
   (segment (start 30.238 59.03) (end 30.238 63.76401) (width 2) (layer F.Cu) (net 1) (status 30))
@@
   (segment (start 23.179 59.03) (end 20.712 61.497) (width 2) (layer F.Cu) (net 1) (status 30))
   (segment (start 20.712 70.647) (end 20.712 61.497) (width 2) (layer F.Cu) (net 1) (status 30))
-  (segment (start 32.634 64.11) (end 34.174 64.11) (width 1.7) (layer F.Cu) (net 2) (status 10))
-  (via (at 34.174 64.11) (size 0.8) (drill 0.4) (layers F.Cu B.Cu) (net 2))
-  (segment (start 33.118 71.984) (end 36.206 71.984) (width 1.7) (layer F.Cu) (net 2) (status 10))
-  (via (at 36.206 71.984) (size 0.8) (drill 0.4) (layers F.Cu B.Cu) (net 2))
-  (segment (start 33.538 59.03) (end 35.19 59.03) (width 1.7) (layer F.Cu) (net 2) (status 10))
-  (via (at 35.19 59.03) (size 0.8) (drill 0.4) (layers F.Cu B.Cu) (net 2))
-  (segment (start 147.458 70.647) (end 145.239 70.647) (width 1.7) (layer F.Cu) (net 2) (status 10))
-  (segment (start 145.239 70.647) (end 145.172 70.714) (width 1.7) (layer F.Cu) (net 2))
-  (via (at 145.172 70.714) (size 0.8) (drill 0.4) (layers F.Cu B.Cu) (net 2))
-  (segment (start 161.92 64.11) (end 163.714 64.11) (width 1.7) (layer F.Cu) (net 2) (status 10))
-  (via (at 163.714 64.11) (size 0.8) (drill 0.4) (layers F.Cu B.Cu) (net 2))
-  (segment (start 162.824 59.03) (end 164.222 59.03) (width 1.7) (layer F.Cu) (net 2) (status 10))
-  (via (at 164.222 59.03) (size 0.8) (drill 0.4) (layers F.Cu B.Cu) (net 2))
-  (segment (start 162.404 71.984) (end 165.492 71.984) (width 1.7) (layer F.Cu) (net 2) (status 10))
-  (via (at 165.492 71.984) (size 0.8) (drill 0.4) (layers F.Cu B.Cu) (net 2))
-  (segment (start 152.538 77.556) (end 152.538 79.096) (width 1.7) (layer F.Cu) (net 2) (status 10))
-  (via (at 152.538 79.096) (size 0.8) (drill 0.4) (layers F.Cu B.Cu) (net 2))
-  (segment (start 23.252 77.556) (end 23.252 79.096) (width 1.7) (layer F.Cu) (net 2) (status 10))
-  (via (at 23.252 79.096) (size 0.8) (drill 0.4) (layers F.Cu B.Cu) (net 2))
-  (segment (start 18.172 70.647) (end 16.327 70.647) (width 1.7) (layer F.Cu) (net 2) (status 10))
-  (segment (start 16.327 70.647) (end 16.14 70.46) (width 1.7) (layer F.Cu) (net 2))
-  (via (at 16.14 70.46) (size 0.8) (drill 0.4) (layers F.Cu B.Cu) (net 2))
   (segment (start 159.524 59.03) (end 159.524 63.76401) (width 2) (layer F.Cu) (net 3) (status 30))
   (segment (start 159.524 63.76401) (end 159.86999 64.11) (width 2) (layer F.Cu) (net 3) (status 30))
@@
     (polygon
       (pts
-        (xy 12.584 98.908) (xy 168.286 98.908) (xy 168.286 12.802) (xy 12.838 12.802) (xy 12.584 12.802)
+        (xy 12.63 12.61) (xy 12.63 188.51) (xy 168.43 188.51) (xy 168.43 12.61)
       )
     )
@@
     (polygon
       (pts
-        (xy 12.584 98.908) (xy 168.286 98.908) (xy 168.286 12.802) (xy 12.584 12.802)
+        (xy 12.63 12.61) (xy 12.63 188.51) (xy 168.43 188.51) (xy 168.43 12.61)
       )
     )

Commit message: Added ground vias
Parts:
- added FL201: EMI_Filter_LCL, Pin_Headers:Pin_Header_Straight_1x03_Pitch2.54mm, F.Cu at (23.3, 83.1)
- moved C204 0.40 mm to (160.5, 64.1)
- moved C206 0.39 mm to (159.5, 72.0)
- moved C203 0.39 mm to (31.2, 64.1)
- moved C205 0.39 mm to (30.2, 72.0)
Connections:
- net /BackPlane/3.3V-Feed renamed Net-(C201-Pad1)
- net /BackPlane/5V-Feed renamed Net-(C202-Pad1)
- D201 pad 2: +12V -> /Power/12V
- D202 pad 2: +12V -> /Power/12V
Routing:
- net /Power/12V: track 0.00 -> 203.2 mm
- net +12V: track 196.1 -> 10.9 mm
- net GND: track 0.00 -> 18.5 mm, vias 0 -> 201

Commit message: Completed digital IO. Begun analog sensing.
Parts:
- renumbered J201 to J301, J202 to J302, J203 to J303, J204 to J304, J205 to J305, J206 to J306
Routing:
- net GND: vias 201 -> 232

Commit message: Begun layout.
Parts:
- added C301: 10u, Capacitors_SMD:CP_Elec_5x4.5, F.Cu at (62.2, -31.5)
- added C302: 10u, Capacitors_SMD:CP_Elec_5x4.5, F.Cu at (53.9, -24.4)
- added C303: 10u, Capacitors_SMD:CP_Elec_5x4.5, F.Cu at (79.8, -45.6)
- added C304: 10u, Capacitors_SMD:CP_Elec_5x4.5, F.Cu at (62.2, -21.6)
- added C305: 10u, Capacitors_SMD:CP_Elec_5x4.5, F.Cu at (70.6, -31.5)
- added C306: 10u, Capacitors_SMD:CP_Elec_5x4.5, F.Cu at (51.6, -14.1)
- added C307: 10u, Capacitors_SMD:CP_Elec_5x4.5, F.Cu at (92.2, -57.4)
- added C308: 10u, Capacitors_SMD:CP_Elec_5x4.5, F.Cu at (43.2, -14.1)
- added C309: 100n, Capacitors_SMD:C_0805, F.Cu at (108.0, -19.5)
- added C401: 100n, Capacitors_SMD:C_0805, B.Cu at (46.4, 107.7)
- added C402: 100n, Capacitors_SMD:C_0805, B.Cu at (50.8, 107.7)
- added C501: 100n, Capacitors_SMD:C_0805, F.Cu at (206.9, -100.5)
- added C502: 100n, Capacitors_SMD:C_0805, F.Cu at (211.1, -106.7)
- added C503: 100n, Capacitors_SMD:C_0805, F.Cu at (202.5, -95.1)
- added C504: 100n, Capacitors_SMD:C_0805, F.Cu at (193.7, -87.2)
- added C505: 100n, Capacitors_SMD:C_0805, F.Cu at (193.7, -92.5)
- added C506: 100n, Capacitors_SMD:C_0805, F.Cu at (198.1, -94.9)
- added C507: 100n, Capacitors_SMD:C_0805, F.Cu at (202.5, -100.4)
- added C508: 100n, Capacitors_SMD:C_0805, F.Cu at (189.1, -87.1)
- added C509: 100n, Capacitors_SMD:C_0805, F.Cu at (206.7, -105.8)
- added C510: 100n, Capacitors_SMD:C_0805, F.Cu at (211.1, -112.0)
- added C601: 100n, Capacitors_SMD:C_0805, B.Cu at (62.1, 161.9)
- added C602: 100n, Capacitors_SMD:C_0805, B.Cu at (62.4, 151.0)
- added C603: 100n, Capacitors_SMD:C_0805, B.Cu at (72.8, 160.3)
- added C604: 100n, Capacitors_SMD:C_0805, B.Cu at (82.7, 160.3)
- added C605: 100n, Capacitors_SMD:C_0805, B.Cu at (92.6, 160.3)
- added C606: 100n, Capacitors_SMD:C_0805, B.Cu at (102.5, 160.3)
- added C607: 100n, Capacitors_SMD:C_0805, B.Cu at (112.4, 160.3)
- added CON401: AVR-JTAG-10, Pin_Headers:Pin_Header_Straight_2x05_Pitch2.54mm, B.Cu at (152.8, 116.0)
- added D301: MBR0580, Diodes_SMD:D_SOD-123, F.Cu at (88.0, 74.5)
- added D302: MBR0580, Diodes_SMD:D_SOD-123, F.Cu at (81.7, 74.5)
- added D303: MBR0580, Diodes_SMD:D_SOD-123, F.Cu at (75.3, 74.5)
- added D304: MBR0580, Diodes_SMD:D_SOD-123, F.Cu at (69.0, 74.5)
- added D305: MBR0580, Diodes_SMD:D_SOD-123, F.Cu at (62.6, 74.5)
- added D306: MBR0580, Diodes_SMD:D_SOD-123, F.Cu at (56.3, 74.8)
- added D307: MBR0580, Diodes_SMD:D_SOD-123, F.Cu at (49.9, 74.5)
- added D308: MBR0580, Diodes_SMD:D_SOD-123, F.Cu at (43.6, 74.5)
- added D501: CDBA3100-HF, Diodes_SMD:D_SMA, F.Cu at (181.2, -127.3)
- added D502: CDBA3100-HF, Diodes_SMD:D_SMA, F.Cu at (150.1, -102.3)
- added D503: CDBA3100-HF, Diodes_SMD:D_SMA, F.Cu at (179.6, -120.2)
- added D504: CDBA3100-HF, Diodes_SMD:D_SMA, F.Cu at (137.1, -91.7)
- added D505: CDBA3100-HF, Diodes_SMD:D_SMA, F.Cu at (168.3, -122.0)
- added D506: CDBA3100-HF, Diodes_SMD:D_SMA, F.Cu at (150.1, -95.1)
- added D507: STPS0560Z, Diodes_SMD:D_SOD-123, F.Cu at (173.2, -108.2)
- added D508: STPS0560Z, Diodes_SMD:D_SOD-123, F.Cu at (156.3, -88.5)
- added D509: STPS0560Z, Diodes_SMD:D_SOD-123, F.Cu at (165.2, -88.8)
- added D510: STPS0560Z, Diodes_SMD:D_SOD-123, F.Cu at (189.8, -120.7)
- added D511: STPS0560Z, Diodes_SMD:D_SOD-123, F.Cu at (160.3, -94.9)
- added D512: STPS0560Z, Diodes_SMD:D_SOD-123, F.Cu at (191.4, -127.8)
- added D513: STPS0560Z, Diodes_SMD:D_SOD-123, F.Cu at (200.4, -127.8)
- added D514: STPS0560Z, Diodes_SMD:D_SOD-123, F.Cu at (182.2, -113.5)
- added D515: STPS0560Z, Diodes_SMD:D_SOD-123, F.Cu at (182.2, -107.4)
- added D516: STPS0560Z, Diodes_SMD:D_SOD-123, F.Cu at (178.2, -101.2)
- added D517: STPS0560Z, Diodes_SMD:D_SOD-123, F.Cu at (169.2, -101.1)
- added D518: STPS0560Z, Diodes_SMD:D_SOD-123, F.Cu at (169.2, -94.9)
- added D519: CDBA3100-HF, Diodes_SMD:D_SMA, F.Cu at (163.1, -107.7)
- added D520: CDBA3100-HF, Diodes_SMD:D_SMA, F.Cu at (168.3, -114.9)
- added D521: STPS0560Z, Diodes_SMD:D_SOD-123, F.Cu at (160.3, -101.1)
- added D522: STPS0560Z, Diodes_SMD:D_SOD-123, F.Cu at (147.3, -88.5)
- added D523: STPS0560Z, Diodes_SMD:D_SOD-123, F.Cu at (191.2, -114.5)
- added D524: STPS0560Z, Diodes_SMD:D_SOD-123, F.Cu at (198.7, -121.7)
- added D601: Green, LEDs:LED_0805, F.Cu at (20.5, 152.2)
- added D602: Green, LEDs:LED_0805, F.Cu at (20.5, 157.0)
- added D603: Green, LEDs:LED_0805, F.Cu at (20.5, 161.8)
- added D604: Green, LEDs:LED_0805, F.Cu at (20.5, 166.5)
- added D605: Green, LEDs:LED_0805, F.Cu at (20.5, 171.3)
- added D606: Green, LEDs:LED_0805, F.Cu at (20.5, 176.0)
- added D607: Green, LEDs:LED_0805, F.Cu at (20.5, 180.8)
- added D608: Green, LEDs:LED_0805, F.Cu at (20.5, 185.5)
- added D609: Red, LEDs:LED_0805, F.Cu at (31.2, 152.2)
- added D610: Red, LEDs:LED_0805, F.Cu at (31.2, 157.0)
- added D611: Red, LEDs:LED_0805, F.Cu at (31.2, 161.8)
- added D612: Red, LEDs:LED_0805, F.Cu at (31.2, 166.5)
- added D613: Red, LEDs:LED_0805, F.Cu at (31.2, 171.3)
- added D614: Red, LEDs:LED_0805, F.Cu at (31.2, 176.0)
- added D615: Red, LEDs:LED_0805, F.Cu at (31.2, 180.8)
- added D616: Red, LEDs:LED_0805, F.Cu at (31.1, 185.5)
- added J201: GS2, Pin_Headers:Pin_Header_Straight_1x02_Pitch2.54mm, F.Cu at (28.6, 53.7)
- added J202: GS2, Pin_Headers:Pin_Header_Straight_1x02_Pitch2.54mm, F.Cu at (158.4, 53.7)
- added J301: GS3, Pin_Headers:Pin_Header_Straight_1x03_Pitch2.54mm, F.Cu at (43.1, 56.5)
- added J302: GS3, Pin_Headers:Pin_Header_Straight_1x03_Pitch2.54mm, F.Cu at (48.1, 56.5)
- added J303: GS3, Pin_Headers:Pin_Header_Straight_1x03_Pitch2.54mm, F.Cu at (53.2, 56.5)
- added J304: GS3, Pin_Headers:Pin_Header_Straight_1x03_Pitch2.54mm, F.Cu at (58.3, 56.5)
- added J305: GS3, Pin_Headers:Pin_Header_Straight_1x03_Pitch2.54mm, F.Cu at (63.6, 56.5)
- added J306: GS3, Pin_Headers:Pin_Header_Straight_1x03_Pitch2.54mm, F.Cu at (68.7, 56.5)
- added J307: GS3, Pin_Headers:Pin_Header_Straight_1x03_Pitch2.54mm, F.Cu at (73.8, 56.5)
- added J308: GS3, Pin_Headers:Pin_Header_Straight_1x03_Pitch2.54mm, F.Cu at (78.9, 56.5)
- added J309: Conn_02x08_Counter_Clockwise, Pin_Headers:Pin_Header_Straight_2x08_Pitch2.54mm, F.Cu at (42.6, 82.7)
- added J310: Conn_02x08_Counter_Clockwise, Pin_Headers:Pin_Header_Straight_2x08_Pitch2.54mm, F.Cu at (85.2, 32.6)
- added J401: Conn_02x06_Counter_Clockwise, Pin_Headers:Pin_Header_Straight_2x06_Pitch2.54mm, B.Cu at (164.7, 140.3)
- added J402: Conn_02x08_Counter_Clockwise, Pin_Headers:Pin_Header_Straight_2x08_Pitch2.54mm, B.Cu at (85.2, 103.0)
- added J403: Conn_02x04_Counter_Clockwise, Housings_DIP:DIP-8_W9.53mm_SMD, B.Cu at (135.8, 111.9)
- added J601: Conn_02x08_Counter_Clockwise, Pin_Headers:Pin_Header_Straight_2x08_Pitch2.54mm_SMD, B.Cu at (51.5, 182.1)
- added J602: Conn_02x06_Counter_Clockwise, Pin_Headers:Pin_Header_Straight_2x06_Pitch2.54mm_SMD, B.Cu at (157.1, 180.9)
- added J603: GS3, Pin_Headers:Pin_Header_Straight_1x03_Pitch2.54mm, F.Cu at (72.0, 176.4)
- added J604: Conn_01x06, Pin_Headers:Pin_Header_Straight_1x06_Pitch2.54mm, F.Cu at (64.9, 181.5)
- added JP401: Jumper, Pin_Headers:Pin_Header_Straight_1x02_Pitch2.54mm, B.Cu at (114.9, 109.3)
- added LED601: WS2812B, LEDs:LED_WS2812B-PLCC4, F.Cu at (72.8, 152.9)
- added LED602: WS2812B, LEDs:LED_WS2812B-PLCC4, F.Cu at (82.7, 152.9)
- added LED603: WS2812B, LEDs:LED_WS2812B-PLCC4, F.Cu at (92.6, 152.9)
- added LED604: WS2812B, LEDs:LED_WS2812B-PLCC4, F.Cu at (102.5, 152.9)
- added LED605: WS2812B, LEDs:LED_WS2812B-PLCC4, F.Cu at (112.4, 152.9)
- added Q301: ZXTN25050DFHTA, TO_SOT_Packages_SMD:SOT-23, F.Cu at (88.0, 70.0)
- added Q302: ZXTN25050DFHTA, TO_SOT_Packages_SMD:SOT-23, F.Cu at (81.7, 70.0)
- added Q303: ZXTN25050DFHTA, TO_SOT_Packages_SMD:SOT-23, F.Cu at (75.3, 70.0)
- added Q304: ZXTN25050DFHTA, TO_SOT_Packages_SMD:SOT-23, F.Cu at (69.0, 70.0)
- added Q305: ZXTN25050DFHTA, TO_SOT_Packages_SMD:SOT-23, F.Cu at (62.6, 70.0)
- added Q306: ZXTN25050DFHTA, TO_SOT_Packages_SMD:SOT-23, F.Cu at (56.3, 70.0)
- added Q307: ZXTN25050DFHTA, TO_SOT_Packages_SMD:SOT-23, F.Cu at (49.9, 70.0)
- added Q308: ZXTN25050DFHTA, TO_SOT_Packages_SMD:SOT-23, F.Cu at (43.6, 70.0)
- added Q309: ZXTN25050DFHTA, TO_SOT_Packages_SMD:SOT-23, F.Cu at (61.4, -56.3)
- added Q310: ZXTN25050DFHTA, TO_SOT_Packages_SMD:SOT-23, F.Cu at (60.3, -48.2)
- added R301: 1k, Resistors_SMD:R_2512, F.Cu at (70.5, -15.4)
- added R302: 1k, Resistors_SMD:R_2512, F.Cu at (79.7, -22.1)
- added R303: 1k, Resistors_SMD:R_2512, F.Cu at (106.5, -51.1)
- added R304: 1k, Resistors_SMD:R_2512, F.Cu at (106.5, -43.7)
- added R305: 1k, Resistors_SMD:R_2512, F.Cu at (88.1, -31.8)
- added R306: 1k, Resistors_SMD:R_2512, F.Cu at (79.7, -29.5)
- added R307: 1k, Resistors_SMD:R_2512, F.Cu at (69.1, -7.95)
- added R308: 1k, Resistors_SMD:R_2512, F.Cu at (97.3, -41.2)
- added R309: 100, Resistors_SMD:R_0805, F.Cu at (88.6, -13.7)
- added R310: 100, Resistors_SMD:R_0805, F.Cu at (94.3, -28.6)
- added R311: 100, Resistors_SMD:R_0805, F.Cu at (112.8, -46.6)
- added R312: 100, Resistors_SMD:R_0805, F.Cu at (97.4, -12.3)
- added R313: 100, Resistors_SMD:R_0805, F.Cu at (103.6, -20.2)
- added R314: 100, Resistors_SMD:R_0805, F.Cu at (103.1, -31.1)
- added R315: 100, Resistors_SMD:R_0805, F.Cu at (93.0, -12.3)
- added R316: 100, Resistors_SMD:R_0805, F.Cu at (99.2, -23.2)
- added R317: 10k, Resistors_SMD:R_0805, F.Cu at (94.8, -23.2)
- added R318: 10k, Resistors_SMD:R_0805, F.Cu at (84.2, -13.7)
- added R319: 10k, Resistors_SMD:R_0805, F.Cu at (107.5, -31.1)
- added R320: 10k, Resistors_SMD:R_0805, F.Cu at (87.2, -8.29)
- added R321: 10k, Resistors_SMD:R_0805, F.Cu at (112.4, -24.8)
- added R322: 10k, Resistors_SMD:R_0805, F.Cu at (103.6, -14.8)
- added R323: 10k, Resistors_SMD:R_0805, F.Cu at (86.0, -19.2)
- added R324: 10k, Resistors_SMD:R_0805, F.Cu at (112.8, -52.1)
- added R325: 470, Resistors_SMD:R_0805, F.Cu at (90.4, -19.2)
- added R326: 470, Resistors_SMD:R_0805, F.Cu at (98.7, -28.6)
- added R327: 470, Resistors_SMD:R_0805, F.Cu at (111.9, -30.3)
- added R328: 470, Resistors_SMD:R_0805, F.Cu at (82.8, -8.29)
- added R329: 470, Resistors_SMD:R_0805, F.Cu at (108.0, -24.8)
- added R330: 470, Resistors_SMD:R_0805, F.Cu at (111.9, -35.7)
- added R331: 470, Resistors_SMD:R_0805, F.Cu at (94.8, -17.7)
- added R332: 470, Resistors_SMD:R_0805, F.Cu at (112.8, -41.2)
- added R333: 10k, Resistors_SMD:R_0805, F.Cu at (103.6, -25.7)
- added R334: 470, Resistors_SMD:R_0805, F.Cu at (99.2, -17.7)
- added R335: 470, Resistors_SMD:R_0805, F.Cu at (91.6, -6.84)
- added R401: 10k, Resistors_SMD:R_0805, B.Cu at (162.1, 117.5)
- added R402: 10k, Resistors_SMD:R_0805, B.Cu at (162.1, 113.3)
- added R403: 10k, Resistors_SMD:R_0805, B.Cu at (162.1, 109.1)
- added R404: 10k, Resistors_SMD:R_0805, B.Cu at (162.1, 104.8)
- added R405: 10k, Resistors_SMD:R_0805, B.Cu at (95.0, 142.6)
- added R406: 10k, Resistors_SMD:R_0805, B.Cu at (106.2, 142.3)
- added R407: 10k, Resistors_SMD:R_0805, B.Cu at (87.3, 111.2)
- added R408: 10k, Resistors_SMD:R_0805, B.Cu at (101.1, 142.6)
- added R409: 10k, Resistors_SMD:R_0805, B.Cu at (91.9, 111.2)
- added R410: 10k, Resistors_SMD:R_0805, B.Cu at (145.5, 119.3)
- added R411: 10k, Resistors_SMD:R_0805, B.Cu at (145.5, 114.6)
- added R412: 10k, Resistors_SMD:R_0805, B.Cu at (80.7, 141.8)
- added R413: 10k, Resistors_SMD:R_0805, B.Cu at (145.5, 109.9)
- added R414: 10k, Resistors_SMD:R_0805, B.Cu at (145.5, 105.3)
- added R501: 1k, Resistors_SMD:R_0805, F.Cu at (206.7, -111.1)
- added R502: 1k, Resistors_SMD:R_0805, F.Cu at (207.1, -128.2)
- added R503: 1k, Resistors_SMD:R_0805, F.Cu at (198.1, -100.2)
- added R504: 1k, Resistors_SMD:R_0805, F.Cu at (184.9, -101.6)
- added R505: 1k, Resistors_SMD:R_0805, F.Cu at (211.5, -128.2)
- added R506: 1k, Resistors_SMD:R_0805, F.Cu at (205.4, -122.0)
- added R507: 2k, Resistors_SMD:R_0805, F.Cu at (209.8, -117.3)
- added R508: 2k, Resistors_SMD:R_0805, F.Cu at (175.9, -95.4)
- added R509: 2k, Resistors_SMD:R_0805, F.Cu at (197.9, -115.9)
- added R510: 2k, Resistors_SMD:R_0805, F.Cu at (189.3, -97.8)
- added R511: 2k, Resistors_SMD:R_0805, F.Cu at (188.9, -108.7)
- added R512: 2k, Resistors_SMD:R_0805, F.Cu at (171.9, -89.1)
- added R513: 100, Resistors_SMD:R_0805, F.Cu at (180.3, -95.4)
- added R514: 100, Resistors_SMD:R_0805, F.Cu at (193.7, -97.8)
- added R515: 100, Resistors_SMD:R_0805, F.Cu at (202.3, -105.7)
- added R516: 100, Resistors_SMD:R_0805, F.Cu at (193.7, -103.3)
- added R517: 100, Resistors_SMD:R_0805, F.Cu at (184.7, -90.7)
- added R518: 100, Resistors_SMD:R_0805, F.Cu at (205.4, -116.6)
- added R519: 1k, Resistors_SMD:R_0805, F.Cu at (197.9, -110.4)
- added R520: 1k, Resistors_SMD:R_0805, F.Cu at (176.3, -90.0)
- added R521: 2k, Resistors_SMD:R_0805, F.Cu at (189.3, -103.3)
- added R522: 2k, Resistors_SMD:R_0805, F.Cu at (184.9, -96.1)
- added R523: 100, Resistors_SMD:R_0805, F.Cu at (209.8, -122.7)
- added R524: 100, Resistors_SMD:R_0805, F.Cu at (189.3, -92.4)
- added R525: 10k, Resistors_SMD:R_0805, F.Cu at (202.3, -111.1)
- added R526: 10k, Resistors_SMD:R_0805, F.Cu at (193.3, -108.7)
- added R601: 56, Resistors_SMD:R_0805, B.Cu at (25.8, 152.2)
- added R602: 56, Resistors_SMD:R_0805, B.Cu at (25.8, 157.0)
- added R603: 56, Resistors_SMD:R_0805, B.Cu at (25.8, 161.8)
- added R604: 56, Resistors_SMD:R_0805, B.Cu at (25.8, 166.5)
- added R605: 56, Resistors_SMD:R_0805, B.Cu at (25.8, 171.3)
- added R606: 56, Resistors_SMD:R_0805, B.Cu at (25.8, 176.0)
- added R607: 56, Resistors_SMD:R_0805, B.Cu at (25.8, 180.8)
- added R608: 56, Resistors_SMD:R_0805, B.Cu at (25.8, 185.5)
- added R609: 68, Resistors_SMD:R_0805, B.Cu at (37.2, 152.2)
- added R610: 68, Resistors_SMD:R_0805, B.Cu at (37.2, 157.0)
- added R611: 68, Resistors_SMD:R_0805, B.Cu at (37.2, 161.8)
- added R612: 68, Resistors_SMD:R_0805, B.Cu at (37.2, 166.5)
- added R613: 68, Resistors_SMD:R_0805, B.Cu at (37.2, 171.3)
- added R614: 68, Resistors_SMD:R_0805, B.Cu at (37.2, 176.0)
- added R615: 68, Resistors_SMD:R_0805, B.Cu at (37.2, 180.8)
- added R616: 68, Resistors_SMD:R_0805, B.Cu at (37.2, 185.5)
- added RV501: B72510E250K62, Capacitors_SMD:C_0805, F.Cu at (156.1, -123.0)
- added RV502: B72510E250K62, Capacitors_SMD:C_0805, F.Cu at (137.9, -108.6)
- added RV503: B72510E250K62, Capacitors_SMD:C_0805, F.Cu at (137.9, -103.3)
- added RV504: B72510E250K62, Capacitors_SMD:C_0805, F.Cu at (156.1, -128.3)
- added RV505: B72510E250K62, Capacitors_SMD:C_0805, F.Cu at (169.1, -128.3)
- added RV506: B72510E250K62, Capacitors_SMD:C_0805, F.Cu at (137.9, -98.0)
- added RV507: B72510E250K62, Capacitors_SMD:C_0805, F.Cu at (150.9, -108.6)
- added RV508: B72510E250K62, Capacitors_SMD:C_0805, F.Cu at (156.1, -117.7)
- added SPRKESP32401: Spark_ESP32Thing, spark_esp32thing:Sparkfun_ESP32Thing, B.Cu at (120.3, 115.4)
- added U301: LTV-354T, Housings_SOIC:SO-4_4.4x3.6mm_Pitch2.54mm, F.Cu at (88.6, -39.2)
- added U302: LTV-354T, Housings_SOIC:SO-4_4.4x3.6mm_Pitch2.54mm, F.Cu at (110.3, -58.6)
- added U303: LTV-354T, Housings_SOIC:SO-4_4.4x3.6mm_Pitch2.54mm, F.Cu at (88.6, -46.8)
- added U304: LTV-354T, Housings_SOIC:SO-4_4.4x3.6mm_Pitch2.54mm, F.Cu at (97.8, -48.7)
- added U305: LTV-354T, Housings_SOIC:SO-4_4.4x3.6mm_Pitch2.54mm, F.Cu at (60.4, -12.9)
- added U306: LTV-354T, Housings_SOIC:SO-4_4.4x3.6mm_Pitch2.54mm, F.Cu at (79.4, -36.9)
- added U307: LTV-354T, Housings_SOIC:SO-4_4.4x3.6mm_Pitch2.54mm, F.Cu at (71.0, -22.8)
- added U308: LTV-354T, Housings_SOIC:SO-4_4.4x3.6mm_Pitch2.54mm, F.Cu at (101.0, -58.6)
- added U309: MCP23017, Housings_SOIC:SOIC-28W_7.5x17.9mm_Pitch1.27mm, F.Cu at (42.3, -51.2)
- added U401: TXB0102DCU, Housings_SSOP:VSSOP-8_2.4x2.1mm_Pitch0.5mm, B.Cu at (48.8, 112.9)
- added U501: ADS1115IDGST, SOP50P490X110-10N, F.Cu at (138.8, -115.9)
- added U502: ADS1115IDGST, SOP50P490X110-10N, F.Cu at (138.8, -125.8)
- added U601: TXB0102DCU, Housings_SSOP:VSSOP-8_2.4x2.1mm_Pitch0.5mm, B.Cu at (62.2, 156.3)
- moved C204 1.02 mm to (159.5, 64.1)
- moved D204 1.02 mm to (160.2, 59.0)
- moved C205 1.02 mm to (29.2, 72.0)
- moved D203 1.02 mm to (30.9, 59.0)
- moved C203 1.02 mm to (30.2, 64.1)
- moved C206 1.02 mm to (158.5, 72.0)
- renumbered J301 to J311, J302 to J312, J303 to J313, J304 to J314, J305 to J315, J306 to J316
Connections:
- J311 pad 3: Net-(J301-Pad3) -> DO1_PWR
- J311 pad 4: Net-(J301-Pad4) -> DO1_GND_CTRL
- J311 pad 5: Net-(J301-Pad5) -> DO2_PWR
- J311 pad 6: Net-(J301-Pad6) -> DO2_GND_CTRL
- J311 pad 7: Net-(J301-Pad7) -> DO3_PWR
- J311 pad 8: Net-(J301-Pad8) -> DO3_GND_CTRL
- J311 pad 9: Net-(J301-Pad9) -> DO4_PWR
- J312 pad 1: Net-(J302-Pad1) -> DO4_GND_CTRL
- J312 pad 2: Net-(J302-Pad2) -> DO5_PWR
- J312 pad 3: Net-(J302-Pad3) -> DO5_GND_CTRL
- J312 pad 4: Net-(J302-Pad4) -> DO6_PWR
- J312 pad 5: Net-(J302-Pad5) -> DO6_GND_CTRL
- J312 pad 6: Net-(J302-Pad6) -> DO7_PWR
- J312 pad 7: Net-(J302-Pad7) -> DO7_GND_CTRL
- J312 pad 8: Net-(J302-Pad8) -> DO8_PWR
- J312 pad 9: Net-(J302-Pad9) -> DO8_GND_CTRL
- J313 pad 1: Net-(J303-Pad1) -> Sense1_DUT
- J313 pad 2: Net-(J303-Pad2) -> GND
- J313 pad 3: Net-(J303-Pad3) -> Sense2_DUT
- J313 pad 4: Net-(J303-Pad4) -> Sense3_DUT
- J313 pad 5: Net-(J303-Pad5) -> GND
- J313 pad 6: Net-(J303-Pad6) -> Sense4_DUT
- J313 pad 7: Net-(J303-Pad7) -> Sense5_DUT
- J313 pad 8: Net-(J303-Pad8) -> GND
- J313 pad 9: Net-(J303-Pad9) -> Sense6_DUT
- J314 pad 1: Net-(J304-Pad1) -> DI1_1
- J314 pad 2: Net-(J304-Pad2) -> DI1_2
- J314 pad 3: Net-(J304-Pad3) -> DI2_1
- J314 pad 4: Net-(J304-Pad4) -> DI2_2
- J314 pad 5: Net-(J304-Pad5) -> DI3_1
- J314 pad 6: Net-(J304-Pad6) -> DI3_2
- J314 pad 7: Net-(J304-Pad7) -> DI4_1
- J314 pad 8: Net-(J304-Pad8) -> DI4_2
- J314 pad 9: Net-(J304-Pad9) -> DI5_1
- J315 pad 1: Net-(J305-Pad1) -> DI5_2
- J315 pad 2: Net-(J305-Pad2) -> DI6_1
- J315 pad 3: Net-(J305-Pad3) -> DI6_2
- J315 pad 4: Net-(J305-Pad4) -> DI7_1
- J315 pad 5: Net-(J305-Pad5) -> DI7_2
- J315 pad 6: Net-(J305-Pad6) -> DI8_1
- J315 pad 7: Net-(J305-Pad7) -> DI8_2
- J315 pad 8: Net-(J305-Pad8) -> Wiegand_D1
- J315 pad 9: Net-(J305-Pad9) -> Wiegand_D2
- J316 pad 1: Net-(J306-Pad1) -> Sense7_DUT
- J316 pad 2: Net-(J306-Pad2) -> GND
- J316 pad 3: Net-(J306-Pad3) -> Sense8_DUT
- J316 pad 9: Net-(J306-Pad9) -> BELL
- U201 pad 2: +3V3 -> Net-(J201-Pad2)
- U202 pad 2: +5V -> Net-(J202-Pad2)
Routing:
- net Net-(J201-Pad2): track 0.00 -> 22.6 mm
- net Net-(J202-Pad2): track 0.00 -> 15.9 mm
- net +3V3: track 32.6 -> 18.5 mm
- net +5V: track 28.9 -> 18.3 mm
- net /Power/12V: track 203.2 -> 199.2 mm
- net GND: vias 232 -> 75
- added copper zone on B.Cu, net GND_C
- added copper zone on F.Cu, net GND_C
- added copper zone on B.Cu, net GND_S
- added copper zone on F.Cu, net GND_S
Other:
- outline, holes or cut-outs redrawn
- net class DigitalOutput added: clearance 0.2, trace_width 1.7, via_dia 0.8, via_drill 0.4
- net class RGB_LED_PWR added: clearance 0.2, trace_width 0.25, via_dia 0.8, via_drill 0.4
- board text added: "1"
- board text added: "2"
- board text added: "3"
- board text added: "4"
- board text added: "5"
- board text added: "6"
- board text added: "7"
- board text added: "8"
- board text added: "ESP PWR"
- board text added: "Inputs"
- board text added: "Outputs"
- board text added: "To MCU"
- board text added: "To backplane"
- board text removed: "Mount component side towards DIN rail"

Commit message: All components placed
Parts:
- moved R502 236.3 mm to (107.5, 86.1), turned to 90 degrees
- moved R505 224.5 mm to (145.1, 86.3), turned to 90 degrees
- moved C502 215.9 mm to (104.0, 80.8), turned to 90 degrees
- moved RV505 215.4 mm to (149.9, 86.2), turned to 270 degrees
- moved RV504 215.2 mm to (137.6, 86.1), turned to 270 degrees
- moved D513 214.3 mm to (135.0, 76.3)
- moved R506 213.3 mm to (159.0, 86.2), turned to 90 degrees
- moved D512 211.3 mm to (122.9, 72.0)
- moved D503 209.0 mm to (122.7, 80.9)
- moved D510 208.7 mm to (109.9, 72.1)
- moved R509 208.2 mm to (118.0, 76.4), turned to 90 degrees
- moved D505 204.5 mm to (147.2, 81.3)
- moved R503 201.7 mm to (120.6, 86.0), turned to 90 degrees
- moved R515 196.5 mm to (118.1, 71.9), turned to 90 degrees
- moved RV502 196.4 mm to (112.3, 86.1), turned to 270 degrees
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Routing:
- net /Power/12V: track 199.2 -> 229.1 mm
- net Net-(J202-Pad2): track 15.9 -> 25.5 mm
Other:
- board text added: "3.3V"
- board text added: "5V"
- board text added: "SPI_CLK"
- board text added: "SPI_CS0"
- board text added: "SPI_D/MOSI"
- board text added: "SPI_GND"
- board text added: "SPI_Q/MISO"
- board text added: "SPI_V_SELECT"
- board text added: "SPI_Vcc"
- board text added: "To status"

Commit message: More layout
Parts:
- moved D308 60.0 mm to (102.5, 85.7), turned to 90 degrees
- moved D301 56.8 mm to (32.1, 84.7), turned to 90 degrees
- moved Q308 54.1 mm to (96.9, 78.9), turned to 90 degrees
- moved R332 54.1 mm to (97.7, 74.3)
- moved D307 47.8 mm to (96.4, 85.7), turned to 90 degrees
- moved D302 45.1 mm to (37.7, 84.7), turned to 90 degrees
- moved Q307 41.1 mm to (90.0, 79.1), turned to 90 degrees
- moved R331 41.1 mm to (90.7, 74.3)
- moved D306 34.8 mm to (89.3, 85.7), turned to 90 degrees
- moved Q306 28.7 mm to (83.5, 79.1), turned to 90 degrees
- moved R330 28.7 mm to (84.2, 74.3)
- moved D305 21.0 mm to (80.4, 85.7), turned to 90 degrees
- moved Q303 19.9 mm to (55.5, 71.5)
- moved R327 19.9 mm to (56.3, 66.9)
- moved Q301 19.9 mm to (68.2, 71.5)
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Connections:
- J310 pad 12: ANALOG_RDY1 -> ANALOG_RDY_1
- J310 pad 13: ANALOG_RDY2 -> ANALOG_RDY_2
Routing:
- net +5V: track 18.6 -> 294.2 mm, vias 0 -> 11
- net +3V3: track 18.5 -> 211.0 mm, vias 0 -> 3
- net Sense1_DUT: track 0.00 -> 76.6 mm
- net DI3: track 0.00 -> 73.2 mm, vias 0 -> 4
- net DI4: track 0.00 -> 62.4 mm, vias 0 -> 2
- net DI5: track 0.00 -> 54.2 mm, vias 0 -> 2
- net ANALOG_I2C_SDA: track 0.00 -> 49.5 mm, vias 0 -> 2
- net I2C_PWR: track 0.00 -> 47.5 mm, vias 0 -> 4
- net Sense6: track 0.00 -> 46.5 mm, vias 0 -> 6
- net DI6: track 0.00 -> 45.9 mm, vias 0 -> 2
- net ANALOG_I2C_SCL: track 0.00 -> 45.2 mm, vias 0 -> 2
- net DI7: track 0.00 -> 44.9 mm, vias 0 -> 2
- net DI8: track 0.00 -> 40.5 mm, vias 0 -> 4
- net DI1: track 0.00 -> 39.8 mm, vias 0 -> 3
- net ANALOG_RDY_2: track 0.00 -> 39.0 mm, vias 0 -> 4
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Other:
- net class 3.3V-Rail-regular added: clearance 0.2, trace_width 0.25, via_dia 0.8, via_drill 0.4
