File: G2/G2.kicad_pcb (KiCad board)
At the start: 2 copper layers, 156.2 x 187.5 mm, 242 parts, among them CON401 AVR-JTAG-10, J201 GS2, J202 GS2, J301 GS3, J302 GS3, J303 GS3, J304 GS3, J305 GS3, J306 GS3, J307 GS3, J308 GS3, J309 Conn_02x08_Odd_Even, J310 Conn_02x08_Odd_Even, J311 Conn_01x09, J312 Conn_01x09, J313 Conn_01x09, J314 Conn_01x09, J315 Conn_01x09, J316 Conn_01x09, J401 Conn_01x07, J402 Conn_02x08_Odd_Even, J403 Conn_02x04_Counter_Clockwise, J601 Conn_02x08_Odd_Even, Q301 ZXTN25050DFHTA, Q302 ZXTN25050DFHTA, Q303 ZXTN25050DFHTA, Q304 ZXTN25050DFHTA, Q305 ZXTN25050DFHTA, Q306 ZXTN25050DFHTA, Q307 ZXTN25050DFHTA, Q308 ZXTN25050DFHTA, Q309 ZXTN25050DFHTA, Q310 ZXTN25050DFHTA, U201 LM1084-3.3, U202 LM1084-5.0, U301 LTV-354T, U302 LTV-354T, U303 LTV-354T, U304 LTV-354T, U305 LTV-354T, U306 LTV-354T, U307 LTV-354T, U308 LTV-354T, U309 MCP23017, U401 TXB0102DCU, U501 ADS1115IDGST, U502 ADS1115IDGST, U601 TXB0102DCU

Commit message: Added name information
Other:
- board text added: "G2 Backplane 2017-10-03 PerMalmberg @ Github"
- board text added: "G2 MCU 2017-10-03 PerMalmberg @ Github"
- board text added: "G2 Status 2017-10-03 PerMalmberg @ Github"
Changed lines of the file:
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@@
   (general
     (thickness 1.6)
-    (drawings 45)
+    (drawings 48)
     (tracks 2720)
     (zones 0)
@@
     (pcbplotparams
       (layerselection 0x011f0_ffffffff)
-      (usegerberextensions false)
+      (usegerberextensions true)
       (usegerberattributes true)
       (usegerberadvancedattributes true)
@@
       (plotinvisibletext false)
       (padsonsilk false)
-      (subtractmaskfromsilk false)
+      (subtractmaskfromsilk true)
       (outputformat 1)
       (mirror false)
@@
     )
   )
+  (gr_text "G2\nStatus\n2017-10-03\nPerMalmberg @ Github" (at 164.45 192.12) (layer B.SilkS)
+    (effects (font (size 1.5 1.5) (thickness 0.3)) (justify left mirror))
+  )
+  (gr_text "G2\nMCU\n2017-10-03\nPerMalmberg @ Github" (at 15.61 107.21) (layer F.SilkS)
+    (effects (font (size 1.5 1.5) (thickness 0.3)) (justify left))
+  )
+  (gr_text "G2\nBackplane\n2017-10-03\nPerMalmberg @ Github" (at 160.98 46.45 90) (layer F.SilkS)
+    (effects (font (size 1.5 1.5) (thickness 0.3)) (justify left))
+  )
   (gr_line (start 167.9 199.93) (end 167.9 99.32) (layer B.SilkS) (width 0.1))

Commit message: Fixed a via issue
Routing:
- net GND_C: vias 92 -> 93
- net (no net): vias 1 -> 0
Changed lines of the file:
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@@
     (pcbplotparams
       (layerselection 0x011f0_ffffffff)
-      (usegerberextensions true)
+      (usegerberextensions false)
       (usegerberattributes true)
       (usegerberadvancedattributes true)
@@
   (segment (start 152.57 118.86) (end 152.57 120.11) (width 0.25) (layer F.Cu) (net 29))
   (segment (start 152.57 120.11) (end 152.57 141.72) (width 0.25) (layer F.Cu) (net 29))
+  (via (at 150.75 100.87) (size 0.8) (drill 0.4) (layers F.Cu B.Cu) (net 187))
   (via (at 93.5 118.68) (size 0.8) (drill 0.4) (layers F.Cu B.Cu) (net 187))
   (via (at 88.36 118.72) (size 0.8) (drill 0.4) (layers F.Cu B.Cu) (net 187))
@@
   (via (at 160.99 100.87) (size 0.8) (drill 0.4) (layers F.Cu B.Cu) (net 187))
   (via (at 155.91 100.87) (size 0.8) (drill 0.4) (layers F.Cu B.Cu) (net 187))
-  (via (at 150.83 100.87) (size 0.8) (drill 0.4) (layers F.Cu B.Cu) (net 0))
   (via (at 145.75 100.87) (size 0.8) (drill 0.4) (layers F.Cu B.Cu) (net 187))
   (via (at 140.67 100.87) (size 0.8) (drill 0.4) (layers F.Cu B.Cu) (net 187))

Commit message: Fixed backwards connected TXB0102DCUs. Fixed rgb led ctrl being connected instead of level shift enable to TXB0102DCU. Made the hole for IRD contact larger. Increased hole size for screw terminals
Parts:
- removed D301, D302, D303, D304, D305, D306, D307, D308: MBR0580, Diodes_SMD:D_SOD-123
- moved R405 1.17 mm to (129.0, 148.7), turned to 180 degrees
Connections:
- C401 pad 1: +5V_C -> Net-(C401-Pad1)
- C402 pad 2: +3V3_C -> +5V_C
- R405 pad 1: /MCU/RGB_LED_DATA_CTRL -> /MCU/LEVEL_SHIFTER_ENABLE
- U401 pad 1: Net-(SPRKESP32401-Pad29) -> /MCU/Wiegand_D2
- U401 pad 3: +5V_C -> Net-(C401-Pad1)
- U401 pad 4: /MCU/Wiegand_D2 -> Net-(SPRKESP32401-Pad28)
- U401 pad 5: /MCU/Wiegand_D1 -> Net-(SPRKESP32401-Pad29)
- U401 pad 6: /MCU/RGB_LED_DATA_CTRL -> /MCU/LEVEL_SHIFTER_ENABLE
- U401 pad 7: +3V3_C -> +5V_C
- U401 pad 8: Net-(SPRKESP32401-Pad28) -> /MCU/Wiegand_D1
- U601 pad 3: +5V_S -> +3V3_S
- U601 pad 5: Net-(LED601-Pad4) -> /Status/RGB_LED_DATA_CTRL
- U601 pad 7: +3V3_S -> +5V_S
- U601 pad 8: /Status/RGB_LED_DATA_CTRL -> Net-(LED601-Pad4)
Routing:
- net +3V3_C: track 258.6 -> 206.2 mm, vias 6 -> 5
- net /MCU/LEVEL_SHIFTER_ENABLE: track 67.4 -> 89.8 mm
- net +5V_C: track 116.4 -> 104.9 mm
- net Net-(C401-Pad1): track 0.00 -> 7.65 mm
- net /MCU/RGB_LED_DATA_CTRL: track 81.1 -> 73.9 mm, vias 3 -> 2
- net +5V_S: track 157.2 -> 163.0 mm
- net /Status/RGB_LED_DATA_CTRL: track 26.5 -> 29.5 mm
- net Sense1_DUT: track 78.9 -> 76.4 mm
- net Net-(SPRKESP32401-Pad29): track 8.69 -> 10.9 mm, vias 2 -> 1
- net /MCU/Wiegand_D1: track 80.6 -> 79.0 mm, vias 0 -> 2
- net /MCU/Wiegand_D2: track 85.5 -> 87.0 mm
- net Net-(SPRKESP32401-Pad28): track 13.2 -> 11.8 mm
- net +3V3_S: track 213.3 -> 214.5 mm
- net /Status/LEVEL_SHIFTER_ENABLE: track 23.9 -> 24.5 mm
- net Net-(LED601-Pad4): track 14.4 -> 15.0 mm
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Other:
- outline, holes or cut-outs redrawn

Commit message: No longer uses Pogo pins
Parts:
- removed PG401: PogoPins02x06_Pitch5.08, PogoPins02x06_Pitch5:PogoPins02x06_Pitch5.08
- removed PG601: PogoPins02x06_Pitch5.08_ContactSurface, PogoPins02x06_Pitch5:PogoPins02x06_Pitch5.08_ContactSurface
- added J404: Conn_01x08, LocalComponents:WE68710814022_8x0.50mm_SMT_ZIF_Horizontal_Top, F.Cu at (81.0, 128.8)
- added J602: Conn_01x08, LocalComponents:WE68710814022_8x0.50mm_SMT_ZIF_Horizontal_Top, B.Cu at (108.7, 179.6)
- moved C402 7.22 mm to (139.1, 154.2), turned to 180 degrees
Routing:
- net /MCU/IO_4: track 176.9 -> 115.0 mm, vias 1 -> 0
- net /MCU/IO_3: track 176.2 -> 116.8 mm, vias 1 -> 0
- net /MCU/IO_2: track 171.3 -> 118.8 mm, vias 1 -> 0
- net /MCU/IO_1: track 172.6 -> 121.2 mm, vias 1 -> 0
- net +3V3_C: track 206.2 -> 179.7 mm, vias 5 -> 3
- net /MCU/RGB_LED_DATA_CTRL: track 73.9 -> 99.0 mm, vias 2 -> 1
- net +5V_C: track 104.9 -> 125.6 mm
- net /Status/RGB_LED_DATA_CTRL: track 29.5 -> 48.3 mm
- net +3V3_S: track 214.5 -> 232.2 mm
- net +5V_S: track 163.0 -> 146.1 mm, vias 7 -> 6
- net /DigitalIO/DO8_GND_CTRL: track 70.5 -> 59.2 mm
- net /DigitalIO/DO3_GND_CTRL: track 59.1 -> 48.5 mm
- net /DigitalIO/DO7_GND_CTRL: track 56.1 -> 47.1 mm
- net /DigitalIO/DO6_GND_CTRL: track 50.4 -> 41.6 mm
- net /MCU/ANALOG_RDY_2: track 50.9 -> 59.4 mm, vias 1 -> 0
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
Commit message: Swapped wires on flat cable socket since it is mounted on the backside
Parts:
- J401: value Conn_01x07 -> Conn_01x08; footprint Pin_Headers:Pin_Header_Straight_1x07_Pitch2.54mm -> Pin_Headers:Pin_Header_Straight_1x08_Pitch2.54mm
- moved C602 10.8 mm to (76.2, 176.5), turned to 90 degrees
- moved C601 8.76 mm to (75.5, 182.8), turned to 0 degrees
Connections:
- C401 pad 1: Net-(C401-Pad1) -> +3V3_C
- J401 pad 1: /MCU/IO_1 -> GND_C
- J401 pad 2: /MCU/IO_2 -> /MCU/IO_1
- J401 pad 3: /MCU/IO_3 -> /MCU/IO_2
- J401 pad 4: /MCU/IO_4 -> /MCU/IO_3
- J401 pad 5: /MCU/IO_5 -> /MCU/IO_4
- J401 pad 6: /MCU/IO_6 -> /MCU/IO_5
- J401 pad 7: /MCU/IO_7 -> /MCU/IO_6
- U401 pad 3: Net-(C401-Pad1) -> +3V3_C
Routing:
- net +3V3_C: track 179.7 -> 238.4 mm, vias 3 -> 5
- net /MCU/IO_7: track 104.9 -> 122.9 mm
- net /MCU/IO_6: track 107.2 -> 124.2 mm
- net /Status/RGB_LED_DATA_CTRL: track 48.3 -> 32.9 mm, vias 0 -> 2
- net /MCU/ANALOG_RDY_2: track 59.4 -> 47.4 mm
- net /MCU/IO_5: track 113.1 -> 125.0 mm
- net /MCU/IO_4: track 115.0 -> 124.6 mm
- net Net-(C401-Pad1): track 7.65 -> 0.00 mm
- net /MCU/IO_3: track 116.8 -> 124.3 mm
- net +5V_S: track 146.1 -> 138.9 mm
- net +3V3_S: track 232.2 -> 226.1 mm
- net /MCU/IO_2: track 118.8 -> 124.0 mm
- net Net-(Q304-Pad1): track 59.7 -> 54.7 mm
- net Net-(D610-Pad1): track 35.9 -> 40.7 mm
- net /MCU/DIGITAL_I2C_SDA: track 116.3 -> 112.1 mm
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
Commit message: Minor layout changes
Routing:
- net /MCU/DIGITAL_I2C_SCL: track 84.4 -> 81.0 mm
- net +3V3_C: track 238.4 -> 241.4 mm
- net GND_S: track 5.63 -> 6.60 mm
- net Net-(SPRKESP32401-Pad28): track 11.8 -> 11.2 mm
- net /MCU/DIGITAL_I2C_SDA: vias 1 -> 0
Changed lines of the file:
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@@
     (thickness 1.6)
     (drawings 48)
-    (tracks 2659)
+    (tracks 2657)
     (zones 0)
     (modules 234)
@@
   (gr_line (start 12.4 12.4) (end 12.4062 199.9238) (layer Edge.Cuts) (width 0.15))
   (gr_line (start 12.4 12.4) (end 168.6 12.4) (layer Edge.Cuts) (width 0.15))
+  (segment (start 142.367 149.733) (end 144.95 147.15) (width 0.25) (layer F.Cu) (net 23))
+  (segment (start 144.95 147.15) (end 144.95 141.72) (width 0.25) (layer F.Cu) (net 23))
+  (segment (start 140.704 149.966) (end 142.134 149.966) (width 0.25) (layer B.Cu) (net 23))
+  (segment (start 142.134 149.966) (end 142.367 149.733) (width 0.25) (layer B.Cu) (net 23))
+  (via (at 142.367 149.733) (size 0.8) (drill 0.4) (layers F.Cu B.Cu) (net 23))
+  (segment (start 90.308 109.512) (end 92.297 111.501) (width 0.25) (layer B.Cu) (net 25))
+  (segment (start 137.49001 130.44001) (end 147.49 140.44) (width 0.25) (layer B.Cu) (net 25))
+  (segment (start 92.297 111.501) (end 100.081588 111.501) (width 0.25) (layer B.Cu) (net 25))
+  (segment (start 100.081588 111.501) (end 103.860597 115.280009) (width 0.25) (layer B.Cu) (net 25))
+  (segment (start 103.860597 115.280009) (end 112.850548 115.28001) (width 0.25) (layer B.Cu) (net 25))
+  (segment (start 112.850548 115.28001) (end 115.62942 118.058882) (width 0.25) (layer B.Cu) (net 25))
+  (segment (start 115.62942 118.058882) (end 115.62942 119.832891) (width 0.25) (layer B.Cu) (net 25))
+  (segment (start 115.62942 119.832891) (end 116.456538 120.660009) (width 0.25) (layer B.Cu) (net 25))
+  (segment (start 116.456538 120.660009) (end 117.723719 120.66001) (width 0.25) (layer B.Cu) (net 25))
+  (segment (start 117.723719 120.66001) (end 127.503718 130.440009) (width 0.25) (layer B.Cu) (net 25))
+  (segment (start 147.49 140.44) (end 147.49 141.72) (width 0.25) (layer B.Cu) (net 25))
+  (segment (start 127.503718 130.440009) (end 137.49001 130.44001) (width 0.25) (layer B.Cu) (net 25))
+  (segment (start 147.484153 139.408847) (end 149.795306 141.72) (width 0.25) (layer F.Cu) (net 27))
+  (segment (start 149.795306 141.72) (end 150.03 141.72) (width 0.25) (layer F.Cu) (net 27))
+  (segment (start 127.690119 129.99) (end 138.065306 129.99) (width 0.25) (layer B.Cu) (net 27))
+  (segment (start 138.065306 129.99) (end 147.484153 139.408847) (width 0.25) (layer B.Cu) (net 27))
+  (via (at 147.484153 139.408847) (size 0.8) (drill 0.4) (layers F.Cu B.Cu) (net 27))
   (via (at 84.663 142.78) (size 0.8) (drill 0.4) (layers F.Cu B.Cu) (net 187))
   (via (at 75.519 134.144) (size 0.8) (drill 0.4) (layers F.Cu B.Cu) (net 187))
@@
   (segment (start 130.5481 115.094) (end 130.5354 115.0813) (width 0.25) (layer B.Cu) (net 22))
   (via (at 130.5354 115.0813) (size 0.8) (drill 0.4) (layers F.Cu B.Cu) (net 22))
-  (segment (start 142.31 149.95) (end 141.744315 149.95) (width 0.25) (layer B.Cu) (net 23))
-  (segment (start 141.744315 149.95) (end 141.728315 149.966) (width 0.25) (layer B.Cu) (net 23))
-  (segment (start 141.728315 149.966) (end 141.329 149.966) (width 0.25) (layer B.Cu) (net 23))
-  (segment (start 144.95 142.12) (end 145.8 142.97) (width 0.25) (layer F.Cu) (net 23) (status 10))
-  (segment (start 145.8 142.97) (end 145.8 146.673002) (width 0.25) (layer F.Cu) (net 23))
-  (segment (start 145.8 146.673002) (end 142.523002 149.95) (width 0.25) (layer F.Cu) (net 23))
-  (segment (start 142.523002 149.95) (end 142.31 149.95) (width 0.25) (layer F.Cu) (net 23))
-  (via (at 142.31 149.95) (size 0.8) (drill 0.4) (layers F.Cu B.Cu) (net 23))
   (segment (start 144.95 142.12) (end 144.95 141.72) (width 0.25) (layer F.Cu) (net 23) (status 30))
   (segment (start 140.713999 114.223999) (end 120.241999 114.223999) (width 0.25) (layer B.Cu) (net 24))
@@
   (segment (start 161.75001 113.014992) (end 159.715018 110.98) (width 0.25) (layer B.Cu) (net 25))
   (segment (start 159.715018 110.98) (end 157.4 110.98) (width 0.25) (layer B.Cu) (net 25))
-  (segment (start 143.22 136.17) (end 137.49001 130.44001) (width 0.25) (layer B.Cu) (net 25))
-  (segment (start 137.49001 130.44001) (end 127.503718 130.440009) (width 0.25) (layer B.Cu) (net 25))
-  (segment (start 115.62942 118.058882) (end 112.850548 115.28001) (width 0.25) (layer B.Cu) (net 25))
-  (segment (start 127.503718 130.440009) (end 117.723719 120.66001) (width 0.25) (layer B.Cu) (net 25))
-  (segment (start 117.723719 120.66001) (end 116.456538 120.660009) (width 0.25) (layer B.Cu) (net 25))
-  (segment (start 116.456538 120.660009) (end 115.62942 119.832891) (width 0.25) (layer B.Cu) (net 25))
-  (segment (start 115.62942 119.832891) (end 115.62942 118.058882) (width 0.25) (layer B.Cu) (net 25))
-  (segment (start 112.850548 115.28001) (end 103.860597 115.280009) (width 0.25) (layer B.Cu) (net 25))
-  (segment (start 103.860597 115.280009) (end 100.081588 111.501) (width 0.25) (layer B.Cu) (net 25))
-  (segment (start 100.081588 111.501) (end 92.297 111.501) (width 0.25) (layer B.Cu) (net 25))
-  (segment (start 92.297 111.501) (end 90.308 109.512) (width 0.25) (layer B.Cu) (net 25))
-  (segment (start 147.49 141.72) (end 147.49 140.44) (width 0.25) (layer F.Cu) (net 25) (status 10))
-  (segment (start 147.49 140.44) (end 143.22 136.17) (width 0.25) (layer F.Cu) (net 25))
   (segment (start 161.75001 126.19777) (end 147.49 140.45778) (width 0.25) (layer B.Cu) (net 25))
   (segment (start 147.49 140.45778) (end 147.49 141.72) (width 0.25) (layer B.Cu) (net 25) (status 20))
@@
   (segment (start 150.95501 119.643151) (end 150.95501 118.076849) (width 0.25) (layer B.Cu) (net 26))
   (segment (start 139.623581 106.74542) (end 128.376542 106.74542) (width 0.25) (layer B.Cu) (net 26) (status 20))
-  (segment (start 146.89 132.73) (end 150.03 135.87) (width 0.25) (layer F.Cu) (net 27))
-  (segment (start 150.03 135.87) (end 150.03 141.72) (width 0.25) (layer F.Cu) (net 27) (status 20))
   (segment (start 150.03 118.86) (end 150.03 118.46) (width 0.25) (layer B.Cu) (net 28) (status 30))
   (segment (start 150.03 118.46) (end 142.971421 111.401421) (width 0.25) (layer B.Cu) (net 28) (status 10))
@@
   (segment (start 140.994 148.966) (end 141.043999 148.916001) (width 0.25) (layer B.Cu) (net 187) (status 30))
   (segment (start 141.043999 148.916001) (end 142.193999 148.916001) (width 0.25) (layer B.Cu) (net 187) (status 10))
+  (segment (start 80.98 128.06) (end 78.682 128.06) (width 0.25) (layer F.Cu) (net 188))
+  (segment (start 78.682 128.06) (end 78.186 128.556) (width 0.25) (layer F.Cu) (net 188))
   (segment (start 78.186 141.383) (end 76.3258 143.2432) (width 2) (layer B.Cu) (net 188))
   (segment (start 76.3258 143.2432) (end 72.1817 143.2432) (width 2) (layer B.Cu) (net 188))
@@
   (via (at 77.6 169.08) (size 0.8) (drill 0.4) (layers F.Cu B.Cu) (net 191))
   (segment (start 77.6 165.94) (end 77.6 169.08) (width 2) (layer B.Cu) (net 191))
+  (segment (start 108.666 181.36) (end 110.998 181.36) (width 0.25) (layer B.Cu) (net 192))
+  (segment (start 110.998 181.36) (end 111.121 181.36) (width 0.25) (layer B.Cu) (net 192))
+  (segment (start 108.666 180.86) (end 109.516 180.86) (width 0.25) (layer B.Cu) (net 192))
+  (segment (start 109.516 180.86) (end 110.016 181.36) (width 0.25) (layer B.Cu) (net 192))
+  (segment (start 110.016 181.36) (end 110.998 181.36) (width 0.25) (layer B.Cu) (net 192))
+  (segment (start 111.121 181.36) (end 111.252 181.229) (width 0.25) (layer B.Cu) (net 192))
   (segment (start 79.112 183.108) (end 79.112 184.5238) (width 0.25) (layer B.Cu) (net 192))
-  (segment (start 108.666 180.86) (end 110.17 180.86) (width 0.25) (layer B.Cu) (net 192))
-  (segment (start 110.17 180.86) (end 110.67 181.36) (width 0.25) (layer B.Cu) (net 192))
-  (segment (start 110.67 181.36) (end 108.666 181.36) (width 0.25) (layer B.Cu) (net 192))
   (via (at 102.062 170.212) (size 0.8) (drill 0.4) (layers F.Cu B.Cu) (net 192))
   (via (at 102.316 165.894) (size 0.8) (drill 0.4) (layers F.Cu B.Cu) (net 192))
@@
   (segment (start 118.216542 106.74542) (end 118.216542 110.44842) (width 0.25) (layer B.Cu) (net 24) (status 30))
   (segment (start 118.216542 110.44842) (end 117.938542 110.72642) (width 0.25) (layer B.Cu) (net 24) (status 30))
-  (segment (start 143.22 136.1989) (end 143.22 136.17) (width 0.25) (layer F.Cu) (net 25))
-  (via (at 143.22 136.17) (size 0.8) (drill 0.4) (layers F.Cu B.Cu) (net 25))
   (segment (start 161.75001 113.014992) (end 161.75001 126.19777) (width 0.25) (layer B.Cu) (net 25))
   (segment (start 147.48444 118.86334) (end 147.48444 120.11334) (width 0.25) (layer B.Cu) (net 26) (status 10))
   (segment (start 128.37794 110.72642) (end 128.37794 106.746818) (width 0.25) (layer B.Cu) (net 26) (status 30))
   (segment (start 128.37794 106.746818) (end 128.376542 106.74542) (width 0.25) (layer B.Cu) (net 26) (status 30))
-  (segment (start 127.690119 129.99) (end 144.15 129.99) (width 0.25) (layer B.Cu) (net 27))
-  (segment (start 144.15 129.99) (end 146.89 132.73) (width 0.25) (layer B.Cu) (net 27))
-  (via (at 146.89 132.73) (size 0.8) (drill 0.4) (layers F.Cu B.Cu) (net 27))
   (segment (start 116.642939 120.21) (end 117.910119 120.21) (width 0.25) (layer B.Cu) (net 27))
   (segment (start 117.910119 120.21) (end 127.690119 129.99) (width 0.25) (layer B.Cu) (net 27))
@@
   (segment (start 100.468 28.804) (end 100.468 30.074) (width 0.25) (layer F.Cu) (net 134) (status 20))
   (segment (start 137.604 149.966) (end 137.354 149.966) (width 0.25) (layer B.Cu) (net 21) (status 30))
-  (segment (start 141.329 149.966) (end 140.704 149.966) (width 0.25) (layer B.Cu) (net 23) (status 20))
   (segment (start 24.311 164.7702) (end 22.1598 164.7702) (width 0.25) (layer F.Cu) (net 143) (status 10))
   (via (at 21.29 165.64) (size 0.8) (drill 0.4) (layers F.Cu B.Cu) (net 143))

Commit message: Connected unconnected GND zones.
Routing:
- net GND: vias 132 -> 142

Commit message: Updated Wiegand nets; D2 -> D1, D1 -> D0. Updated PCB
Parts:
- D201, D202: value D -> RBR3MM30ATR
- RV501, RV502, RV503, RV505, RV506, RV507, RV508: value B72510E250K62 -> B72510E250K062
Connections:
- J310 pad 7: Wiegand_D1 -> Wiegand_D0
- J310 pad 8: Wiegand_D2 -> Wiegand_D1
- J315 pad 8: Wiegand_D1 -> Wiegand_D0
- J315 pad 9: Wiegand_D2 -> Wiegand_D1
- J402 pad 7: /MCU/Wiegand_D1 -> /MCU/Wiegand_D0
- J402 pad 8: /MCU/Wiegand_D2 -> /MCU/Wiegand_D1
- U401 pad 1: /MCU/Wiegand_D2 -> /MCU/Wiegand_D1
- U401 pad 8: /MCU/Wiegand_D1 -> /MCU/Wiegand_D0
Routing:
- net /MCU/Wiegand_D2: track 83.8 -> 0.00 mm, vias 1 -> 0
- net /MCU/Wiegand_D0: track 0.00 -> 80.4 mm, vias 0 -> 2
- net Wiegand_D2: track 31.4 -> 0.00 mm
- net Wiegand_D0: track 0.00 -> 25.6 mm
- net Wiegand_D1: track 25.6 -> 31.4 mm
- net /MCU/Wiegand_D1: track 80.4 -> 83.8 mm, vias 2 -> 1
