File: G2/MCU.sch (KiCad schematic (older format))
At the start: 2 parts

Commit message: Most things connected to MCU
Parts:
- added C? (x2): 100n, Capacitors_SMD:C_0805, symbol C
- added CON?: AVR-JTAG-10, Pin_Headers:Pin_Header_Straight_2x05_Pitch2.54mm, symbol AVR-JTAG-10
- added J?: Conn_02x04_Counter_Clockwise, Housings_DIP:DIP-8_W9.53mm_SMD, symbol Conn_02x04_Counter_Clockwise
- added JP?: Jumper, Pin_Headers:Pin_Header_Straight_1x02_Pitch2.54mm, symbol Jumper
- added Q?: ZXTN25050DFHTA, TO_SOT_Packages_SMD:SOT-23, symbol Q_NPN_BCE
- added R? (x11): 10k, Resistors_SMD:R_0805, symbol R
- added R?: 10k, symbol R
- added R?: 470, Resistors_SMD:R_0805, symbol R
- added SPRKESP32?: Spark_ESP32Thing, symbol Spark_ESP32Thing
- added U?: TXB0102DCU, Housings_SSOP:VSSOP-8_2.4x2.1mm_Pitch0.5mm, symbol TXB0102DCU
Connections:
- net +3V3: now reaches R?.1
- net +3V3: now also R?.1, C?.2, CON?.4, J?.1 (Pin_1), J?.2 (Pin_2), J?.3 (Pin_3), J?.4 (Pin_4), JP?.1, Q?.2 (C), R?.1, R?.1, R?.1, R?.1, R?.1, R?.1, R?.1, U?.7 (VCCB)
- net I2C_SCL renamed DIGITAL_I2C_SCL
- net DIGITAL_I2C_SCL: now also SPRKESP32?.26 (U2_RXD/GPIO16)
- net I2C_SDA renamed DIGITAL_I2C_SDA
- net DIGITAL_I2C_SDA: now also SPRKESP32?.27 (U2_TXD/GPIO17)
- new net: J?.8 (Pin_8), R?.2, SPRKESP32?.1 (ADC1_0/GPI36/SenseVP)
- new net: JP?.2, SPRKESP32?.16 (3V3), SPRKESP32?.25 (3V3)
- new net: J?.7 (Pin_7), R?.2, SPRKESP32?.2 (ADC1_1/GPI37/CapVP)
- new net: J?.6 (Pin_6), R?.2, SPRKESP32?.3 (ACD1_2/GPI38/CapVN)
- new net: J?.5 (Pin_5), R?.2, SPRKESP32?.4 (ADC1_3/GPI39/SensVN)
- new net: Q?.1 (B), R?.1
- new net +5V: C?.1, U?.3 (VCCA)
- new net ANALOG_I2C_SCL: R?.2, SPRKESP32?.9 (DAC1/ADC2_8/GPIO25)
- new net ANALOG_I2C_SDA: R?.2, SPRKESP32?.10 (DAC2/ADC2_9/GPIO26)
- new net ANALOG_RDY_1: SPRKESP32?.7 (VDETI/ADC1_6/GPI34)
- new net ANALOG_RDY_2: SPRKESP32?.8 (VDET2/ADC1_7/GPI35)
- new net DIA_Interrupt: SPRKESP32?.6 (Touch8/ADC1_5/GPIO33/XTAL32)
- new net GND: C?.1, C?.2, CON?.10, CON?.2, R?.1, R?.1, R?.1, R?.1, R?.2, SPRKESP32?.17 (GND), SPRKESP32?.20 (GND), SPRKESP32?.21 (GND), SPRKESP32?.24 (GND), SPRKESP32?.40 (GND), U?.1 (B2), U?.2 (GND)
- new net I2C_PWR: Q?.3 (E)
- new net I2C_PWR_CTRL: R?.2, SPRKESP32?.11 (Touch7/ADC2_7/GPIO27)
- new net JTAG:MTCK: CON?.1, R?.2, SPRKESP32?.14 (Touch4/HSP_ID/ADC2_4/GPIO13)
- new net JTAG:MTDO: CON?.3, R?.2, SPRKESP32?.31 (Touch3/HSPI_CS0/ADC2_3/GPIO15)
- new net JTAG_MTDI: CON?.9, R?.2, SPRKESP32?.13 (Touch5/HSPI_Q/ADC2_5/GPIO12)
- new net JTAG_MTMS: CON?.5, R?.2, SPRKESP32?.12 (Touch6/HSPI_CLK/ADC2_6/GPIO14)
- new net RGB_LED_DATA: SPRKESP32?.30 (Touch2/HSPI_WP/ADC2_2/GPIO2/CS), U?.5 (A1), U?.8 (B1)
- new net RGB_LED_ENABLE: R?.1, SPRKESP32?.32 (LED(blue)/V_SPI_CS0/GPIO5), U?.6 (OE)
- new net VSPI_CLK: SPRKESP32?.33 (V_SPI_CLK/GPIO18/SCK)
- new net VSPI_CS0: R?.2, SPRKESP32?.36 (U0_RTS/V_SPI_WP/GPIO22/SCL)
- new net VSPI_D/MOSI: SPRKESP32?.34 (V_SPI_D/GPIO23/MOSI)
- new net VSPI_Q/MISO: SPRKESP32?.35 (U0_CTS/V_SPI_Q/GPIO19/MISO)
- new net Wiegand_D1: SPRKESP32?.28 (Touch0/HSPI_HD/ADC2_0/GPIO4)
- new net Wiegand_D2: SPRKESP32?.29 (Button/Touch1/ADC2_1/GPIO0/CLK1)
- new net ~RESET: CON?.6, SPRKESP32?.15 (~RST)
- no-connect marks 0 -> 9
Other:
- moved on the sheet: R?

Commit message: Begun layout.
Parts:
- removed C? (x2): 100n, Capacitors_SMD:C_0805, symbol C
- removed Q?: ZXTN25050DFHTA, TO_SOT_Packages_SMD:SOT-23, symbol Q_NPN_BCE
- removed R?: 10k, symbol R
- removed R?: 470, Resistors_SMD:R_0805, symbol R
- removed U?: TXB0102DCU, Housings_SSOP:VSSOP-8_2.4x2.1mm_Pitch0.5mm, symbol TXB0102DCU
- added C401, C402: 100n, Capacitors_SMD:C_0805, symbol C
- added J401: Conn_02x06_Counter_Clockwise, Pin_Headers:Pin_Header_Straight_2x06_Pitch2.54mm, symbol Conn_02x06_Counter_Clockwise
- added J402: Conn_02x08_Counter_Clockwise, Pin_Headers:Pin_Header_Straight_2x08_Pitch2.54mm, symbol Conn_02x08_Counter_Clockwise
- added R405: 10k, Resistors_SMD:R_0805, symbol R
- added U401: TXB0102DCU, Housings_SSOP:VSSOP-8_2.4x2.1mm_Pitch0.5mm, symbol TXB0102DCU
- SPRKESP32401: renamed from SPRKESP32?; footprint (none) -> spark_esp32thing:Sparkfun_ESP32Thing
- gave numbers to parts that had none: 16
Connections:
- net labels added: +3V3_C, +5V_C, BELL_CTRL, GND_C, LEVEL_SHIFTER_ENABLE, RGB_LED_DATA_CTRL
- net labels removed: +3.3V, +5V, GND, I2C_PWR, RGB_LED_DATA, RGB_LED_ENABLE
- wire segments 74 -> 100
Other:
- note added: "To Status"
- note added: "To backplane"
- moved on the sheet: CON401, J403, JP401, R401, R402, R403, R404, R406, R407, R408, R409, R410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

Commit message: Layout of IO board completed, except bell transistor.
Parts:
- removed J402: Conn_02x08_Counter_Clockwise, Pin_Headers:Pin_Header_Straight_2x08_Pitch2.54mm, symbol Conn_02x08_Counter_Clockwise
- added J402: Conn_02x08_Odd_Even, Pin_Headers:Pin_Header_Straight_2x08_Pitch2.54mm, symbol Conn_02x08_Odd_Even
Connections:
- wire segments 100 -> 106

Commit message: Layout nearly complete, only LCD left
Parts:
- removed J401: Conn_02x06_Counter_Clockwise, Pin_Headers:Pin_Header_Straight_2x06_Pitch2.54mm, symbol Conn_02x06_Counter_Clockwise
- added PG401: PogoPins02x06_Pitch5.08, PogoPins02x06_Pitch5:PogoPins02x06_Pitch5.08, symbol PogoPins02x06_Pitch5.08
Other:
- note added: "To MCU"
Changed lines of the file:
@@
 LIBS:Worldsemi
 LIBS:LocalPower
+LIBS:pogopins02x06_pitch5.08
 LIBS:G2-cache
 EELAYER 26 0
@@
 Text Label 8850 4900 2    60   ~ 0
 VSPI_CS0
-Text Notes 2900 4450 0    60   ~ 0
+Text Notes 2850 4350 0    60   ~ 0
 To Status
 Text Notes 3850 3500 0    60   ~ 0
@@
 Text Label 3550 2750 2    60   ~ 0
 DIGITAL_I2C_SCL
-$Comp
-L Conn_02x06_Counter_Clockwise J401
-U 1 1 59C908D7
-P 3050 4850
-F 0 "J401" H 3100 5175 50  0000 C CNN
-F 1 "Conn_02x06_Counter_Clockwise" H 3100 5176 50  0001 C CNN
-F 2 "Pin_Headers:Pin_Header_Straight_2x06_Pitch2.54mm" H 3050 4850 50  0001 C CNN
-F 3 "" H 3050 4850 50  0001 C CNN
-	1    3050 4850
-	1    0    0    -1
-$EndComp
-Text Label 3450 4850 0    60   ~ 0
-VSPI_CLK
-Text Label 3450 4950 0    60   ~ 0
-VSPI_D/MOSI
-Text Label 3450 5050 0    60   ~ 0
-VSPI_Q/MISO
-Text Label 3450 5150 0    60   ~ 0
-VSPI_CS0
-Text Label 2800 5050 2    60   ~ 0
+Text Label 2650 5050 2    60   ~ 0
 LEVEL_SHIFTER_ENABLE
-Text Label 2800 5150 2    60   ~ 0
+Text Label 2650 5150 2    60   ~ 0
 RGB_LED_DATA_CTRL
-Entry Wire Line
-	4150 5150 4250 5250
-Entry Wire Line
-	4250 5150 4350 5250
-Entry Wire Line
-	4350 5150 4450 5250
-Entry Wire Line
-	4450 5150 4550 5250
 Text Label 5600 4150 0    60   ~ 0
 RGB_LED_DATA_CTRL
 Entry Wire Line
-	2750 5150 2850 5250
-Entry Wire Line
-	2650 5150 2750 5250
+	2600 5150 2700 5250
+Entry Wire Line
+	2500 5150 2600 5250
 Entry Wire Line
 	7850 4400 7950 4300
@@
 L GND_C #PWR075
 U 1 1 59CA6266
-P 2850 4650
-F 0 "#PWR075" H 2850 4400 50  0001 C CNN
-F 1 "GND_C" V 2855 4522 50  0000 R CNN
-F 2 "" H 2850 4650 50  0001 C CNN
-F 3 "" H 2850 4650 50  0001 C CNN
-	1    2850 4650
+P 2700 4650
+F 0 "#PWR075" H 2700 4400 50  0001 C CNN
+F 1 "GND_C" V 2705 4522 50  0000 R CNN
+F 2 "" H 2700 4650 50  0001 C CNN
+F 3 "" H 2700 4650 50  0001 C CNN
+	1    2700 4650
 	0    1    1    0
 $EndComp
@@
 L GND_C #PWR076
 U 1 1 59CA62B6
-P 2850 4750
-F 0 "#PWR076" H 2850 4500 50  0001 C CNN
-F 1 "GND_C" V 2855 4622 50  0000 R CNN
-F 2 "" H 2850 4750 50  0001 C CNN
-F 3 "" H 2850 4750 50  0001 C CNN
-	1    2850 4750
+P 2700 4750
+F 0 "#PWR076" H 2700 4500 50  0001 C CNN
+F 1 "GND_C" V 2705 4622 50  0000 R CNN
+F 2 "" H 2700 4750 50  0001 C CNN
+F 3 "" H 2700 4750 50  0001 C CNN
+	1    2700 4750
 	0    1    1    0
 $EndComp
@@
 L +5V_C #PWR0124
 U 1 1 59CA75DF
-P 2850 4850
-F 0 "#PWR0124" H 2850 4700 50  0001 C CNN
-F 1 "+5V_C" V 2850 5100 50  0000 C CNN
-F 2 "" H 2850 4850 50  0001 C CNN
-F 3 "" H 2850 4850 50  0001 C CNN
-	1    2850 4850
+P 2700 4850
+F 0 "#PWR0124" H 2700 4700 50  0001 C CNN
+F 1 "+5V_C" V 2700 5100 50  0000 C CNN
+F 2 "" H 2700 4850 50  0001 C CNN
+F 3 "" H 2700 4850 50  0001 C CNN
+	1    2700 4850
 	0    -1   -1   0
 $EndComp
@@
 L +5V_C #PWR0125
 U 1 1 59CA770A
-P 2850 4950
-F 0 "#PWR0125" H 2850 4800 50  0001 C CNN
-F 1 "+5V_C" V 2850 5200 50  0000 C CNN
-F 2 "" H 2850 4950 50  0001 C CNN
-F 3 "" H 2850 4950 50  0001 C CNN
-	1    2850 4950
+P 2700 4950
+F 0 "#PWR0125" H 2700 4800 50  0001 C CNN
+F 1 "+5V_C" V 2700 5200 50  0000 C CNN
+F 2 "" H 2700 4950 50  0001 C CNN
+F 3 "" H 2700 4950 50  0001 C CNN
+	1    2700 4950
 	0    -1   -1   0
 $EndComp
@@
 Wire Bus Line
 	7850 5250 7850 4250
-Wire Bus Line
-	2600 5250 7850 5250
 Wire Wire Line
 	7950 4600 8950 4600
@@
 Wire Wire Line
 	7950 4800 8950 4800
-Wire Wire Line
-	3350 5150 4150 5150
-Wire Wire Line
-	3350 5050 4250 5050
-Wire Wire Line
-	4250 5050 4250 5150
-Wire Wire Line
-	4350 4950 4350 5150
-Wire Wire Line
-	3350 4950 4350 4950
-Wire Wire Line
-	3350 4850 4450 4850
-Wire Wire Line
-	4450 4850 4450 5150
 Wire Wire Line
 	7950 4300 8950 4300
@@
 	8950 4350 8950 4400
 Wire Wire Line
-	2750 5150 2850 5150
-Wire Wire Line
-	2650 5150 2650 5050
-Wire Wire Line
-	2650 5050 2850 5050
+	2600 5150 2700 5150
+Wire Wire Line
+	2500 5150 2500 5050
+Wire Wire Line
+	2500 5050 2700 5050
 Wire Wire Line
 	5600 4200 5550 4200
@@
 	1900 3150 2000 3250
 $Comp
-L GND_C #PWR?
+L GND_C #PWR048
 U 1 1 59CEF416
 P 3600 2550
-F 0 "#PWR?" H 3600 2300 50  0001 C CNN
+F 0 "#PWR048" H 3600 2300 50  0001 C CNN
 F 1 "GND_C" V 3605 2422 50  0000 R CNN
 F 2 "" H 3600 2550 50  0001 C CNN
@@
 $EndComp
 $Comp
-L GND_C #PWR?
+L GND_C #PWR050
 U 1 1 59CEF4CD
 P 4100 3250
-F 0 "#PWR?" H 4100 3000 50  0001 C CNN
+F 0 "#PWR050" H 4100 3000 50  0001 C CNN
 F 1 "GND_C" V 4105 3122 50  0000 R CNN
 F 2 "" H 4100 3250 50  0001 C CNN
@@
 $EndComp
 $Comp
-L +5V_C #PWR?
+L +5V_C #PWR052
 U 1 1 59CEF6CC
 P 3600 2650
-F 0 "#PWR?" H 3600 2500 50  0001 C CNN
+F 0 "#PWR052" H 3600 2500 50  0001 C CNN
 F 1 "+5V_C" V 3600 2900 50  0000 C CNN
 F 2 "" H 3600 2650 50  0001 C CNN
@@
 $EndComp
 $Comp
-L +3V3_C #PWR?
+L +3V3_C #PWR054
 U 1 1 59CEF71D
 P 4100 2550
-F 0 "#PWR?" H 4100 2400 50  0001 C CNN
+F 0 "#PWR054" H 4100 2400 50  0001 C CNN
 F 1 "+3V3_C" V 4100 2800 50  0000 C CNN
 F 2 "" H 4100 2550 50  0001 C CNN
@@
 	0    1    -1   0
 $EndComp
+Wire Wire Line
+	4450 4850 4450 5150
+Wire Wire Line
+	4350 4950 4350 5150
+Wire Wire Line
+	4250 5050 4250 5150
+Entry Wire Line
+	4450 5150 4550 5250
+Entry Wire Line
+	4350 5150 4450 5250
+Entry Wire Line
+	4250 5150 4350 5250
+Entry Wire Line
+	4150 5150 4250 5250
+Wire Wire Line
+	3350 4850 4450 4850
+Wire Wire Line
+	3350 4950 4350 4950
+Wire Wire Line
+	3350 5050 4250 5050
+Wire Wire Line
+	3350 5150 4150 5150
+Text Label 3850 5150 0    60   ~ 0
+VSPI_CS0
+Text Label 3850 5050 0    60   ~ 0
+VSPI_Q/MISO
+Text Label 3850 4950 0    60   ~ 0
+VSPI_D/MOSI
+Text Label 3850 4850 0    60   ~ 0
+VSPI_CLK
+Text Notes 3300 6100 0    60   ~ 0
+To MCU
+$Comp
+L PogoPins02x06_Pitch5.08 PG401
+U 1 1 59CF7820
+P 2900 4550
+F 0 "PG401" H 3025 4697 60  0000 C CNN
+F 1 "PogoPins02x06_Pitch5.08" H 3025 4591 60  0000 C CNN
+F 2 "PogoPins02x06_Pitch5:PogoPins02x06_Pitch5.08" H 2900 4550 60  0001 C CNN
+F 3 "" H 2900 4550 60  0001 C CNN
+	1    2900 4550
+	1    0    0    -1
+$EndComp
+Wire Bus Line
+	1900 5250 7850 5250
 $EndSCHEMATC

Commit message: Layout completed. No display - it won't fit in the enclosure
Parts:
- removed R412: 10k, Resistors_SMD:R_0805, symbol R
- added J401: Conn_01x07, Pin_Headers:Pin_Header_Straight_1x07_Pitch2.54mm, symbol Conn_01x07
Connections:
- net IO_5: now reaches SPRKESP32401.37 (U0_RXD/GPIO3/CLK2)
- net IO_5: now also J401.5 (Pin_5)
- net IO_6: now reaches SPRKESP32401.38 (U0_TXD/GPIO1/CLK3)
- net IO_6: now also J401.6 (Pin_6)
- net IO_7: now reaches SPRKESP32401.39 (V_SPI_HD/GPIO21/SDA)
- net IO_7: now also J401.7 (Pin_7)
- net VSPI_CLK renamed IO_1
- net IO_1: now also J401.1 (Pin_1)
- net VSPI_CS0 renamed IO_4
- net IO_4: now also J401.4 (Pin_4)
- net VSPI_D/MOSI renamed IO_2
- net IO_2: now also J401.2 (Pin_2)
- net VSPI_Q/MISO renamed IO_3
- net IO_3: now also J401.3 (Pin_3)
- no-connect marks 9 -> 7

Commit message: Fixed backwards connected TXB0102DCUs. Fixed rgb led ctrl being connected instead of level shift enable to TXB0102DCU. Made the hole for IRD contact larger. Increased hole size for screw terminals
Connections:
- net +3V3_C: no longer C402.2, U401.7 (VCCB)
- net +5V_C: now also C402.2, U401.7 (VCCB); no longer C401.1, U401.3 (VCCA)
- net LEVEL_SHIFTER_ENABLE: now also R405.1, U401.6 (OE)
- net RGB_LED_DATA_CTRL: no longer R405.1, U401.6 (OE)
- net Wiegand_D1: now also U401.8 (B1); no longer U401.5 (A1)
- net Wiegand_D2: now also U401.1 (B2); no longer U401.4 (A2)
- net at SPRKESP32401.28 (Touch0/HSPI_HD/ADC2_0/GPIO4): now also U401.4 (A2); no longer U401.8 (B1)
- net at SPRKESP32401.29 (Button/Touch1/ADC2_1/GPIO0/CLK1): now also U401.5 (A1); no longer U401.1 (B2)
- new net: C401.1, U401.3 (VCCA)
Other:
- moved on the sheet: C401, C402, R405, U401

Commit message: No longer uses Pogo pins
Parts:
- removed PG401: PogoPins02x06_Pitch5.08, PogoPins02x06_Pitch5:PogoPins02x06_Pitch5.08, symbol PogoPins02x06_Pitch5.08
- added J404: Conn_01x08, LocalComponents:WE68710814022_8x0.50mm_SMT_ZIF_Horizontal_Top, symbol Conn_01x08
Connections:
- net +3V3_C: now also J404.5 (Pin_5), J404.6 (Pin_6)
- net +5V_C: now also J404.3 (Pin_3), J404.4 (Pin_4)
- net GND_C: now also J404.1 (Pin_1), J404.2 (Pin_2)
- net LEVEL_SHIFTER_ENABLE: now also J404.7 (Pin_7)
- net RGB_LED_DATA_CTRL: now also J404.8 (Pin_8)
Changed lines of the file:
@@
 Text Label 3550 2750 2    60   ~ 0
 DIGITAL_I2C_SCL
-Text Label 2650 5050 2    60   ~ 0
+Text Label 3850 5050 2    60   ~ 0
 LEVEL_SHIFTER_ENABLE
-Text Label 2650 5150 2    60   ~ 0
+Text Label 3950 5150 2    60   ~ 0
 RGB_LED_DATA_CTRL
 Entry Wire Line
-	2600 5150 2700 5250
-Entry Wire Line
-	2500 5150 2600 5250
+	3900 5150 4000 5250
+Entry Wire Line
+	3800 5150 3900 5250
 Entry Wire Line
 	7850 4400 7950 4300
@@
 L GND_C #PWR075
 U 1 1 59CA6266
-P 2700 4650
-F 0 "#PWR075" H 2700 4400 50  0001 C CNN
-F 1 "GND_C" V 2705 4522 50  0000 R CNN
-F 2 "" H 2700 4650 50  0001 C CNN
-F 3 "" H 2700 4650 50  0001 C CNN
-	1    2700 4650
+P 4000 4450
+F 0 "#PWR075" H 4000 4200 50  0001 C CNN
+F 1 "GND_C" V 4005 4322 50  0000 R CNN
+F 2 "" H 4000 4450 50  0001 C CNN
+F 3 "" H 4000 4450 50  0001 C CNN
+	1    4000 4450
 	0    1    1    0
 $EndComp
@@
 L GND_C #PWR076
 U 1 1 59CA62B6
-P 2700 4750
-F 0 "#PWR076" H 2700 4500 50  0001 C CNN
-F 1 "GND_C" V 2705 4622 50  0000 R CNN
-F 2 "" H 2700 4750 50  0001 C CNN
-F 3 "" H 2700 4750 50  0001 C CNN
-	1    2700 4750
+P 4000 4550
+F 0 "#PWR076" H 4000 4300 50  0001 C CNN
+F 1 "GND_C" V 4005 4422 50  0000 R CNN
+F 2 "" H 4000 4550 50  0001 C CNN
+F 3 "" H 4000 4550 50  0001 C CNN
+	1    4000 4550
 	0    1    1    0
 $EndComp
@@
 L +3V3_C #PWR0122
 U 1 1 59CA73CD
-P 3350 4750
-F 0 "#PWR0122" H 3350 4600 50  0001 C CNN
-F 1 "+3V3_C" V 3350 5000 50  0000 C CNN
-F 2 "" H 3350 4750 50  0001 C CNN
-F 3 "" H 3350 4750 50  0001 C CNN
-	1    3350 4750
-	0    1    -1   0
+P 4000 4850
+F 0 "#PWR0122" H 4000 4700 50  0001 C CNN
+F 1 "+3V3_C" V 4000 5100 50  0000 C CNN
+F 2 "" H 4000 4850 50  0001 C CNN
+F 3 "" H 4000 4850 50  0001 C CNN
+	1    4000 4850
+	0    -1   1    0
 $EndComp
 $Comp
 L +3V3_C #PWR0123
 U 1 1 59CA7406
-P 3350 4650
-F 0 "#PWR0123" H 3350 4500 50  0001 C CNN
-F 1 "+3V3_C" V 3350 4900 50  0000 C CNN
-F 2 "" H 3350 4650 50  0001 C CNN
-F 3 "" H 3350 4650 50  0001 C CNN
-	1    3350 4650
-	0    1    -1   0
+P 4000 4950
+F 0 "#PWR0123" H 4000 4800 50  0001 C CNN
+F 1 "+3V3_C" V 4000 5200 50  0000 C CNN
+F 2 "" H 4000 4950 50  0001 C CNN
+F 3 "" H 4000 4950 50  0001 C CNN
+	1    4000 4950
+	0    -1   1    0
 $EndComp
 $Comp
 L +5V_C #PWR0124
 U 1 1 59CA75DF
-P 2700 4850
-F 0 "#PWR0124" H 2700 4700 50  0001 C CNN
-F 1 "+5V_C" V 2700 5100 50  0000 C CNN
-F 2 "" H 2700 4850 50  0001 C CNN
-F 3 "" H 2700 4850 50  0001 C CNN
-	1    2700 4850
+P 4000 4650
+F 0 "#PWR0124" H 4000 4500 50  0001 C CNN
+F 1 "+5V_C" V 4000 4900 50  0000 C CNN
+F 2 "" H 4000 4650 50  0001 C CNN
+F 3 "" H 4000 4650 50  0001 C CNN
+	1    4000 4650
 	0    -1   -1   0
 $EndComp
@@
 L +5V_C #PWR0125
 U 1 1 59CA770A
-P 2700 4950
-F 0 "#PWR0125" H 2700 4800 50  0001 C CNN
-F 1 "+5V_C" V 2700 5200 50  0000 C CNN
-F 2 "" H 2700 4950 50  0001 C CNN
-F 3 "" H 2700 4950 50  0001 C CNN
-	1    2700 4950
+P 4000 4750
+F 0 "#PWR0125" H 4000 4600 50  0001 C CNN
+F 1 "+5V_C" V 4000 5000 50  0000 C CNN
+F 2 "" H 4000 4750 50  0001 C CNN
+F 3 "" H 4000 4750 50  0001 C CNN
+	1    4000 4750
 	0    -1   -1   0
 $EndComp
@@
 Text Notes 3300 6100 0    60   ~ 0
 To MCU
-$Comp
-L PogoPins02x06_Pitch5.08 PG401
-U 1 1 59CF7820
-P 2900 4550
-F 0 "PG401" H 3025 4697 60  0000 C CNN
-F 1 "PogoPins02x06_Pitch5.08" H 3025 4591 60  0000 C CNN
-F 2 "PogoPins02x06_Pitch5:PogoPins02x06_Pitch5.08" H 2900 4550 60  0001 C CNN
-F 3 "" H 2900 4550 60  0001 C CNN
-	1    2900 4550
-	1    0    0    -1
-$EndComp
 $Comp
 L Conn_01x07 J401
@@
 Text Label 8600 5200 0    60   ~ 0
 IO_7
-Entry Wire Line
-	3900 5150 4000 5250
-Entry Wire Line
-	3800 5150 3900 5250
-Entry Wire Line
-	3700 5150 3800 5250
-Entry Wire Line
-	3600 5150 3700 5250
-Text Label 3350 4850 0    60   ~ 0
-IO_1
-Text Label 3350 4950 0    60   ~ 0
-IO_2
-Text Label 3350 5050 0    60   ~ 0
-IO_3
-Text Label 3350 5150 0    60   ~ 0
-IO_4
 Text Label 5600 4350 0    60   ~ 0
 LEVEL_SHIFTER_ENABLE
@@
 	8950 4350 8950 4400
 Wire Wire Line
-	2600 5150 2700 5150
-Wire Wire Line
-	2500 5150 2500 5050
-Wire Wire Line
-	2500 5050 2700 5050
+	3900 5150 4000 5150
+Wire Wire Line
+	3800 5150 3800 5050
+Wire Wire Line
+	3800 5050 4000 5050
 Wire Wire Line
 	5600 4650 5550 4650
@@
 Wire Wire Line
 	4900 3150 4900 2150
-Wire Bus Line
-	1900 5250 7850 5250
 Wire Wire Line
 	7950 4600 8950 4600
@@
 Connection ~ 8250 4900
 Wire Wire Line
-	3600 5150 3350 5150
-Wire Wire Line
-	3350 5050 3700 5050
-Wire Wire Line
-	3350 4950 3800 4950
-Wire Wire Line
-	3350 4850 3900 4850
-Wire Wire Line
-	3700 5050 3700 5150
-Wire Wire Line
-	3800 4950 3800 5150
-Wire Wire Line
-	3900 4850 3900 5150
-Wire Wire Line
 	5350 1450 5350 1500
 Wire Wire Line
@@
 Wire Wire Line
 	6800 2850 6300 2850
+$Comp
+L Conn_01x08 J404
+U 1 1 5A081331
+P 4200 4750
+F 0 "J404" H 4280 4742 50  0000 L CNN
+F 1 "Conn_01x08" H 4280 4651 50  0000 L CNN
+F 2 "LocalComponents:WE68710814022_8x0.50mm_SMT_ZIF_Horizontal_Top" H 4200 4750 50  0001 C CNN
+F 3 "https://www.mouser.se/Search/ProductDetail.aspx?qs=ZtY9WdtwX54hJHBraEAPJw%3d%3d" H 4200 4750 50  0001 C CNN
+	1    4200 4750
+	1    0    0    -1
+$EndComp
+Wire Bus Line
+	3400 5250 7850 5250
 $EndSCHEMATC

Commit message: Swapped wires on flat cable socket since it is mounted on the backside
Parts:
- removed J401: Conn_01x07, Pin_Headers:Pin_Header_Straight_1x07_Pitch2.54mm, symbol Conn_01x07
- added J401: Conn_01x08, Pin_Headers:Pin_Header_Straight_1x08_Pitch2.54mm, symbol Conn_01x08
Connections:
- net +3V3_C: now also C401.1, U401.3 (VCCA)
- net GND_C: now also J401.1 (Pin_1)
- net IO_1: now also J401.2 (Pin_2)
- net IO_2: now also J401.3 (Pin_3)
- net IO_3: now also J401.4 (Pin_4)
- net IO_4: now also J401.5 (Pin_5)
- net IO_5: now also J401.6 (Pin_6)
- net IO_6: now also J401.7 (Pin_7)
- net IO_7: now also J401.8 (Pin_8)
