File: G2/MCU.sch (KiCad schematic (older format))
At the start: 23 parts, among them CON401 AVR-JTAG-10, J401 Conn_01x08, J402 Conn_02x08_Odd_Even, J403 Conn_02x04_Counter_Clockwise, J404 Conn_01x08, U401 TXB0102DCU

Commit message: Minor layout changes
Changed lines of the file:
@@
 Text Notes 2850 4350 0    60   ~ 0
 To Status
-Text Notes 3850 3500 0    60   ~ 0
+Text Notes 3600 3400 0    60   ~ 0
 To backplane
 Text Label 8100 2200 0    60   ~ 0

Commit message: Removed leftover traces in schematic
Connections:
- wire segments 110 -> 108
Changed lines of the file:
@@
 	7850 2400 7850 2150
-Wire Wire Line
-	5350 1500 5450 1500
-Connection ~ 5350 1500
 Wire Wire Line
 	6800 4100 8950 4100
@@
 	7950 5200 7950 5700
 Wire Wire Line
-	5350 1450 5350 1500
-Wire Wire Line
 	5600 4150 6550 4150

Commit message: Updated Wiegand nets; D2 -> D1, D1 -> D0. Updated PCB
Connections:
- net labels added: Wiegand_D0
- net labels removed: Wiegand_D2
Changed lines of the file:
@@
 LIBS:diode
 LIBS:analog_devices
+LIBS:ADS1115IDGST
+LIBS:spark_esp32thing
 LIBS:sensors
 LIBS:Worldsemi
 LIBS:LocalPower
+LIBS:pogopins02x06_pitch5.08
 LIBS:G2-cache
 EELAYER 26 0
@@
 $EndComp
 Text Label 4200 2850 0    60   ~ 0
-Wiegand_D2
+Wiegand_D1
 Text Label 3550 2850 2    60   ~ 0
-Wiegand_D1
+Wiegand_D0
 Text Label 4200 2750 0    60   ~ 0
 DIGITAL_I2C_SDA

Commit message: Removed I2C power control
Connections:
- net labels removed: I2C_PWR_CTRL
- wire segments 108 -> 104
- no-connect marks 7 -> 9
Changed lines of the file:
@@
 NoConn ~ 8950 3200
 NoConn ~ 8950 3100
-Text Label 8100 2400 0    60   ~ 0
-I2C_PWR_CTRL
 Text Label 7750 4000 0    60   ~ 0
 DIGITAL_I2C_SDA
@@
 Text Label 8100 1900 0    60   ~ 0
 DIA_Interrupt
-Text Label 4200 2650 0    60   ~ 0
-I2C_PWR_CTRL
 Text Label 4200 3150 0    60   ~ 0
 ANALOG_I2C_SDA
@@
 Entry Wire Line
 	6800 2050 6900 2150
-Entry Wire Line
-	7750 2050 7850 2150
 Text Label 8100 1800 0    60   ~ 0
 BELL_CTRL
@@
 	-1   0    0    1
 $EndComp
-Entry Wire Line
-	4400 2050 4500 2150
 Entry Wire Line
 	4500 2050 4600 2150
@@
 	7550 1800 8950 1800
 Wire Wire Line
-	7850 2400 8950 2400
-Wire Wire Line
-	7850 2400 7850 2150
-Wire Wire Line
 	6800 4100 8950 4100
 Wire Wire Line
@@
 Wire Wire Line
 	3600 2750 2000 2750
-Wire Wire Line
-	4100 2650 4500 2650
-Wire Wire Line
-	4500 2650 4500 2150
 Wire Wire Line
 	4100 2750 4600 2750
@@
 $EndComp
 $Comp
-L GND_C #PWR?
+L GND_C #PWR0165
 U 1 1 5A085C87
 P 8650 5700
-F 0 "#PWR?" H 8650 5450 50  0001 C CNN
+F 0 "#PWR0165" H 8650 5450 50  0001 C CNN
 F 1 "GND_C" V 8655 5572 50  0000 R CNN
 F 2 "" H 8650 5700 50  0001 C CNN
@@
 	-1   0    0    1
 $EndComp
+NoConn ~ 8950 2400
+NoConn ~ 4100 2650
 $EndSCHEMATC
