File: G2/DigitalIO.sch (KiCad schematic (older format))
At the start: 107 parts

Commit message: Most things connected to MCU
Parts:
- removed D? (x8): Green, LEDs:LED_0805, symbol LED
- removed D? (x8): Red, LEDs:LED_0805, symbol LED
- removed R? (x8): 56, Resistors_SMD:R_0805, symbol R
- removed R? (x8): 68, Resistors_SMD:R_0805, symbol R
Connections:
- net I2C_Reset is gone; now on net +3V3: U?.18 (~RESET)
- net +3V3: no longer C?.1, U?.9 (VCC)
- net DO1_GND renamed DO1_GND_CTRL
- net DO2_GND renamed DO2_GND_CTRL
- net DO3_GND renamed DO3_GND_CTRL
- net DO4_GND renamed DO4_GND_CTRL
- net DO5_GND renamed DO5_GND_CTRL
- net DO6_GND renamed DO6_GND_CTRL
- net DO7_GND renamed DO7_GND_CTRL
- net DO8_GND: no longer names the net of Q?.2 (C)
- net DO8_GND: no longer D?.1 (K)
- net I2C_SCL renamed DIGITAL_I2C_SCL
- net I2C_SDA renamed DIGITAL_I2C_SDA
- new net DO8_GND_CTRL: D?.1 (K)
- new net I2C_PWR: C?.1, U?.9 (VCC)
Other:
- moved on the sheet: C?, D?, J?, Q?, R?, U?

Commit message: Begun layout.
Parts:
- added J309, J310: Conn_02x08_Counter_Clockwise, Pin_Headers:Pin_Header_Straight_2x08_Pitch2.54mm, symbol Conn_02x08_Counter_Clockwise
- added J311, J312, J313, J314, J315, J316: Conn_01x09, LocalComponents:MOLEX_1x9_39544-3009, symbol Conn_01x09
- added Q309, Q310: ZXTN25050DFHTA, TO_SOT_Packages_SMD:SOT-23, symbol Q_NPN_BCE
- added R334, R335: 470, Resistors_SMD:R_0805, symbol R
- D301, D302, D303, D304, D305, D306, D307, D308: renamed from D?; footprint Diodes_SMD:SOD-123 -> Diodes_SMD:D_SOD-123
- U309: renamed from U?; footprint (none) -> Housings_SOIC:SOIC-28W_7.5x17.9mm_Pitch1.27mm
- gave numbers to parts that had none: 66
Connections:
- net labels added: ANALOG_I2C_SCL, ANALOG_I2C_SDA, ANALOG_RDY1, ANALOG_RDY2, BELL, BELL_CTRL, I2C_PWR_CTRL, Sense1_DUT, Sense2_DUT, Sense3_DUT, Sense4_DUT, Sense5_DUT, Sense6_DUT, Sense7_DUT, Sense8_DUT, Wiegand_D1, Wiegand_D2
- wire segments 89 -> 102
- no-connect marks 1 -> 2
Other:
- note added: "QQQ Hög eller låg?"
- note added: "To MCU"
- note added: "To status card"
- moved on the sheet: D301, D302, D303, D304, D305, D306, D307, D308, Q301, Q302, Q303, Q304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

Commit message: More layout
Connections:
- net labels added: ANALOG_RDY_1, ANALOG_RDY_2
- net labels removed: ANALOG_RDY1, ANALOG_RDY2
Changed lines of the file:
@@
 Wiegand_D2
 Text GLabel 10300 1600 0    60   Input ~ 0
-ANALOG_RDY2
+ANALOG_RDY_2
 Text GLabel 10300 1700 0    60   Input ~ 0
-ANALOG_RDY1
+ANALOG_RDY_1
 Text GLabel 10300 1800 0    60   Input ~ 0
 DIA_Interrupt

Commit message: Layout of IO board completed, except bell transistor.
Parts:
- removed J309, J310: Conn_02x08_Counter_Clockwise, Pin_Headers:Pin_Header_Straight_2x08_Pitch2.54mm, symbol Conn_02x08_Counter_Clockwise
- added J309, J310: Conn_02x08_Odd_Even, Pin_Headers:Pin_Header_Straight_2x08_Pitch2.54mm, symbol Conn_02x08_Odd_Even
Connections:
- net labels added: +12V_Filtered
- wire segments 102 -> 118

Commit message: Layout completed. No display - it won't fit in the enclosure
Connections:
- net +5V: now also J316.6 (Pin_6), J316.7 (Pin_7), J316.8 (Pin_8)
- net GND: now also J316.4 (Pin_4), J316.5 (Pin_5)
Other:
- note removed: "QQQ Hög eller låg?"
Changed lines of the file:
@@
 Text GLabel 10250 2950 2    60   Input ~ 0
 I2C_PWR_CTRL
-Text Notes 13350 6550 0    60   ~ 0
-QQQ Hög eller låg?
 $Comp
 L Conn_01x09 J316
@@
 Text GLabel 13650 1250 0    60   Input ~ 0
 DO1_PWR
-Text GLabel 13650 1350 0    60   Input ~ 0
-DO1_GND_CTRL
-Text GLabel 13650 1550 0    60   Input ~ 0
-DO2_GND_CTRL
-Text GLabel 13650 1750 0    60   Input ~ 0
-DO3_GND_CTRL
-Text GLabel 13650 2000 0    60   Input ~ 0
-DO4_GND_CTRL
-Text GLabel 13650 2200 0    60   Input ~ 0
-DO5_GND_CTRL
-Text GLabel 13650 2400 0    60   Input ~ 0
-DO6_GND_CTRL
-Text GLabel 13650 2600 0    60   Input ~ 0
-DO7_GND_CTRL
-Text GLabel 13650 2800 0    60   Input ~ 0
-DO8_GND_CTRL
 Text GLabel 13650 2950 0    60   Input ~ 0
 Sense1_DUT
@@
 $EndComp
 NoConn ~ 10650 1450
+$Comp
+L GND #PWR058
+U 1 1 59D14971
+P 15350 3300
+F 0 "#PWR058" H 15350 3050 50  0001 C CNN
+F 1 "GND" V 15355 3172 50  0000 R CNN
+F 2 "" H 15350 3300 50  0001 C CNN
+F 3 "" H 15350 3300 50  0001 C CNN
+	1    15350 3300
+	0    1    1    0
+$EndComp
+$Comp
+L GND #PWR060
+U 1 1 59D14A2A
+P 15350 3400
+F 0 "#PWR060" H 15350 3150 50  0001 C CNN
+F 1 "GND" V 15355 3272 50  0000 R CNN
+F 2 "" H 15350 3400 50  0001 C CNN
+F 3 "" H 15350 3400 50  0001 C CNN
+	1    15350 3400
+	0    1    1    0
+$EndComp
+$Comp
+L +5V #PWR062
+U 1 1 59D15929
+P 15350 3500
+F 0 "#PWR062" H 15350 3350 50  0001 C CNN
+F 1 "+5V" V 15365 3628 50  0000 L CNN
+F 2 "" H 15350 3500 50  0001 C CNN
+F 3 "" H 15350 3500 50  0001 C CNN
+	1    15350 3500
+	0    -1   1    0
+$EndComp
+$Comp
+L +5V #PWR072
+U 1 1 59D1620A
+P 15350 3600
+F 0 "#PWR072" H 15350 3450 50  0001 C CNN
+F 1 "+5V" V 15365 3728 50  0000 L CNN
+F 2 "" H 15350 3600 50  0001 C CNN
+F 3 "" H 15350 3600 50  0001 C CNN
+	1    15350 3600
+	0    -1   1    0
+$EndComp
+$Comp
+L +5V #PWR073
+U 1 1 59D162C3
+P 15350 3700
+F 0 "#PWR073" H 15350 3550 50  0001 C CNN
+F 1 "+5V" V 15365 3828 50  0000 L CNN
+F 2 "" H 15350 3700 50  0001 C CNN
+F 3 "" H 15350 3700 50  0001 C CNN
+	1    15350 3700
+	0    -1   1    0
+$EndComp
+Text GLabel 10100 3900 1    60   Input ~ 0
+I2C_PWR
+$Comp
+L PWR_FLAG #FLG03
+U 1 1 59D17995
+P 10100 3900
+F 0 "#FLG03" H 10100 3975 50  0001 C CNN
+F 1 "PWR_FLAG" H 10100 4073 50  0000 C CNN
+F 2 "" H 10100 3900 50  0001 C CNN
+F 3 "" H 10100 3900 50  0001 C CNN
+	1    10100 3900
+	-1   0    0    1
+$EndComp
+Text Label 13650 1350 2    60   ~ 0
+DO1_GND_CTRL
+Text Label 13650 1550 2    60   ~ 0
+DO2_GND_CTRL
+Text Label 13650 1750 2    60   ~ 0
+DO3_GND_CTRL
+Text Label 13650 2000 2    60   ~ 0
+DO4_GND_CTRL
+Text Label 13650 2200 2    60   ~ 0
+DO5_GND_CTRL
+Text Label 13650 2400 2    60   ~ 0
+DO6_GND_CTRL
+Text Label 13650 2600 2    60   ~ 0
+DO7_GND_CTRL
+Text Label 13650 2800 2    60   ~ 0
+DO8_GND_CTRL
 $EndSCHEMATC

Commit message: Fixed backwards connected TXB0102DCUs. Fixed rgb led ctrl being connected instead of level shift enable to TXB0102DCU. Made the hole for IRD contact larger. Increased hole size for screw terminals
Parts:
- removed D301, D302, D303, D304, D305, D306, D307, D308: MBR0580, Diodes_SMD:D_SOD-123, symbol MBR0580
Changed lines of the file:
@@
-$EndComp
-$Comp
-L MBR0580 D301
-U 1 1 59C35761
-P 4900 1200
-F 0 "D301" V 4854 1279 50  0000 L CNN
-F 1 "MBR0580" H 4900 1300 50  0000 L CNN
-F 2 "Diodes_SMD:D_SOD-123" H 4900 1025 50  0001 C CNN
-F 3 "" H 4900 1200 50  0001 C CNN
-	1    4900 1200
-	0    1    1    0
 $EndComp
 $Comp
@@
 $EndComp
 $Comp
-L MBR0580 D302
-U 1 1 59C3ACC6
-P 4900 2200
-F 0 "D302" V 4854 2279 50  0000 L CNN
-F 1 "MBR0580" H 4900 2300 50  0000 L CNN
-F 2 "Diodes_SMD:D_SOD-123" H 4900 2025 50  0001 C CNN
-F 3 "" H 4900 2200 50  0001 C CNN
-	1    4900 2200
-	0    1    1    0
-$EndComp
-$Comp
 L GND #PWR029
 U 1 1 59C3ACCD
@@
 $EndComp
 $Comp
-L MBR0580 D303
-U 1 1 59C3B127
-P 4900 3200
-F 0 "D303" V 4854 3279 50  0000 L CNN
-F 1 "MBR0580" H 4900 3300 50  0000 L CNN
-F 2 "Diodes_SMD:D_SOD-123" H 4900 3025 50  0001 C CNN
-F 3 "" H 4900 3200 50  0001 C CNN
-	1    4900 3200
-	0    1    1    0
-$EndComp
-$Comp
 L GND #PWR031
 U 1 1 59C3B12E
@@
 $EndComp
 $Comp
-L MBR0580 D304
-U 1 1 59C3B4DD
-P 4900 4200
-F 0 "D304" V 4854 4279 50  0000 L CNN
-F 1 "MBR0580" H 4900 4300 50  0000 L CNN
-F 2 "Diodes_SMD:D_SOD-123" H 4900 4025 50  0001 C CNN
-F 3 "" H 4900 4200 50  0001 C CNN
-	1    4900 4200
-	0    1    1    0
-$EndComp
-$Comp
 L GND #PWR033
 U 1 1 59C3B4E4
@@
 $EndComp
 $Comp
-L MBR0580 D305
-U 1 1 59C3B5B2
-P 4900 5200
-F 0 "D305" V 4854 5279 50  0000 L CNN
-F 1 "MBR0580" H 4900 5300 50  0000 L CNN
-F 2 "Diodes_SMD:D_SOD-123" H 4900 5025 50  0001 C CNN
-F 3 "" H 4900 5200 50  0001 C CNN
-	1    4900 5200
-	0    1    1    0
-$EndComp
-$Comp
 L GND #PWR035
 U 1 1 59C3B5B9
@@
 $EndComp
 $Comp
-L MBR0580 D306
-U 1 1 59C3BCC7
-P 4900 6200
-F 0 "D306" V 4854 6279 50  0000 L CNN
-F 1 "MBR0580" H 4900 6300 50  0000 L CNN
-F 2 "Diodes_SMD:D_SOD-123" H 4900 6025 50  0001 C CNN
-F 3 "" H 4900 6200 50  0001 C CNN
-	1    4900 6200
-	0    1    1    0
-$EndComp
-$Comp
 L GND #PWR037
 U 1 1 59C3BCCE
@@
 $EndComp
 $Comp
-L MBR0580 D307
-U 1 1 59C3C5E0
-P 6950 1000
-F 0 "D307" V 6904 1079 50  0000 L CNN
-F 1 "MBR0580" H 6950 1100 50  0000 L CNN
-F 2 "Diodes_SMD:D_SOD-123" H 6950 825 50  0001 C CNN
-F 3 "" H 6950 1000 50  0001 C CNN
-	1    6950 1000
-	0    1    1    0
-$EndComp
-$Comp
 L GND #PWR039
 U 1 1 59C3C5E7
@@
 	1    6550 2000
 	1    0    0    -1
-$EndComp
-$Comp
-L MBR0580 D308
-U 1 1 59C3C6CE
-P 6950 2000
-F 0 "D308" V 6904 2079 50  0000 L CNN
-F 1 "MBR0580" H 6950 2100 50  0000 L CNN
-F 2 "Diodes_SMD:D_SOD-123" H 6950 1825 50  0001 C CNN
-F 3 "" H 6950 2000 50  0001 C CNN
-	1    6950 2000
-	0    1    1    0
 $EndComp
 $Comp
@@
 	4600 1500 4600 1400
 Wire Wire Line
-	4900 1350 4900 1400
-Wire Wire Line
-	4900 1400 4600 1400
-Wire Wire Line
-	4900 1050 4900 1000
-Wire Wire Line
 	4250 1200 4300 1200
 Wire Wire Line
 	4600 2500 4600 2400
 Wire Wire Line
-	4900 2350 4900 2400
-Wire Wire Line
-	4900 2400 4600 2400
-Wire Wire Line
-	4900 2050 4900 2000
-Wire Wire Line
 	4250 2200 4300 2200
 Wire Wire Line
 	4600 3500 4600 3400
 Wire Wire Line
-	4900 3350 4900 3400
-Wire Wire Line
-	4900 3400 4600 3400
-Wire Wire Line
-	4900 3050 4900 3000
-Wire Wire Line
 	4250 3200 4300 3200
 Wire Wire Line
 	4600 4500 4600 4400
 Wire Wire Line
-	4900 4350 4900 4400
-Wire Wire Line
-	4900 4400 4600 4400
-Wire Wire Line
-	4900 4050 4900 4000
-Wire Wire Line
 	4250 4200 4300 4200
 Wire Wire Line
 	4600 5500 4600 5400
 Wire Wire Line
-	4900 5350 4900 5400
-Wire Wire Line
-	4900 5400 4600 5400
-Wire Wire Line
-	4900 5050 4900 5000
-Wire Wire Line
 	4250 5200 4300 5200
 Wire Wire Line
 	4600 6500 4600 6400
 Wire Wire Line
-	4900 6350 4900 6400
-Wire Wire Line
-	4900 6400 4600 6400
-Wire Wire Line
-	4900 6050 4900 6000
-Wire Wire Line
 	4250 6200 4300 6200
 Wire Wire Line
 	6650 1300 6650 1200
 Wire Wire Line
-	6950 1150 6950 1200
-Wire Wire Line
-	6950 1200 6650 1200
-Wire Wire Line
-	6950 850  6950 800
-Wire Wire Line
 	6300 1000 6350 1000
 Wire Wire Line
 	6650 2300 6650 2200
-Wire Wire Line
-	6950 2150 6950 2200
-Wire Wire Line
-	6950 2200 6650 2200
-Wire Wire Line
-	6950 1850 6950 1800
 Wire Wire Line
 	6300 2000 6350 2000
@@
 Wire Bus Line
 	5250 650  5250 8850
-Connection ~ 4900 1000
-Connection ~ 4900 2000
-Connection ~ 4900 3000
-Connection ~ 6950 1800
-Connection ~ 4900 4000
-Connection ~ 4900 5000
-Connection ~ 4900 6000
-Connection ~ 6950 800
 Wire Wire Line
 	5350 7850 6400 7850
@@
 Wire Wire Line
 	6400 8150 5350 8150
-Wire Wire Line
-	4600 2000 5150 2000
 Wire Wire Line
 	4600 1000 5150 1000
@@
 Text Label 13650 2800 2    60   ~ 0
 DO8_GND_CTRL
+Wire Wire Line
+	4600 2000 5150 2000
 $EndSCHEMATC
