File: G2/DigitalIO.sch (KiCad schematic (older format))
At the start: 79 parts, among them J301 GS3, J302 GS3, J303 GS3, J304 GS3, J305 GS3, J306 GS3, J307 GS3, J308 GS3, J309 Conn_02x08_Odd_Even, J310 Conn_02x08_Odd_Even, J311 Conn_01x09, J312 Conn_01x09, J313 Conn_01x09, J314 Conn_01x09, J315 Conn_01x09, J316 Conn_01x09, Q301 ZXTN25050DFHTA, Q302 ZXTN25050DFHTA, Q303 ZXTN25050DFHTA, Q304 ZXTN25050DFHTA, Q305 ZXTN25050DFHTA, Q306 ZXTN25050DFHTA, Q307 ZXTN25050DFHTA, Q308 ZXTN25050DFHTA, Q309 ZXTN25050DFHTA, Q310 ZXTN25050DFHTA, U301 LTV-354T, U302 LTV-354T, U303 LTV-354T, U304 LTV-354T, U305 LTV-354T, U306 LTV-354T, U307 LTV-354T, U308 LTV-354T, U309 MCP23017

Commit message: Updated Wiegand nets; D2 -> D1, D1 -> D0. Updated PCB
Connections:
- net Wiegand_D2 is gone; now on net Wiegand_D1: J310.8 (Pin_8), J315.9 (Pin_9)
- net Wiegand_D1: no longer J310.7 (Pin_7), J315.8 (Pin_8)
- new net Wiegand_D0: J310.7 (Pin_7), J315.8 (Pin_8)
Changed lines of the file:
@@
 LIBS:diode
 LIBS:analog_devices
+LIBS:ADS1115IDGST
+LIBS:spark_esp32thing
 LIBS:sensors
 LIBS:Worldsemi
 LIBS:LocalPower
+LIBS:pogopins02x06_pitch5.08
 LIBS:G2-cache
 EELAYER 26 0
@@
 $EndComp
 Text GLabel 15350 2750 0    60   Input ~ 0
+Wiegand_D0
+Text GLabel 15350 2850 0    60   Input ~ 0
 Wiegand_D1
-Text GLabel 15350 2850 0    60   Input ~ 0
-Wiegand_D2
 Text GLabel 15350 3800 0    60   Input ~ 0
 BELL
@@
 I2C_PWR_CTRL
 Text GLabel 10650 1350 0    60   Input ~ 0
+Wiegand_D0
+Text GLabel 11150 1350 2    60   Input ~ 0
 Wiegand_D1
-Text GLabel 11150 1350 2    60   Input ~ 0
-Wiegand_D2
 Text GLabel 10650 1750 0    60   Input ~ 0
 ANALOG_I2C_SCL

Commit message: Removed I2C power control
Parts:
- removed Q309: ZXTN25050DFHTA, TO_SOT_Packages_SMD:SOT-23, symbol Q_NPN_BCE
- removed R334: 470, Resistors_SMD:R_0805, symbol R
Connections:
- net I2C_PWR is gone; now on net +3V3: C309.1, U309.9 (VCC)
- net I2C_PWR_CTRL: no longer names the net of J310.4 (Pin_4)
- no-connect marks 2 -> 3
Other:
- moved on the sheet: C309, Q310, R335
Changed lines of the file:
@@
 L C C309
 U 1 1 59C4102A
-P 8050 3250
-F 0 "C309" H 8165 3296 50  0000 L CNN
-F 1 "100n" H 8165 3205 50  0000 L CNN
-F 2 "Capacitors_SMD:C_0805" H 8088 3100 50  0001 C CNN
-F 3 "" H 8050 3250 50  0001 C CNN
-	1    8050 3250
+P 8050 3200
+F 0 "C309" H 8165 3246 50  0000 L CNN
+F 1 "100n" H 8165 3155 50  0000 L CNN
+F 2 "Capacitors_SMD:C_0805" H 8088 3050 50  0001 C CNN
+F 3 "" H 8050 3200 50  0001 C CNN
+	1    8050 3200
 	1    0    0    -1
 $EndComp
@@
 L GND #PWR044
 U 1 1 59C42024
-P 8050 3400
-F 0 "#PWR044" H 8050 3150 50  0001 C CNN
-F 1 "GND" H 8055 3227 50  0000 C CNN
-F 2 "" H 8050 3400 50  0001 C CNN
-F 3 "" H 8050 3400 50  0001 C CNN
-	1    8050 3400
+P 8050 3350
+F 0 "#PWR044" H 8050 3100 50  0001 C CNN
+F 1 "GND" H 8055 3177 50  0000 C CNN
+F 2 "" H 8050 3350 50  0001 C CNN
+F 3 "" H 8050 3350 50  0001 C CNN
+	1    8050 3350
 	1    0    0    -1
 $EndComp
@@
 Text Notes 8550 3550 1    60   ~ 0
 Near MCP23017
-Text GLabel 8050 4150 1    60   Input ~ 0
-I2C_PWR
 $Comp
 L +3.3V #PWR019
@@
 	0    1    1    0
 $EndComp
-Text GLabel 8050 3100 1    60   Input ~ 0
-I2C_PWR
 $Comp
 L Q_NPN_BCE Q310
 U 1 1 59CCBF12
-P 13500 6800
-F 0 "Q310" V 13700 6750 50  0000 L CNN
-F 1 "ZXTN25050DFHTA" H 12900 6650 50  0000 L CNN
-F 2 "TO_SOT_Packages_SMD:SOT-23" H 13700 6900 50  0001 C CNN
-F 3 "" H 13500 6800 50  0001 C CNN
-	1    13500 6800
+P 11500 4350
+F 0 "Q310" V 11700 4300 50  0000 L CNN
+F 1 "ZXTN25050DFHTA" H 10900 4200 50  0000 L CNN
+F 2 "TO_SOT_Packages_SMD:SOT-23" H 11700 4450 50  0001 C CNN
+F 3 "" H 11500 4350 50  0001 C CNN
+	1    11500 4350
 	1    0    0    -1
 $EndComp
@@
 L GND #PWR020
 U 1 1 59CCBF1E
-P 13600 7100
-F 0 "#PWR020" H 13600 6850 50  0001 C CNN
-F 1 "GND" H 13605 6927 50  0000 C CNN
-F 2 "" H 13600 7100 50  0001 C CNN
-F 3 "" H 13600 7100 50  0001 C CNN
-	1    13600 7100
+P 11600 4650
+F 0 "#PWR020" H 11600 4400 50  0001 C CNN
+F 1 "GND" H 11605 4477 50  0000 C CNN
+F 2 "" H 11600 4650 50  0001 C CNN
+F 3 "" H 11600 4650 50  0001 C CNN
+	1    11600 4650
 	1    0    0    -1
 $EndComp
@@
 L R R335
 U 1 1 59CCBF29
-P 13100 6800
-F 0 "R335" V 13000 6800 50  0000 C CNN
-F 1 "470" V 13100 6800 50  0000 C CNN
-F 2 "Resistors_SMD:R_0805" V 13030 6800 50  0001 C CNN
-F 3 "" H 13100 6800 50  0001 C CNN
-	1    13100 6800
-	0    1    1    0
-$EndComp
-Text GLabel 13900 6600 2    60   Input ~ 0
+P 11100 4350
+F 0 "R335" V 11000 4350 50  0000 C CNN
+F 1 "470" V 11100 4350 50  0000 C CNN
+F 2 "Resistors_SMD:R_0805" V 11030 4350 50  0001 C CNN
+F 3 "" H 11100 4350 50  0001 C CNN
+	1    11100 4350
+	0    1    1    0
+$EndComp
+Text GLabel 11900 4150 2    60   Input ~ 0
 BELL
-Text GLabel 12950 6800 0    60   Input ~ 0
+Text GLabel 10950 4350 0    60   Input ~ 0
 BELL_CTRL
 Text GLabel 6400 7450 0    60   Input ~ 0
@@
 Text Notes 7950 9500 2    60   ~ 0
 To status card
-$Comp
-L Q_NPN_BCE Q309
-U 1 1 59CF0CB0
-P 9700 2950
-F 0 "Q309" V 9900 2900 50  0000 L CNN
-F 1 "ZXTN25050DFHTA" H 9100 2800 50  0000 L CNN
-F 2 "TO_SOT_Packages_SMD:SOT-23" H 9900 3050 50  0001 C CNN
-F 3 "" H 9700 2950 50  0001 C CNN
-	1    9700 2950
-	-1   0    0    -1
-$EndComp
-$Comp
-L R R334
-U 1 1 59CF0CB7
-P 10100 2950
-F 0 "R334" V 10000 2950 50  0000 C CNN
-F 1 "470" V 10100 2950 50  0000 C CNN
-F 2 "Resistors_SMD:R_0805" V 10030 2950 50  0001 C CNN
-F 3 "" H 10100 2950 50  0001 C CNN
-	1    10100 2950
-	0    -1   1    0
-$EndComp
-$Comp
-L +3.3V #PWR021
-U 1 1 59CF0CBE
-P 9600 2750
-F 0 "#PWR021" H 9600 2600 50  0001 C CNN
-F 1 "+3.3V" H 9615 2923 50  0000 C CNN
-F 2 "" H 9600 2750 50  0001 C CNN
-F 3 "" H 9600 2750 50  0001 C CNN
-	1    9600 2750
-	1    0    0    -1
-$EndComp
-Text GLabel 9600 3150 3    60   Input ~ 0
-I2C_PWR
-Text GLabel 10250 2950 2    60   Input ~ 0
-I2C_PWR_CTRL
 $Comp
 L Conn_01x09 J316
@@
 	7750 2750 7750 3650
 Wire Wire Line
-	13600 7100 13600 7000
-Wire Wire Line
-	13900 6600 13600 6600
-Wire Wire Line
-	13250 6800 13300 6800
-Wire Wire Line
-	9950 2950 9900 2950
+	11600 4650 11600 4550
+Wire Wire Line
+	11900 4150 11600 4150
+Wire Wire Line
+	11250 4350 11300 4350
 Wire Bus Line
 	7300 650  7300 1650
@@
 Text GLabel 11150 1250 2    60   Input ~ 0
 DIGITAL_I2C_SDA
-Text GLabel 11150 1150 2    60   Input ~ 0
-I2C_PWR_CTRL
 Text GLabel 10650 1350 0    60   Input ~ 0
 Wiegand_D0
@@
 	0    -1   1    0
 $EndComp
-Text GLabel 10100 3900 1    60   Input ~ 0
-I2C_PWR
-$Comp
-L PWR_FLAG #FLG03
-U 1 1 59D17995
-P 10100 3900
-F 0 "#FLG03" H 10100 3975 50  0001 C CNN
-F 1 "PWR_FLAG" H 10100 4073 50  0000 C CNN
-F 2 "" H 10100 3900 50  0001 C CNN
-F 3 "" H 10100 3900 50  0001 C CNN
-	1    10100 3900
-	-1   0    0    1
-$EndComp
 Text Label 13650 1350 2    60   ~ 0
 DO1_GND_CTRL
@@
 Wire Wire Line
 	4600 2000 5150 2000
+$Comp
+L +3.3V #PWR021
+U 1 1 5A53CE41
+P 8050 4150
+F 0 "#PWR021" H 8050 4000 50  0001 C CNN
+F 1 "+3.3V" V 8050 4400 50  0000 C CNN
+F 2 "" H 8050 4150 50  0001 C CNN
+F 3 "" H 8050 4150 50  0001 C CNN
+	1    8050 4150
+	1    0    0    -1
+$EndComp
+$Comp
+L +3.3V #PWR0162
+U 1 1 5A53D1F2
+P 8050 3050
+F 0 "#PWR0162" H 8050 2900 50  0001 C CNN
+F 1 "+3.3V" H 8050 3250 50  0000 C CNN
+F 2 "" H 8050 3050 50  0001 C CNN
+F 3 "" H 8050 3050 50  0001 C CNN
+	1    8050 3050
+	1    0    0    -1
+$EndComp
+NoConn ~ 11150 1150
 $EndSCHEMATC
