File: G2/Power.sch (KiCad schematic (older format))
At the start: 18 parts, among them J201 Conn_01x09, J202 Conn_01x09, J203 Conn_01x09, J204 Conn_01x09, J205 Conn_01x09, J206 Conn_01x09, U201 LM1084-3.3, U202 LM1084-5.0

Commit message: Added ground vias
Parts:
- added FL201: EMI_Filter_LCL, Pin_Headers:Pin_Header_Straight_1x03_Pitch2.54mm, symbol EMI_Filter_LCL
Connections:
- net +12V: now also FL201.1; no longer D201.2 (A), D202.2 (A)
- net +3V3: no longer J201.4 (Pin_4)
- net +5V: no longer J201.6 (Pin_6)
- net GND: now also FL201.2; no longer J201.3 (Pin_3), J201.5 (Pin_5)
- new net 12V: D201.2 (A), D202.2 (A), FL201.3
Changed lines of the file:
@@
 $EndDescr
-$Comp
-L +12V #PWR0203
-U 1 1 59BF8056
-P 2200 2350
-F 0 "#PWR0203" H 2200 2200 50  0001 C CNN
-F 1 "+12V" H 2215 2523 50  0000 C CNN
-F 2 "" H 2200 2350 50  0001 C CNN
-F 3 "" H 2200 2350 50  0001 C CNN
-	1    2200 2350
-	1    0    0    -1
-$EndComp
 $Comp
 L GND #PWR0204
@@
 Connection ~ 4950 2500
 Wire Wire Line
-	2200 2350 2200 3200
-Wire Wire Line
 	3700 3200 4950 3200
 Connection ~ 4450 3500
@@
 Connection ~ 2800 3200
 Wire Wire Line
-	2200 2500 2350 2500
+	1950 2500 2350 2500
 Wire Wire Line
 	2200 3200 2350 3200
@@
 $EndComp
 $Comp
-L +3.3V #PWR0211
-U 1 1 59BFF8FD
-P 6400 1150
-F 0 "#PWR0211" H 6400 1000 50  0001 C CNN
-F 1 "+3.3V" V 6415 1278 50  0000 L CNN
-F 2 "" H 6400 1150 50  0001 C CNN
-F 3 "" H 6400 1150 50  0001 C CNN
-	1    6400 1150
+L EMI_Filter_LCL FL201
+U 1 1 59C1AAEC
+P 1650 2600
+F 0 "FL201" H 1650 2917 50  0000 C CNN
+F 1 "EMI_Filter_LCL" H 1650 2826 50  0000 C CNN
+F 2 "Pin_Headers:Pin_Header_Straight_1x03_Pitch2.54mm" V 1650 2600 50  0001 C CNN
+F 3 "http://www.mouser.se/Search/ProductDetail.aspx?R=DSS1NB31H104Q91Avirtualkey64800000virtualkey81-DSS1NB31H104Q91A" V 1650 2600 50  0001 C CNN
+	1    1650 2600
+	1    0    0    -1
+$EndComp
+$Comp
+L GND #PWR01
+U 1 1 59C1AD14
+P 1650 2700
+F 0 "#PWR01" H 1650 2450 50  0001 C CNN
+F 1 "GND" H 1655 2527 50  0000 C CNN
+F 2 "" H 1650 2700 50  0001 C CNN
+F 3 "" H 1650 2700 50  0001 C CNN
+	1    1650 2700
+	1    0    0    -1
+$EndComp
+$Comp
+L +12V #PWR02
+U 1 1 59C1AE88
+P 1350 2500
+F 0 "#PWR02" H 1350 2350 50  0001 C CNN
+F 1 "+12V" H 1365 2673 50  0000 C CNN
+F 2 "" H 1350 2500 50  0001 C CNN
+F 3 "" H 1350 2500 50  0001 C CNN
+	1    1350 2500
 	0    -1   -1   0
 $EndComp
-$Comp
-L +5V #PWR0213
-U 1 1 59BFF9BC
-P 6400 1350
-F 0 "#PWR0213" H 6400 1200 50  0001 C CNN
-F 1 "+5V" V 6415 1478 50  0000 L CNN
-F 2 "" H 6400 1350 50  0001 C CNN
-F 3 "" H 6400 1350 50  0001 C CNN
-	1    6400 1350
-	0    -1   -1   0
-$EndComp
-$Comp
-L GND #PWR0210
-U 1 1 59BFFA21
-P 6400 1050
-F 0 "#PWR0210" H 6400 800 50  0001 C CNN
-F 1 "GND" V 6405 922 50  0000 R CNN
-F 2 "" H 6400 1050 50  0001 C CNN
-F 3 "" H 6400 1050 50  0001 C CNN
-	1    6400 1050
-	0    1    1    0
-$EndComp
-$Comp
-L GND #PWR0212
-U 1 1 59BFFA50
-P 6400 1250
-F 0 "#PWR0212" H 6400 1000 50  0001 C CNN
-F 1 "GND" V 6405 1122 50  0000 R CNN
-F 2 "" H 6400 1250 50  0001 C CNN
-F 3 "" H 6400 1250 50  0001 C CNN
-	1    6400 1250
-	0    1    1    0
-$EndComp
+Text Label 1350 2500 1    60   ~ 0
+12V_Source
+Wire Wire Line
+	2200 3200 2200 2500
 $EndSCHEMATC

Commit message: Completed digital IO. Begun analog sensing.
Parts:
- removed J201, J202, J203, J204, J205, J206: Conn_01x09, LocalComponents:MOLEX_1x9_39544-3009, symbol Conn_01x09
- added J? (x2): GS2, Pin_Headers:Pin_Header_Straight_1x02_Pitch2.54mm, symbol GS2
Connections:
- net +3V3: now also J?.1 (G1); no longer U201.2 (VO)
- net +5V: now also J?.1 (G1); no longer U202.2 (VO)
- new net: J?.2 (G2), U201.2 (VO)
- new net: J?.2 (G2), U202.2 (VO)
Other:
- moved on the sheet: C203, C204, C205, C206, D203, D204

Commit message: Begun layout.
Parts:
- gave numbers to parts that had none: 2
Changed lines of the file:
@@
 LIBS:sensors
 LIBS:Worldsemi
+LIBS:LocalPower
 LIBS:G2-cache
 EELAYER 26 0
@@
 $Descr A4 11693 8268
 encoding utf-8
-Sheet 2 7
+Sheet 2 6
 Title ""
 Date ""
@@
 	2200 3200 2200 2500
 $Comp
-L GS2 J?
+L GS2 J201
 U 1 1 59C6A7C3
 P 3900 2500
-F 0 "J?" V 3695 2500 50  0000 C CNN
+F 0 "J201" V 3695 2500 50  0000 C CNN
 F 1 "GS2" V 3786 2500 50  0000 C CNN
 F 2 "Pin_Headers:Pin_Header_Straight_1x02_Pitch2.54mm" V 3974 2500 50  0001 C CNN
@@
 $EndComp
 $Comp
-L GS2 J?
+L GS2 J202
 U 1 1 59C6AA5F
 P 3900 3200
-F 0 "J?" V 3695 3200 50  0000 C CNN
+F 0 "J202" V 3695 3200 50  0000 C CNN
 F 1 "GS2" V 3786 3200 50  0000 C CNN
 F 2 "Pin_Headers:Pin_Header_Straight_1x02_Pitch2.54mm" V 3974 3200 50  0001 C CNN

Commit message: Layout of IO board completed, except bell transistor.
Connections:
- net 12V renamed +12V_Filtered
Changed lines of the file:
@@
 	-1   0    0    1
 $EndComp
-Text Notes 1950 2100 0    60   ~ 0
+Text Notes 1450 2150 0    60   ~ 0
 3.5A / 41.5W
 $Comp
@@
 Text Label 1350 2500 1    60   ~ 0
 12V_Source
+$Comp
+L GS2 J201
+U 1 1 59C6A7C3
+P 3900 2500
+F 0 "J201" V 3695 2500 50  0000 C CNN
+F 1 "GS2" V 3786 2500 50  0000 C CNN
+F 2 "Pin_Headers:Pin_Header_Straight_1x02_Pitch2.54mm" V 3974 2500 50  0001 C CNN
+F 3 "" H 3900 2500 50  0001 C CNN
+	1    3900 2500
+	0    1    1    0
+$EndComp
+$Comp
+L GS2 J202
+U 1 1 59C6AA5F
+P 3900 3200
+F 0 "J202" V 3695 3200 50  0000 C CNN
+F 1 "GS2" V 3786 3200 50  0000 C CNN
+F 2 "Pin_Headers:Pin_Header_Straight_1x02_Pitch2.54mm" V 3974 3200 50  0001 C CNN
+F 3 "" H 3900 3200 50  0001 C CNN
+	1    3900 3200
+	0    1    1    0
+$EndComp
+Text GLabel 2200 2400 1    60   Input ~ 0
++12V_Filtered
 Wire Wire Line
 	2800 2800 5200 2800
@@
 	2650 3200 3100 3200
 Wire Wire Line
-	2200 3200 2200 2500
-$Comp
-L GS2 J201
-U 1 1 59C6A7C3
-P 3900 2500
-F 0 "J201" V 3695 2500 50  0000 C CNN
-F 1 "GS2" V 3786 2500 50  0000 C CNN
-F 2 "Pin_Headers:Pin_Header_Straight_1x02_Pitch2.54mm" V 3974 2500 50  0001 C CNN
-F 3 "" H 3900 2500 50  0001 C CNN
-	1    3900 2500
-	0    1    1    0
-$EndComp
-$Comp
-L GS2 J202
-U 1 1 59C6AA5F
-P 3900 3200
-F 0 "J202" V 3695 3200 50  0000 C CNN
-F 1 "GS2" V 3786 3200 50  0000 C CNN
-F 2 "Pin_Headers:Pin_Header_Straight_1x02_Pitch2.54mm" V 3974 3200 50  0001 C CNN
-F 3 "" H 3900 3200 50  0001 C CNN
-	1    3900 3200
-	0    1    1    0
-$EndComp
+	2200 2400 2200 3200
 $EndSCHEMATC

Commit message: Layout completed. No display - it won't fit in the enclosure
Changed lines of the file:
@@
 L PWR_FLAG #FLG0201
 U 1 1 59BFAAB0
-P 1750 1550
-F 0 "#FLG0201" H 1750 1625 50  0001 C CNN
-F 1 "PWR_FLAG" H 1750 1723 50  0000 C CNN
-F 2 "" H 1750 1550 50  0001 C CNN
-F 3 "" H 1750 1550 50  0001 C CNN
-	1    1750 1550
+P 1700 1250
+F 0 "#FLG0201" H 1700 1325 50  0001 C CNN
+F 1 "PWR_FLAG" H 1700 1423 50  0000 C CNN
+F 2 "" H 1700 1250 50  0001 C CNN
+F 3 "" H 1700 1250 50  0001 C CNN
+	1    1700 1250
 	-1   0    0    1
 $EndComp
@@
 L +12V #PWR0201
 U 1 1 59BFBDEF
-P 1750 1550
-F 0 "#PWR0201" H 1750 1400 50  0001 C CNN
-F 1 "+12V" H 1765 1723 50  0000 C CNN
-F 2 "" H 1750 1550 50  0001 C CNN
-F 3 "" H 1750 1550 50  0001 C CNN
-	1    1750 1550
+P 1700 1250
+F 0 "#PWR0201" H 1700 1100 50  0001 C CNN
+F 1 "+12V" H 1715 1423 50  0000 C CNN
+F 2 "" H 1700 1250 50  0001 C CNN
+F 3 "" H 1700 1250 50  0001 C CNN
+	1    1700 1250
 	1    0    0    -1
 $EndComp
@@
 L PWR_FLAG #FLG0202
 U 1 1 59BFBE64
-P 2100 1550
-F 0 "#FLG0202" H 2100 1625 50  0001 C CNN
-F 1 "PWR_FLAG" H 2100 1724 50  0000 C CNN
-F 2 "" H 2100 1550 50  0001 C CNN
-F 3 "" H 2100 1550 50  0001 C CNN
-	1    2100 1550
+P 2050 1250
+F 0 "#FLG0202" H 2050 1325 50  0001 C CNN
+F 1 "PWR_FLAG" H 2050 1424 50  0000 C CNN
+F 2 "" H 2050 1250 50  0001 C CNN
+F 3 "" H 2050 1250 50  0001 C CNN
+	1    2050 1250
 	1    0    0    -1
 $EndComp
@@
 L GND #PWR0202
 U 1 1 59BFBE9F
-P 2100 1550
-F 0 "#PWR0202" H 2100 1300 50  0001 C CNN
-F 1 "GND" H 2105 1377 50  0000 C CNN
-F 2 "" H 2100 1550 50  0001 C CNN
-F 3 "" H 2100 1550 50  0001 C CNN
-	1    2100 1550
+P 2050 1250
+F 0 "#PWR0202" H 2050 1000 50  0001 C CNN
+F 1 "GND" H 2055 1077 50  0000 C CNN
+F 2 "" H 2050 1250 50  0001 C CNN
+F 3 "" H 2050 1250 50  0001 C CNN
+	1    2050 1250
 	1    0    0    -1
 $EndComp
@@
 Wire Wire Line
 	2200 2400 2200 3200
+$Comp
+L PWR_FLAG #FLG01
+U 1 1 59D10DB1
+P 2500 1250
+F 0 "#FLG01" H 2500 1325 50  0001 C CNN
+F 1 "PWR_FLAG" H 2500 1423 50  0000 C CNN
+F 2 "" H 2500 1250 50  0001 C CNN
+F 3 "" H 2500 1250 50  0001 C CNN
+	1    2500 1250
+	-1   0    0    1
+$EndComp
+$Comp
+L +3.3V #PWR056
+U 1 1 59D10DDA
+P 2500 1250
+F 0 "#PWR056" H 2500 1100 50  0001 C CNN
+F 1 "+3.3V" H 2515 1423 50  0000 C CNN
+F 2 "" H 2500 1250 50  0001 C CNN
+F 3 "" H 2500 1250 50  0001 C CNN
+	1    2500 1250
+	1    0    0    -1
+$EndComp
+$Comp
+L +5V #PWR074
+U 1 1 59D17336
+P 2850 1250
+F 0 "#PWR074" H 2850 1100 50  0001 C CNN
+F 1 "+5V" H 2865 1423 50  0000 C CNN
+F 2 "" H 2850 1250 50  0001 C CNN
+F 3 "" H 2850 1250 50  0001 C CNN
+	1    2850 1250
+	1    0    0    -1
+$EndComp
+$Comp
+L PWR_FLAG #FLG02
+U 1 1 59D1735F
+P 2850 1250
+F 0 "#FLG02" H 2850 1325 50  0001 C CNN
+F 1 "PWR_FLAG" H 2850 1423 50  0000 C CNN
+F 2 "" H 2850 1250 50  0001 C CNN
+F 3 "" H 2850 1250 50  0001 C CNN
+	1    2850 1250
+	-1   0    0    1
+$EndComp
 $EndSCHEMATC

Commit message: Added component data sheets and names
Parts:
- D201, D202: value D -> RBR3MM30ATR
Changed lines of the file:
@@
 LIBS:diode
 LIBS:analog_devices
-LIBS:ADS1115IDGST
-LIBS:spark_esp32thing
 LIBS:sensors
 LIBS:Worldsemi
 LIBS:LocalPower
-LIBS:pogopins02x06_pitch5.08
 LIBS:G2-cache
 EELAYER 26 0
@@
 U 1 1 59BF993D
 P 2500 2500
-F 0 "D201" H 2500 2284 50  0000 C CNN
-F 1 "D" H 2500 2375 50  0000 C CNN
+F 0 "D201" H 2550 2400 50  0000 C CNN
+F 1 "RBR3MM30ATR" H 2600 2650 50  0000 C CNN
 F 2 "Diodes_SMD:D_SOD-123F" H 2500 2500 50  0001 C CNN
 F 3 "http://www.mouser.se/ProductDetail/ROHM-Semiconductor/RBR3MM30ATR/?qs=sGAEpiMZZMtQ8nqTKtFS%2fI%2fhdhCnE2X2fXNJX4qgoABnAExEb9ZEtQ%3d%3d" H 2500 2500 50  0001 C CNN
@@
 U 1 1 59BF9A8A
 P 2500 3200
-F 0 "D202" H 2500 2984 50  0000 C CNN
-F 1 "D" H 2500 3075 50  0000 C CNN
+F 0 "D202" H 2550 3050 50  0000 C CNN
+F 1 "RBR3MM30ATR" H 2650 3350 50  0000 C CNN
 F 2 "Diodes_SMD:D_SOD-123F" H 2500 3200 50  0001 C CNN
 F 3 "http://www.mouser.se/ProductDetail/ROHM-Semiconductor/RBR3MM30ATR/?qs=sGAEpiMZZMtQ8nqTKtFS%2fI%2fhdhCnE2X2fXNJX4qgoABnAExEb9ZEtQ%3d%3d" H 2500 3200 50  0001 C CNN
