File: G2/Status.sch (KiCad schematic (older format))
At the start: 37 parts

Commit message: Begun layout.
Parts:
- added C601, C602, C603, C604, C605, C606, C607: 100n, Capacitors_SMD:C_0805, symbol C
- added J601: Conn_02x08_Counter_Clockwise, Pin_Headers:Pin_Header_Straight_2x08_Pitch2.54mm_SMD, symbol Conn_02x08_Counter_Clockwise
- added J602: Conn_02x06_Counter_Clockwise, Pin_Headers:Pin_Header_Straight_2x06_Pitch2.54mm_SMD, symbol Conn_02x06_Counter_Clockwise
- added J603: GS3, Pin_Headers:Pin_Header_Straight_1x03_Pitch2.54mm, symbol GS3
- added J604: Conn_01x06, Pin_Headers:Pin_Header_Straight_1x06_Pitch2.54mm, symbol Conn_01x06
- added U601: TXB0102DCU, Housings_SSOP:VSSOP-8_2.4x2.1mm_Pitch0.5mm, symbol TXB0102DCU
- gave numbers to parts that had none: 37
Connections:
- net labels added: +3V3_S, +5V_S, GND_S, LEVEL_SHIFTER_ENABLE, RGB_LED_DATA_CTRL
- net labels removed: +3.3V, +5V, DI1, DI2, DI3, DI4, DI5, DI6, DI7, DI8, DO1_GND_CTRL, DO3_GND_CTRL, DO4_GND_CTRL, DO5_GND_CTRL, DO6_GND_CTRL, DO7_GND_CTRL, DO8_GND_CTRL, GND, RGB_LED_DATA
- wire segments 36 -> 106
- no-connect marks 0 -> 2
Other:
- note added: "Digial inputs"
- note added: "Digital outputs"
- note added: "SPI"
- note added: "To Backplane"
- note added: "To MCU"
- moved on the sheet: D601, D602, D603, D604, D605, D606, D607, D608, D609, D610, D611, D612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

Commit message: Layout of IO board completed, except bell transistor.
Parts:
- removed J601: Conn_02x08_Counter_Clockwise, Pin_Headers:Pin_Header_Straight_2x08_Pitch2.54mm_SMD, symbol Conn_02x08_Counter_Clockwise
- added J601: Conn_02x08_Odd_Even, Pin_Headers:Pin_Header_Straight_2x08_Pitch2.54mm_SMD, symbol Conn_02x08_Odd_Even
Connections:
- wire segments 106 -> 125
Other:
- moved on the sheet: D601, D602, D603, D604, D605, D606, D607, D608, D609, D610, D611, D612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

Commit message: Layout nearly complete, only LCD left
Parts:
- removed J602: Conn_02x06_Counter_Clockwise, Pin_Headers:Pin_Header_Straight_2x06_Pitch2.54mm_SMD, symbol Conn_02x06_Counter_Clockwise
- added PG601: PogoPins02x06_Pitch5.08_ContactSurface, PogoPins02x06_Pitch5:PogoPins02x06_Pitch5.08_ContactSurface, symbol PogoPins02x06_Pitch5.08_ContactSurface
Other:
- moved on the sheet: J603
Changed lines of the file:
@@
 LIBS:Worldsemi
 LIBS:LocalPower
+LIBS:pogopins02x06_pitch5.08
 LIBS:G2-cache
 EELAYER 26 0
@@
 $EndComp
 NoConn ~ 2450 1700
-$Comp
-L Conn_01x06 J604
-U 1 1 59CD2565
-P 8950 2650
-F 0 "J604" H 9030 2642 50  0000 L CNN
-F 1 "Conn_01x06" H 9030 2551 50  0000 L CNN
-F 2 "Pin_Headers:Pin_Header_Straight_1x06_Pitch2.54mm" H 8950 2650 50  0001 C CNN
-F 3 "" H 8950 2650 50  0001 C CNN
-	1    8950 2650
-	1    0    0    -1
-$EndComp
-$Comp
-L GS3 J603
-U 1 1 59CD27C9
-P 7850 2550
-F 0 "J603" H 7850 2855 50  0000 C CNN
-F 1 "GS3" H 7850 2764 50  0000 C CNN
-F 2 "Pin_Headers:Pin_Header_Straight_1x03_Pitch2.54mm" V 7938 2476 50  0001 C CNN
-F 3 "" H 7850 2550 50  0001 C CNN
-	1    7850 2550
-	1    0    0    -1
-$EndComp
 NoConn ~ 9000 1400
 Text Label 3800 2950 0    60   ~ 0
@@
 Text Label 3800 1900 0    60   ~ 0
 LEVEL_SHIFTER_ENABLE
-Text Notes 8900 3100 0    60   ~ 0
-SPI
-Text Label 6700 2650 0    60   ~ 0
-VSPI_CLK
-Text Label 6700 2750 0    60   ~ 0
-VSPI_D/MOSI
-Text Label 6700 2850 0    60   ~ 0
-VSPI_Q/MISO
-Text Label 6700 2950 0    60   ~ 0
-VSPI_CS0
-Text Notes 5750 3150 0    60   ~ 0
-To MCU
 Text Notes 2160 5500 3    60   ~ 0
 To Backplane
@@
 	1    8600 950
 	0    -1   1    0
-$EndComp
-$Comp
-L Conn_02x06_Counter_Clockwise J602
-U 1 1 59C8EF69
-P 5850 2650
-F 0 "J602" H 5900 3067 50  0000 C CNN
-F 1 "Conn_02x06_Counter_Clockwise" H 5900 2976 50  0000 C CNN
-F 2 "Pin_Headers:Pin_Header_Straight_2x06_Pitch2.54mm_SMD" H 5850 2650 50  0001 C CNN
-F 3 "" H 5850 2650 50  0001 C CNN
-	1    5850 2650
-	1    0    0    -1
 $EndComp
 Text Notes 1260 3350 3    60   ~ 0
@@
 L +3V3_S #PWR0130
 U 1 1 59CAE1C1
-P 6150 2450
-F 0 "#PWR0130" H 6150 2300 50  0001 C CNN
-F 1 "+3V3_S" V 6165 2578 50  0000 L CNN
-F 2 "" H 6150 2450 50  0001 C CNN
-F 3 "" H 6150 2450 50  0001 C CNN
-	1    6150 2450
+P 6000 2450
+F 0 "#PWR0130" H 6000 2300 50  0001 C CNN
+F 1 "+3V3_S" V 6000 2600 50  0000 L CNN
+F 2 "" H 6000 2450 50  0001 C CNN
+F 3 "" H 6000 2450 50  0001 C CNN
+	1    6000 2450
 	0    1    1    0
 $EndComp
@@
 L GND_S #PWR0131
 U 1 1 59CAE2F4
-P 5650 2450
-F 0 "#PWR0131" H 5650 2200 50  0001 C CNN
-F 1 "GND_S" V 5655 2322 50  0000 R CNN
-F 2 "" H 5650 2450 50  0001 C CNN
-F 3 "" H 5650 2450 50  0001 C CNN
-	1    5650 2450
+P 5350 2450
+F 0 "#PWR0131" H 5350 2200 50  0001 C CNN
+F 1 "GND_S" V 5355 2322 50  0000 R CNN
+F 2 "" H 5350 2450 50  0001 C CNN
+F 3 "" H 5350 2450 50  0001 C CNN
+	1    5350 2450
 	0    1    1    0
 $EndComp
@@
 L +3V3_S #PWR0132
 U 1 1 59CAE368
-P 6150 2550
-F 0 "#PWR0132" H 6150 2400 50  0001 C CNN
-F 1 "+3V3_S" V 6165 2678 50  0000 L CNN
-F 2 "" H 6150 2550 50  0001 C CNN
-F 3 "" H 6150 2550 50  0001 C CNN
-	1    6150 2550
+P 6000 2550
+F 0 "#PWR0132" H 6000 2400 50  0001 C CNN
+F 1 "+3V3_S" V 6000 2700 50  0000 L CNN
+F 2 "" H 6000 2550 50  0001 C CNN
+F 3 "" H 6000 2550 50  0001 C CNN
+	1    6000 2550
 	0    1    1    0
 $EndComp
@@
 L GND_S #PWR0133
 U 1 1 59CAE815
-P 5650 2550
-F 0 "#PWR0133" H 5650 2300 50  0001 C CNN
-F 1 "GND_S" V 5655 2422 50  0000 R CNN
-F 2 "" H 5650 2550 50  0001 C CNN
-F 3 "" H 5650 2550 50  0001 C CNN
-	1    5650 2550
+P 5350 2550
+F 0 "#PWR0133" H 5350 2300 50  0001 C CNN
+F 1 "GND_S" V 5355 2422 50  0000 R CNN
+F 2 "" H 5350 2550 50  0001 C CNN
+F 3 "" H 5350 2550 50  0001 C CNN
+	1    5350 2550
 	0    1    1    0
 $EndComp
@@
 L +5V_S #PWR0134
 U 1 1 59CAED7D
-P 5650 2650
-F 0 "#PWR0134" H 5650 2500 50  0001 C CNN
-F 1 "+5V_S" V 5665 2778 50  0000 L CNN
-F 2 "" H 5650 2650 50  0001 C CNN
-F 3 "" H 5650 2650 50  0001 C CNN
-	1    5650 2650
+P 5350 2650
+F 0 "#PWR0134" H 5350 2500 50  0001 C CNN
+F 1 "+5V_S" V 5365 2778 50  0000 L CNN
+F 2 "" H 5350 2650 50  0001 C CNN
+F 3 "" H 5350 2650 50  0001 C CNN
+	1    5350 2650
 	0    -1   -1   0
 $EndComp
@@
 L +5V_S #PWR0135
 U 1 1 59CAEEB5
-P 5650 2750
-F 0 "#PWR0135" H 5650 2600 50  0001 C CNN
-F 1 "+5V_S" V 5665 2878 50  0000 L CNN
-F 2 "" H 5650 2750 50  0001 C CNN
-F 3 "" H 5650 2750 50  0001 C CNN
-	1    5650 2750
+P 5350 2750
+F 0 "#PWR0135" H 5350 2600 50  0001 C CNN
+F 1 "+5V_S" V 5365 2878 50  0000 L CNN
+F 2 "" H 5350 2750 50  0001 C CNN
+F 3 "" H 5350 2750 50  0001 C CNN
+	1    5350 2750
 	0    -1   -1   0
 $EndComp
@@
 $EndComp
 $Comp
-L +3V3_S #PWR0159
-U 1 1 59CB3349
-P 7700 2450
-F 0 "#PWR0159" H 7700 2300 50  0001 C CNN
-F 1 "+3V3_S" V 7715 2578 50  0000 L CNN
-F 2 "" H 7700 2450 50  0001 C CNN
-F 3 "" H 7700 2450 50  0001 C CNN
-	1    7700 2450
-	0    -1   -1   0
-$EndComp
-$Comp
-L +5V_S #PWR0160
-U 1 1 59CB3519
-P 7700 2650
-F 0 "#PWR0160" H 7700 2500 50  0001 C CNN
-F 1 "+5V_S" V 7700 2900 50  0000 C CNN
-F 2 "" H 7700 2650 50  0001 C CNN
-F 3 "" H 7700 2650 50  0001 C CNN
-	1    7700 2650
-	0    -1   -1   0
-$EndComp
-$Comp
 L GND_S #PWR0161
 U 1 1 59CB38C7
@@
 $EndComp
 $Comp
-L GND_S #PWR0163
-U 1 1 59CB489A
-P 8750 2450
-F 0 "#PWR0163" H 8750 2200 50  0001 C CNN
-F 1 "GND_S" V 8755 2322 50  0000 R CNN
-F 2 "" H 8750 2450 50  0001 C CNN
-F 3 "" H 8750 2450 50  0001 C CNN
-	1    8750 2450
-	0    1    1    0
-$EndComp
-$Comp
 L GND_S #PWR0127
 U 1 1 59CB54ED
@@
 	1500 6750 1500 6700
 Wire Wire Line
-	2450 1900 5200 1900
-Wire Wire Line
 	2150 1000 2150 1100
 Wire Wire Line
@@
 	2450 1500 3200 1500
 Wire Wire Line
-	8000 2550 8750 2550
-Wire Wire Line
 	2600 4450 2600 5000
 Wire Wire Line
@@
 	3650 5550 3650 6400
 Wire Wire Line
-	5200 1900 5200 2850
-Wire Wire Line
-	5200 2850 5650 2850
-Wire Wire Line
 	1650 1500 1250 1500
 Wire Wire Line
 	1250 1500 1250 2950
-Wire Wire Line
-	1250 2950 5650 2950
-Wire Wire Line
-	8750 2650 8000 2650
-Wire Wire Line
-	8000 2650 8000 2750
-Wire Wire Line
-	8000 2750 7350 2750
-Wire Wire Line
-	7350 2750 7350 2650
-Wire Wire Line
-	7350 2650 6150 2650
-Wire Wire Line
-	8750 2750 8050 2750
-Wire Wire Line
-	8050 2750 8050 2800
-Wire Wire Line
-	8050 2800 7300 2800
-Wire Wire Line
-	7300 2800 7300 2750
-Wire Wire Line
-	7300 2750 6150 2750
-Wire Wire Line
-	8750 2850 6150 2850
-Wire Wire Line
-	6150 2950 8750 2950
 Wire Notes Line
 	1150 3250 1150 4900
@@
 Wire Wire Line
 	2750 6200 2750 6400
+Wire Wire Line
+	6000 2950 8600 2950
+Wire Wire Line
+	8600 2850 6000 2850
+Wire Wire Line
+	7150 2750 6000 2750
+Wire Wire Line
+	7150 2800 7150 2750
+Wire Wire Line
+	7900 2800 7150 2800
+Wire Wire Line
+	7900 2750 7900 2800
+Wire Wire Line
+	8600 2750 7900 2750
+Wire Wire Line
+	7200 2650 6000 2650
+Wire Wire Line
+	7200 2750 7200 2650
+Wire Wire Line
+	7850 2750 7200 2750
+Wire Wire Line
+	7850 2650 7850 2750
+Wire Wire Line
+	8600 2650 7850 2650
+Wire Wire Line
+	7850 2550 8600 2550
+$Comp
+L GND_S #PWR0163
+U 1 1 59CB489A
+P 8600 2450
+F 0 "#PWR0163" H 8600 2200 50  0001 C CNN
+F 1 "GND_S" V 8605 2322 50  0000 R CNN
+F 2 "" H 8600 2450 50  0001 C CNN
+F 3 "" H 8600 2450 50  0001 C CNN
+	1    8600 2450
+	0    1    1    0
+$EndComp
+$Comp
+L +5V_S #PWR0160
+U 1 1 59CB3519
+P 7550 2650
+F 0 "#PWR0160" H 7550 2500 50  0001 C CNN
+F 1 "+5V_S" V 7550 2900 50  0000 C CNN
+F 2 "" H 7550 2650 50  0001 C CNN
+F 3 "" H 7550 2650 50  0001 C CNN
+	1    7550 2650
+	0    -1   -1   0
+$EndComp
+$Comp
+L +3V3_S #PWR0159
+U 1 1 59CB3349
+P 7550 2450
+F 0 "#PWR0159" H 7550 2300 50  0001 C CNN
+F 1 "+3V3_S" V 7565 2578 50  0000 L CNN
+F 2 "" H 7550 2450 50  0001 C CNN
+F 3 "" H 7550 2450 50  0001 C CNN
+	1    7550 2450
+	0    -1   -1   0
+$EndComp
+Text Label 6550 2950 0    60   ~ 0
+VSPI_CS0
+Text Label 6550 2850 0    60   ~ 0
+VSPI_Q/MISO
+Text Label 6550 2750 0    60   ~ 0
+VSPI_D/MOSI
+Text Label 6550 2650 0    60   ~ 0
+VSPI_CLK
+Text Notes 8650 3100 0    60   ~ 0
+SPI
+$Comp
+L GS3 J603
+U 1 1 59CD27C9
+P 7700 2550
+F 0 "J603" H 7700 2855 50  0000 C CNN
+F 1 "GS3" H 7700 2764 50  0000 C CNN
+F 2 "Pin_Headers:Pin_Header_Straight_1x03_Pitch2.54mm" V 7788 2476 50  0001 C CNN
+F 3 "" H 7700 2550 50  0001 C CNN
+	1    7700 2550
+	1    0    0    -1
+$EndComp
+$Comp
+L Conn_01x06 J604
+U 1 1 59CD2565
+P 8800 2650
+F 0 "J604" H 8880 2642 50  0000 L CNN
+F 1 "Conn_01x06" H 8880 2551 50  0000 L CNN
+F 2 "Pin_Headers:Pin_Header_Straight_1x06_Pitch2.54mm" H 8800 2650 50  0001 C CNN
+F 3 "" H 8800 2650 50  0001 C CNN
+	1    8800 2650
+	1    0    0    -1
+$EndComp
+Wire Wire Line
+	1250 2950 5350 2950
+Wire Wire Line
+	5350 2850 4850 2850
+Wire Wire Line
+	4850 2850 4850 1900
+Wire Wire Line
+	4850 1900 2450 1900
+$Comp
+L PogoPins02x06_Pitch5.08_ContactSurface PG601
+U 1 1 59CF7341
+P 5550 2350
+F 0 "PG601" H 5675 2497 60  0000 C CNN
+F 1 "PogoPins02x06_Pitch5.08_ContactSurface" H 5675 2391 60  0000 C CNN
+F 2 "PogoPins02x06_Pitch5:PogoPins02x06_Pitch5.08_ContactSurface" H 5550 2350 60  0001 C CNN
+F 3 "" H 5550 2350 60  0001 C CNN
+	1    5550 2350
+	1    0    0    -1
+$EndComp
+Text Notes 5500 3100 0    60   ~ 0
+To MCU
 $EndSCHEMATC

Commit message: Layout completed. No display - it won't fit in the enclosure
Parts:
- removed J603: GS3, Pin_Headers:Pin_Header_Straight_1x03_Pitch2.54mm, symbol GS3
- removed J604: Conn_01x06, Pin_Headers:Pin_Header_Straight_1x06_Pitch2.54mm, symbol Conn_01x06
Connections:
- net labels removed: VSPI_CLK, VSPI_CS0, VSPI_D/MOSI, VSPI_Q/MISO
- wire segments 125 -> 112
- no-connect marks 2 -> 3
Other:
- note removed: "SPI"
- moved on the sheet: C603
Changed lines of the file:
@@
 $EndComp
 NoConn ~ 2450 1700
-NoConn ~ 9000 1400
 Text Label 3800 2950 0    60   ~ 0
 RGB_LED_DATA_CTRL
@@
 L C C603
 U 1 1 59D1E003
-P 3600 900
-F 0 "C603" V 3348 900 50  0000 C CNN
-F 1 "100n" V 3439 900 50  0000 C CNN
-F 2 "Capacitors_SMD:C_0805" H 3638 750 50  0001 C CNN
-F 3 "" H 3600 900 50  0001 C CNN
-	1    3600 900
+P 3600 950
+F 0 "C603" V 3348 950 50  0000 C CNN
+F 1 "100n" V 3439 950 50  0000 C CNN
+F 2 "Capacitors_SMD:C_0805" H 3638 800 50  0001 C CNN
+F 3 "" H 3600 950 50  0001 C CNN
+	1    3600 950
 	0    -1   1    0
 $EndComp
@@
 L +5V_S #PWR0141
 U 1 1 59CB1AF8
-P 3450 900
-F 0 "#PWR0141" H 3450 750 50  0001 C CNN
-F 1 "+5V_S" V 3450 1150 50  0000 C CNN
-F 2 "" H 3450 900 50  0001 C CNN
-F 3 "" H 3450 900 50  0001 C CNN
-	1    3450 900
+P 3450 950
+F 0 "#PWR0141" H 3450 800 50  0001 C CNN
+F 1 "+5V_S" V 3450 1200 50  0000 C CNN
+F 2 "" H 3450 950 50  0001 C CNN
+F 3 "" H 3450 950 50  0001 C CNN
+	1    3450 950
 	0    -1   -1   0
 $EndComp
@@
 L GND_S #PWR0161
 U 1 1 59CB38C7
-P 3750 900
-F 0 "#PWR0161" H 3750 650 50  0001 C CNN
-F 1 "GND_S" V 3755 772 50  0000 R CNN
-F 2 "" H 3750 900 50  0001 C CNN
-F 3 "" H 3750 900 50  0001 C CNN
-	1    3750 900
-	0    -1   -1   0
-$EndComp
-$Comp
-L GND_S #PWR0162
-U 1 1 59CB3C13
-P 1650 1700
-F 0 "#PWR0162" H 1650 1450 50  0001 C CNN
-F 1 "GND_S" V 1655 1572 50  0000 R CNN
-F 2 "" H 1650 1700 50  0001 C CNN
-F 3 "" H 1650 1700 50  0001 C CNN
-	1    1650 1700
-	0    1    1    0
+P 3750 950
+F 0 "#PWR0161" H 3750 700 50  0001 C CNN
+F 1 "GND_S" V 3755 822 50  0000 R CNN
+F 2 "" H 3750 950 50  0001 C CNN
+F 3 "" H 3750 950 50  0001 C CNN
+	1    3750 950
+	0    -1   -1   0
 $EndComp
 $Comp
@@
 	1    0    0    -1
 $EndComp
+Text Notes 5500 3100 0    60   ~ 0
+To MCU
 Wire Wire Line
 	4000 1400 4100 1400
@@
 	2750 6200 2750 6400
 Wire Wire Line
-	6000 2950 8600 2950
-Wire Wire Line
-	8600 2850 6000 2850
-Wire Wire Line
-	7150 2750 6000 2750
-Wire Wire Line
-	7150 2800 7150 2750
-Wire Wire Line
-	7900 2800 7150 2800
-Wire Wire Line
-	7900 2750 7900 2800
-Wire Wire Line
-	8600 2750 7900 2750
-Wire Wire Line
-	7200 2650 6000 2650
-Wire Wire Line
-	7200 2750 7200 2650
-Wire Wire Line
-	7850 2750 7200 2750
-Wire Wire Line
-	7850 2650 7850 2750
-Wire Wire Line
-	8600 2650 7850 2650
-Wire Wire Line
-	7850 2550 8600 2550
-$Comp
-L GND_S #PWR0163
-U 1 1 59CB489A
-P 8600 2450
-F 0 "#PWR0163" H 8600 2200 50  0001 C CNN
-F 1 "GND_S" V 8605 2322 50  0000 R CNN
-F 2 "" H 8600 2450 50  0001 C CNN
-F 3 "" H 8600 2450 50  0001 C CNN
-	1    8600 2450
-	0    1    1    0
-$EndComp
-$Comp
-L +5V_S #PWR0160
-U 1 1 59CB3519
-P 7550 2650
-F 0 "#PWR0160" H 7550 2500 50  0001 C CNN
-F 1 "+5V_S" V 7550 2900 50  0000 C CNN
-F 2 "" H 7550 2650 50  0001 C CNN
-F 3 "" H 7550 2650 50  0001 C CNN
-	1    7550 2650
-	0    -1   -1   0
-$EndComp
-$Comp
-L +3V3_S #PWR0159
-U 1 1 59CB3349
-P 7550 2450
-F 0 "#PWR0159" H 7550 2300 50  0001 C CNN
-F 1 "+3V3_S" V 7565 2578 50  0000 L CNN
-F 2 "" H 7550 2450 50  0001 C CNN
-F 3 "" H 7550 2450 50  0001 C CNN
-	1    7550 2450
-	0    -1   -1   0
-$EndComp
-Text Label 6550 2950 0    60   ~ 0
-VSPI_CS0
-Text Label 6550 2850 0    60   ~ 0
-VSPI_Q/MISO
-Text Label 6550 2750 0    60   ~ 0
-VSPI_D/MOSI
-Text Label 6550 2650 0    60   ~ 0
-VSPI_CLK
-Text Notes 8650 3100 0    60   ~ 0
-SPI
-$Comp
-L GS3 J603
-U 1 1 59CD27C9
-P 7700 2550
-F 0 "J603" H 7700 2855 50  0000 C CNN
-F 1 "GS3" H 7700 2764 50  0000 C CNN
-F 2 "Pin_Headers:Pin_Header_Straight_1x03_Pitch2.54mm" V 7788 2476 50  0001 C CNN
-F 3 "" H 7700 2550 50  0001 C CNN
-	1    7700 2550
-	1    0    0    -1
-$EndComp
-$Comp
-L Conn_01x06 J604
-U 1 1 59CD2565
-P 8800 2650
-F 0 "J604" H 8880 2642 50  0000 L CNN
-F 1 "Conn_01x06" H 8880 2551 50  0000 L CNN
-F 2 "Pin_Headers:Pin_Header_Straight_1x06_Pitch2.54mm" H 8800 2650 50  0001 C CNN
-F 3 "" H 8800 2650 50  0001 C CNN
-	1    8800 2650
-	1    0    0    -1
-$EndComp
-Wire Wire Line
 	1250 2950 5350 2950
 Wire Wire Line
@@
 Wire Wire Line
 	4850 1900 2450 1900
+NoConn ~ 9000 1400
+$Comp
+L +3V3_S #PWR0160
+U 1 1 59D34C7D
+P 7750 2750
+F 0 "#PWR0160" H 7750 2600 50  0001 C CNN
+F 1 "+3V3_S" V 7750 2900 50  0000 L CNN
+F 2 "" H 7750 2750 50  0001 C CNN
+F 3 "" H 7750 2750 50  0001 C CNN
+	1    7750 2750
+	1    0    0    -1
+$EndComp
+$Comp
+L +5V_S #PWR0163
+U 1 1 59D3546D
+P 8150 2750
+F 0 "#PWR0163" H 8150 2600 50  0001 C CNN
+F 1 "+5V_S" V 8165 2878 50  0000 L CNN
+F 2 "" H 8150 2750 50  0001 C CNN
+F 3 "" H 8150 2750 50  0001 C CNN
+	1    8150 2750
+	1    0    0    -1
+$EndComp
+$Comp
+L GND_S #PWR0164
+U 1 1 59D355C1
+P 8450 2750
+F 0 "#PWR0164" H 8450 2500 50  0001 C CNN
+F 1 "GND_S" V 8455 2622 50  0000 R CNN
+F 2 "" H 8450 2750 50  0001 C CNN
+F 3 "" H 8450 2750 50  0001 C CNN
+	1    8450 2750
+	1    0    0    -1
+$EndComp
+$Comp
+L PWR_FLAG #FLG08
+U 1 1 59D3575B
+P 7750 2750
+F 0 "#FLG08" H 7750 2825 50  0001 C CNN
+F 1 "PWR_FLAG" H 7750 2923 50  0000 C CNN
+F 2 "" H 7750 2750 50  0001 C CNN
+F 3 "" H 7750 2750 50  0001 C CNN
+	1    7750 2750
+	-1   0    0    1
+$EndComp
+$Comp
+L PWR_FLAG #FLG09
+U 1 1 59D35829
+P 8150 2750
+F 0 "#FLG09" H 8150 2825 50  0001 C CNN
+F 1 "PWR_FLAG" H 8150 2923 50  0000 C CNN
+F 2 "" H 8150 2750 50  0001 C CNN
+F 3 "" H 8150 2750 50  0001 C CNN
+	1    8150 2750
+	-1   0    0    1
+$EndComp
+$Comp
+L PWR_FLAG #FLG010
+U 1 1 59D35892
+P 8450 2750
+F 0 "#FLG010" H 8450 2825 50  0001 C CNN
+F 1 "PWR_FLAG" H 8450 2924 50  0000 C CNN
+F 2 "" H 8450 2750 50  0001 C CNN
+F 3 "" H 8450 2750 50  0001 C CNN
+	1    8450 2750
+	1    0    0    -1
+$EndComp
+NoConn ~ 1650 1700
 $Comp
 L PogoPins02x06_Pitch5.08_ContactSurface PG601
@@
 	1    0    0    -1
 $EndComp
-Text Notes 5500 3100 0    60   ~ 0
-To MCU
 $EndSCHEMATC
