File: G2/Status.sch (KiCad schematic (older format))
At the start: 47 parts, among them J601 Conn_02x08_Odd_Even, J602 Conn_01x08, U601 TXB0102DCU

Commit message: Step two of conversion to v5 format
Parts:
- C601, C602, C603, C604, C605, C606, C607: symbol G2-rescue:C -> Device:C
- D601, D602, D603, D604, D605, D606, D607, D608, D609, D610, D611, D612, D613, D614, D615, D616: symbol G2-rescue:LED -> Device:LED
- J601: symbol G2-rescue:Conn_02x08_Odd_Even -> Connector_Generic:Conn_02x08_Odd_Even
- J602: symbol G2-rescue:Conn_01x08 -> Connector_Generic:Conn_01x08
- LED601, LED602, LED603, LED604, LED605: symbol G2-rescue:WS2812B -> LED:WS2812B
- R601, R602, R603, R604, R605, R606, R607, R608, R609, R610, R611, R612, R613, R614, R615, R616: symbol G2-rescue:R -> Device:R
- U601: symbol G2-rescue:TXB0102DCU -> Logic_LevelTranslator:TXB0102DCU

Commit message: PCB updated to reflect new footprints.
Connections:
- wire segments 109 -> 107
Changed lines of the file:
@@
 L LocalPower:+5V_S #PWR0136
 U 1 1 59CAF048
-P 3200 1400
-F 0 "#PWR0136" H 3200 1250 50  0001 C CNN
-F 1 "+5V_S" V 3215 1528 50  0000 L CNN
-F 2 "" H 3200 1400 50  0001 C CNN
-F 3 "" H 3200 1400 50  0001 C CNN
-	1    3200 1400
+P 3600 1100
+F 0 "#PWR0136" H 3600 950 50  0001 C CNN
+F 1 "+5V_S" V 3615 1228 50  0000 L CNN
+F 2 "" H 3600 1100 50  0001 C CNN
+F 3 "" H 3600 1100 50  0001 C CNN
+	1    3600 1100
 	0    -1   -1   0
 $EndComp
@@
 L LocalPower:+5V_S #PWR0143
 U 1 1 59CB1C65
-P 4450 1400
-F 0 "#PWR0143" H 4450 1250 50  0001 C CNN
-F 1 "+5V_S" V 4450 1650 50  0000 C CNN
-F 2 "" H 4450 1400 50  0001 C CNN
-F 3 "" H 4450 1400 50  0001 C CNN
-	1    4450 1400
+P 4850 1100
+F 0 "#PWR0143" H 4850 950 50  0001 C CNN
+F 1 "+5V_S" V 4850 1350 50  0000 C CNN
+F 2 "" H 4850 1100 50  0001 C CNN
+F 3 "" H 4850 1100 50  0001 C CNN
+	1    4850 1100
 	0    -1   -1   0
 $EndComp
@@
 L LocalPower:+5V_S #PWR0145
 U 1 1 59CB201E
-P 5700 1400
-F 0 "#PWR0145" H 5700 1250 50  0001 C CNN
-F 1 "+5V_S" V 5700 1650 50  0000 C CNN
-F 2 "" H 5700 1400 50  0001 C CNN
-F 3 "" H 5700 1400 50  0001 C CNN
-	1    5700 1400
+P 6100 1100
+F 0 "#PWR0145" H 6100 950 50  0001 C CNN
+F 1 "+5V_S" V 6100 1350 50  0000 C CNN
+F 2 "" H 6100 1100 50  0001 C CNN
+F 3 "" H 6100 1100 50  0001 C CNN
+	1    6100 1100
 	0    -1   -1   0
 $EndComp
@@
 L LocalPower:+5V_S #PWR0146
 U 1 1 59CB208B
-P 6950 1400
-F 0 "#PWR0146" H 6950 1250 50  0001 C CNN
-F 1 "+5V_S" V 6950 1650 50  0000 C CNN
-F 2 "" H 6950 1400 50  0001 C CNN
-F 3 "" H 6950 1400 50  0001 C CNN
-	1    6950 1400
+P 7350 1100
+F 0 "#PWR0146" H 7350 950 50  0001 C CNN
+F 1 "+5V_S" V 7350 1350 50  0000 C CNN
+F 2 "" H 7350 1100 50  0001 C CNN
+F 3 "" H 7350 1100 50  0001 C CNN
+	1    7350 1100
 	0    -1   -1   0
 $EndComp
@@
 L LocalPower:+5V_S #PWR0148
 U 1 1 59CB2413
-P 8200 1400
-F 0 "#PWR0148" H 8200 1250 50  0001 C CNN
-F 1 "+5V_S" V 8200 1650 50  0000 C CNN
-F 2 "" H 8200 1400 50  0001 C CNN
-F 3 "" H 8200 1400 50  0001 C CNN
-	1    8200 1400
+P 8600 1100
+F 0 "#PWR0148" H 8600 950 50  0001 C CNN
+F 1 "+5V_S" V 8600 1350 50  0000 C CNN
+F 2 "" H 8600 1100 50  0001 C CNN
+F 3 "" H 8600 1100 50  0001 C CNN
+	1    8600 1100
 	0    -1   -1   0
 $EndComp
@@
 L LocalPower:GND_S #PWR0150
 U 1 1 59CB26A6
-P 4000 1500
-F 0 "#PWR0150" H 4000 1250 50  0001 C CNN
-F 1 "GND_S" V 4005 1372 50  0000 R CNN
-F 2 "" H 4000 1500 50  0001 C CNN
-F 3 "" H 4000 1500 50  0001 C CNN
-	1    4000 1500
-	0    -1   -1   0
+P 3600 1700
+F 0 "#PWR0150" H 3600 1450 50  0001 C CNN
+F 1 "GND_S" V 3605 1572 50  0000 R CNN
+F 2 "" H 3600 1700 50  0001 C CNN
+F 3 "" H 3600 1700 50  0001 C CNN
+	1    3600 1700
+	1    0    0    -1
 $EndComp
 $Comp
@@
 L LocalPower:GND_S #PWR0152
 U 1 1 59CB2780
-P 5250 1500
-F 0 "#PWR0152" H 5250 1250 50  0001 C CNN
-F 1 "GND_S" V 5255 1372 50  0000 R CNN
-F 2 "" H 5250 1500 50  0001 C CNN
-F 3 "" H 5250 1500 50  0001 C CNN
-	1    5250 1500
-	0    -1   -1   0
+P 4850 1700
+F 0 "#PWR0152" H 4850 1450 50  0001 C CNN
+F 1 "GND_S" V 4855 1572 50  0000 R CNN
+F 2 "" H 4850 1700 50  0001 C CNN
+F 3 "" H 4850 1700 50  0001 C CNN
+	1    4850 1700
+	1    0    0    -1
 $EndComp
 $Comp
@@
 L LocalPower:GND_S #PWR0154
 U 1 1 59CB2B39
-P 6500 1500
-F 0 "#PWR0154" H 6500 1250 50  0001 C CNN
-F 1 "GND_S" V 6505 1372 50  0000 R CNN
-F 2 "" H 6500 1500 50  0001 C CNN
-F 3 "" H 6500 1500 50  0001 C CNN
-	1    6500 1500
-	0    -1   -1   0
+P 6100 1700
+F 0 "#PWR0154" H 6100 1450 50  0001 C CNN
+F 1 "GND_S" V 6105 1572 50  0000 R CNN
+F 2 "" H 6100 1700 50  0001 C CNN
+F 3 "" H 6100 1700 50  0001 C CNN
+	1    6100 1700
+	1    0    0    -1
 $EndComp
 $Comp
@@
 L LocalPower:GND_S #PWR0156
 U 1 1 59CB2C13
-P 7750 1500
-F 0 "#PWR0156" H 7750 1250 50  0001 C CNN
-F 1 "GND_S" V 7755 1372 50  0000 R CNN
-F 2 "" H 7750 1500 50  0001 C CNN
-F 3 "" H 7750 1500 50  0001 C CNN
-	1    7750 1500
-	0    -1   -1   0
+P 7350 1700
+F 0 "#PWR0156" H 7350 1450 50  0001 C CNN
+F 1 "GND_S" V 7355 1572 50  0000 R CNN
+F 2 "" H 7350 1700 50  0001 C CNN
+F 3 "" H 7350 1700 50  0001 C CNN
+	1    7350 1700
+	1    0    0    -1
 $EndComp
 $Comp
@@
 L LocalPower:GND_S #PWR0158
 U 1 1 59CB2CED
-P 9000 1500
-F 0 "#PWR0158" H 9000 1250 50  0001 C CNN
-F 1 "GND_S" V 9005 1372 50  0000 R CNN
-F 2 "" H 9000 1500 50  0001 C CNN
-F 3 "" H 9000 1500 50  0001 C CNN
-	1    9000 1500
-	0    -1   -1   0
+P 8600 1700
+F 0 "#PWR0158" H 8600 1450 50  0001 C CNN
+F 1 "GND_S" V 8605 1572 50  0000 R CNN
+F 2 "" H 8600 1700 50  0001 C CNN
+F 3 "" H 8600 1700 50  0001 C CNN
+	1    8600 1700
+	1    0    0    -1
 $EndComp
 $Comp
@@
 Text Notes 5400 3100 0    60   ~ 0
 To MCU
-NoConn ~ 9000 1400
 $Comp
 L LocalPower:+3V3_S #PWR0160
@@
 $EndComp
 Wire Wire Line
-	4000 1400 4100 1400
-Wire Wire Line
-	4100 1400 4100 1450
-Wire Wire Line
-	4100 1450 4350 1450
-Wire Wire Line
-	4350 1450 4350 1500
-Wire Wire Line
-	4350 1500 4450 1500
-Wire Wire Line
-	5250 1400 5350 1400
-Wire Wire Line
-	5350 1400 5350 1450
-Wire Wire Line
-	5350 1450 5600 1450
-Wire Wire Line
-	5600 1450 5600 1500
-Wire Wire Line
-	5600 1500 5700 1500
-Wire Wire Line
-	6500 1400 6600 1400
-Wire Wire Line
-	6600 1400 6600 1450
-Wire Wire Line
-	6600 1450 6850 1450
-Wire Wire Line
-	6850 1450 6850 1500
-Wire Wire Line
-	6850 1500 6950 1500
-Wire Wire Line
-	7750 1400 7850 1400
-Wire Wire Line
-	7850 1400 7850 1450
-Wire Wire Line
-	7850 1450 8100 1450
-Wire Wire Line
-	8100 1450 8100 1500
-Wire Wire Line
-	8100 1500 8200 1500
-Wire Wire Line
 	3700 4050 3700 4150
 Wire Wire Line
@@
 	1200 6150 1200 7550
 Wire Wire Line
-	3650 7050 1500 7050
+	3650 7050 3350 7050
 Connection ~ 1800 7050
 Connection ~ 2150 7050
@@
 Connection ~ 3350 7050
 Wire Wire Line
-	3700 3750 1350 3750
+	3700 3750 3400 3750
 Connection ~ 1700 3750
 Connection ~ 2050 3750
@@
 Wire Wire Line
 	1550 1700 1650 1700
+Wire Wire Line
+	3200 1500 3300 1500
+Wire Wire Line
+	3300 1500 3300 1400
+Wire Wire Line
+	1800 7050 1500 7050
+Wire Wire Line
+	2150 7050 1800 7050
+Wire Wire Line
+	2450 7050 2150 7050
+Wire Wire Line
+	2750 7050 2450 7050
+Wire Wire Line
+	3050 7050 2750 7050
+Wire Wire Line
+	3350 7050 3050 7050
+Wire Wire Line
+	1700 3750 1350 3750
+Wire Wire Line
+	2050 3750 1700 3750
+Wire Wire Line
+	2400 3750 2050 3750
+Wire Wire Line
+	2750 3750 2400 3750
+Wire Wire Line
+	3100 3750 2750 3750
+Wire Wire Line
+	3400 3750 3100 3750
+Wire Wire Line
+	3900 1400 4550 1400
+Wire Wire Line
+	5150 1400 5800 1400
+Wire Wire Line
+	6400 1400 7050 1400
+Wire Wire Line
+	7650 1400 8300 1400
+NoConn ~ 8900 1400
 $EndSCHEMATC
