File: G2/AnalogSense.sch (KiCad schematic (older format))
At the start: 8 parts

Commit message: Most things connected to MCU
Parts:
- added C? (x9): 100n, Capacitors_SMD:C_0805, symbol C
- added D? (x14): STPS0560Z, Diodes_SMD:D_SOD-123, symbol D_Schottky
- added D? (x7): CDBA3100-HF, Diodes_SMD:D_SMA, symbol D
- added R? (x7): 100, Resistors_SMD:R_0805, symbol R
- added R? (x7): 1k, Resistors_SMD:R_0805, symbol R
- added R? (x7): 2k, symbol R
- added R? (x2): 10k, Resistors_SMD:R_0805, symbol R
- added RV? (x7): B72510E250K62, Capacitors_SMD:C_0805, symbol Varistor
- added U? (x2): ADS1115IDGST, SOP50P490X110-10N, symbol ADS1115IDGST
Connections:
- net +5V: now also D?.1 (K), D?.1 (K), D?.1 (K), D?.1 (K), D?.1 (K), D?.1 (K), D?.1 (K), R?.1, R?.1, R?.1, R?.1, R?.1, R?.1, R?.1
- net GND: now also C?.2, C?.2, C?.2, C?.2, C?.2, C?.2, C?.2, C?.2, C?.2, D?.2 (A), D?.2 (A), D?.2 (A), D?.2 (A), D?.2 (A), D?.2 (A), D?.2 (A), D?.2 (A), D?.2 (A), D?.2 (A), D?.2 (A), D?.2 (A), D?.2 (A), D?.2 (A), RV?.1, RV?.1, RV?.1, RV?.1, RV?.1, RV?.1, RV?.1, U?.1 (ADDR), U?.3 (GND), U?.3 (GND)
- net Sense1: now also U?.4 (AIN0)
- new net: C?.1, D?.1 (K), D?.2 (A), R?.1, R?.2, R?.2 (x7)
- new net +3V3: C?.1, C?.1, R?.1, R?.1, U?.1 (ADDR)
- new net ANALOG_I2C_SCL: U?.10 (SCL), U?.10 (SCL)
- new net ANALOG_I2C_SDA: U?.9 (SDA), U?.9 (SDA)
- new net ANALOG_RDY_1: R?.2, U?.2 (ALERT/RDY)
- new net ANALOG_RDY_2: R?.2, U?.2 (ALERT/RDY)
- new net I2C_PWR: U?.8 (VDD), U?.8 (VDD)
- new net Sense2: R?.2, U?.5 (AIN1)
- new net Sense2_DUT: D?.1 (K), R?.1, RV?.2
- new net Sense3: R?.2, U?.6 (AIN2)
- new net Sense3_DUT: D?.1 (K), R?.1, RV?.2
- new net Sense4: R?.2, U?.7 (AIN3)
- new net Sense4_DUT: D?.1 (K), R?.1, RV?.2
- new net Sense5: R?.2, U?.4 (AIN0)
- new net Sense5_DUT: D?.1 (K), R?.1, RV?.2
- new net Sense6: R?.2, U?.5 (AIN1)
- new net Sense6_DUT: D?.1 (K), R?.1, RV?.2
- new net Sense7: R?.2, U?.6 (AIN2)
- new net Sense7_DUT: D?.1 (K), R?.1, RV?.2
- new net Sense8: R?.2, U?.7 (AIN3)
- new net Sense8_DUT: D?.1 (K), R?.1, RV?.2
Other:
- note added: "I2C address: 0x48"
- note added: "Near ADS1115:1"
- note added: "Near ADS1115:2"
- moved on the sheet: C?, D?, R?, RV?

Commit message: Begun layout.
Parts:
- R507, R508, R509, R510, R511, R512, R521, R522: renamed from R?; footprint (none) -> Resistors_SMD:R_0805
- gave numbers to parts that had none: 62
Connections:
- net +3V3: no longer C509.1, C510.1
- net I2C_PWR: now also C509.1, C510.1
Other:
- note added: "I2C address: 0x49"

Commit message: More layout
Other:
- moved on the sheet: R526
Changed lines of the file:
@@
 L +3.3V #PWR0115
 U 1 1 59C73F9C
-P 6350 3800
-F 0 "#PWR0115" H 6350 3650 50  0001 C CNN
-F 1 "+3.3V" V 6365 3928 50  0000 L CNN
-F 2 "" H 6350 3800 50  0001 C CNN
-F 3 "" H 6350 3800 50  0001 C CNN
-	1    6350 3800
+P 5550 3800
+F 0 "#PWR0115" H 5550 3650 50  0001 C CNN
+F 1 "+3.3V" V 5565 3928 50  0000 L CNN
+F 2 "" H 5550 3800 50  0001 C CNN
+F 3 "" H 5550 3800 50  0001 C CNN
+	1    5550 3800
 	0    -1   -1   0
 $EndComp
@@
 L GND #PWR0109
 U 1 1 59C7135C
-P 6400 2850
-F 0 "#PWR0109" H 6400 2600 50  0001 C CNN
-F 1 "GND" V 6405 2722 50  0000 R CNN
-F 2 "" H 6400 2850 50  0001 C CNN
-F 3 "" H 6400 2850 50  0001 C CNN
-	1    6400 2850
+P 5450 2850
+F 0 "#PWR0109" H 5450 2600 50  0001 C CNN
+F 1 "GND" V 5455 2722 50  0000 R CNN
+F 2 "" H 5450 2850 50  0001 C CNN
+F 3 "" H 5450 2850 50  0001 C CNN
+	1    5450 2850
 	0    1    1    0
 $EndComp
@@
 L GND #PWR0108
 U 1 1 59C70E9B
-P 6350 4800
-F 0 "#PWR0108" H 6350 4550 50  0001 C CNN
-F 1 "GND" V 6355 4672 50  0000 R CNN
-F 2 "" H 6350 4800 50  0001 C CNN
-F 3 "" H 6350 4800 50  0001 C CNN
-	1    6350 4800
+P 5450 4800
+F 0 "#PWR0108" H 5450 4550 50  0001 C CNN
+F 1 "GND" V 5455 4672 50  0000 R CNN
+F 2 "" H 5450 4800 50  0001 C CNN
+F 3 "" H 5450 4800 50  0001 C CNN
+	1    5450 4800
 	0    1    1    0
 $EndComp
@@
 L +3.3V #PWR0106
 U 1 1 59C6D362
-P 5700 3600
-F 0 "#PWR0106" H 5700 3450 50  0001 C CNN
-F 1 "+3.3V" H 5715 3773 50  0000 C CNN
-F 2 "" H 5700 3600 50  0001 C CNN
-F 3 "" H 5700 3600 50  0001 C CNN
-	1    5700 3600
+P 4950 3600
+F 0 "#PWR0106" H 4950 3450 50  0001 C CNN
+F 1 "+3.3V" H 4965 3773 50  0000 C CNN
+F 2 "" H 4950 3600 50  0001 C CNN
+F 3 "" H 4950 3600 50  0001 C CNN
+	1    4950 3600
 	1    0    0    -1
 $EndComp
-Connection ~ 5700 3900
-Wire Wire Line
-	5550 3900 6350 3900
-Text GLabel 5550 3900 0    60   Input ~ 0
+Connection ~ 4950 3900
+Wire Wire Line
+	4800 3900 6350 3900
+Text GLabel 4800 3900 0    60   Input ~ 0
 ANALOG_RDY_2
 $Comp
 L R R526
 U 1 1 59C6CAF7
-P 5700 3750
-F 0 "R526" H 5770 3796 50  0000 L CNN
-F 1 "10k" H 5770 3705 50  0000 L CNN
-F 2 "Resistors_SMD:R_0805" V 5630 3750 50  0001 C CNN
-F 3 "" H 5700 3750 50  0001 C CNN
-	1    5700 3750
+P 4950 3750
+F 0 "R526" H 5020 3796 50  0000 L CNN
+F 1 "10k" H 5020 3705 50  0000 L CNN
+F 2 "Resistors_SMD:R_0805" V 4880 3750 50  0001 C CNN
+F 3 "" H 4950 3750 50  0001 C CNN
+	1    4950 3750
 	1    0    0    -1
 $EndComp
@@
 	0    -1   1    0
 $EndComp
+Text Label 5550 3800 0    60   ~ 0
+3.3V-Rail-regular
+Wire Wire Line
+	5550 3800 6350 3800
+Wire Wire Line
+	6400 2850 5450 2850
+Wire Wire Line
+	6350 4800 5450 4800
+Text Label 5550 4800 0    60   ~ 0
+GND-Regular
+Text Label 5600 2850 0    60   ~ 0
+GND-Regular
 $EndSCHEMATC

Commit message: Updated component name (was missing a digit)
Parts:
- RV501, RV502, RV503, RV505, RV506, RV507, RV508: value B72510E250K62 -> B72510E250K062
Changed lines of the file:
@@
 P 3200 2250
 F 0 "RV508" V 2950 2300 50  0000 C CNN
-F 1 "B72510E250K62" V 3050 2450 50  0000 C CNN
+F 1 "B72510E250K062" V 3050 2450 50  0000 C CNN
 F 2 "Capacitors_SMD:C_0805" V 3130 2250 50  0001 C CNN
 F 3 "http://www.mouser.se/Search/ProductDetail.aspx?R=B72510E250K62virtualkey59250000virtualkey871-B72510E250K62" H 3200 2250 50  0001 C CNN
@@
 P 3200 1100
 F 0 "RV507" V 2950 1150 50  0000 C CNN
-F 1 "B72510E250K62" V 3050 1300 50  0000 C CNN
+F 1 "B72510E250K062" V 3050 1300 50  0000 C CNN
 F 2 "Capacitors_SMD:C_0805" V 3130 1100 50  0001 C CNN
 F 3 "http://www.mouser.se/Search/ProductDetail.aspx?R=B72510E250K62virtualkey59250000virtualkey871-B72510E250K62" H 3200 1100 50  0001 C CNN
@@
 P 1000 6800
 F 0 "RV506" V 750 6850 50  0000 C CNN
-F 1 "B72510E250K62" V 850 7000 50  0000 C CNN
+F 1 "B72510E250K062" V 850 7000 50  0000 C CNN
 F 2 "Capacitors_SMD:C_0805" V 930 6800 50  0001 C CNN
 F 3 "http://www.mouser.se/Search/ProductDetail.aspx?R=B72510E250K62virtualkey59250000virtualkey871-B72510E250K62" H 1000 6800 50  0001 C CNN
@@
 P 1000 5650
 F 0 "RV505" V 750 5700 50  0000 C CNN
-F 1 "B72510E250K62" V 850 5850 50  0000 C CNN
+F 1 "B72510E250K062" V 850 5850 50  0000 C CNN
 F 2 "Capacitors_SMD:C_0805" V 930 5650 50  0001 C CNN
 F 3 "http://www.mouser.se/Search/ProductDetail.aspx?R=B72510E250K62virtualkey59250000virtualkey871-B72510E250K62" H 1000 5650 50  0001 C CNN
@@
 P 1000 3350
 F 0 "RV503" V 750 3400 50  0000 C CNN
-F 1 "B72510E250K62" V 850 3550 50  0000 C CNN
+F 1 "B72510E250K062" V 850 3550 50  0000 C CNN
 F 2 "Capacitors_SMD:C_0805" V 930 3350 50  0001 C CNN
 F 3 "http://www.mouser.se/Search/ProductDetail.aspx?R=B72510E250K62virtualkey59250000virtualkey871-B72510E250K62" H 1000 3350 50  0001 C CNN
@@
 P 1000 2200
 F 0 "RV502" V 750 2250 50  0000 C CNN
-F 1 "B72510E250K62" V 850 2400 50  0000 C CNN
+F 1 "B72510E250K062" V 850 2400 50  0000 C CNN
 F 2 "Capacitors_SMD:C_0805" V 930 2200 50  0001 C CNN
 F 3 "http://www.mouser.se/Search/ProductDetail.aspx?R=B72510E250K62virtualkey59250000virtualkey871-B72510E250K62" H 1000 2200 50  0001 C CNN
@@
 P 1000 1100
 F 0 "RV501" V 750 1150 50  0000 C CNN
-F 1 "B72510E250K62" V 850 1300 50  0000 C CNN
+F 1 "B72510E250K062" V 850 1300 50  0000 C CNN
 F 2 "Capacitors_SMD:C_0805" V 930 1100 50  0001 C CNN
 F 3 "https://www.mouser.se/ProductDetail/EPCOS-TDK/B72510E0250K062/?qs=%2fha2pyFadugVCK9yiqateTD%252bWTZyWxpU55VnsqI3B1Kd%2fbUd9GEicg%3d%3d" H 1000 1100 50  0001 C CNN

Commit message: Removed I2C power control
Connections:
- net I2C_PWR is gone; now on net +3V3: C509.1, C510.1, U501.8 (VDD), U502.8 (VDD)
Changed lines of the file:
@@
 Text Notes 7500 4650 1    60   ~ 0
 I2C address: 0x49
-Text GLabel 8000 2350 1    60   Input ~ 0
-I2C_PWR
-Text GLabel 8000 4300 1    60   Input ~ 0
-I2C_PWR
-Text GLabel 6350 3600 0    60   Input ~ 0
-I2C_PWR
-Text GLabel 6400 1650 0    60   Input ~ 0
-I2C_PWR
 Text GLabel 4350 2250 2    60   Input ~ 0
 Sense8
@@
 Text Label 5600 2850 0    60   ~ 0
 GND-Regular
+$Comp
+L +3.3V #PWR0166
+U 1 1 5A53E0D6
+P 8000 2350
+F 0 "#PWR0166" H 8000 2200 50  0001 C CNN
+F 1 "+3.3V" H 8015 2523 50  0000 C CNN
+F 2 "" H 8000 2350 50  0001 C CNN
+F 3 "" H 8000 2350 50  0001 C CNN
+	1    8000 2350
+	1    0    0    -1
+$EndComp
+$Comp
+L +3.3V #PWR0167
+U 1 1 5A53E39D
+P 8000 4300
+F 0 "#PWR0167" H 8000 4150 50  0001 C CNN
+F 1 "+3.3V" H 8015 4473 50  0000 C CNN
+F 2 "" H 8000 4300 50  0001 C CNN
+F 3 "" H 8000 4300 50  0001 C CNN
+	1    8000 4300
+	1    0    0    -1
+$EndComp
+$Comp
+L +3.3V #PWR0168
+U 1 1 5A53E47A
+P 6350 3600
+F 0 "#PWR0168" H 6350 3450 50  0001 C CNN
+F 1 "+3.3V" H 6365 3773 50  0000 C CNN
+F 2 "" H 6350 3600 50  0001 C CNN
+F 3 "" H 6350 3600 50  0001 C CNN
+	1    6350 3600
+	0    -1   -1   0
+$EndComp
+$Comp
+L +3.3V #PWR0169
+U 1 1 5A53E8E5
+P 6400 1650
+F 0 "#PWR0169" H 6400 1500 50  0001 C CNN
+F 1 "+3.3V" H 6415 1823 50  0000 C CNN
+F 2 "" H 6400 1650 50  0001 C CNN
+F 3 "" H 6400 1650 50  0001 C CNN
+	1    6400 1650
+	0    -1   -1   0
+$EndComp
 $EndSCHEMATC
