File: G2/AnalogSense.sch (KiCad schematic (older format))
At the start: 70 parts, among them U501 ADS1115IDGST, U502 ADS1115IDGST

Commit message: Step two of conversion to v5 format
Parts:
- C501, C502, C503, C504, C505, C506, C507, C508, C509, C510: symbol G2-rescue:C -> Device:C
- D501, D502, D503, D504, D505, D506, D519, D520: symbol G2-rescue:D -> Device:D
- D507, D508, D509, D510, D511, D512, D513, D514, D515, D516, D517, D518, D521, D522, D523, D524: symbol G2-rescue:D_Schottky -> Device:D_Schottky
- R501, R502, R503, R504, R505, R506, R507, R508, R509, R510, R511, R512, R513, R514, R515, R516, R517, R518, R519, R520, R521, R522, R523, R524, R525, R526: symbol G2-rescue:R -> Device:R
- RV501, RV502, RV503, RV504, RV505, RV506, RV507, RV508: symbol G2-rescue:Varistor -> Device:Varistor
