File: G3/Connectors.sch (KiCad schematic (older format))
At the start: 32 parts, among them J3101 Conn_01x09, J3102 Conn_01x09, J3103 Conn_01x09, J3104 Conn_01x09, J3105 Conn_01x09, J3106 GS3, J3107 GS3, J3108 GS3, J3109 GS3, J3110 GS3, J3111 GS3, J3112 GS3, J3113 GS3, J3114 Conn_01x09, J3115 Conn_01x09

Commit message: Touch up
Parts:
- renumbered F3101 to F3501, F3102 to F3502, F3103 to F3503, F3104 to F3504, F3105 to F3505, F3106 to F3506, F3107 to F3507, F3108 to F3508, F3109 to F3509, F3110 to F3510, F3111 to F3511, F3112 to F3512, F3113 to F3513, F3114 to F3514, F3115 to F3515, F3116 to F3516, F3117 to F3517, J3101 to J3501, J3102 to J3502, J3103 to J3503, J3104 to J3504, J3105 to J3505, J3106 to J3506, J3107 to J3507, J3108 to J3508, J3109 to J3509, J3110 to J3510, J3111 to J3511, J3112 to J3512, J3113 to J3513, J3114 to J3514, J3115 to J3515
