File: G3/Connectors.sch (KiCad schematic (older format))
At the start: 32 parts, among them J3501 Conn_01x09, J3502 Conn_01x09, J3503 Conn_01x09, J3504 Conn_01x09, J3505 Conn_01x09, J3506 GS3, J3507 GS3, J3508 GS3, J3509 GS3, J3510 GS3, J3511 GS3, J3512 GS3, J3513 GS3, J3514 Conn_01x09, J3515 Conn_01x09

Commit message: Added SDCard slot.
Parts:
- renumbered F3501 to F3601, F3502 to F3602, F3503 to F3603, F3504 to F3604, F3505 to F3605, F3506 to F3606, F3507 to F3607, F3508 to F3608, F3509 to F3609, F3510 to F3610, F3511 to F3611, F3512 to F3612, F3513 to F3613, F3514 to F3614, F3515 to F3615, F3516 to F3616, F3517 to F3617, J3501 to J3601, J3502 to J3602, J3503 to J3603, J3504 to J3604, J3505 to J3605, J3506 to J3606, J3507 to J3607, J3508 to J3608, J3509 to J3609, J3510 to J3610, J3511 to J3611, J3512 to J3612, J3513 to J3613, J3514 to J3614, J3515 to J3615

Commit message: Using MAX4948 instead of DIPs
Parts:
- J3606: value GS3 -> DO1_PWR
- J3607: value GS3 -> DO2_PWR
- J3608: value GS3 -> DO3_PWR
- J3609: value GS3 -> DO4_PWR
- J3610: value GS3 -> DO5_PWR
- J3611: value GS3 -> DO6_PWR
- J3612: value GS3 -> DO7_PWR
- J3613: value GS3 -> DO8_PWR
Connections:
- wire segments 47 -> 48
Changed lines of the file:
@@
 $Descr A4 11693 8268
 encoding utf-8
-Sheet 35 36
+Sheet 36 36
 Title ""
 Date ""
@@
 Text GLabel 7800 3900 0    50   Input ~ 0
 DO6_GND_BREAK
-Text GLabel 7800 4100 0    50   Input ~ 0
-DO7_GND_BREAK
-Text GLabel 7800 4300 0    50   Input ~ 0
-DO8_GND_BREAK
 Text GLabel 1600 4500 0    50   Input ~ 0
 SIREN_GND_BREAK
@@
 AR Path="/5B72552B/5B7CD677" Ref="J3606"  Part="1"
 F 0 "J3606" H 6100 725 50  0000 C CNN
-F 1 "GS3" H 6100 816 50  0000 C CNN
+F 1 "DO1_PWR" H 6100 816 50  0000 C CNN
 F 2 "Connector_PinHeader_2.54mm:PinHeader_1x03_P2.54mm_Vertical" V 6188 976 50  0001 C CNN
 F 3 "" H 6100 1050 50  0001 C CNN
@@
 AR Path="/5B72552B/5B755D38" Ref="J3607"  Part="1"
 F 0 "J3607" H 6100 1275 50  0000 C CNN
-F 1 "GS3" H 6100 1366 50  0000 C CNN
+F 1 "DO2_PWR" H 6100 1366 50  0000 C CNN
 F 2 "Connector_PinHeader_2.54mm:PinHeader_1x03_P2.54mm_Vertical" V 6188 1526 50  0001 C CNN
 F 3 "" H 6100 1600 50  0001 C CNN
@@
 AR Path="/5B72552B/5B755D91" Ref="J3608"  Part="1"
 F 0 "J3608" H 6100 1825 50  0000 C CNN
-F 1 "GS3" H 6100 1916 50  0000 C CNN
+F 1 "DO3_PWR" H 6100 1916 50  0000 C CNN
 F 2 "Connector_PinHeader_2.54mm:PinHeader_1x03_P2.54mm_Vertical" V 6188 2076 50  0001 C CNN
 F 3 "" H 6100 2150 50  0001 C CNN
@@
 AR Path="/5B72552B/5B755DDE" Ref="J3609"  Part="1"
 F 0 "J3609" H 6100 2375 50  0000 C CNN
-F 1 "GS3" H 6100 2466 50  0000 C CNN
+F 1 "DO4_PWR" H 6100 2466 50  0000 C CNN
 F 2 "Connector_PinHeader_2.54mm:PinHeader_1x03_P2.54mm_Vertical" V 6188 2626 50  0001 C CNN
 F 3 "" H 6100 2700 50  0001 C CNN
@@
 AR Path="/5B72552B/5B755FA6" Ref="J3610"  Part="1"
 F 0 "J3610" H 6100 2925 50  0000 C CNN
-F 1 "GS3" H 6100 3016 50  0000 C CNN
+F 1 "DO5_PWR" H 6100 3016 50  0000 C CNN
 F 2 "Connector_PinHeader_2.54mm:PinHeader_1x03_P2.54mm_Vertical" V 6188 3176 50  0001 C CNN
 F 3 "" H 6100 3250 50  0001 C CNN
@@
 AR Path="/5B72552B/5B756008" Ref="J3611"  Part="1"
 F 0 "J3611" H 6100 3475 50  0000 C CNN
-F 1 "GS3" H 6100 3566 50  0000 C CNN
+F 1 "DO6_PWR" H 6100 3566 50  0000 C CNN
 F 2 "Connector_PinHeader_2.54mm:PinHeader_1x03_P2.54mm_Vertical" V 6188 3726 50  0001 C CNN
 F 3 "" H 6100 3800 50  0001 C CNN
@@
 	6550 3800 6300 3800
 $Comp
-L Connector_Generic:Conn_01x03 J?
-U 1 1 5B7561A3
-P 6100 4350
-AR Path="/5B62EDB8/5B7561A3" Ref="J?"  Part="1"
-AR Path="/5B72552B/5B7561A3" Ref="J3612"  Part="1"
-F 0 "J3612" H 6100 4025 50  0000 C CNN
-F 1 "GS3" H 6100 4116 50  0000 C CNN
-F 2 "Connector_PinHeader_2.54mm:PinHeader_1x03_P2.54mm_Vertical" V 6188 4276 50  0001 C CNN
-F 3 "" H 6100 4350 50  0001 C CNN
-	1    6100 4350
-	-1   0    0    1
-$EndComp
-$Comp
-L power:+5V #PWR?
-U 1 1 5B7561AA
-P 6300 4250
-AR Path="/5B62EDB8/5B7561AA" Ref="#PWR?"  Part="1"
-AR Path="/5B72552B/5B7561AA" Ref="#PWR03623"  Part="1"
-F 0 "#PWR03623" H 6300 4100 50  0001 C CNN
-F 1 "+5V" V 6315 4378 50  0000 L CNN
-F 2 "" H 6300 4250 50  0001 C CNN
-F 3 "" H 6300 4250 50  0001 C CNN
-	1    6300 4250
-	0    1    1    0
-$EndComp
-Text GLabel 6300 4450 2    50   Input ~ 0
-12V_PWR
-$Comp
-L Device:Fuse F?
-U 1 1 5B7561B1
-P 6700 4350
-AR Path="/5B61ECB9/5B7561B1" Ref="F?"  Part="1"
-AR Path="/5B72552B/5B7561B1" Ref="F3616"  Part="1"
-F 0 "F3616" V 6503 4350 50  0000 C CNN
-F 1 "xA" V 6594 4350 50  0000 C CNN
-F 2 "Fuse:Fuseholder_Cylinder-5x20mm_Schurter_0031_8201_Horizontal_Open" V 6630 4350 50  0001 C CNN
-F 3 "https://www.mouser.se/ProductDetail/Schurter/00318201?qs=sGAEpiMZZMtRmoYvq3OwzLrTj1%252b%252bxBWBiZ2DdJg9oKI%3d" H 6700 4350 50  0001 C CNN
-	1    6700 4350
-	0    1    1    0
-$EndComp
-Wire Wire Line
-	6550 4350 6300 4350
-$Comp
-L Connector_Generic:Conn_01x03 J?
-U 1 1 5B75622A
-P 6100 4900
-AR Path="/5B62EDB8/5B75622A" Ref="J?"  Part="1"
-AR Path="/5B72552B/5B75622A" Ref="J3613"  Part="1"
-F 0 "J3613" H 6100 4575 50  0000 C CNN
-F 1 "GS3" H 6100 4666 50  0000 C CNN
-F 2 "Connector_PinHeader_2.54mm:PinHeader_1x03_P2.54mm_Vertical" V 6188 4826 50  0001 C CNN
-F 3 "" H 6100 4900 50  0001 C CNN
-	1    6100 4900
-	-1   0    0    1
-$EndComp
-$Comp
-L power:+5V #PWR?
-U 1 1 5B756231
-P 6300 4800
-AR Path="/5B62EDB8/5B756231" Ref="#PWR?"  Part="1"
-AR Path="/5B72552B/5B756231" Ref="#PWR03624"  Part="1"
-F 0 "#PWR03624" H 6300 4650 50  0001 C CNN
-F 1 "+5V" V 6315 4928 50  0000 L CNN
-F 2 "" H 6300 4800 50  0001 C CNN
-F 3 "" H 6300 4800 50  0001 C CNN
-	1    6300 4800
-	0    1    1    0
-$EndComp
-Text GLabel 6300 5000 2    50   Input ~ 0
-12V_PWR
-$Comp
-L Device:Fuse F?
-U 1 1 5B756238
-P 6700 4900
-AR Path="/5B61ECB9/5B756238" Ref="F?"  Part="1"
-AR Path="/5B72552B/5B756238" Ref="F3617"  Part="1"
-F 0 "F3617" V 6503 4900 50  0000 C CNN
-F 1 "xA" V 6594 4900 50  0000 C CNN
-F 2 "Fuse:Fuseholder_Cylinder-5x20mm_Schurter_0031_8201_Horizontal_Open" V 6630 4900 50  0001 C CNN
-F 3 "https://www.mouser.se/ProductDetail/Schurter/00318201?qs=sGAEpiMZZMtRmoYvq3OwzLrTj1%252b%252bxBWBiZ2DdJg9oKI%3d" H 6700 4900 50  0001 C CNN
-	1    6700 4900
-	0    1    1    0
-$EndComp
-Wire Wire Line
-	6550 4900 6300 4900
-$Comp
 L Device:Fuse F?
 U 1 1 5B75939B
@@
 Wire Wire Line
 	7800 3800 6850 3800
-Wire Wire Line
-	6850 4350 6850 4000
-Wire Wire Line
-	6850 4000 7800 4000
-Wire Wire Line
-	7800 4200 7000 4200
-Wire Wire Line
-	7000 4200 7000 4900
-Wire Wire Line
-	7000 4900 6850 4900
+Text GLabel 7800 4100 0    50   Input ~ 0
+DO7_GND_BREAK
+Text GLabel 7800 4300 0    50   Input ~ 0
+DO8_GND_BREAK
+$Comp
+L Connector_Generic:Conn_01x03 J?
+U 1 1 5BA24D87
+P 6100 4350
+AR Path="/5B62EDB8/5BA24D87" Ref="J?"  Part="1"
+AR Path="/5B72552B/5BA24D87" Ref="J3612"  Part="1"
+F 0 "J3612" H 6100 4025 50  0000 C CNN
+F 1 "DO7_PWR" H 6100 4116 50  0000 C CNN
+F 2 "Connector_PinHeader_2.54mm:PinHeader_1x03_P2.54mm_Vertical" V 6188 4276 50  0001 C CNN
+F 3 "" H 6100 4350 50  0001 C CNN
+	1    6100 4350
+	-1   0    0    1
+$EndComp
+$Comp
+L power:+5V #PWR?
+U 1 1 5BA24D8E
+P 6300 4250
+AR Path="/5B62EDB8/5BA24D8E" Ref="#PWR?"  Part="1"
+AR Path="/5B72552B/5BA24D8E" Ref="#PWR03623"  Part="1"
+F 0 "#PWR03623" H 6300 4100 50  0001 C CNN
+F 1 "+5V" V 6315 4378 50  0000 L CNN
+F 2 "" H 6300 4250 50  0001 C CNN
+F 3 "" H 6300 4250 50  0001 C CNN
+	1    6300 4250
+	0    1    1    0
+$EndComp
+Text GLabel 6300 4450 2    50   Input ~ 0
+12V_PWR
+$Comp
+L Device:Fuse F?
+U 1 1 5BA24D95
+P 6700 4350
+AR Path="/5B61ECB9/5BA24D95" Ref="F?"  Part="1"
+AR Path="/5B72552B/5BA24D95" Ref="F3616"  Part="1"
+F 0 "F3616" V 6503 4350 50  0000 C CNN
+F 1 "xA" V 6594 4350 50  0000 C CNN
+F 2 "Fuse:Fuseholder_Cylinder-5x20mm_Schurter_0031_8201_Horizontal_Open" V 6630 4350 50  0001 C CNN
+F 3 "https://www.mouser.se/ProductDetail/Schurter/00318201?qs=sGAEpiMZZMtRmoYvq3OwzLrTj1%252b%252bxBWBiZ2DdJg9oKI%3d" H 6700 4350 50  0001 C CNN
+	1    6700 4350
+	0    1    1    0
+$EndComp
+Wire Wire Line
+	6550 4350 6300 4350
+$Comp
+L Connector_Generic:Conn_01x03 J?
+U 1 1 5BA25430
+P 6100 4900
+AR Path="/5B62EDB8/5BA25430" Ref="J?"  Part="1"
+AR Path="/5B72552B/5BA25430" Ref="J3613"  Part="1"
+F 0 "J3613" H 6100 4575 50  0000 C CNN
+F 1 "DO8_PWR" H 6100 4666 50  0000 C CNN
+F 2 "Connector_PinHeader_2.54mm:PinHeader_1x03_P2.54mm_Vertical" V 6188 4826 50  0001 C CNN
+F 3 "" H 6100 4900 50  0001 C CNN
+	1    6100 4900
+	-1   0    0    1
+$EndComp
+$Comp
+L power:+5V #PWR?
+U 1 1 5BA25437
+P 6300 4800
+AR Path="/5B62EDB8/5BA25437" Ref="#PWR?"  Part="1"
+AR Path="/5B72552B/5BA25437" Ref="#PWR03624"  Part="1"
+F 0 "#PWR03624" H 6300 4650 50  0001 C CNN
+F 1 "+5V" V 6315 4928 50  0000 L CNN
+F 2 "" H 6300 4800 50  0001 C CNN
+F 3 "" H 6300 4800 50  0001 C CNN
+	1    6300 4800
+	0    1    1    0
+$EndComp
+Text GLabel 6300 5000 2    50   Input ~ 0
+12V_PWR
+$Comp
+L Device:Fuse F?
+U 1 1 5BA2543E
+P 6700 4900
+AR Path="/5B61ECB9/5BA2543E" Ref="F?"  Part="1"
+AR Path="/5B72552B/5BA2543E" Ref="F3617"  Part="1"
+F 0 "F3617" V 6503 4900 50  0000 C CNN
+F 1 "xA" V 6594 4900 50  0000 C CNN
+F 2 "Fuse:Fuseholder_Cylinder-5x20mm_Schurter_0031_8201_Horizontal_Open" V 6630 4900 50  0001 C CNN
+F 3 "https://www.mouser.se/ProductDetail/Schurter/00318201?qs=sGAEpiMZZMtRmoYvq3OwzLrTj1%252b%252bxBWBiZ2DdJg9oKI%3d" H 6700 4900 50  0001 C CNN
+	1    6700 4900
+	0    1    1    0
+$EndComp
+Wire Wire Line
+	6550 4900 6300 4900
+Wire Wire Line
+	6850 4350 6900 4350
+Wire Wire Line
+	6900 4350 6900 4000
+Wire Wire Line
+	6900 4000 7800 4000
+Wire Wire Line
+	6850 4900 7000 4900
+Wire Wire Line
+	7000 4900 7000 4200
+Wire Wire Line
+	7000 4200 7800 4200
 $EndSCHEMATC

Commit message: Use smaller TR5 fuse holders
Parts:
- F3601, F3602, F3603, F3604, F3605, F3606, F3607, F3608, F3609, F3610, F3611, F3612, F3613, F3614, F3615, F3616, F3617: footprint Fuse:Fuseholder_Cylinder-5x20mm_Schurter_0031_8201_Horizontal_Open -> Fuse:Fuseholder_TR5_Littlefuse_No560_No460
Changed lines of the file:
@@
 F 0 "F3610" V 6503 1050 50  0000 C CNN
 F 1 "xA" V 6594 1050 50  0000 C CNN
-F 2 "Fuse:Fuseholder_Cylinder-5x20mm_Schurter_0031_8201_Horizontal_Open" V 6630 1050 50  0001 C CNN
+F 2 "Fuse:Fuseholder_TR5_Littlefuse_No560_No460" V 6630 1050 50  0001 C CNN
 F 3 "https://www.mouser.se/ProductDetail/Schurter/00318201?qs=sGAEpiMZZMtRmoYvq3OwzLrTj1%252b%252bxBWBiZ2DdJg9oKI%3d" H 6700 1050 50  0001 C CNN
 	1    6700 1050
@@
 F 0 "F3611" V 6503 1600 50  0000 C CNN
 F 1 "xA" V 6594 1600 50  0000 C CNN
-F 2 "Fuse:Fuseholder_Cylinder-5x20mm_Schurter_0031_8201_Horizontal_Open" V 6630 1600 50  0001 C CNN
+F 2 "Fuse:Fuseholder_TR5_Littlefuse_No560_No460" V 6630 1600 50  0001 C CNN
 F 3 "https://www.mouser.se/ProductDetail/Schurter/00318201?qs=sGAEpiMZZMtRmoYvq3OwzLrTj1%252b%252bxBWBiZ2DdJg9oKI%3d" H 6700 1600 50  0001 C CNN
 	1    6700 1600
@@
 F 0 "F3612" V 6503 2150 50  0000 C CNN
 F 1 "xA" V 6594 2150 50  0000 C CNN
-F 2 "Fuse:Fuseholder_Cylinder-5x20mm_Schurter_0031_8201_Horizontal_Open" V 6630 2150 50  0001 C CNN
+F 2 "Fuse:Fuseholder_TR5_Littlefuse_No560_No460" V 6630 2150 50  0001 C CNN
 F 3 "https://www.mouser.se/ProductDetail/Schurter/00318201?qs=sGAEpiMZZMtRmoYvq3OwzLrTj1%252b%252bxBWBiZ2DdJg9oKI%3d" H 6700 2150 50  0001 C CNN
 	1    6700 2150
@@
 F 0 "F3613" V 6503 2700 50  0000 C CNN
 F 1 "xA" V 6594 2700 50  0000 C CNN
-F 2 "Fuse:Fuseholder_Cylinder-5x20mm_Schurter_0031_8201_Horizontal_Open" V 6630 2700 50  0001 C CNN
+F 2 "Fuse:Fuseholder_TR5_Littlefuse_No560_No460" V 6630 2700 50  0001 C CNN
 F 3 "https://www.mouser.se/ProductDetail/Schurter/00318201?qs=sGAEpiMZZMtRmoYvq3OwzLrTj1%252b%252bxBWBiZ2DdJg9oKI%3d" H 6700 2700 50  0001 C CNN
 	1    6700 2700
@@
 F 0 "F3614" V 6503 3250 50  0000 C CNN
 F 1 "xA" V 6594 3250 50  0000 C CNN
-F 2 "Fuse:Fuseholder_Cylinder-5x20mm_Schurter_0031_8201_Horizontal_Open" V 6630 3250 50  0001 C CNN
+F 2 "Fuse:Fuseholder_TR5_Littlefuse_No560_No460" V 6630 3250 50  0001 C CNN
 F 3 "https://www.mouser.se/ProductDetail/Schurter/00318201?qs=sGAEpiMZZMtRmoYvq3OwzLrTj1%252b%252bxBWBiZ2DdJg9oKI%3d" H 6700 3250 50  0001 C CNN
 	1    6700 3250
@@
 F 0 "F3615" V 6503 3800 50  0000 C CNN
 F 1 "xA" V 6594 3800 50  0000 C CNN
-F 2 "Fuse:Fuseholder_Cylinder-5x20mm_Schurter_0031_8201_Horizontal_Open" V 6630 3800 50  0001 C CNN
+F 2 "Fuse:Fuseholder_TR5_Littlefuse_No560_No460" V 6630 3800 50  0001 C CNN
 F 3 "https://www.mouser.se/ProductDetail/Schurter/00318201?qs=sGAEpiMZZMtRmoYvq3OwzLrTj1%252b%252bxBWBiZ2DdJg9oKI%3d" H 6700 3800 50  0001 C CNN
 	1    6700 3800
@@
 F 0 "F3604" V 3503 2100 50  0000 C CNN
 F 1 "xA" V 3594 2100 50  0000 C CNN
-F 2 "Fuse:Fuseholder_Cylinder-5x20mm_Schurter_0031_8201_Horizontal_Open" V 3630 2100 50  0001 C CNN
+F 2 "Fuse:Fuseholder_TR5_Littlefuse_No560_No460" V 3630 2100 50  0001 C CNN
 F 3 "https://www.mouser.se/ProductDetail/Schurter/00318201?qs=sGAEpiMZZMtRmoYvq3OwzLrTj1%252b%252bxBWBiZ2DdJg9oKI%3d" H 3700 2100 50  0001 C CNN
 	1    3700 2100
@@
 F 0 "F3605" V 3803 2100 50  0000 C CNN
 F 1 "xA" V 3894 2100 50  0000 C CNN
-F 2 "Fuse:Fuseholder_Cylinder-5x20mm_Schurter_0031_8201_Horizontal_Open" V 3930 2100 50  0001 C CNN
+F 2 "Fuse:Fuseholder_TR5_Littlefuse_No560_No460" V 3930 2100 50  0001 C CNN
 F 3 "https://www.mouser.se/ProductDetail/Schurter/00318201?qs=sGAEpiMZZMtRmoYvq3OwzLrTj1%252b%252bxBWBiZ2DdJg9oKI%3d" H 4000 2100 50  0001 C CNN
 	1    4000 2100
@@
 F 0 "F3606" V 4103 2100 50  0000 C CNN
 F 1 "xA" V 4194 2100 50  0000 C CNN
-F 2 "Fuse:Fuseholder_Cylinder-5x20mm_Schurter_0031_8201_Horizontal_Open" V 4230 2100 50  0001 C CNN
+F 2 "Fuse:Fuseholder_TR5_Littlefuse_No560_No460" V 4230 2100 50  0001 C CNN
 F 3 "https://www.mouser.se/ProductDetail/Schurter/00318201?qs=sGAEpiMZZMtRmoYvq3OwzLrTj1%252b%252bxBWBiZ2DdJg9oKI%3d" H 4300 2100 50  0001 C CNN
 	1    4300 2100
@@
 F 0 "F3607" V 4403 2100 50  0000 C CNN
 F 1 "xA" V 4494 2100 50  0000 C CNN
-F 2 "Fuse:Fuseholder_Cylinder-5x20mm_Schurter_0031_8201_Horizontal_Open" V 4530 2100 50  0001 C CNN
+F 2 "Fuse:Fuseholder_TR5_Littlefuse_No560_No460" V 4530 2100 50  0001 C CNN
 F 3 "https://www.mouser.se/ProductDetail/Schurter/00318201?qs=sGAEpiMZZMtRmoYvq3OwzLrTj1%252b%252bxBWBiZ2DdJg9oKI%3d" H 4600 2100 50  0001 C CNN
 	1    4600 2100
@@
 F 0 "F3608" V 4703 2100 50  0000 C CNN
 F 1 "xA" V 4794 2100 50  0000 C CNN
-F 2 "Fuse:Fuseholder_Cylinder-5x20mm_Schurter_0031_8201_Horizontal_Open" V 4830 2100 50  0001 C CNN
+F 2 "Fuse:Fuseholder_TR5_Littlefuse_No560_No460" V 4830 2100 50  0001 C CNN
 F 3 "https://www.mouser.se/ProductDetail/Schurter/00318201?qs=sGAEpiMZZMtRmoYvq3OwzLrTj1%252b%252bxBWBiZ2DdJg9oKI%3d" H 4900 2100 50  0001 C CNN
 	1    4900 2100
@@
 F 0 "F3609" V 5003 2100 50  0000 C CNN
 F 1 "xA" V 5094 2100 50  0000 C CNN
-F 2 "Fuse:Fuseholder_Cylinder-5x20mm_Schurter_0031_8201_Horizontal_Open" V 5130 2100 50  0001 C CNN
+F 2 "Fuse:Fuseholder_TR5_Littlefuse_No560_No460" V 5130 2100 50  0001 C CNN
 F 3 "https://www.mouser.se/ProductDetail/Schurter/00318201?qs=sGAEpiMZZMtRmoYvq3OwzLrTj1%252b%252bxBWBiZ2DdJg9oKI%3d" H 5200 2100 50  0001 C CNN
 	1    5200 2100
@@
 F 0 "F3603" V 3203 2100 50  0000 C CNN
 F 1 "xA" V 3294 2100 50  0000 C CNN
-F 2 "Fuse:Fuseholder_Cylinder-5x20mm_Schurter_0031_8201_Horizontal_Open" V 3330 2100 50  0001 C CNN
+F 2 "Fuse:Fuseholder_TR5_Littlefuse_No560_No460" V 3330 2100 50  0001 C CNN
 F 3 "https://www.mouser.se/ProductDetail/Schurter/00318201?qs=sGAEpiMZZMtRmoYvq3OwzLrTj1%252b%252bxBWBiZ2DdJg9oKI%3d" H 3400 2100 50  0001 C CNN
 	1    3400 2100
@@
 F 0 "F3602" V 2903 2100 50  0000 C CNN
 F 1 "xA" V 2994 2100 50  0000 C CNN
-F 2 "Fuse:Fuseholder_Cylinder-5x20mm_Schurter_0031_8201_Horizontal_Open" V 3030 2100 50  0001 C CNN
+F 2 "Fuse:Fuseholder_TR5_Littlefuse_No560_No460" V 3030 2100 50  0001 C CNN
 F 3 "https://www.mouser.se/ProductDetail/Schurter/00318201?qs=sGAEpiMZZMtRmoYvq3OwzLrTj1%252b%252bxBWBiZ2DdJg9oKI%3d" H 3100 2100 50  0001 C CNN
 	1    3100 2100
@@
 F 0 "F3601" V 2603 2100 50  0000 C CNN
 F 1 "xA" V 2694 2100 50  0000 C CNN
-F 2 "Fuse:Fuseholder_Cylinder-5x20mm_Schurter_0031_8201_Horizontal_Open" V 2730 2100 50  0001 C CNN
+F 2 "Fuse:Fuseholder_TR5_Littlefuse_No560_No460" V 2730 2100 50  0001 C CNN
 F 3 "https://www.mouser.se/ProductDetail/Schurter/00318201?qs=sGAEpiMZZMtRmoYvq3OwzLrTj1%252b%252bxBWBiZ2DdJg9oKI%3d" H 2800 2100 50  0001 C CNN
 	1    2800 2100
@@
 F 0 "F3616" V 6503 4350 50  0000 C CNN
 F 1 "xA" V 6594 4350 50  0000 C CNN
-F 2 "Fuse:Fuseholder_Cylinder-5x20mm_Schurter_0031_8201_Horizontal_Open" V 6630 4350 50  0001 C CNN
+F 2 "Fuse:Fuseholder_TR5_Littlefuse_No560_No460" V 6630 4350 50  0001 C CNN
 F 3 "https://www.mouser.se/ProductDetail/Schurter/00318201?qs=sGAEpiMZZMtRmoYvq3OwzLrTj1%252b%252bxBWBiZ2DdJg9oKI%3d" H 6700 4350 50  0001 C CNN
 	1    6700 4350
@@
 F 0 "F3617" V 6503 4900 50  0000 C CNN
 F 1 "xA" V 6594 4900 50  0000 C CNN
-F 2 "Fuse:Fuseholder_Cylinder-5x20mm_Schurter_0031_8201_Horizontal_Open" V 6630 4900 50  0001 C CNN
+F 2 "Fuse:Fuseholder_TR5_Littlefuse_No560_No460" V 6630 4900 50  0001 C CNN
 F 3 "https://www.mouser.se/ProductDetail/Schurter/00318201?qs=sGAEpiMZZMtRmoYvq3OwzLrTj1%252b%252bxBWBiZ2DdJg9oKI%3d" H 6700 4900 50  0001 C CNN
 	1    6700 4900

Commit message: Changes to input and outputs
Parts:
- removed F3603, F3606, F3609, F3610, F3611, F3612, F3613, F3614, F3615, F3616, F3617: xA, Fuse:Fuseholder_TR5_Littlefuse_No560_No460, symbol Device:Fuse
- removed J3606: DO1_PWR, Connector_PinHeader_2.54mm:PinHeader_1x03_P2.54mm_Vertical, symbol Connector_Generic:Conn_01x03
- removed J3607: DO2_PWR, Connector_PinHeader_2.54mm:PinHeader_1x03_P2.54mm_Vertical, symbol Connector_Generic:Conn_01x03
- removed J3608: DO3_PWR, Connector_PinHeader_2.54mm:PinHeader_1x03_P2.54mm_Vertical, symbol Connector_Generic:Conn_01x03
- removed J3609: DO4_PWR, Connector_PinHeader_2.54mm:PinHeader_1x03_P2.54mm_Vertical, symbol Connector_Generic:Conn_01x03
- removed J3610: DO5_PWR, Connector_PinHeader_2.54mm:PinHeader_1x03_P2.54mm_Vertical, symbol Connector_Generic:Conn_01x03
- removed J3611: DO6_PWR, Connector_PinHeader_2.54mm:PinHeader_1x03_P2.54mm_Vertical, symbol Connector_Generic:Conn_01x03
- removed J3612: DO7_PWR, Connector_PinHeader_2.54mm:PinHeader_1x03_P2.54mm_Vertical, symbol Connector_Generic:Conn_01x03
- removed J3613: DO8_PWR, Connector_PinHeader_2.54mm:PinHeader_1x03_P2.54mm_Vertical, symbol Connector_Generic:Conn_01x03
- added J3506: Digital input, PerMalmberg:MOLEX_1x9_39544-3009, symbol Connector_Generic:Conn_01x09
- added J3509: Digital output, PerMalmberg:MOLEX_1x9_39544-3009, symbol Connector_Generic:Conn_01x09
- J3501: renamed from J3601; value Conn_01x09 -> Sense
- J3502: renamed from J3603; value Conn_01x09 -> Digital Input
- J3503: renamed from J3602; value Conn_01x09 -> Sense
- J3504: renamed from J3604; value Conn_01x09 -> Digital input
- J3505: renamed from J3605; value Conn_01x09 -> Power 12/5/3
- J3507: renamed from J3614; value Conn_01x09 -> Digital Output
- J3508: renamed from J3615; value Conn_01x09 -> Digital output
- renumbered F3601 to F3501, F3602 to F3502, F3604 to F3503, F3605 to F3504, F3607 to F3505, F3608 to F3506
Connections:
- net labels added: BELL_PWR, DI1_PWR, DI2_PWR, DI3_PWR, DI4_PWR, DI5_PWR, DI6_PWR, DI7_PWR, DI8_PWR, DO1_PWR, DO2_PWR, DO3_PWR, DO4_PWR, DO5_PWR, DO6_PWR, DO7_PWR, DO8_PWR, SIREN_PWR
- net labels removed: +12V, BELL_GND_BREAK, DO1_GND_BREAK, DO2_GND_BREAK, DO3_GND_BREAK, DO4_GND_BREAK, DO5_GND_BREAK, DO6_GND_BREAK, DO7_GND_BREAK, DO8_GND_BREAK, SIREN_GND_BREAK
- wire segments 48 -> 14
- no-connect marks 0 -> 2
Other:
- note added: "Analog sensors sense voltage level based on\n resistance between SenseN_DUT and GND"

Commit message: Changed special power supply connector to free contacts at regular connector. Moved power LEDs.
Connections:
- net labels added: POWER_SUPPLY_12V
- wire segments 14 -> 17
Changed lines of the file:
@@
 $Descr A4 11693 8268
 encoding utf-8
-Sheet 35 34
+Sheet 34 34
 Title ""
 Date ""
@@
 $EndComp
 $Comp
-L power:GND #PWR03510
-U 1 1 5BA116DF
-P 3950 1600
-F 0 "#PWR03510" H 3950 1350 50  0001 C CNN
-F 1 "GND" H 3955 1427 50  0000 C CNN
-F 2 "" H 3950 1600 50  0001 C CNN
-F 3 "" H 3950 1600 50  0001 C CNN
-	1    3950 1600
-	1    0    0    -1
-$EndComp
-$Comp
 L power:GND #PWR03512
 U 1 1 5BA11728
@@
 	1    0    0    -1
 $EndComp
+Text GLabel 3600 1550 1    50   Input ~ 0
+POWER_SUPPLY_12V
+Wire Wire Line
+	3600 1550 3600 1850
+Wire Wire Line
+	3600 1850 3950 1850
+Wire Wire Line
+	3950 1850 3950 1600
 $EndSCHEMATC
