File: G3/DigitalOutput.sch (KiCad schematic (older format))
At the start: 2 parts, among them Q2201 ZXTN25050DFHTA

Commit message: More touch ups
Parts:
- added R2202: 10k, Resistor_SMD:R_0805_2012Metric, symbol Device:R
Connections:
- net labels added: CTRL, ~Out
- net labels removed: gnd_break, output_control
- wire segments 5 -> 2
Changed lines of the file:
@@
 $Descr A4 11693 8268
 encoding utf-8
-Sheet 22 35
+Sheet 30 35
 Title ""
 Date ""
@@
 $Comp
 L Device:Q_NPN_BCE Q?
-U 1 1 5B6C08F9
-P 1800 1150
-AR Path="/5B62EDB8/5B6C08F9" Ref="Q?"  Part="1"
-AR Path="/5B62EDB8/5B6C04D0/5B6C08F9" Ref="Q2201"  Part="1"
-AR Path="/5B62EDB8/5B6C94C6/5B6C08F9" Ref="Q2301"  Part="1"
-AR Path="/5B62EDB8/5B6CA292/5B6C08F9" Ref="Q2401"  Part="1"
-AR Path="/5B62EDB8/5B6CB22A/5B6C08F9" Ref="Q2501"  Part="1"
-AR Path="/5B62EDB8/5B6CC0CE/5B6C08F9" Ref="Q2601"  Part="1"
-AR Path="/5B62EDB8/5B6CCE9A/5B6C08F9" Ref="Q2701"  Part="1"
-AR Path="/5B62EDB8/5B6CDC66/5B6C08F9" Ref="Q2801"  Part="1"
-AR Path="/5B62EDB8/5B6CEB95/5B6C08F9" Ref="Q2901"  Part="1"
-F 0 "Q2901" V 2000 1100 50  0000 L CNN
-F 1 "ZXTN25050DFHTA" H 1200 1000 50  0000 L CNN
-F 2 "Package_TO_SOT_SMD:SOT-23" H 2000 1250 50  0001 C CNN
-F 3 "" H 1800 1150 50  0001 C CNN
-	1    1800 1150
-	1    0    0    -1
-$EndComp
-$Comp
-L power:GND #PWR?
-U 1 1 5B6C0900
-P 1900 1450
-AR Path="/5B62EDB8/5B6C0900" Ref="#PWR?"  Part="1"
-AR Path="/5B62EDB8/5B6C04D0/5B6C0900" Ref="#PWR02201"  Part="1"
-AR Path="/5B62EDB8/5B6C94C6/5B6C0900" Ref="#PWR02301"  Part="1"
-AR Path="/5B62EDB8/5B6CA292/5B6C0900" Ref="#PWR02401"  Part="1"
-AR Path="/5B62EDB8/5B6CB22A/5B6C0900" Ref="#PWR02501"  Part="1"
-AR Path="/5B62EDB8/5B6CC0CE/5B6C0900" Ref="#PWR02601"  Part="1"
-AR Path="/5B62EDB8/5B6CCE9A/5B6C0900" Ref="#PWR02701"  Part="1"
-AR Path="/5B62EDB8/5B6CDC66/5B6C0900" Ref="#PWR02801"  Part="1"
-AR Path="/5B62EDB8/5B6CEB95/5B6C0900" Ref="#PWR02901"  Part="1"
-F 0 "#PWR02901" H 1900 1200 50  0001 C CNN
-F 1 "GND" H 1905 1277 50  0000 C CNN
-F 2 "" H 1900 1450 50  0001 C CNN
-F 3 "" H 1900 1450 50  0001 C CNN
-	1    1900 1450
+U 1 1 5B8D6899
+P 1700 1050
+AR Path="/5B62EDB8/5B8D6899" Ref="Q?"  Part="1"
+AR Path="/5B62EDB8/5B8B425B/5B8D6899" Ref="Q?"  Part="1"
+AR Path="/5B62EDB8/5B8BDF9E/5B8D6899" Ref="Q?"  Part="1"
+AR Path="/5B62EDB8/5B8CC011/5B8D6899" Ref="Q?"  Part="1"
+AR Path="/5B62EDB8/5B8CD7E8/5B8D6899" Ref="Q?"  Part="1"
+AR Path="/5B62EDB8/5B6C04D0/5B8D6899" Ref="Q2201"  Part="1"
+AR Path="/5B62EDB8/5B8DFA1F/5B8D6899" Ref="Q3001"  Part="1"
+AR Path="/5B62EDB8/5B8D6A51/5B8D6899" Ref="Q2401"  Part="1"
+AR Path="/5B62EDB8/5B8D8275/5B8D6899" Ref="Q2501"  Part="1"
+AR Path="/5B62EDB8/5B8D9A4C/5B8D6899" Ref="Q2601"  Part="1"
+AR Path="/5B62EDB8/5B8DB29A/5B8D6899" Ref="Q2701"  Part="1"
+AR Path="/5B62EDB8/5B8DCA71/5B8D6899" Ref="Q2801"  Part="1"
+AR Path="/5B62EDB8/5B8DE248/5B8D6899" Ref="Q2901"  Part="1"
+AR Path="/5B62EDB8/5B8EE9B3/5B8D6899" Ref="Q3101"  Part="1"
+AR Path="/5B62EDB8/5B8F19D7/5B8D6899" Ref="Q3201"  Part="1"
+AR Path="/5B62EDB8/5B8F31AE/5B8D6899" Ref="Q3301"  Part="1"
+AR Path="/5B62EDB8/5B8F4985/5B8D6899" Ref="Q3401"  Part="1"
+F 0 "Q3001" V 1900 1000 50  0000 L CNN
+F 1 "ZXTN25050DFHTA" H 1950 950 50  0000 L CNN
+F 2 "Package_TO_SOT_SMD:SOT-23" H 1900 1150 50  0001 C CNN
+F 3 "" H 1700 1050 50  0001 C CNN
+	1    1700 1050
 	1    0    0    -1
 $EndComp
 $Comp
 L Device:R R?
-U 1 1 5B6C0906
-P 1400 1150
-AR Path="/5B62EDB8/5B6C0906" Ref="R?"  Part="1"
-AR Path="/5B62EDB8/5B6C04D0/5B6C0906" Ref="R2201"  Part="1"
-AR Path="/5B62EDB8/5B6C94C6/5B6C0906" Ref="R2301"  Part="1"
-AR Path="/5B62EDB8/5B6CA292/5B6C0906" Ref="R2401"  Part="1"
-AR Path="/5B62EDB8/5B6CB22A/5B6C0906" Ref="R2501"  Part="1"
-AR Path="/5B62EDB8/5B6CC0CE/5B6C0906" Ref="R2601"  Part="1"
-AR Path="/5B62EDB8/5B6CCE9A/5B6C0906" Ref="R2701"  Part="1"
-AR Path="/5B62EDB8/5B6CDC66/5B6C0906" Ref="R2801"  Part="1"
-AR Path="/5B62EDB8/5B6CEB95/5B6C0906" Ref="R2901"  Part="1"
-F 0 "R2901" V 1300 1150 50  0000 C CNN
-F 1 "470" V 1400 1150 50  0000 C CNN
-F 2 "Resistor_SMD:R_0805_2012Metric" V 1330 1150 50  0001 C CNN
-F 3 "" H 1400 1150 50  0001 C CNN
-	1    1400 1150
+U 1 1 5B8D68A0
+P 950 1050
+AR Path="/5B62EDB8/5B8D68A0" Ref="R?"  Part="1"
+AR Path="/5B62EDB8/5B8B425B/5B8D68A0" Ref="R?"  Part="1"
+AR Path="/5B62EDB8/5B8BDF9E/5B8D68A0" Ref="R?"  Part="1"
+AR Path="/5B62EDB8/5B8CC011/5B8D68A0" Ref="R?"  Part="1"
+AR Path="/5B62EDB8/5B8CD7E8/5B8D68A0" Ref="R?"  Part="1"
+AR Path="/5B62EDB8/5B6C04D0/5B8D68A0" Ref="R2201"  Part="1"
+AR Path="/5B62EDB8/5B8DFA1F/5B8D68A0" Ref="R3001"  Part="1"
+AR Path="/5B62EDB8/5B8D6A51/5B8D68A0" Ref="R2401"  Part="1"
+AR Path="/5B62EDB8/5B8D8275/5B8D68A0" Ref="R2501"  Part="1"
+AR Path="/5B62EDB8/5B8D9A4C/5B8D68A0" Ref="R2601"  Part="1"
+AR Path="/5B62EDB8/5B8DB29A/5B8D68A0" Ref="R2701"  Part="1"
+AR Path="/5B62EDB8/5B8DCA71/5B8D68A0" Ref="R2801"  Part="1"
+AR Path="/5B62EDB8/5B8DE248/5B8D68A0" Ref="R2901"  Part="1"
+AR Path="/5B62EDB8/5B8EE9B3/5B8D68A0" Ref="R3101"  Part="1"
+AR Path="/5B62EDB8/5B8F19D7/5B8D68A0" Ref="R3201"  Part="1"
+AR Path="/5B62EDB8/5B8F31AE/5B8D68A0" Ref="R3301"  Part="1"
+AR Path="/5B62EDB8/5B8F4985/5B8D68A0" Ref="R3401"  Part="1"
+F 0 "R3001" V 850 1050 50  0000 C CNN
+F 1 "470" V 950 1050 50  0000 C CNN
+F 2 "Resistor_SMD:R_0805_2012Metric" V 880 1050 50  0001 C CNN
+F 3 "" H 950 1050 50  0001 C CNN
+	1    950  1050
 	0    1    1    0
 $EndComp
+$Comp
+L power:GND #PWR?
+U 1 1 5B8D68A7
+P 1800 1250
+AR Path="/5B62EDB8/5B8D68A7" Ref="#PWR?"  Part="1"
+AR Path="/5B62EDB8/5B8B425B/5B8D68A7" Ref="#PWR?"  Part="1"
+AR Path="/5B62EDB8/5B8BDF9E/5B8D68A7" Ref="#PWR?"  Part="1"
+AR Path="/5B62EDB8/5B8CC011/5B8D68A7" Ref="#PWR?"  Part="1"
+AR Path="/5B62EDB8/5B8CD7E8/5B8D68A7" Ref="#PWR?"  Part="1"
+AR Path="/5B62EDB8/5B6C04D0/5B8D68A7" Ref="#PWR02202"  Part="1"
+AR Path="/5B62EDB8/5B8DFA1F/5B8D68A7" Ref="#PWR03002"  Part="1"
+AR Path="/5B62EDB8/5B8D6A51/5B8D68A7" Ref="#PWR02402"  Part="1"
+AR Path="/5B62EDB8/5B8D8275/5B8D68A7" Ref="#PWR02502"  Part="1"
+AR Path="/5B62EDB8/5B8D9A4C/5B8D68A7" Ref="#PWR02602"  Part="1"
+AR Path="/5B62EDB8/5B8DB29A/5B8D68A7" Ref="#PWR02702"  Part="1"
+AR Path="/5B62EDB8/5B8DCA71/5B8D68A7" Ref="#PWR02802"  Part="1"
+AR Path="/5B62EDB8/5B8DE248/5B8D68A7" Ref="#PWR02902"  Part="1"
+AR Path="/5B62EDB8/5B8EE9B3/5B8D68A7" Ref="#PWR03102"  Part="1"
+AR Path="/5B62EDB8/5B8F19D7/5B8D68A7" Ref="#PWR03202"  Part="1"
+AR Path="/5B62EDB8/5B8F31AE/5B8D68A7" Ref="#PWR03302"  Part="1"
+AR Path="/5B62EDB8/5B8F4985/5B8D68A7" Ref="#PWR03402"  Part="1"
+F 0 "#PWR03002" H 1800 1000 50  0001 C CNN
+F 1 "GND" H 1805 1077 50  0000 C CNN
+F 2 "" H 1800 1250 50  0001 C CNN
+F 3 "" H 1800 1250 50  0001 C CNN
+	1    1800 1250
+	1    0    0    -1
+$EndComp
+$Comp
+L Device:R R?
+U 1 1 5B8D68AD
+P 1350 1200
+AR Path="/5B62EDB8/5B8D68AD" Ref="R?"  Part="1"
+AR Path="/5B62EDB8/5B8B425B/5B8D68AD" Ref="R?"  Part="1"
+AR Path="/5B62EDB8/5B8BDF9E/5B8D68AD" Ref="R?"  Part="1"
+AR Path="/5B62EDB8/5B8CC011/5B8D68AD" Ref="R?"  Part="1"
+AR Path="/5B62EDB8/5B8CD7E8/5B8D68AD" Ref="R?"  Part="1"
+AR Path="/5B62EDB8/5B6C04D0/5B8D68AD" Ref="R2202"  Part="1"
+AR Path="/5B62EDB8/5B8DFA1F/5B8D68AD" Ref="R3002"  Part="1"
+AR Path="/5B62EDB8/5B8D6A51/5B8D68AD" Ref="R2402"  Part="1"
+AR Path="/5B62EDB8/5B8D8275/5B8D68AD" Ref="R2502"  Part="1"
+AR Path="/5B62EDB8/5B8D9A4C/5B8D68AD" Ref="R2602"  Part="1"
+AR Path="/5B62EDB8/5B8DB29A/5B8D68AD" Ref="R2702"  Part="1"
+AR Path="/5B62EDB8/5B8DCA71/5B8D68AD" Ref="R2802"  Part="1"
+AR Path="/5B62EDB8/5B8DE248/5B8D68AD" Ref="R2902"  Part="1"
+AR Path="/5B62EDB8/5B8EE9B3/5B8D68AD" Ref="R3102"  Part="1"
+AR Path="/5B62EDB8/5B8F19D7/5B8D68AD" Ref="R3202"  Part="1"
+AR Path="/5B62EDB8/5B8F31AE/5B8D68AD" Ref="R3302"  Part="1"
+AR Path="/5B62EDB8/5B8F4985/5B8D68AD" Ref="R3402"  Part="1"
+F 0 "R3002" H 1420 1246 50  0000 L CNN
+F 1 "10k" H 1420 1155 50  0000 L CNN
+F 2 "Resistor_SMD:R_0805_2012Metric" V 1280 1200 50  0001 C CNN
+F 3 "" H 1350 1200 50  0001 C CNN
+	1    1350 1200
+	-1   0    0    1
+$EndComp
+$Comp
+L power:GND #PWR?
+U 1 1 5B8D68B4
+P 1350 1350
+AR Path="/5B62EDB8/5B8D68B4" Ref="#PWR?"  Part="1"
+AR Path="/5B62EDB8/5B8B425B/5B8D68B4" Ref="#PWR?"  Part="1"
+AR Path="/5B62EDB8/5B8BDF9E/5B8D68B4" Ref="#PWR?"  Part="1"
+AR Path="/5B62EDB8/5B8CC011/5B8D68B4" Ref="#PWR?"  Part="1"
+AR Path="/5B62EDB8/5B8CD7E8/5B8D68B4" Ref="#PWR?"  Part="1"
+AR Path="/5B62EDB8/5B6C04D0/5B8D68B4" Ref="#PWR02201"  Part="1"
+AR Path="/5B62EDB8/5B8DFA1F/5B8D68B4" Ref="#PWR03001"  Part="1"
+AR Path="/5B62EDB8/5B8D6A51/5B8D68B4" Ref="#PWR02401"  Part="1"
+AR Path="/5B62EDB8/5B8D8275/5B8D68B4" Ref="#PWR02501"  Part="1"
+AR Path="/5B62EDB8/5B8D9A4C/5B8D68B4" Ref="#PWR02601"  Part="1"
+AR Path="/5B62EDB8/5B8DB29A/5B8D68B4" Ref="#PWR02701"  Part="1"
+AR Path="/5B62EDB8/5B8DCA71/5B8D68B4" Ref="#PWR02801"  Part="1"
+AR Path="/5B62EDB8/5B8DE248/5B8D68B4" Ref="#PWR02901"  Part="1"
+AR Path="/5B62EDB8/5B8EE9B3/5B8D68B4" Ref="#PWR03101"  Part="1"
+AR Path="/5B62EDB8/5B8F19D7/5B8D68B4" Ref="#PWR03201"  Part="1"
+AR Path="/5B62EDB8/5B8F31AE/5B8D68B4" Ref="#PWR03301"  Part="1"
+AR Path="/5B62EDB8/5B8F4985/5B8D68B4" Ref="#PWR03401"  Part="1"
+F 0 "#PWR03001" H 1350 1100 50  0001 C CNN
+F 1 "GND" H 1355 1177 50  0000 C CNN
+F 2 "" H 1350 1350 50  0001 C CNN
+F 3 "" H 1350 1350 50  0001 C CNN
+	1    1350 1350
+	1    0    0    -1
+$EndComp
 Wire Wire Line
-	1900 1450 1900 1350
+	1100 1050 1350 1050
+Connection ~ 1350 1050
 Wire Wire Line
-	1550 1150 1600 1150
-Text HLabel 1200 1150 0    50   Input ~ 0
-output_control
-Wire Wire Line
-	1250 1150 1200 1150
-Text HLabel 2000 800  2    50   Output ~ 0
-gnd_break
-Wire Wire Line
-	1900 950  1900 800
-Wire Wire Line
-	1900 800  2000 800
+	1350 1050 1500 1050
+Text HLabel 800  1050 0    50   Input ~ 0
+CTRL
+Text HLabel 1800 850  1    50   Input ~ 0
+~Out
 $EndSCHEMATC

Commit message: Added SDCard slot.
Parts:
- renumbered Q2201 to Q2301, R2201 to R2301, R2202 to R2302
Changed lines of the file:
@@
 $Descr A4 11693 8268
 encoding utf-8
-Sheet 30 35
+Sheet 30 36
 Title ""
 Date ""
@@
 AR Path="/5B62EDB8/5B8CC011/5B8D6899" Ref="Q?"  Part="1"
 AR Path="/5B62EDB8/5B8CD7E8/5B8D6899" Ref="Q?"  Part="1"
-AR Path="/5B62EDB8/5B6C04D0/5B8D6899" Ref="Q2201"  Part="1"
-AR Path="/5B62EDB8/5B8DFA1F/5B8D6899" Ref="Q3001"  Part="1"
-AR Path="/5B62EDB8/5B8D6A51/5B8D6899" Ref="Q2401"  Part="1"
-AR Path="/5B62EDB8/5B8D8275/5B8D6899" Ref="Q2501"  Part="1"
-AR Path="/5B62EDB8/5B8D9A4C/5B8D6899" Ref="Q2601"  Part="1"
-AR Path="/5B62EDB8/5B8DB29A/5B8D6899" Ref="Q2701"  Part="1"
-AR Path="/5B62EDB8/5B8DCA71/5B8D6899" Ref="Q2801"  Part="1"
-AR Path="/5B62EDB8/5B8DE248/5B8D6899" Ref="Q2901"  Part="1"
-AR Path="/5B62EDB8/5B8EE9B3/5B8D6899" Ref="Q3101"  Part="1"
-AR Path="/5B62EDB8/5B8F19D7/5B8D6899" Ref="Q3201"  Part="1"
-AR Path="/5B62EDB8/5B8F31AE/5B8D6899" Ref="Q3301"  Part="1"
-AR Path="/5B62EDB8/5B8F4985/5B8D6899" Ref="Q3401"  Part="1"
-F 0 "Q3401" V 1900 1000 50  0000 L CNN
+AR Path="/5B62EDB8/5B6C04D0/5B8D6899" Ref="Q2301"  Part="1"
+AR Path="/5B62EDB8/5B8DFA1F/5B8D6899" Ref="Q3101"  Part="1"
+AR Path="/5B62EDB8/5B8D6A51/5B8D6899" Ref="Q2501"  Part="1"
+AR Path="/5B62EDB8/5B8D8275/5B8D6899" Ref="Q2601"  Part="1"
+AR Path="/5B62EDB8/5B8D9A4C/5B8D6899" Ref="Q2701"  Part="1"
+AR Path="/5B62EDB8/5B8DB29A/5B8D6899" Ref="Q2801"  Part="1"
+AR Path="/5B62EDB8/5B8DCA71/5B8D6899" Ref="Q2901"  Part="1"
+AR Path="/5B62EDB8/5B8DE248/5B8D6899" Ref="Q3001"  Part="1"
+AR Path="/5B62EDB8/5B8EE9B3/5B8D6899" Ref="Q3201"  Part="1"
+AR Path="/5B62EDB8/5B8F19D7/5B8D6899" Ref="Q3301"  Part="1"
+AR Path="/5B62EDB8/5B8F31AE/5B8D6899" Ref="Q3401"  Part="1"
+AR Path="/5B62EDB8/5B8F4985/5B8D6899" Ref="Q3501"  Part="1"
+F 0 "Q3501" V 1900 1000 50  0000 L CNN
 F 1 "ZXTN25050DFHTA" H 1950 950 50  0000 L CNN
 F 2 "Package_TO_SOT_SMD:SOT-23" H 1900 1150 50  0001 C CNN
@@
 AR Path="/5B62EDB8/5B8CC011/5B8D68A0" Ref="R?"  Part="1"
 AR Path="/5B62EDB8/5B8CD7E8/5B8D68A0" Ref="R?"  Part="1"
-AR Path="/5B62EDB8/5B6C04D0/5B8D68A0" Ref="R2201"  Part="1"
-AR Path="/5B62EDB8/5B8DFA1F/5B8D68A0" Ref="R3001"  Part="1"
-AR Path="/5B62EDB8/5B8D6A51/5B8D68A0" Ref="R2401"  Part="1"
-AR Path="/5B62EDB8/5B8D8275/5B8D68A0" Ref="R2501"  Part="1"
-AR Path="/5B62EDB8/5B8D9A4C/5B8D68A0" Ref="R2601"  Part="1"
-AR Path="/5B62EDB8/5B8DB29A/5B8D68A0" Ref="R2701"  Part="1"
-AR Path="/5B62EDB8/5B8DCA71/5B8D68A0" Ref="R2801"  Part="1"
-AR Path="/5B62EDB8/5B8DE248/5B8D68A0" Ref="R2901"  Part="1"
-AR Path="/5B62EDB8/5B8EE9B3/5B8D68A0" Ref="R3101"  Part="1"
-AR Path="/5B62EDB8/5B8F19D7/5B8D68A0" Ref="R3201"  Part="1"
-AR Path="/5B62EDB8/5B8F31AE/5B8D68A0" Ref="R3301"  Part="1"
-AR Path="/5B62EDB8/5B8F4985/5B8D68A0" Ref="R3401"  Part="1"
-F 0 "R3401" V 850 1050 50  0000 C CNN
+AR Path="/5B62EDB8/5B6C04D0/5B8D68A0" Ref="R2301"  Part="1"
+AR Path="/5B62EDB8/5B8DFA1F/5B8D68A0" Ref="R3101"  Part="1"
+AR Path="/5B62EDB8/5B8D6A51/5B8D68A0" Ref="R2501"  Part="1"
+AR Path="/5B62EDB8/5B8D8275/5B8D68A0" Ref="R2601"  Part="1"
+AR Path="/5B62EDB8/5B8D9A4C/5B8D68A0" Ref="R2701"  Part="1"
+AR Path="/5B62EDB8/5B8DB29A/5B8D68A0" Ref="R2801"  Part="1"
+AR Path="/5B62EDB8/5B8DCA71/5B8D68A0" Ref="R2901"  Part="1"
+AR Path="/5B62EDB8/5B8DE248/5B8D68A0" Ref="R3001"  Part="1"
+AR Path="/5B62EDB8/5B8EE9B3/5B8D68A0" Ref="R3201"  Part="1"
+AR Path="/5B62EDB8/5B8F19D7/5B8D68A0" Ref="R3301"  Part="1"
+AR Path="/5B62EDB8/5B8F31AE/5B8D68A0" Ref="R3401"  Part="1"
+AR Path="/5B62EDB8/5B8F4985/5B8D68A0" Ref="R3501"  Part="1"
+F 0 "R3501" V 850 1050 50  0000 C CNN
 F 1 "470" V 950 1050 50  0000 C CNN
 F 2 "Resistor_SMD:R_0805_2012Metric" V 880 1050 50  0001 C CNN
@@
 AR Path="/5B62EDB8/5B8CC011/5B8D68A7" Ref="#PWR?"  Part="1"
 AR Path="/5B62EDB8/5B8CD7E8/5B8D68A7" Ref="#PWR?"  Part="1"
-AR Path="/5B62EDB8/5B6C04D0/5B8D68A7" Ref="#PWR02202"  Part="1"
-AR Path="/5B62EDB8/5B8DFA1F/5B8D68A7" Ref="#PWR03002"  Part="1"
-AR Path="/5B62EDB8/5B8D6A51/5B8D68A7" Ref="#PWR02402"  Part="1"
-AR Path="/5B62EDB8/5B8D8275/5B8D68A7" Ref="#PWR02502"  Part="1"
-AR Path="/5B62EDB8/5B8D9A4C/5B8D68A7" Ref="#PWR02602"  Part="1"
-AR Path="/5B62EDB8/5B8DB29A/5B8D68A7" Ref="#PWR02702"  Part="1"
-AR Path="/5B62EDB8/5B8DCA71/5B8D68A7" Ref="#PWR02802"  Part="1"
-AR Path="/5B62EDB8/5B8DE248/5B8D68A7" Ref="#PWR02902"  Part="1"
-AR Path="/5B62EDB8/5B8EE9B3/5B8D68A7" Ref="#PWR03102"  Part="1"
-AR Path="/5B62EDB8/5B8F19D7/5B8D68A7" Ref="#PWR03202"  Part="1"
-AR Path="/5B62EDB8/5B8F31AE/5B8D68A7" Ref="#PWR03302"  Part="1"
-AR Path="/5B62EDB8/5B8F4985/5B8D68A7" Ref="#PWR03402"  Part="1"
-F 0 "#PWR03402" H 1800 1000 50  0001 C CNN
+AR Path="/5B62EDB8/5B6C04D0/5B8D68A7" Ref="#PWR02302"  Part="1"
+AR Path="/5B62EDB8/5B8DFA1F/5B8D68A7" Ref="#PWR03102"  Part="1"
+AR Path="/5B62EDB8/5B8D6A51/5B8D68A7" Ref="#PWR02502"  Part="1"
+AR Path="/5B62EDB8/5B8D8275/5B8D68A7" Ref="#PWR02602"  Part="1"
+AR Path="/5B62EDB8/5B8D9A4C/5B8D68A7" Ref="#PWR02702"  Part="1"
+AR Path="/5B62EDB8/5B8DB29A/5B8D68A7" Ref="#PWR02802"  Part="1"
+AR Path="/5B62EDB8/5B8DCA71/5B8D68A7" Ref="#PWR02902"  Part="1"
+AR Path="/5B62EDB8/5B8DE248/5B8D68A7" Ref="#PWR03002"  Part="1"
+AR Path="/5B62EDB8/5B8EE9B3/5B8D68A7" Ref="#PWR03202"  Part="1"
+AR Path="/5B62EDB8/5B8F19D7/5B8D68A7" Ref="#PWR03302"  Part="1"
+AR Path="/5B62EDB8/5B8F31AE/5B8D68A7" Ref="#PWR03402"  Part="1"
+AR Path="/5B62EDB8/5B8F4985/5B8D68A7" Ref="#PWR03502"  Part="1"
+F 0 "#PWR03502" H 1800 1000 50  0001 C CNN
 F 1 "GND" H 1805 1077 50  0000 C CNN
 F 2 "" H 1800 1250 50  0001 C CNN
@@
 AR Path="/5B62EDB8/5B8CC011/5B8D68AD" Ref="R?"  Part="1"
 AR Path="/5B62EDB8/5B8CD7E8/5B8D68AD" Ref="R?"  Part="1"
-AR Path="/5B62EDB8/5B6C04D0/5B8D68AD" Ref="R2202"  Part="1"
-AR Path="/5B62EDB8/5B8DFA1F/5B8D68AD" Ref="R3002"  Part="1"
-AR Path="/5B62EDB8/5B8D6A51/5B8D68AD" Ref="R2402"  Part="1"
-AR Path="/5B62EDB8/5B8D8275/5B8D68AD" Ref="R2502"  Part="1"
-AR Path="/5B62EDB8/5B8D9A4C/5B8D68AD" Ref="R2602"  Part="1"
-AR Path="/5B62EDB8/5B8DB29A/5B8D68AD" Ref="R2702"  Part="1"
-AR Path="/5B62EDB8/5B8DCA71/5B8D68AD" Ref="R2802"  Part="1"
-AR Path="/5B62EDB8/5B8DE248/5B8D68AD" Ref="R2902"  Part="1"
-AR Path="/5B62EDB8/5B8EE9B3/5B8D68AD" Ref="R3102"  Part="1"
-AR Path="/5B62EDB8/5B8F19D7/5B8D68AD" Ref="R3202"  Part="1"
-AR Path="/5B62EDB8/5B8F31AE/5B8D68AD" Ref="R3302"  Part="1"
-AR Path="/5B62EDB8/5B8F4985/5B8D68AD" Ref="R3402"  Part="1"
-F 0 "R3402" H 1420 1246 50  0000 L CNN
+AR Path="/5B62EDB8/5B6C04D0/5B8D68AD" Ref="R2302"  Part="1"
+AR Path="/5B62EDB8/5B8DFA1F/5B8D68AD" Ref="R3102"  Part="1"
+AR Path="/5B62EDB8/5B8D6A51/5B8D68AD" Ref="R2502"  Part="1"
+AR Path="/5B62EDB8/5B8D8275/5B8D68AD" Ref="R2602"  Part="1"
+AR Path="/5B62EDB8/5B8D9A4C/5B8D68AD" Ref="R2702"  Part="1"
+AR Path="/5B62EDB8/5B8DB29A/5B8D68AD" Ref="R2802"  Part="1"
+AR Path="/5B62EDB8/5B8DCA71/5B8D68AD" Ref="R2902"  Part="1"
+AR Path="/5B62EDB8/5B8DE248/5B8D68AD" Ref="R3002"  Part="1"
+AR Path="/5B62EDB8/5B8EE9B3/5B8D68AD" Ref="R3202"  Part="1"
+AR Path="/5B62EDB8/5B8F19D7/5B8D68AD" Ref="R3302"  Part="1"
+AR Path="/5B62EDB8/5B8F31AE/5B8D68AD" Ref="R3402"  Part="1"
+AR Path="/5B62EDB8/5B8F4985/5B8D68AD" Ref="R3502"  Part="1"
+F 0 "R3502" H 1420 1246 50  0000 L CNN
 F 1 "10k" H 1420 1155 50  0000 L CNN
 F 2 "Resistor_SMD:R_0805_2012Metric" V 1280 1200 50  0001 C CNN
-F 3 "" H 1350 1200 50  0001 C CNN
+F 3 "https://www.mouser.se/ProductDetail/Panasonic-Industrial-Devices/ERJ-6ENF1002V?qs=sGAEpiMZZMu61qfTUdNhGzRxdwze5h8ZcGDx6geba20%3d" H 1350 1200 50  0001 C CNN
 	1    1350 1200
 	-1   0    0    1
@@
 AR Path="/5B62EDB8/5B8CC011/5B8D68B4" Ref="#PWR?"  Part="1"
 AR Path="/5B62EDB8/5B8CD7E8/5B8D68B4" Ref="#PWR?"  Part="1"
-AR Path="/5B62EDB8/5B6C04D0/5B8D68B4" Ref="#PWR02201"  Part="1"
-AR Path="/5B62EDB8/5B8DFA1F/5B8D68B4" Ref="#PWR03001"  Part="1"
-AR Path="/5B62EDB8/5B8D6A51/5B8D68B4" Ref="#PWR02401"  Part="1"
-AR Path="/5B62EDB8/5B8D8275/5B8D68B4" Ref="#PWR02501"  Part="1"
-AR Path="/5B62EDB8/5B8D9A4C/5B8D68B4" Ref="#PWR02601"  Part="1"
-AR Path="/5B62EDB8/5B8DB29A/5B8D68B4" Ref="#PWR02701"  Part="1"
-AR Path="/5B62EDB8/5B8DCA71/5B8D68B4" Ref="#PWR02801"  Part="1"
-AR Path="/5B62EDB8/5B8DE248/5B8D68B4" Ref="#PWR02901"  Part="1"
-AR Path="/5B62EDB8/5B8EE9B3/5B8D68B4" Ref="#PWR03101"  Part="1"
-AR Path="/5B62EDB8/5B8F19D7/5B8D68B4" Ref="#PWR03201"  Part="1"
-AR Path="/5B62EDB8/5B8F31AE/5B8D68B4" Ref="#PWR03301"  Part="1"
-AR Path="/5B62EDB8/5B8F4985/5B8D68B4" Ref="#PWR03401"  Part="1"
-F 0 "#PWR03401" H 1350 1100 50  0001 C CNN
+AR Path="/5B62EDB8/5B6C04D0/5B8D68B4" Ref="#PWR02301"  Part="1"
+AR Path="/5B62EDB8/5B8DFA1F/5B8D68B4" Ref="#PWR03101"  Part="1"
+AR Path="/5B62EDB8/5B8D6A51/5B8D68B4" Ref="#PWR02501"  Part="1"
+AR Path="/5B62EDB8/5B8D8275/5B8D68B4" Ref="#PWR02601"  Part="1"
+AR Path="/5B62EDB8/5B8D9A4C/5B8D68B4" Ref="#PWR02701"  Part="1"
+AR Path="/5B62EDB8/5B8DB29A/5B8D68B4" Ref="#PWR02801"  Part="1"
+AR Path="/5B62EDB8/5B8DCA71/5B8D68B4" Ref="#PWR02901"  Part="1"
+AR Path="/5B62EDB8/5B8DE248/5B8D68B4" Ref="#PWR03001"  Part="1"
+AR Path="/5B62EDB8/5B8EE9B3/5B8D68B4" Ref="#PWR03201"  Part="1"
+AR Path="/5B62EDB8/5B8F19D7/5B8D68B4" Ref="#PWR03301"  Part="1"
+AR Path="/5B62EDB8/5B8F31AE/5B8D68B4" Ref="#PWR03401"  Part="1"
+AR Path="/5B62EDB8/5B8F4985/5B8D68B4" Ref="#PWR03501"  Part="1"
+F 0 "#PWR03501" H 1350 1100 50  0001 C CNN
 F 1 "GND" H 1355 1177 50  0000 C CNN
 F 2 "" H 1350 1350 50  0001 C CNN
