File: G3/MCU.sch (KiCad schematic (older format))
At the start: 25 parts, among them J301 Conn_02x07_Odd_Even, SW301 Boot option, SW302 Reset, SW303 Adress, U301 ESP32_WROVER, U302 TXB0102DCU

Commit message: Changed from DIP swtich to pin header for address setting.
Parts:
- removed SW303: Adress, Package_DIP:DIP-6_W8.89mm_SMDSocket_LongPads, symbol Switch:SW_DIP_x03
- added J?: Conn_02x03_Counter_Clockwise, Connector_PinHeader_2.54mm:PinHeader_2x03_P2.54mm_Vertical, symbol Connector_Generic:Conn_02x03_Counter_Clockwise
Connections:
- wire segments 94 -> 92
Changed lines of the file:
@@
 MTDO
-$Comp
-L Switch:SW_DIP_x03 SW303
-U 1 1 5B73292F
-P 9400 1450
-F 0 "SW303" H 9400 1917 50  0000 C CNN
-F 1 "Adress" H 9400 1826 50  0000 C CNN
-F 2 "Package_DIP:DIP-6_W8.89mm_SMDSocket_LongPads" H 9400 1450 50  0001 C CNN
-F 3 "https://www.mouser.se/ProductDetail/Apem/DMR03T?qs=sGAEpiMZZMv%2f%252b2JhlA6ysJSm%252bcOQqpSgWoOP1dvNuLA%3d" H 9400 1450 50  0001 C CNN
-	1    9400 1450
-	1    0    0    -1
-$EndComp
 $Comp
 L Device:R R313
@@
 L power:+3.3V #PWR0321
 U 1 1 5B73AAEB
-P 9850 1400
-F 0 "#PWR0321" H 9850 1250 50  0001 C CNN
-F 1 "+3.3V" H 9865 1573 50  0000 C CNN
-F 2 "" H 9850 1400 50  0001 C CNN
-F 3 "" H 9850 1400 50  0001 C CNN
-	1    9850 1400
+P 9750 1350
+F 0 "#PWR0321" H 9750 1200 50  0001 C CNN
+F 1 "+3.3V" H 9765 1523 50  0000 C CNN
+F 2 "" H 9750 1350 50  0001 C CNN
+F 3 "" H 9750 1350 50  0001 C CNN
+	1    9750 1350
 	0    1    1    0
 $EndComp
-Wire Wire Line
-	9700 1250 9700 1350
-Connection ~ 9700 1350
-Wire Wire Line
-	9700 1350 9700 1400
-Connection ~ 9700 1450
-Wire Wire Line
-	9700 1450 9700 1550
-Wire Wire Line
-	9700 1400 9850 1400
-Connection ~ 9700 1400
-Wire Wire Line
-	9700 1400 9700 1450
 Text Label 8850 1250 0    50   ~ 0
 ADDR_0
@@
 Wire Wire Line
 	3250 3400 1500 3400
+$Comp
+L Connector_Generic:Conn_02x03_Counter_Clockwise J?
+U 1 1 5B7B0A2D
+P 9300 1350
+F 0 "J?" H 9350 1667 50  0000 C CNN
+F 1 "Conn_02x03_Counter_Clockwise" H 9350 1576 50  0000 C CNN
+F 2 "Connector_PinHeader_2.54mm:PinHeader_2x03_P2.54mm_Vertical" H 9300 1350 50  0001 C CNN
+F 3 "~" H 9300 1350 50  0001 C CNN
+	1    9300 1350
+	1    0    0    -1
+$EndComp
+Wire Wire Line
+	9600 1250 9600 1350
+Connection ~ 9600 1350
+Wire Wire Line
+	9600 1350 9600 1450
+Wire Wire Line
+	9600 1350 9750 1350
 $EndSCHEMATC

Commit message: Touch up
Parts:
- gave numbers to parts that had none: 1
Connections:
- net labels added: StatusLED
- wire segments 92 -> 85
- no-connect marks 2 -> 1
Changed lines of the file:
@@
 $Descr A4 11693 8268
 encoding utf-8
-Sheet 3 31
+Sheet 3 35
 Title ""
 Date ""
@@
 Text GLabel 7550 3300 2    60   Input ~ 0
 ANALOG_I2C_SDA
-Text GLabel 5500 2700 2    60   Input ~ 0
+Text GLabel 5250 2800 2    60   Input ~ 0
 ANALOG_RDY_2
-Text GLabel 5500 2800 2    60   Input ~ 0
+Text GLabel 5250 3600 2    60   Input ~ 0
 ANALOG_RDY_1
 Wire Wire Line
@@
 Wire Wire Line
 	6550 3200 5250 3200
-Wire Wire Line
-	5250 2800 5500 2800
-Wire Wire Line
-	5500 2700 5250 2700
-Text GLabel 5500 2600 2    60   Input ~ 0
+Text GLabel 5250 3700 2    60   Input ~ 0
 DIA_Interrupt
-Wire Wire Line
-	5500 2600 5250 2600
 $Comp
 L power:GND #PWR0309
@@
 Wire Wire Line
 	8500 1950 8500 1850
-Text Label 5400 3700 0    50   ~ 0
+Text Label 5250 2700 0    50   ~ 0
 ADDR_0
-Text Label 5400 3600 0    50   ~ 0
+Text Label 5250 2600 0    50   ~ 0
 ADDR_1
-Text Label 5400 3500 0    50   ~ 0
+Text Label 5250 2500 0    50   ~ 0
 ADDR_2
-Wire Wire Line
-	5400 3400 5250 3400
-Wire Wire Line
-	5250 3500 5400 3500
-Wire Wire Line
-	5400 3600 5250 3600
-Wire Wire Line
-	5250 3700 5400 3700
 $Comp
 L power:GND #PWR0316
@@
 Wire Wire Line
 	8350 1950 8500 1950
-NoConn ~ 5250 2500
-Text GLabel 5400 3400 2    50   Input ~ 0
+Text GLabel 5250 3500 2    50   Input ~ 0
 I2C_Reset
 $Comp
@@
 	3250 3400 1500 3400
 $Comp
-L Connector_Generic:Conn_02x03_Counter_Clockwise J?
+L Connector_Generic:Conn_02x03_Counter_Clockwise J302
 U 1 1 5B7B0A2D
 P 9300 1350
-F 0 "J?" H 9350 1667 50  0000 C CNN
+F 0 "J302" H 9350 1667 50  0000 C CNN
 F 1 "Conn_02x03_Counter_Clockwise" H 9350 1576 50  0000 C CNN
 F 2 "Connector_PinHeader_2.54mm:PinHeader_2x03_P2.54mm_Vertical" H 9300 1350 50  0001 C CNN
@@
 Wire Wire Line
 	9600 1350 9750 1350
+Text GLabel 5250 3400 2    50   Input ~ 0
+StatusLED
 $EndSCHEMATC

Commit message: More touch ups
Parts:
- added J?: BME280, symbol Connector_Generic:Conn_01x04
Connections:
- wire segments 85 -> 89
Changed lines of the file:
@@
 Text GLabel 5250 3400 2    50   Input ~ 0
 StatusLED
+$Comp
+L Connector_Generic:Conn_01x04 J?
+U 1 1 5B903FBD
+P 7750 3550
+F 0 "J?" H 7830 3542 50  0000 L CNN
+F 1 "BME280" H 7830 3451 50  0000 L CNN
+F 2 "" H 7750 3550 50  0001 C CNN
+F 3 "~" H 7750 3550 50  0001 C CNN
+	1    7750 3550
+	1    0    0    -1
+$EndComp
+Wire Wire Line
+	7450 3100 7450 3450
+Wire Wire Line
+	7450 3450 7550 3450
+Wire Wire Line
+	7150 3000 7150 3550
+Wire Wire Line
+	7150 3550 7550 3550
+$Comp
+L power:+5V #PWR?
+U 1 1 5B909304
+P 7550 3650
+F 0 "#PWR?" H 7550 3500 50  0001 C CNN
+F 1 "+5V" V 7565 3778 50  0000 L CNN
+F 2 "" H 7550 3650 50  0001 C CNN
+F 3 "" H 7550 3650 50  0001 C CNN
+	1    7550 3650
+	0    -1   -1   0
+$EndComp
+$Comp
+L power:GND #PWR?
+U 1 1 5B9093BD
+P 7550 3750
+F 0 "#PWR?" H 7550 3500 50  0001 C CNN
+F 1 "GND" V 7555 3622 50  0000 R CNN
+F 2 "" H 7550 3750 50  0001 C CNN
+F 3 "" H 7550 3750 50  0001 C CNN
+	1    7550 3750
+	0    1    1    0
+$EndComp
 $EndSCHEMATC

Commit message: Added header for BME280
Parts:
- J301: value Conn_02x07_Odd_Even -> Debug
- gave numbers to parts that had none: 1
- renumbered J302 to J303
Connections:
- wire segments 89 -> 82
Changed lines of the file:
@@
 $EndComp
 $Comp
-L power:+3.3V #PWR0317
+L power:+3.3V #PWR0319
 U 1 1 5B73B74B
 P 8400 4150
-F 0 "#PWR0317" H 8400 4000 50  0001 C CNN
+F 0 "#PWR0319" H 8400 4000 50  0001 C CNN
 F 1 "+3.3V" H 8415 4323 50  0000 C CNN
 F 2 "" H 8400 4150 50  0001 C CNN
@@
 $EndComp
 $Comp
-L power:+5V #PWR0319
+L power:+5V #PWR0321
 U 1 1 5B73B784
 P 8600 4150
-F 0 "#PWR0319" H 8600 4000 50  0001 C CNN
+F 0 "#PWR0321" H 8600 4000 50  0001 C CNN
 F 1 "+5V" H 8615 4323 50  0000 C CNN
 F 2 "" H 8600 4150 50  0001 C CNN
@@
 $EndComp
 $Comp
-L power:GND #PWR0315
+L power:GND #PWR0317
 U 1 1 5B73C2C7
 P 8100 4200
-F 0 "#PWR0315" H 8100 3950 50  0001 C CNN
+F 0 "#PWR0317" H 8100 3950 50  0001 C CNN
 F 1 "GND" V 8105 4072 50  0000 R CNN
 F 2 "" H 8100 4200 50  0001 C CNN
@@
 $EndComp
 $Comp
-L power:GND #PWR0320
+L power:GND #PWR0322
 U 1 1 5B73C2E7
 P 8900 4200
-F 0 "#PWR0320" H 8900 3950 50  0001 C CNN
+F 0 "#PWR0322" H 8900 3950 50  0001 C CNN
 F 1 "GND" V 8905 4072 50  0000 R CNN
 F 2 "" H 8900 4200 50  0001 C CNN
@@
 Wiegand_D1
 $Comp
-L power:GND #PWR0318
+L power:GND #PWR0320
 U 1 1 5B73CB5F
 P 8500 5250
-F 0 "#PWR0318" H 8500 5000 50  0001 C CNN
+F 0 "#PWR0320" H 8500 5000 50  0001 C CNN
 F 1 "GND" H 8505 5077 50  0000 C CNN
 F 2 "" H 8500 5250 50  0001 C CNN
@@
 U 1 1 5B6A5C70
 P 5650 5700
-F 0 "J301" H 5700 6217 50  0000 C CNN
-F 1 "Conn_02x07_Odd_Even" H 5700 6126 50  0000 C CNN
+F 0 "J301" H 5700 6100 50  0000 C CNN
+F 1 "Debug" H 5700 6000 50  0000 C CNN
 F 2 "Connector_PinHeader_2.54mm:PinHeader_2x05_P2.54mm_Vertical" H 5650 5700 50  0001 C CNN
 F 3 "~" H 5650 5700 50  0001 C CNN
@@
 P 5450 5500
 F 0 "#PWR0311" H 5450 5250 50  0001 C CNN
-F 1 "GND" H 5455 5327 50  0000 C CNN
+F 1 "GND" H 5400 5350 50  0000 C CNN
 F 2 "" H 5450 5500 50  0001 C CNN
 F 3 "" H 5450 5500 50  0001 C CNN
@@
 Text Label 2650 2650 0    50   ~ 0
 CH_Enable
-Text Label 6100 5600 0    50   ~ 0
+Text Label 5950 5600 0    50   ~ 0
 MTMS
-Text Label 6100 5700 0    50   ~ 0
+Text Label 5950 5700 0    50   ~ 0
 MTDI
-Text Label 6100 5900 0    50   ~ 0
+Text Label 5950 5900 0    50   ~ 0
 MTCK
-Text Label 6100 5800 0    50   ~ 0
+Text Label 5950 5800 0    50   ~ 0
 MTDO
 Text Label 2950 2900 0    50   ~ 0
@@
 Text Label 5950 5500 0    50   ~ 0
 Boot_option
-Text Label 5200 5700 2    50   ~ 0
+Text Label 5450 5700 2    50   ~ 0
 TDX0
-Text Label 5200 5800 2    50   ~ 0
+Text Label 5450 5800 2    50   ~ 0
 RDX0
 Wire Wire Line
@@
 Wire Wire Line
 	3250 3000 2950 3000
-Text Label 5200 5600 2    50   ~ 0
+Text Label 5450 5600 2    50   ~ 0
 CH_Enable
 Text Label 2700 3400 0    50   ~ 0
@@
 Wire Wire Line
 	2100 2650 3250 2650
-Wire Wire Line
-	5450 5600 5200 5600
-Wire Wire Line
-	5200 5700 5450 5700
-Wire Wire Line
-	5200 5800 5450 5800
 NoConn ~ 5450 5900
-Wire Wire Line
-	6200 5900 5950 5900
-Wire Wire Line
-	5950 5800 6200 5800
-Wire Wire Line
-	6200 5700 5950 5700
-Wire Wire Line
-	5950 5600 6200 5600
 Wire Wire Line
 	2900 5150 2900 3650
@@
 	7800 1250 7800 1550
 $Comp
-L power:+3.3V #PWR0321
+L power:+3.3V #PWR0323
 U 1 1 5B73AAEB
 P 9750 1350
-F 0 "#PWR0321" H 9750 1200 50  0001 C CNN
+F 0 "#PWR0323" H 9750 1200 50  0001 C CNN
 F 1 "+3.3V" H 9765 1523 50  0000 C CNN
 F 2 "" H 9750 1350 50  0001 C CNN
@@
 ADDR_2
 $Comp
-L power:GND #PWR0316
+L power:GND #PWR0318
 U 1 1 5B75512D
 P 8350 1950
-F 0 "#PWR0316" H 8350 1700 50  0001 C CNN
+F 0 "#PWR0318" H 8350 1700 50  0001 C CNN
 F 1 "GND" H 8355 1777 50  0000 C CNN
 F 2 "" H 8350 1950 50  0001 C CNN
@@
 	3250 3400 1500 3400
 $Comp
-L Connector_Generic:Conn_02x03_Counter_Clockwise J302
+L Connector_Generic:Conn_02x03_Counter_Clockwise J303
 U 1 1 5B7B0A2D
 P 9300 1350
-F 0 "J302" H 9350 1667 50  0000 C CNN
+F 0 "J303" H 9350 1667 50  0000 C CNN
 F 1 "Conn_02x03_Counter_Clockwise" H 9350 1576 50  0000 C CNN
 F 2 "Connector_PinHeader_2.54mm:PinHeader_2x03_P2.54mm_Vertical" H 9300 1350 50  0001 C CNN
@@
 StatusLED
 $Comp
-L Connector_Generic:Conn_01x04 J?
+L Connector_Generic:Conn_01x04 J302
 U 1 1 5B903FBD
-P 7750 3550
-F 0 "J?" H 7830 3542 50  0000 L CNN
-F 1 "BME280" H 7830 3451 50  0000 L CNN
-F 2 "" H 7750 3550 50  0001 C CNN
-F 3 "~" H 7750 3550 50  0001 C CNN
-	1    7750 3550
-	1    0    0    -1
-$EndComp
-Wire Wire Line
-	7450 3100 7450 3450
-Wire Wire Line
-	7450 3450 7550 3450
-Wire Wire Line
-	7150 3000 7150 3550
-Wire Wire Line
-	7150 3550 7550 3550
-$Comp
-L power:+5V #PWR?
+P 8300 3550
+F 0 "J302" H 8380 3542 50  0000 L CNN
+F 1 "BME280" H 8380 3451 50  0000 L CNN
+F 2 "" H 8300 3550 50  0001 C CNN
+F 3 "~" H 8300 3550 50  0001 C CNN
+	1    8300 3550
+	1    0    0    -1
+$EndComp
+$Comp
+L power:+5V #PWR0315
 U 1 1 5B909304
-P 7550 3650
-F 0 "#PWR?" H 7550 3500 50  0001 C CNN
-F 1 "+5V" V 7565 3778 50  0000 L CNN
-F 2 "" H 7550 3650 50  0001 C CNN
-F 3 "" H 7550 3650 50  0001 C CNN
-	1    7550 3650
+P 8100 3450
+F 0 "#PWR0315" H 8100 3300 50  0001 C CNN
+F 1 "+5V" V 8115 3578 50  0000 L CNN
+F 2 "" H 8100 3450 50  0001 C CNN
+F 3 "" H 8100 3450 50  0001 C CNN
+	1    8100 3450
 	0    -1   -1   0
 $EndComp
 $Comp
-L power:GND #PWR?
+L power:GND #PWR0316
 U 1 1 5B9093BD
-P 7550 3750
-F 0 "#PWR?" H 7550 3500 50  0001 C CNN
-F 1 "GND" V 7555 3622 50  0000 R CNN
-F 2 "" H 7550 3750 50  0001 C CNN
-F 3 "" H 7550 3750 50  0001 C CNN
-	1    7550 3750
-	0    1    1    0
-$EndComp
+P 8100 3550
+F 0 "#PWR0316" H 8100 3300 50  0001 C CNN
+F 1 "GND" V 8105 3422 50  0000 R CNN
+F 2 "" H 8100 3550 50  0001 C CNN
+F 3 "" H 8100 3550 50  0001 C CNN
+	1    8100 3550
+	0    1    1    0
+$EndComp
+Wire Wire Line
+	7150 3000 7150 3650
+Wire Wire Line
+	7150 3650 8100 3650
+Wire Wire Line
+	7450 3100 7450 3750
+Wire Wire Line
+	7450 3750 8100 3750
 $EndSCHEMATC

Commit message: added Factory reset switch
Parts:
- added SW303: Factory reset, Button_Switch_SMD:SW_SPST_CK_KXT3, symbol Switch:SW_Push
Connections:
- wire segments 82 -> 86
Changed lines of the file:
@@
 	7150 3000 5250 3000
 $Comp
-L power:+3.3V #PWR0313
+L power:+3.3V #PWR0314
 U 1 1 5B73B348
 P 7300 2650
-F 0 "#PWR0313" H 7300 2500 50  0001 C CNN
+F 0 "#PWR0314" H 7300 2500 50  0001 C CNN
 F 1 "+3.3V" H 7315 2823 50  0000 C CNN
 F 2 "" H 7300 2650 50  0001 C CNN
@@
 $EndComp
 $Comp
-L power:+3.3V #PWR0319
+L power:+3.3V #PWR0320
 U 1 1 5B73B74B
 P 8400 4150
-F 0 "#PWR0319" H 8400 4000 50  0001 C CNN
+F 0 "#PWR0320" H 8400 4000 50  0001 C CNN
 F 1 "+3.3V" H 8415 4323 50  0000 C CNN
 F 2 "" H 8400 4150 50  0001 C CNN
@@
 $EndComp
 $Comp
-L power:+5V #PWR0321
+L power:+5V #PWR0322
 U 1 1 5B73B784
 P 8600 4150
-F 0 "#PWR0321" H 8600 4000 50  0001 C CNN
+F 0 "#PWR0322" H 8600 4000 50  0001 C CNN
 F 1 "+5V" H 8615 4323 50  0000 C CNN
 F 2 "" H 8600 4150 50  0001 C CNN
@@
 Connection ~ 7300 5050
 $Comp
-L power:GND #PWR0314
+L power:GND #PWR0315
 U 1 1 5B73C2A7
 P 7300 5350
-F 0 "#PWR0314" H 7300 5100 50  0001 C CNN
+F 0 "#PWR0315" H 7300 5100 50  0001 C CNN
 F 1 "GND" H 7305 5177 50  0000 C CNN
 F 2 "" H 7300 5350 50  0001 C CNN
@@
 $EndComp
 $Comp
-L power:GND #PWR0317
+L power:GND #PWR0318
 U 1 1 5B73C2C7
 P 8100 4200
-F 0 "#PWR0317" H 8100 3950 50  0001 C CNN
+F 0 "#PWR0318" H 8100 3950 50  0001 C CNN
 F 1 "GND" V 8105 4072 50  0000 R CNN
 F 2 "" H 8100 4200 50  0001 C CNN
@@
 $EndComp
 $Comp
-L power:GND #PWR0322
+L power:GND #PWR0323
 U 1 1 5B73C2E7
 P 8900 4200
-F 0 "#PWR0322" H 8900 3950 50  0001 C CNN
+F 0 "#PWR0323" H 8900 3950 50  0001 C CNN
 F 1 "GND" V 8905 4072 50  0000 R CNN
 F 2 "" H 8900 4200 50  0001 C CNN
@@
 Wiegand_D1
 $Comp
-L power:GND #PWR0320
+L power:GND #PWR0321
 U 1 1 5B73CB5F
 P 8500 5250
-F 0 "#PWR0320" H 8500 5000 50  0001 C CNN
+F 0 "#PWR0321" H 8500 5000 50  0001 C CNN
 F 1 "GND" H 8505 5077 50  0000 C CNN
 F 2 "" H 8500 5250 50  0001 C CNN
@@
 Text GLabel 7550 3300 2    60   Input ~ 0
 ANALOG_I2C_SDA
-Text GLabel 5250 2800 2    60   Input ~ 0
+Text GLabel 5750 2800 2    60   Input ~ 0
 ANALOG_RDY_2
 Text GLabel 5250 3600 2    60   Input ~ 0
@@
 $EndComp
 $Comp
-L power:+3.3V #PWR0312
+L power:+3.3V #PWR0313
 U 1 1 5B741A1B
 P 6700 2650
-F 0 "#PWR0312" H 6700 2500 50  0001 C CNN
+F 0 "#PWR0313" H 6700 2500 50  0001 C CNN
 F 1 "+3.3V" H 6715 2823 50  0000 C CNN
 F 2 "" H 6700 2650 50  0001 C CNN
@@
 Text GLabel 5250 3800 2    60   Input ~ 0
 SIREN_CTRL
-Text Notes 6000 6300 0    50   ~ 0
+Text Notes 5200 6250 0    50   ~ 0
 Check placement of pins so othey\nare easy to wire with flat cable
 $Comp
@@
 	7800 1250 7800 1550
 $Comp
-L power:+3.3V #PWR0323
+L power:+3.3V #PWR0324
 U 1 1 5B73AAEB
 P 9750 1350
-F 0 "#PWR0323" H 9750 1200 50  0001 C CNN
+F 0 "#PWR0324" H 9750 1200 50  0001 C CNN
 F 1 "+3.3V" H 9765 1523 50  0000 C CNN
 F 2 "" H 9750 1350 50  0001 C CNN
@@
 ADDR_2
 $Comp
-L power:GND #PWR0318
+L power:GND #PWR0319
 U 1 1 5B75512D
 P 8350 1950
-F 0 "#PWR0318" H 8350 1700 50  0001 C CNN
+F 0 "#PWR0319" H 8350 1700 50  0001 C CNN
 F 1 "GND" H 8355 1777 50  0000 C CNN
 F 2 "" H 8350 1950 50  0001 C CNN
@@
 $EndComp
 $Comp
-L power:+5V #PWR0315
+L power:+5V #PWR0316
 U 1 1 5B909304
 P 8100 3450
-F 0 "#PWR0315" H 8100 3300 50  0001 C CNN
+F 0 "#PWR0316" H 8100 3300 50  0001 C CNN
 F 1 "+5V" V 8115 3578 50  0000 L CNN
 F 2 "" H 8100 3450 50  0001 C CNN
@@
 $EndComp
 $Comp
-L power:GND #PWR0316
+L power:GND #PWR0317
 U 1 1 5B9093BD
 P 8100 3550
-F 0 "#PWR0316" H 8100 3300 50  0001 C CNN
+F 0 "#PWR0317" H 8100 3300 50  0001 C CNN
 F 1 "GND" V 8105 3422 50  0000 R CNN
 F 2 "" H 8100 3550 50  0001 C CNN
@@
 Wire Wire Line
 	7450 3750 8100 3750
+$Comp
+L Switch:SW_Push SW303
+U 1 1 5B9494D5
+P 6000 2200
+F 0 "SW303" H 6000 2485 50  0000 C CNN
+F 1 "Factory reset" H 6000 2394 50  0000 C CNN
+F 2 "Button_Switch_SMD:SW_SPST_CK_KXT3" H 6000 2400 50  0001 C CNN
+F 3 "https://www.mouser.se/ProductDetail/CK/KXT331LHS?qs=sGAEpiMZZMsgGjVA3toVBICuw%2fFQq%2fBnDsOBIRFitAg%3d" H 6000 2400 50  0001 C CNN
+	1    6000 2200
+	1    0    0    -1
+$EndComp
+Wire Wire Line
+	5250 2800 5650 2800
+Wire Wire Line
+	5800 2200 5650 2200
+Wire Wire Line
+	5650 2200 5650 2800
+Connection ~ 5650 2800
+Wire Wire Line
+	5650 2800 5750 2800
+$Comp
+L power:GND #PWR0312
+U 1 1 5B953711
+P 6200 2200
+F 0 "#PWR0312" H 6200 1950 50  0001 C CNN
+F 1 "GND" H 6205 2027 50  0000 C CNN
+F 2 "" H 6200 2200 50  0001 C CNN
+F 3 "" H 6200 2200 50  0001 C CNN
+	1    6200 2200
+	0    -1   -1   0
+$EndComp
 $EndSCHEMATC

Commit message: UART TX/RX fixed
Connections:
- net labels added: RDX, TDX
- net labels removed: RDX0, TDX0
Other:
- note added: "Near Wrover module"
- note added: "Note: RX<->TX"
- note removed: "Check placement of pins so othey\nare easy to wire with flat cable"
Changed lines of the file:
@@
 Text GLabel 5250 3800 2    60   Input ~ 0
 SIREN_CTRL
-Text Notes 5200 6250 0    50   ~ 0
-Check placement of pins so othey\nare easy to wire with flat cable
 $Comp
 L Connector_Generic:Conn_02x05_Odd_Even J301
@@
 Text Label 2650 2650 0    50   ~ 0
 CH_Enable
-Text Label 5950 5600 0    50   ~ 0
+Text Label 5950 5900 0    50   ~ 0
 MTMS
 Text Label 5950 5700 0    50   ~ 0
 MTDI
-Text Label 5950 5900 0    50   ~ 0
+Text Label 5950 5600 0    50   ~ 0
 MTCK
 Text Label 5950 5800 0    50   ~ 0
 MTDO
-Text Label 2950 2900 0    50   ~ 0
-TDX0
-Text Label 2950 3000 0    50   ~ 0
-RDX0
+Text Label 3000 3000 2    50   ~ 0
+TDX
+Text Label 3000 2900 2    50   ~ 0
+RDX
 Text Label 5950 5500 0    50   ~ 0
 Boot_option
 Text Label 5450 5700 2    50   ~ 0
-TDX0
+TDX
 Text Label 5450 5800 2    50   ~ 0
-RDX0
-Wire Wire Line
-	3250 2900 2950 2900
-Wire Wire Line
-	3250 3000 2950 3000
+RDX
 Text Label 5450 5600 2    50   ~ 0
 CH_Enable
@@
 	0    -1   -1   0
 $EndComp
+Wire Wire Line
+	3000 2900 3250 2900
+Wire Wire Line
+	3000 3000 3250 3000
+Text Notes 2600 3100 0    50   ~ 0
+Note: RX<->TX
+Wire Notes Line
+	2500 2750 3250 2750
+Wire Notes Line
+	3250 2750 3250 3150
+Wire Notes Line
+	3250 3150 2500 3150
+Wire Notes Line
+	2500 3150 2500 2750
+Wire Notes Line
+	3100 1550 3100 900
+Wire Notes Line
+	3100 900  4250 900
+Wire Notes Line
+	4250 900  4250 1550
+Wire Notes Line
+	4250 1550 3100 1550
+Text Notes 3150 1050 0    50   ~ 0
+Near Wrover module
 $EndSCHEMATC

Commit message: Added SDCard slot.
Parts:
- removed J303: Conn_02x03_Counter_Clockwise, Connector_PinHeader_2.54mm:PinHeader_2x03_P2.54mm_Vertical, symbol Connector_Generic:Conn_02x03_Counter_Clockwise
- removed R303, R304, R305, R311, R312, R313: 10k, Resistor_SMD:R_0805_2012Metric, symbol Device:R
- J302: footprint (none) -> Connector_PinHeader_2.54mm:PinHeader_1x04_P2.54mm_Vertical
- renumbered R306 to R303, R307 to R304, R308 to R305, R309 to R306, R310 to R307
Connections:
- net labels added: Factory_reset, SD_CD, SD_CLK, SD_CMD, SD_DATA0, SD_DATA1, SD_DATA2, SD_DATA3
- net labels removed: ADDR_0, ADDR_1, ADDR_2
- wire segments 86 -> 63
Other:
- note added: "Pin layout according to\nESP32-Wrover-kit-debug-breakout"
- note removed: "Optional, solder if not present on the JTAG debugger."

Commit message: Using MAX4948 instead of DIPs
Parts:
- removed R303, R304: 10k, Resistor_SMD:R_0805_2012Metric, symbol Device:R
- added R306, R307: 10k, Resistor_SMD:R_0805_2012Metric, symbol Device:R
- renumbered R305 to R303, R306 to R304, R307 to R305
Connections:
- net labels added: I2C_SCL, I2C_SDA, SD_SPI_CLK, SD_SPI_CS, SD_SPI_MISO, SD_SPI_MOSI
- net labels removed: ANALOG_I2C_SCL, ANALOG_I2C_SDA, BELL_CTRL, DIGITAL_I2C_SCL, DIGITAL_I2C_SDA, SIREN_CTRL
- wire segments 63 -> 55
