File: G3/DigitalInput.sch (KiCad schematic (older format))
At the start: 5 parts, among them U1401 LTV-354T

Commit message: Changed label on signal for digital input schema.
Connections:
- net labels added: ~signal
- net labels removed: O1
Changed lines of the file:
@@
 AR Path="/5B62EDB8/5B68BAA8/5B66E449" Ref="U2001"  Part="1"
 AR Path="/5B62EDB8/5B68D1A7/5B66E449" Ref="U2101"  Part="1"
-F 0 "U1901" H 1650 1825 50  0000 C CNN
+F 0 "U1401" H 1650 1825 50  0000 C CNN
 F 1 "LTV-354T" H 1650 1734 50  0000 C CNN
 F 2 "Package_SO:SO-4_4.4x3.6mm_P2.54mm" H 1450 1300 50  0001 L CIN
@@
 AR Path="/5B62EDB8/5B68BAA8/5B66E450" Ref="R2001"  Part="1"
 AR Path="/5B62EDB8/5B68D1A7/5B66E450" Ref="R2101"  Part="1"
-F 0 "R1901" V 1000 1400 50  0000 C CNN
+F 0 "R1401" V 1000 1400 50  0000 C CNN
 F 1 "1k" V 1100 1400 50  0000 C CNN
 F 2 "Resistor_SMD:R_2512_6332Metric" V 1030 1400 50  0001 C CNN
@@
 AR Path="/5B62EDB8/5B68BAA8/5B66E457" Ref="R2002"  Part="1"
 AR Path="/5B62EDB8/5B68D1A7/5B66E457" Ref="R2102"  Part="1"
-F 0 "R1902" V 2500 1600 50  0000 C CNN
+F 0 "R1402" V 2500 1600 50  0000 C CNN
 F 1 "100" V 2600 1600 50  0000 C CNN
 F 2 "Resistor_SMD:R_0805_2012Metric" V 2530 1600 50  0001 C CNN
@@
 AR Path="/5B62EDB8/5B68BAA8/5B66E45E" Ref="C2001"  Part="1"
 AR Path="/5B62EDB8/5B68D1A7/5B66E45E" Ref="C2101"  Part="1"
-F 0 "C1901" V 2050 1600 50  0000 C CNN
+F 0 "C1401" V 2050 1600 50  0000 C CNN
 F 1 "10u" H 2300 1700 50  0000 C CNN
 F 2 "Capacitor_SMD:CP_Elec_5x4.5" H 2238 1450 50  0001 C CNN
@@
 AR Path="/5B62EDB8/5B68BAA8/5B66E465" Ref="R2003"  Part="1"
 AR Path="/5B62EDB8/5B68D1A7/5B66E465" Ref="R2103"  Part="1"
-F 0 "R1903" H 3150 1350 50  0000 C CNN
+F 0 "R1403" H 3150 1350 50  0000 C CNN
 F 1 "10k" H 3150 1450 50  0000 C CNN
 F 2 "Resistor_SMD:R_0805_2012Metric" V 2930 1400 50  0001 C CNN
@@
 AR Path="/5B62EDB8/5B68BAA8/5B66E46C" Ref="#PWR02001"  Part="1"
 AR Path="/5B62EDB8/5B68D1A7/5B66E46C" Ref="#PWR02101"  Part="1"
-F 0 "#PWR01901" H 2000 1350 50  0001 C CNN
+F 0 "#PWR01401" H 2000 1350 50  0001 C CNN
 F 1 "GND" H 2005 1427 50  0000 C CNN
 F 2 "" H 2000 1600 50  0001 C CNN
@@
 AR Path="/5B62EDB8/5B68BAA8/5B66E473" Ref="#PWR02002"  Part="1"
 AR Path="/5B62EDB8/5B68D1A7/5B66E473" Ref="#PWR02102"  Part="1"
-F 0 "#PWR01902" H 3150 1250 50  0001 C CNN
+F 0 "#PWR01402" H 3150 1250 50  0001 C CNN
 F 1 "+3.3V" V 3165 1528 50  0000 L CNN
 F 2 "" H 3150 1400 50  0001 C CNN
@@
 	950  1600 1350 1600
 Text HLabel 2750 1200 1    50   Output ~ 0
-O1
+~signal
 Wire Wire Line
 	2750 1400 2750 1200

Commit message: Added SDCard slot.
Parts:
- renumbered C1401 to C1501, R1401 to R1501, R1402 to R1502, R1403 to R1503, U1401 to U1501
Changed lines of the file:
@@
 $Descr A4 11693 8268
 encoding utf-8
-Sheet 15 35
+Sheet 15 36
 Title ""
 Date ""
@@
 P 1650 1500
 AR Path="/5B62EDB8/5B66E449" Ref="U?"  Part="1"
-AR Path="/5B62EDB8/5B66E27E/5B66E449" Ref="U1401"  Part="1"
-AR Path="/5B62EDB8/5B66FC5D/5B66E449" Ref="U1501"  Part="1"
-AR Path="/5B62EDB8/5B685B64/5B66E449" Ref="U1601"  Part="1"
-AR Path="/5B62EDB8/5B687263/5B66E449" Ref="U1701"  Part="1"
-AR Path="/5B62EDB8/5B688B1A/5B66E449" Ref="U1801"  Part="1"
-AR Path="/5B62EDB8/5B68A219/5B66E449" Ref="U1901"  Part="1"
-AR Path="/5B62EDB8/5B68BAA8/5B66E449" Ref="U2001"  Part="1"
-AR Path="/5B62EDB8/5B68D1A7/5B66E449" Ref="U2101"  Part="1"
-F 0 "U2101" H 1650 1825 50  0000 C CNN
+AR Path="/5B62EDB8/5B66E27E/5B66E449" Ref="U1501"  Part="1"
+AR Path="/5B62EDB8/5B66FC5D/5B66E449" Ref="U1601"  Part="1"
+AR Path="/5B62EDB8/5B685B64/5B66E449" Ref="U1701"  Part="1"
+AR Path="/5B62EDB8/5B687263/5B66E449" Ref="U1801"  Part="1"
+AR Path="/5B62EDB8/5B688B1A/5B66E449" Ref="U1901"  Part="1"
+AR Path="/5B62EDB8/5B68A219/5B66E449" Ref="U2001"  Part="1"
+AR Path="/5B62EDB8/5B68BAA8/5B66E449" Ref="U2101"  Part="1"
+AR Path="/5B62EDB8/5B68D1A7/5B66E449" Ref="U2201"  Part="1"
+F 0 "U2201" H 1650 1825 50  0000 C CNN
 F 1 "LTV-354T" H 1650 1734 50  0000 C CNN
 F 2 "Package_SO:SO-4_4.4x3.6mm_P2.54mm" H 1450 1300 50  0001 L CIN
@@
 P 1100 1400
 AR Path="/5B62EDB8/5B66E450" Ref="R?"  Part="1"
-AR Path="/5B62EDB8/5B66E27E/5B66E450" Ref="R1401"  Part="1"
-AR Path="/5B62EDB8/5B66FC5D/5B66E450" Ref="R1501"  Part="1"
-AR Path="/5B62EDB8/5B685B64/5B66E450" Ref="R1601"  Part="1"
-AR Path="/5B62EDB8/5B687263/5B66E450" Ref="R1701"  Part="1"
-AR Path="/5B62EDB8/5B688B1A/5B66E450" Ref="R1801"  Part="1"
-AR Path="/5B62EDB8/5B68A219/5B66E450" Ref="R1901"  Part="1"
-AR Path="/5B62EDB8/5B68BAA8/5B66E450" Ref="R2001"  Part="1"
-AR Path="/5B62EDB8/5B68D1A7/5B66E450" Ref="R2101"  Part="1"
-F 0 "R2101" V 1000 1400 50  0000 C CNN
+AR Path="/5B62EDB8/5B66E27E/5B66E450" Ref="R1501"  Part="1"
+AR Path="/5B62EDB8/5B66FC5D/5B66E450" Ref="R1601"  Part="1"
+AR Path="/5B62EDB8/5B685B64/5B66E450" Ref="R1701"  Part="1"
+AR Path="/5B62EDB8/5B687263/5B66E450" Ref="R1801"  Part="1"
+AR Path="/5B62EDB8/5B688B1A/5B66E450" Ref="R1901"  Part="1"
+AR Path="/5B62EDB8/5B68A219/5B66E450" Ref="R2001"  Part="1"
+AR Path="/5B62EDB8/5B68BAA8/5B66E450" Ref="R2101"  Part="1"
+AR Path="/5B62EDB8/5B68D1A7/5B66E450" Ref="R2201"  Part="1"
+F 0 "R2201" V 1000 1400 50  0000 C CNN
 F 1 "1k" V 1100 1400 50  0000 C CNN
 F 2 "Resistor_SMD:R_2512_6332Metric" V 1030 1400 50  0001 C CNN
@@
 P 2600 1600
 AR Path="/5B62EDB8/5B66E457" Ref="R?"  Part="1"
-AR Path="/5B62EDB8/5B66E27E/5B66E457" Ref="R1402"  Part="1"
-AR Path="/5B62EDB8/5B66FC5D/5B66E457" Ref="R1502"  Part="1"
-AR Path="/5B62EDB8/5B685B64/5B66E457" Ref="R1602"  Part="1"
-AR Path="/5B62EDB8/5B687263/5B66E457" Ref="R1702"  Part="1"
-AR Path="/5B62EDB8/5B688B1A/5B66E457" Ref="R1802"  Part="1"
-AR Path="/5B62EDB8/5B68A219/5B66E457" Ref="R1902"  Part="1"
-AR Path="/5B62EDB8/5B68BAA8/5B66E457" Ref="R2002"  Part="1"
-AR Path="/5B62EDB8/5B68D1A7/5B66E457" Ref="R2102"  Part="1"
-F 0 "R2102" V 2500 1600 50  0000 C CNN
+AR Path="/5B62EDB8/5B66E27E/5B66E457" Ref="R1502"  Part="1"
+AR Path="/5B62EDB8/5B66FC5D/5B66E457" Ref="R1602"  Part="1"
+AR Path="/5B62EDB8/5B685B64/5B66E457" Ref="R1702"  Part="1"
+AR Path="/5B62EDB8/5B687263/5B66E457" Ref="R1802"  Part="1"
+AR Path="/5B62EDB8/5B688B1A/5B66E457" Ref="R1902"  Part="1"
+AR Path="/5B62EDB8/5B68A219/5B66E457" Ref="R2002"  Part="1"
+AR Path="/5B62EDB8/5B68BAA8/5B66E457" Ref="R2102"  Part="1"
+AR Path="/5B62EDB8/5B68D1A7/5B66E457" Ref="R2202"  Part="1"
+F 0 "R2202" V 2500 1600 50  0000 C CNN
 F 1 "100" V 2600 1600 50  0000 C CNN
 F 2 "Resistor_SMD:R_0805_2012Metric" V 2530 1600 50  0001 C CNN
@@
 P 2200 1600
 AR Path="/5B62EDB8/5B66E45E" Ref="C?"  Part="1"
-AR Path="/5B62EDB8/5B66E27E/5B66E45E" Ref="C1401"  Part="1"
-AR Path="/5B62EDB8/5B66FC5D/5B66E45E" Ref="C1501"  Part="1"
-AR Path="/5B62EDB8/5B685B64/5B66E45E" Ref="C1601"  Part="1"
-AR Path="/5B62EDB8/5B687263/5B66E45E" Ref="C1701"  Part="1"
-AR Path="/5B62EDB8/5B688B1A/5B66E45E" Ref="C1801"  Part="1"
-AR Path="/5B62EDB8/5B68A219/5B66E45E" Ref="C1901"  Part="1"
-AR Path="/5B62EDB8/5B68BAA8/5B66E45E" Ref="C2001"  Part="1"
-AR Path="/5B62EDB8/5B68D1A7/5B66E45E" Ref="C2101"  Part="1"
-F 0 "C2101" V 2050 1600 50  0000 C CNN
+AR Path="/5B62EDB8/5B66E27E/5B66E45E" Ref="C1501"  Part="1"
+AR Path="/5B62EDB8/5B66FC5D/5B66E45E" Ref="C1601"  Part="1"
+AR Path="/5B62EDB8/5B685B64/5B66E45E" Ref="C1701"  Part="1"
+AR Path="/5B62EDB8/5B687263/5B66E45E" Ref="C1801"  Part="1"
+AR Path="/5B62EDB8/5B688B1A/5B66E45E" Ref="C1901"  Part="1"
+AR Path="/5B62EDB8/5B68A219/5B66E45E" Ref="C2001"  Part="1"
+AR Path="/5B62EDB8/5B68BAA8/5B66E45E" Ref="C2101"  Part="1"
+AR Path="/5B62EDB8/5B68D1A7/5B66E45E" Ref="C2201"  Part="1"
+F 0 "C2201" V 2050 1600 50  0000 C CNN
 F 1 "10u" H 2300 1700 50  0000 C CNN
 F 2 "Capacitor_SMD:CP_Elec_5x4.5" H 2238 1450 50  0001 C CNN
@@
 P 3000 1400
 AR Path="/5B62EDB8/5B66E465" Ref="R?"  Part="1"
-AR Path="/5B62EDB8/5B66E27E/5B66E465" Ref="R1403"  Part="1"
-AR Path="/5B62EDB8/5B66FC5D/5B66E465" Ref="R1503"  Part="1"
-AR Path="/5B62EDB8/5B685B64/5B66E465" Ref="R1603"  Part="1"
-AR Path="/5B62EDB8/5B687263/5B66E465" Ref="R1703"  Part="1"
-AR Path="/5B62EDB8/5B688B1A/5B66E465" Ref="R1803"  Part="1"
-AR Path="/5B62EDB8/5B68A219/5B66E465" Ref="R1903"  Part="1"
-AR Path="/5B62EDB8/5B68BAA8/5B66E465" Ref="R2003"  Part="1"
-AR Path="/5B62EDB8/5B68D1A7/5B66E465" Ref="R2103"  Part="1"
-F 0 "R2103" H 3150 1350 50  0000 C CNN
+AR Path="/5B62EDB8/5B66E27E/5B66E465" Ref="R1503"  Part="1"
+AR Path="/5B62EDB8/5B66FC5D/5B66E465" Ref="R1603"  Part="1"
+AR Path="/5B62EDB8/5B685B64/5B66E465" Ref="R1703"  Part="1"
+AR Path="/5B62EDB8/5B687263/5B66E465" Ref="R1803"  Part="1"
+AR Path="/5B62EDB8/5B688B1A/5B66E465" Ref="R1903"  Part="1"
+AR Path="/5B62EDB8/5B68A219/5B66E465" Ref="R2003"  Part="1"
+AR Path="/5B62EDB8/5B68BAA8/5B66E465" Ref="R2103"  Part="1"
+AR Path="/5B62EDB8/5B68D1A7/5B66E465" Ref="R2203"  Part="1"
+F 0 "R2203" H 3150 1350 50  0000 C CNN
 F 1 "10k" H 3150 1450 50  0000 C CNN
 F 2 "Resistor_SMD:R_0805_2012Metric" V 2930 1400 50  0001 C CNN
-F 3 "" H 3000 1400 50  0001 C CNN
+F 3 "https://www.mouser.se/ProductDetail/Panasonic-Industrial-Devices/ERJ-6ENF1002V?qs=sGAEpiMZZMu61qfTUdNhGzRxdwze5h8ZcGDx6geba20%3d" H 3000 1400 50  0001 C CNN
 	1    3000 1400
 	0    1    1    0
@@
 P 2000 1600
 AR Path="/5B62EDB8/5B66E46C" Ref="#PWR?"  Part="1"
-AR Path="/5B62EDB8/5B66E27E/5B66E46C" Ref="#PWR01401"  Part="1"
-AR Path="/5B62EDB8/5B66FC5D/5B66E46C" Ref="#PWR01501"  Part="1"
-AR Path="/5B62EDB8/5B685B64/5B66E46C" Ref="#PWR01601"  Part="1"
-AR Path="/5B62EDB8/5B687263/5B66E46C" Ref="#PWR01701"  Part="1"
-AR Path="/5B62EDB8/5B688B1A/5B66E46C" Ref="#PWR01801"  Part="1"
-AR Path="/5B62EDB8/5B68A219/5B66E46C" Ref="#PWR01901"  Part="1"
-AR Path="/5B62EDB8/5B68BAA8/5B66E46C" Ref="#PWR02001"  Part="1"
-AR Path="/5B62EDB8/5B68D1A7/5B66E46C" Ref="#PWR02101"  Part="1"
-F 0 "#PWR02101" H 2000 1350 50  0001 C CNN
+AR Path="/5B62EDB8/5B66E27E/5B66E46C" Ref="#PWR01501"  Part="1"
+AR Path="/5B62EDB8/5B66FC5D/5B66E46C" Ref="#PWR01601"  Part="1"
+AR Path="/5B62EDB8/5B685B64/5B66E46C" Ref="#PWR01701"  Part="1"
+AR Path="/5B62EDB8/5B687263/5B66E46C" Ref="#PWR01801"  Part="1"
+AR Path="/5B62EDB8/5B688B1A/5B66E46C" Ref="#PWR01901"  Part="1"
+AR Path="/5B62EDB8/5B68A219/5B66E46C" Ref="#PWR02001"  Part="1"
+AR Path="/5B62EDB8/5B68BAA8/5B66E46C" Ref="#PWR02101"  Part="1"
+AR Path="/5B62EDB8/5B68D1A7/5B66E46C" Ref="#PWR02201"  Part="1"
+F 0 "#PWR02201" H 2000 1350 50  0001 C CNN
 F 1 "GND" H 2005 1427 50  0000 C CNN
 F 2 "" H 2000 1600 50  0001 C CNN
@@
 P 3150 1400
 AR Path="/5B62EDB8/5B66E473" Ref="#PWR?"  Part="1"
-AR Path="/5B62EDB8/5B66E27E/5B66E473" Ref="#PWR01402"  Part="1"
-AR Path="/5B62EDB8/5B66FC5D/5B66E473" Ref="#PWR01502"  Part="1"
-AR Path="/5B62EDB8/5B685B64/5B66E473" Ref="#PWR01602"  Part="1"
-AR Path="/5B62EDB8/5B687263/5B66E473" Ref="#PWR01702"  Part="1"
-AR Path="/5B62EDB8/5B688B1A/5B66E473" Ref="#PWR01802"  Part="1"
-AR Path="/5B62EDB8/5B68A219/5B66E473" Ref="#PWR01902"  Part="1"
-AR Path="/5B62EDB8/5B68BAA8/5B66E473" Ref="#PWR02002"  Part="1"
-AR Path="/5B62EDB8/5B68D1A7/5B66E473" Ref="#PWR02102"  Part="1"
-F 0 "#PWR02102" H 3150 1250 50  0001 C CNN
+AR Path="/5B62EDB8/5B66E27E/5B66E473" Ref="#PWR01502"  Part="1"
+AR Path="/5B62EDB8/5B66FC5D/5B66E473" Ref="#PWR01602"  Part="1"
+AR Path="/5B62EDB8/5B685B64/5B66E473" Ref="#PWR01702"  Part="1"
+AR Path="/5B62EDB8/5B687263/5B66E473" Ref="#PWR01802"  Part="1"
+AR Path="/5B62EDB8/5B688B1A/5B66E473" Ref="#PWR01902"  Part="1"
+AR Path="/5B62EDB8/5B68A219/5B66E473" Ref="#PWR02002"  Part="1"
+AR Path="/5B62EDB8/5B68BAA8/5B66E473" Ref="#PWR02102"  Part="1"
+AR Path="/5B62EDB8/5B68D1A7/5B66E473" Ref="#PWR02202"  Part="1"
+F 0 "#PWR02202" H 3150 1250 50  0001 C CNN
 F 1 "+3.3V" V 3165 1528 50  0000 L CNN
 F 2 "" H 3150 1400 50  0001 C CNN

Commit message: PCB started
Connections:
- net labels added: DI_in, DigitalInput3
- wire segments 9 -> 10
Changed lines of the file:
@@
 L Isolator:LTV-354T U?
 U 1 1 5B66E449
-P 1650 1500
+P 2100 1500
 AR Path="/5B62EDB8/5B66E449" Ref="U?"  Part="1"
 AR Path="/5B62EDB8/5B66E27E/5B66E449" Ref="U1501"  Part="1"
@@
 AR Path="/5B62EDB8/5B68BAA8/5B66E449" Ref="U2101"  Part="1"
 AR Path="/5B62EDB8/5B68D1A7/5B66E449" Ref="U2201"  Part="1"
-F 0 "U2201" H 1650 1825 50  0000 C CNN
-F 1 "LTV-354T" H 1650 1734 50  0000 C CNN
-F 2 "Package_SO:SO-4_4.4x3.6mm_P2.54mm" H 1450 1300 50  0001 L CIN
-F 3 "" H 1675 1500 50  0001 L CNN
-	1    1650 1500
+F 0 "U1501" H 2100 1825 50  0000 C CNN
+F 1 "LTV-354T" H 2100 1734 50  0000 C CNN
+F 2 "Package_SO:SO-4_4.4x3.6mm_P2.54mm" H 1900 1300 50  0001 L CIN
+F 3 "" H 2125 1500 50  0001 L CNN
+	1    2100 1500
 	1    0    0    -1
 $EndComp
@@
 L Device:R R?
 U 1 1 5B66E450
-P 1100 1400
+P 1150 1400
 AR Path="/5B62EDB8/5B66E450" Ref="R?"  Part="1"
 AR Path="/5B62EDB8/5B66E27E/5B66E450" Ref="R1501"  Part="1"
@@
 AR Path="/5B62EDB8/5B68BAA8/5B66E450" Ref="R2101"  Part="1"
 AR Path="/5B62EDB8/5B68D1A7/5B66E450" Ref="R2201"  Part="1"
-F 0 "R2201" V 1000 1400 50  0000 C CNN
-F 1 "1k" V 1100 1400 50  0000 C CNN
-F 2 "Resistor_SMD:R_2512_6332Metric" V 1030 1400 50  0001 C CNN
-F 3 "" H 1100 1400 50  0001 C CNN
-	1    1100 1400
+F 0 "R1501" V 1050 1400 50  0000 C CNN
+F 1 "1k" V 1150 1400 50  0000 C CNN
+F 2 "Resistor_SMD:R_2512_6332Metric" V 1080 1400 50  0001 C CNN
+F 3 "" H 1150 1400 50  0001 C CNN
+	1    1150 1400
 	0    1    1    0
 $EndComp
@@
 L Device:R R?
 U 1 1 5B66E457
-P 2600 1600
+P 3050 1600
 AR Path="/5B62EDB8/5B66E457" Ref="R?"  Part="1"
 AR Path="/5B62EDB8/5B66E27E/5B66E457" Ref="R1502"  Part="1"
@@
 AR Path="/5B62EDB8/5B68BAA8/5B66E457" Ref="R2102"  Part="1"
 AR Path="/5B62EDB8/5B68D1A7/5B66E457" Ref="R2202"  Part="1"
-F 0 "R2202" V 2500 1600 50  0000 C CNN
-F 1 "100" V 2600 1600 50  0000 C CNN
-F 2 "Resistor_SMD:R_0805_2012Metric" V 2530 1600 50  0001 C CNN
-F 3 "" H 2600 1600 50  0001 C CNN
-	1    2600 1600
+F 0 "R1502" V 2950 1600 50  0000 C CNN
+F 1 "100" V 3050 1600 50  0000 C CNN
+F 2 "Resistor_SMD:R_0805_2012Metric" V 2980 1600 50  0001 C CNN
+F 3 "" H 3050 1600 50  0001 C CNN
+	1    3050 1600
 	0    1    1    0
 $EndComp
@@
 L Device:CP C?
 U 1 1 5B66E45E
-P 2200 1600
+P 2650 1600
 AR Path="/5B62EDB8/5B66E45E" Ref="C?"  Part="1"
 AR Path="/5B62EDB8/5B66E27E/5B66E45E" Ref="C1501"  Part="1"
@@
 AR Path="/5B62EDB8/5B68BAA8/5B66E45E" Ref="C2101"  Part="1"
 AR Path="/5B62EDB8/5B68D1A7/5B66E45E" Ref="C2201"  Part="1"
-F 0 "C2201" V 2050 1600 50  0000 C CNN
-F 1 "10u" H 2300 1700 50  0000 C CNN
-F 2 "Capacitor_SMD:CP_Elec_5x4.5" H 2238 1450 50  0001 C CNN
-F 3 "" H 2200 1600 50  0001 C CNN
-	1    2200 1600
+F 0 "C1501" V 2500 1600 50  0000 C CNN
+F 1 "10u" H 2750 1700 50  0000 C CNN
+F 2 "Capacitor_SMD:CP_Elec_5x4.5" H 2688 1450 50  0001 C CNN
+F 3 "" H 2650 1600 50  0001 C CNN
+	1    2650 1600
 	0    1    1    0
 $EndComp
@@
 L Device:R R?
 U 1 1 5B66E465
-P 3000 1400
+P 3450 1400
 AR Path="/5B62EDB8/5B66E465" Ref="R?"  Part="1"
 AR Path="/5B62EDB8/5B66E27E/5B66E465" Ref="R1503"  Part="1"
@@
 AR Path="/5B62EDB8/5B68BAA8/5B66E465" Ref="R2103"  Part="1"
 AR Path="/5B62EDB8/5B68D1A7/5B66E465" Ref="R2203"  Part="1"
-F 0 "R2203" H 3150 1350 50  0000 C CNN
-F 1 "10k" H 3150 1450 50  0000 C CNN
-F 2 "Resistor_SMD:R_0805_2012Metric" V 2930 1400 50  0001 C CNN
-F 3 "https://www.mouser.se/ProductDetail/Panasonic-Industrial-Devices/ERJ-6ENF1002V?qs=sGAEpiMZZMu61qfTUdNhGzRxdwze5h8ZcGDx6geba20%3d" H 3000 1400 50  0001 C CNN
-	1    3000 1400
+F 0 "R1503" H 3600 1350 50  0000 C CNN
+F 1 "10k" H 3600 1450 50  0000 C CNN
+F 2 "Resistor_SMD:R_0805_2012Metric" V 3380 1400 50  0001 C CNN
+F 3 "https://www.mouser.se/ProductDetail/Panasonic-Industrial-Devices/ERJ-6ENF1002V?qs=sGAEpiMZZMu61qfTUdNhGzRxdwze5h8ZcGDx6geba20%3d" H 3450 1400 50  0001 C CNN
+	1    3450 1400
 	0    1    1    0
 $EndComp
@@
 L power:GND #PWR?
 U 1 1 5B66E46C
-P 2000 1600
+P 2450 1600
 AR Path="/5B62EDB8/5B66E46C" Ref="#PWR?"  Part="1"
 AR Path="/5B62EDB8/5B66E27E/5B66E46C" Ref="#PWR01501"  Part="1"
@@
 AR Path="/5B62EDB8/5B68BAA8/5B66E46C" Ref="#PWR02101"  Part="1"
 AR Path="/5B62EDB8/5B68D1A7/5B66E46C" Ref="#PWR02201"  Part="1"
-F 0 "#PWR02201" H 2000 1350 50  0001 C CNN
-F 1 "GND" H 2005 1427 50  0000 C CNN
-F 2 "" H 2000 1600 50  0001 C CNN
-F 3 "" H 2000 1600 50  0001 C CNN
-	1    2000 1600
+F 0 "#PWR02201" H 2450 1350 50  0001 C CNN
+F 1 "GND" H 2455 1427 50  0000 C CNN
+F 2 "" H 2450 1600 50  0001 C CNN
+F 3 "" H 2450 1600 50  0001 C CNN
+	1    2450 1600
 	1    0    0    -1
 $EndComp
@@
 L power:+3.3V #PWR?
 U 1 1 5B66E473
-P 3150 1400
+P 3600 1400
 AR Path="/5B62EDB8/5B66E473" Ref="#PWR?"  Part="1"
 AR Path="/5B62EDB8/5B66E27E/5B66E473" Ref="#PWR01502"  Part="1"
@@
 AR Path="/5B62EDB8/5B68BAA8/5B66E473" Ref="#PWR02102"  Part="1"
 AR Path="/5B62EDB8/5B68D1A7/5B66E473" Ref="#PWR02202"  Part="1"
-F 0 "#PWR02202" H 3150 1250 50  0001 C CNN
-F 1 "+3.3V" V 3165 1528 50  0000 L CNN
-F 2 "" H 3150 1400 50  0001 C CNN
-F 3 "" H 3150 1400 50  0001 C CNN
-	1    3150 1400
+F 0 "#PWR02202" H 3600 1250 50  0001 C CNN
+F 1 "+3.3V" V 3615 1528 50  0000 L CNN
+F 2 "" H 3600 1400 50  0001 C CNN
+F 3 "" H 3600 1400 50  0001 C CNN
+	1    3600 1400
 	0    1    1    0
 $EndComp
 Wire Wire Line
-	1350 1400 1250 1400
+	1800 1400 1300 1400
 Wire Wire Line
-	2750 1600 2750 1400
+	3200 1600 3200 1400
 Wire Wire Line
-	1950 1400 2750 1400
+	2400 1400 3200 1400
 Wire Wire Line
-	1950 1600 2000 1600
+	2400 1600 2450 1600
 Wire Wire Line
-	2350 1600 2450 1600
-Connection ~ 2000 1600
-Connection ~ 2750 1400
+	2800 1600 2900 1600
+Connection ~ 2450 1600
+Connection ~ 3200 1400
 Wire Wire Line
-	2000 1600 2050 1600
+	2450 1600 2500 1600
 Wire Wire Line
-	2750 1400 2850 1400
-Text HLabel 950  1400 0    50   BiDi ~ 0
+	3200 1400 3300 1400
+Text HLabel 750  1400 0    50   BiDi ~ 0
 In1
-Text HLabel 950  1600 0    50   BiDi ~ 0
+Text HLabel 750  1600 0    50   BiDi ~ 0
 In2
-Wire Wire Line
-	950  1600 1350 1600
-Text HLabel 2750 1200 1    50   Output ~ 0
+Text HLabel 3200 1200 1    50   Output ~ 0
 ~signal
 Wire Wire Line
-	2750 1400 2750 1200
-Text Notes 1000 1100 0    60   ~ 0
+	3200 1400 3200 1200
+Text Notes 1450 1100 0    60   ~ 0
 Select input resistor based on input voltage.\nMax 50mA.\n1k should allow for \nvoltages 3.3 - 48V\n2.4W
+Wire Wire Line
+	1000 1400 750  1400
+Text Label 1300 1400 0    50   ~ 0
+DI_in
+Text Label 900  1400 1    50   ~ 0
+DigitalInput3
+Wire Wire Line
+	750  1600 1800 1600
 $EndSCHEMATC

Commit message: Changes to input and outputs
Parts:
- added D1501: Red, LED_THT:LED_D5.0mm_Clear, symbol Device:LED
- added F1501: xA, Fuse:Fuseholder_TR5_Littlefuse_No560_No460, symbol Device:Fuse
- added J1501: Digital input supply, Connector_PinHeader_2.54mm:PinHeader_1x03_P2.54mm_Vertical, symbol Connector_Generic:Conn_01x03
- added J1502: Digital input GND, Connector_PinHeader_2.54mm:PinHeader_1x02_P2.54mm_Vertical_SMD_Pin1Left, symbol Connector_Generic:Conn_01x02
- added R1502: 165, Resistor_SMD:R_0805_2012Metric, symbol Device:R
- renumbered R1502 to R1503, R1503 to R1504
Connections:
- net labels added: +3V3, +5V, 12V_PWR, DI_in1, DI_in2, Pwr
- net labels removed: DI_in, DigitalInput3
- wire segments 10 -> 15
Other:
- note added: "Either connect a dry contact between Pwr and In1 and enable \npower and ground jumpers, or disable both jumpers and feed\nIn1 and In2 from external source."
- note added: "Select input resistor based on input voltage.\nMax 50mA.\n1k should allow for voltages 3.3 - 48V\n2.4W"
- note removed: "Select input resistor based on input voltage.\nMax 50mA.\n1k should allow for \nvoltages 3.3 - 48V\n2.4W"
