File: G3/StatusIndication.sch (KiCad schematic (older format))
At the start: 32 parts

Commit message: More touch ups
Parts:
- renumbered D3001 to D2301, D3002 to D2302, D3003 to D2303, D3004 to D2304, D3005 to D2305, D3006 to D2306, D3007 to D2307, D3008 to D2308, D3009 to D2309, D3010 to D2310, D3011 to D2311, D3012 to D2312, D3013 to D2313, D3014 to D2314, D3015 to D2315, D3016 to D2316, R3001 to R2301, R3002 to R2302, R3003 to R2303, R3004 to R2304, R3005 to R2305, R3006 to R2306, R3007 to R2307, R3008 to R2308, R3009 to R2309, R3010 to R2310, R3011 to R2311, R3012 to R2312, R3013 to R2313, R3014 to R2314, R3015 to R2315, R3016 to R2316
Changed lines of the file:
@@
 $EndDescr
 $Comp
-L Device:R R3001
+L Device:R R2301
 U 1 1 5B780F33
 P 3000 1800
-F 0 "R3001" V 2793 1800 50  0000 C CNN
+F 0 "R2301" V 2793 1800 50  0000 C CNN
 F 1 "165" V 2884 1800 50  0000 C CNN
 F 2 "Resistor_SMD:R_0805_2012Metric" V 2930 1800 50  0001 C CNN
@@
 $EndComp
 $Comp
-L Device:LED D3001
+L Device:LED D2301
 U 1 1 5B780FD6
 P 3400 1800
-F 0 "D3001" H 3392 1545 50  0000 C CNN
+F 0 "D2301" H 3392 1545 50  0000 C CNN
 F 1 "Green" H 3392 1636 50  0000 C CNN
 F 2 "LED_THT:LED_D5.0mm_Clear" H 3400 1800 50  0001 C CNN
@@
 $EndComp
 $Comp
-L power:+3V3 #PWR03001
+L power:+3V3 #PWR02301
 U 1 1 5B78108C
 P 2850 1800
-F 0 "#PWR03001" H 2850 1650 50  0001 C CNN
+F 0 "#PWR02301" H 2850 1650 50  0001 C CNN
 F 1 "+3V3" V 2865 1928 50  0000 L CNN
 F 2 "" H 2850 1800 50  0001 C CNN
@@
 	3550 1800 3750 1800
 $Comp
-L Device:LED D3009
+L Device:LED D2309
 U 1 1 5B781A9E
 P 5500 1800
-F 0 "D3009" H 5492 1545 50  0000 C CNN
+F 0 "D2309" H 5492 1545 50  0000 C CNN
 F 1 "Red" H 5492 1636 50  0000 C CNN
 F 2 "LED_THT:LED_D5.0mm_Clear" H 5500 1800 50  0001 C CNN
@@
 	5650 1800 5850 1800
 $Comp
-L Device:R R3009
+L Device:R R2309
 U 1 1 5B7821D4
 P 5100 1800
-F 0 "R3009" V 4893 1800 50  0000 C CNN
+F 0 "R2309" V 4893 1800 50  0000 C CNN
 F 1 "165" V 4984 1800 50  0000 C CNN
 F 2 "Resistor_SMD:R_0805_2012Metric" V 5030 1800 50  0001 C CNN
@@
 $EndComp
 $Comp
-L Device:R R3002
+L Device:R R2302
 U 1 1 5B78227E
 P 3000 2200
-F 0 "R3002" V 2793 2200 50  0000 C CNN
+F 0 "R2302" V 2793 2200 50  0000 C CNN
 F 1 "165" V 2884 2200 50  0000 C CNN
 F 2 "Resistor_SMD:R_0805_2012Metric" V 2930 2200 50  0001 C CNN
@@
 $EndComp
 $Comp
-L Device:LED D3002
+L Device:LED D2302
 U 1 1 5B782285
 P 3400 2200
-F 0 "D3002" H 3392 1945 50  0000 C CNN
+F 0 "D2302" H 3392 1945 50  0000 C CNN
 F 1 "Green" H 3392 2036 50  0000 C CNN
 F 2 "LED_THT:LED_D5.0mm_Clear" H 3400 2200 50  0001 C CNN
@@
 	3550 2200 3750 2200
 $Comp
-L Device:R R3003
+L Device:R R2303
 U 1 1 5B782300
 P 3000 2650
-F 0 "R3003" V 2793 2650 50  0000 C CNN
+F 0 "R2303" V 2793 2650 50  0000 C CNN
 F 1 "165" V 2884 2650 50  0000 C CNN
 F 2 "Resistor_SMD:R_0805_2012Metric" V 2930 2650 50  0001 C CNN
@@
 $EndComp
 $Comp
-L Device:LED D3003
+L Device:LED D2303
 U 1 1 5B782307
 P 3400 2650
-F 0 "D3003" H 3392 2395 50  0000 C CNN
+F 0 "D2303" H 3392 2395 50  0000 C CNN
 F 1 "Green" H 3392 2486 50  0000 C CNN
 F 2 "LED_THT:LED_D5.0mm_Clear" H 3400 2650 50  0001 C CNN
@@
 	3550 2650 3750 2650
 $Comp
-L Device:R R3004
+L Device:R R2304
 U 1 1 5B782445
 P 3000 3150
-F 0 "R3004" V 2793 3150 50  0000 C CNN
+F 0 "R2304" V 2793 3150 50  0000 C CNN
 F 1 "165" V 2884 3150 50  0000 C CNN
 F 2 "Resistor_SMD:R_0805_2012Metric" V 2930 3150 50  0001 C CNN
@@
 $EndComp
 $Comp
-L Device:LED D3004
+L Device:LED D2304
 U 1 1 5B78244C
 P 3400 3150
-F 0 "D3004" H 3392 2895 50  0000 C CNN
+F 0 "D2304" H 3392 2895 50  0000 C CNN
 F 1 "Green" H 3392 2986 50  0000 C CNN
 F 2 "LED_THT:LED_D5.0mm_Clear" H 3400 3150 50  0001 C CNN
@@
 	3550 3150 3750 3150
 $Comp
-L Device:R R3005
+L Device:R R2305
 U 1 1 5B782544
 P 3000 3600
-F 0 "R3005" V 2793 3600 50  0000 C CNN
+F 0 "R2305" V 2793 3600 50  0000 C CNN
 F 1 "165" V 2884 3600 50  0000 C CNN
 F 2 "Resistor_SMD:R_0805_2012Metric" V 2930 3600 50  0001 C CNN
@@
 $EndComp
 $Comp
-L Device:LED D3005
+L Device:LED D2305
 U 1 1 5B78254B
 P 3400 3600
-F 0 "D3005" H 3392 3345 50  0000 C CNN
+F 0 "D2305" H 3392 3345 50  0000 C CNN
 F 1 "Green" H 3392 3436 50  0000 C CNN
 F 2 "LED_THT:LED_D5.0mm_Clear" H 3400 3600 50  0001 C CNN
@@
 	3550 3600 3750 3600
 $Comp
-L Device:R R3006
+L Device:R R2306
 U 1 1 5B78269C
 P 3000 4050
-F 0 "R3006" V 2793 4050 50  0000 C CNN
+F 0 "R2306" V 2793 4050 50  0000 C CNN
 F 1 "165" V 2884 4050 50  0000 C CNN
 F 2 "Resistor_SMD:R_0805_2012Metric" V 2930 4050 50  0001 C CNN
@@
 $EndComp
 $Comp
-L Device:LED D3006
+L Device:LED D2306
 U 1 1 5B7826A3
 P 3400 4050
-F 0 "D3006" H 3392 3795 50  0000 C CNN
+F 0 "D2306" H 3392 3795 50  0000 C CNN
 F 1 "Green" H 3392 3886 50  0000 C CNN
 F 2 "LED_THT:LED_D5.0mm_Clear" H 3400 4050 50  0001 C CNN
@@
 	3550 4050 3750 4050
 $Comp
-L Device:R R3007
+L Device:R R2307
 U 1 1 5B78285C
 P 3000 4500
-F 0 "R3007" V 2793 4500 50  0000 C CNN
+F 0 "R2307" V 2793 4500 50  0000 C CNN
 F 1 "165" V 2884 4500 50  0000 C CNN
 F 2 "Resistor_SMD:R_0805_2012Metric" V 2930 4500 50  0001 C CNN
@@
 $EndComp
 $Comp
-L Device:LED D3007
+L Device:LED D2307
 U 1 1 5B782863
 P 3400 4500
-F 0 "D3007" H 3392 4245 50  0000 C CNN
+F 0 "D2307" H 3392 4245 50  0000 C CNN
 F 1 "Green" H 3392 4336 50  0000 C CNN
 F 2 "LED_THT:LED_D5.0mm_Clear" H 3400 4500 50  0001 C CNN
@@
 	3550 4500 3750 4500
 $Comp
-L Device:R R3008
+L Device:R R2308
 U 1 1 5B782A93
 P 3000 4950
-F 0 "R3008" V 2793 4950 50  0000 C CNN
+F 0 "R2308" V 2793 4950 50  0000 C CNN
 F 1 "165" V 2884 4950 50  0000 C CNN
 F 2 "Resistor_SMD:R_0805_2012Metric" V 2930 4950 50  0001 C CNN
@@
 $EndComp
 $Comp
-L Device:LED D3008
+L Device:LED D2308
 U 1 1 5B782A9A
 P 3400 4950
-F 0 "D3008" H 3392 4695 50  0000 C CNN
+F 0 "D2308" H 3392 4695 50  0000 C CNN
 F 1 "Green" H 3392 4786 50  0000 C CNN
 F 2 "LED_THT:LED_D5.0mm_Clear" H 3400 4950 50  0001 C CNN
@@
 	3550 4950 3750 4950
 $Comp
-L Device:LED D3010
+L Device:LED D2310
 U 1 1 5B782D8A
 P 5500 2200
-F 0 "D3010" H 5492 1945 50  0000 C CNN
+F 0 "D2310" H 5492 1945 50  0000 C CNN
 F 1 "Red" H 5492 2036 50  0000 C CNN
 F 2 "LED_THT:LED_D5.0mm_Clear" H 5500 2200 50  0001 C CNN
@@
 	5650 2200 5850 2200
 $Comp
-L Device:R R3010
+L Device:R R2310
 U 1 1 5B782D93
 P 5100 2200
-F 0 "R3010" V 4893 2200 50  0000 C CNN
+F 0 "R2310" V 4893 2200 50  0000 C CNN
 F 1 "165" V 4984 2200 50  0000 C CNN
 F 2 "Resistor_SMD:R_0805_2012Metric" V 5030 2200 50  0001 C CNN
@@
 $EndComp
 $Comp
-L Device:LED D3011
+L Device:LED D2311
 U 1 1 5B7830C7
 P 5500 2700
-F 0 "D3011" H 5492 2445 50  0000 C CNN
+F 0 "D2311" H 5492 2445 50  0000 C CNN
 F 1 "Red" H 5492 2536 50  0000 C CNN
 F 2 "LED_THT:LED_D5.0mm_Clear" H 5500 2700 50  0001 C CNN
@@
 	5650 2700 5850 2700
 $Comp
-L Device:R R3011
+L Device:R R2311
 U 1 1 5B7830D0
 P 5100 2700
-F 0 "R3011" V 4893 2700 50  0000 C CNN
+F 0 "R2311" V 4893 2700 50  0000 C CNN
 F 1 "165" V 4984 2700 50  0000 C CNN
 F 2 "Resistor_SMD:R_0805_2012Metric" V 5030 2700 50  0001 C CNN
@@
 $EndComp
 $Comp
-L Device:LED D3012
+L Device:LED D2312
 U 1 1 5B78347B
 P 5500 3150
-F 0 "D3012" H 5492 2895 50  0000 C CNN
+F 0 "D2312" H 5492 2895 50  0000 C CNN
 F 1 "Red" H 5492 2986 50  0000 C CNN
 F 2 "LED_THT:LED_D5.0mm_Clear" H 5500 3150 50  0001 C CNN
@@
 	5650 3150 5850 3150
 $Comp
-L Device:R R3012
+L Device:R R2312
 U 1 1 5B783484
 P 5100 3150
-F 0 "R3012" V 4893 3150 50  0000 C CNN
+F 0 "R2312" V 4893 3150 50  0000 C CNN
 F 1 "165" V 4984 3150 50  0000 C CNN
 F 2 "Resistor_SMD:R_0805_2012Metric" V 5030 3150 50  0001 C CNN
@@
 $EndComp
 $Comp
-L Device:LED D3013
+L Device:LED D2313
 U 1 1 5B7838C9
 P 5500 3600
-F 0 "D3013" H 5492 3345 50  0000 C CNN
+F 0 "D2313" H 5492 3345 50  0000 C CNN
 F 1 "Red" H 5492 3436 50  0000 C CNN
 F 2 "LED_THT:LED_D5.0mm_Clear" H 5500 3600 50  0001 C CNN
@@
 	5650 3600 5850 3600
 $Comp
-L Device:R R3013
+L Device:R R2313
 U 1 1 5B7838D2
 P 5100 3600
-F 0 "R3013" V 4893 3600 50  0000 C CNN
+F 0 "R2313" V 4893 3600 50  0000 C CNN
 F 1 "165" V 4984 3600 50  0000 C CNN
 F 2 "Resistor_SMD:R_0805_2012Metric" V 5030 3600 50  0001 C CNN
@@
 $EndComp
 $Comp
-L Device:LED D3014
+L Device:LED D2314
 U 1 1 5B783DB0
 P 5500 4050
-F 0 "D3014" H 5492 3795 50  0000 C CNN
+F 0 "D2314" H 5492 3795 50  0000 C CNN
 F 1 "Red" H 5492 3886 50  0000 C CNN
 F 2 "LED_THT:LED_D5.0mm_Clear" H 5500 4050 50  0001 C CNN
@@
 	5650 4050 5850 4050
 $Comp
-L Device:R R3014
+L Device:R R2314
 U 1 1 5B783DB9
 P 5100 4050
-F 0 "R3014" V 4893 4050 50  0000 C CNN
+F 0 "R2314" V 4893 4050 50  0000 C CNN
 F 1 "165" V 4984 4050 50  0000 C CNN
 F 2 "Resistor_SMD:R_0805_2012Metric" V 5030 4050 50  0001 C CNN
@@
 $EndComp
 $Comp
-L Device:LED D3015
+L Device:LED D2315
 U 1 1 5B784347
 P 5500 4500
-F 0 "D3015" H 5492 4245 50  0000 C CNN
+F 0 "D2315" H 5492 4245 50  0000 C CNN
 F 1 "Red" H 5492 4336 50  0000 C CNN
 F 2 "LED_THT:LED_D5.0mm_Clear" H 5500 4500 50  0001 C CNN
@@
 	5650 4500 5850 4500
 $Comp
-L Device:R R3015
+L Device:R R2315
 U 1 1 5B784350
 P 5100 4500
-F 0 "R3015" V 4893 4500 50  0000 C CNN
+F 0 "R2315" V 4893 4500 50  0000 C CNN
 F 1 "165" V 4984 4500 50  0000 C CNN
 F 2 "Resistor_SMD:R_0805_2012Metric" V 5030 4500 50  0001 C CNN
@@
 $EndComp
 $Comp
-L Device:LED D3016
+L Device:LED D2316
 U 1 1 5B7849A5
 P 5500 5000
-F 0 "D3016" H 5492 4745 50  0000 C CNN
+F 0 "D2316" H 5492 4745 50  0000 C CNN
 F 1 "Red" H 5492 4836 50  0000 C CNN
 F 2 "LED_THT:LED_D5.0mm_Clear" H 5500 5000 50  0001 C CNN
@@
 	5650 5000 5850 5000
 $Comp
-L Device:R R3016
+L Device:R R2316
 U 1 1 5B7849AE
 P 5100 5000
-F 0 "R3016" V 4893 5000 50  0000 C CNN
+F 0 "R2316" V 4893 5000 50  0000 C CNN
 F 1 "165" V 4984 5000 50  0000 C CNN
 F 2 "Resistor_SMD:R_0805_2012Metric" V 5030 5000 50  0001 C CNN
@@
 	2850 4500 2850 4950
 $Comp
-L power:+3V3 #PWR03002
+L power:+3V3 #PWR02302
 U 1 1 5B787261
 P 4950 1800
-F 0 "#PWR03002" H 4950 1650 50  0001 C CNN
+F 0 "#PWR02302" H 4950 1650 50  0001 C CNN
 F 1 "+3V3" V 4965 1928 50  0000 L CNN
 F 2 "" H 4950 1800 50  0001 C CNN

Commit message: Added SDCard slot.
Parts:
- renumbered D2301 to D2401, D2302 to D2402, D2303 to D2403, D2304 to D2404, D2305 to D2405, D2306 to D2406, D2307 to D2407, D2308 to D2408, D2309 to D2409, D2310 to D2410, D2311 to D2411, D2312 to D2412, D2313 to D2413, D2314 to D2414, D2315 to D2415, D2316 to D2416, R2301 to R2401, R2302 to R2402, R2303 to R2403, R2304 to R2404, R2305 to R2405, R2306 to R2406, R2307 to R2407, R2308 to R2408, R2309 to R2409, R2310 to R2410, R2311 to R2411, R2312 to R2412, R2313 to R2413, R2314 to R2414, R2315 to R2415, R2316 to R2416
Changed lines of the file:
@@
 $Descr A4 11693 8268
 encoding utf-8
-Sheet 30 35
+Sheet 30 36
 Title ""
 Date ""
@@
 $EndDescr
 $Comp
-L Device:R R2301
+L Device:R R2401
 U 1 1 5B780F33
 P 3000 1800
-F 0 "R2301" V 2793 1800 50  0000 C CNN
+F 0 "R2401" V 2793 1800 50  0000 C CNN
 F 1 "165" V 2884 1800 50  0000 C CNN
 F 2 "Resistor_SMD:R_0805_2012Metric" V 2930 1800 50  0001 C CNN
@@
 $EndComp
 $Comp
-L Device:LED D2301
+L Device:LED D2401
 U 1 1 5B780FD6
 P 3400 1800
-F 0 "D2301" H 3392 1545 50  0000 C CNN
+F 0 "D2401" H 3392 1545 50  0000 C CNN
 F 1 "Green" H 3392 1636 50  0000 C CNN
 F 2 "LED_THT:LED_D5.0mm_Clear" H 3400 1800 50  0001 C CNN
@@
 $EndComp
 $Comp
-L power:+3V3 #PWR02301
+L power:+3V3 #PWR02401
 U 1 1 5B78108C
 P 2850 1800
-F 0 "#PWR02301" H 2850 1650 50  0001 C CNN
+F 0 "#PWR02401" H 2850 1650 50  0001 C CNN
 F 1 "+3V3" V 2865 1928 50  0000 L CNN
 F 2 "" H 2850 1800 50  0001 C CNN
@@
 	3550 1800 3750 1800
 $Comp
-L Device:LED D2309
+L Device:LED D2409
 U 1 1 5B781A9E
 P 5500 1800
-F 0 "D2309" H 5492 1545 50  0000 C CNN
+F 0 "D2409" H 5492 1545 50  0000 C CNN
 F 1 "Red" H 5492 1636 50  0000 C CNN
 F 2 "LED_THT:LED_D5.0mm_Clear" H 5500 1800 50  0001 C CNN
@@
 	5650 1800 5850 1800
 $Comp
-L Device:R R2309
+L Device:R R2409
 U 1 1 5B7821D4
 P 5100 1800
-F 0 "R2309" V 4893 1800 50  0000 C CNN
+F 0 "R2409" V 4893 1800 50  0000 C CNN
 F 1 "165" V 4984 1800 50  0000 C CNN
 F 2 "Resistor_SMD:R_0805_2012Metric" V 5030 1800 50  0001 C CNN
@@
 $EndComp
 $Comp
-L Device:R R2302
+L Device:R R2402
 U 1 1 5B78227E
 P 3000 2200
-F 0 "R2302" V 2793 2200 50  0000 C CNN
+F 0 "R2402" V 2793 2200 50  0000 C CNN
 F 1 "165" V 2884 2200 50  0000 C CNN
 F 2 "Resistor_SMD:R_0805_2012Metric" V 2930 2200 50  0001 C CNN
@@
 $EndComp
 $Comp
-L Device:LED D2302
+L Device:LED D2402
 U 1 1 5B782285
 P 3400 2200
-F 0 "D2302" H 3392 1945 50  0000 C CNN
+F 0 "D2402" H 3392 1945 50  0000 C CNN
 F 1 "Green" H 3392 2036 50  0000 C CNN
 F 2 "LED_THT:LED_D5.0mm_Clear" H 3400 2200 50  0001 C CNN
@@
 	3550 2200 3750 2200
 $Comp
-L Device:R R2303
+L Device:R R2403
 U 1 1 5B782300
 P 3000 2650
-F 0 "R2303" V 2793 2650 50  0000 C CNN
+F 0 "R2403" V 2793 2650 50  0000 C CNN
 F 1 "165" V 2884 2650 50  0000 C CNN
 F 2 "Resistor_SMD:R_0805_2012Metric" V 2930 2650 50  0001 C CNN
@@
 $EndComp
 $Comp
-L Device:LED D2303
+L Device:LED D2403
 U 1 1 5B782307
 P 3400 2650
-F 0 "D2303" H 3392 2395 50  0000 C CNN
+F 0 "D2403" H 3392 2395 50  0000 C CNN
 F 1 "Green" H 3392 2486 50  0000 C CNN
 F 2 "LED_THT:LED_D5.0mm_Clear" H 3400 2650 50  0001 C CNN
@@
 	3550 2650 3750 2650
 $Comp
-L Device:R R2304
+L Device:R R2404
 U 1 1 5B782445
 P 3000 3150
-F 0 "R2304" V 2793 3150 50  0000 C CNN
+F 0 "R2404" V 2793 3150 50  0000 C CNN
 F 1 "165" V 2884 3150 50  0000 C CNN
 F 2 "Resistor_SMD:R_0805_2012Metric" V 2930 3150 50  0001 C CNN
@@
 $EndComp
 $Comp
-L Device:LED D2304
+L Device:LED D2404
 U 1 1 5B78244C
 P 3400 3150
-F 0 "D2304" H 3392 2895 50  0000 C CNN
+F 0 "D2404" H 3392 2895 50  0000 C CNN
 F 1 "Green" H 3392 2986 50  0000 C CNN
 F 2 "LED_THT:LED_D5.0mm_Clear" H 3400 3150 50  0001 C CNN
@@
 	3550 3150 3750 3150
 $Comp
-L Device:R R2305
+L Device:R R2405
 U 1 1 5B782544
 P 3000 3600
-F 0 "R2305" V 2793 3600 50  0000 C CNN
+F 0 "R2405" V 2793 3600 50  0000 C CNN
 F 1 "165" V 2884 3600 50  0000 C CNN
 F 2 "Resistor_SMD:R_0805_2012Metric" V 2930 3600 50  0001 C CNN
@@
 $EndComp
 $Comp
-L Device:LED D2305
+L Device:LED D2405
 U 1 1 5B78254B
 P 3400 3600
-F 0 "D2305" H 3392 3345 50  0000 C CNN
+F 0 "D2405" H 3392 3345 50  0000 C CNN
 F 1 "Green" H 3392 3436 50  0000 C CNN
 F 2 "LED_THT:LED_D5.0mm_Clear" H 3400 3600 50  0001 C CNN
@@
 	3550 3600 3750 3600
 $Comp
-L Device:R R2306
+L Device:R R2406
 U 1 1 5B78269C
 P 3000 4050
-F 0 "R2306" V 2793 4050 50  0000 C CNN
+F 0 "R2406" V 2793 4050 50  0000 C CNN
 F 1 "165" V 2884 4050 50  0000 C CNN
 F 2 "Resistor_SMD:R_0805_2012Metric" V 2930 4050 50  0001 C CNN
@@
 $EndComp
 $Comp
-L Device:LED D2306
+L Device:LED D2406
 U 1 1 5B7826A3
 P 3400 4050
-F 0 "D2306" H 3392 3795 50  0000 C CNN
+F 0 "D2406" H 3392 3795 50  0000 C CNN
 F 1 "Green" H 3392 3886 50  0000 C CNN
 F 2 "LED_THT:LED_D5.0mm_Clear" H 3400 4050 50  0001 C CNN
@@
 	3550 4050 3750 4050
 $Comp
-L Device:R R2307
+L Device:R R2407
 U 1 1 5B78285C
 P 3000 4500
-F 0 "R2307" V 2793 4500 50  0000 C CNN
+F 0 "R2407" V 2793 4500 50  0000 C CNN
 F 1 "165" V 2884 4500 50  0000 C CNN
 F 2 "Resistor_SMD:R_0805_2012Metric" V 2930 4500 50  0001 C CNN
@@
 $EndComp
 $Comp
-L Device:LED D2307
+L Device:LED D2407
 U 1 1 5B782863
 P 3400 4500
-F 0 "D2307" H 3392 4245 50  0000 C CNN
+F 0 "D2407" H 3392 4245 50  0000 C CNN
 F 1 "Green" H 3392 4336 50  0000 C CNN
 F 2 "LED_THT:LED_D5.0mm_Clear" H 3400 4500 50  0001 C CNN
@@
 	3550 4500 3750 4500
 $Comp
-L Device:R R2308
+L Device:R R2408
 U 1 1 5B782A93
 P 3000 4950
-F 0 "R2308" V 2793 4950 50  0000 C CNN
+F 0 "R2408" V 2793 4950 50  0000 C CNN
 F 1 "165" V 2884 4950 50  0000 C CNN
 F 2 "Resistor_SMD:R_0805_2012Metric" V 2930 4950 50  0001 C CNN
@@
 $EndComp
 $Comp
-L Device:LED D2308
+L Device:LED D2408
 U 1 1 5B782A9A
 P 3400 4950
-F 0 "D2308" H 3392 4695 50  0000 C CNN
+F 0 "D2408" H 3392 4695 50  0000 C CNN
 F 1 "Green" H 3392 4786 50  0000 C CNN
 F 2 "LED_THT:LED_D5.0mm_Clear" H 3400 4950 50  0001 C CNN
@@
 	3550 4950 3750 4950
 $Comp
-L Device:LED D2310
+L Device:LED D2410
 U 1 1 5B782D8A
 P 5500 2200
-F 0 "D2310" H 5492 1945 50  0000 C CNN
+F 0 "D2410" H 5492 1945 50  0000 C CNN
 F 1 "Red" H 5492 2036 50  0000 C CNN
 F 2 "LED_THT:LED_D5.0mm_Clear" H 5500 2200 50  0001 C CNN
@@
 	5650 2200 5850 2200
 $Comp
-L Device:R R2310
+L Device:R R2410
 U 1 1 5B782D93
 P 5100 2200
-F 0 "R2310" V 4893 2200 50  0000 C CNN
+F 0 "R2410" V 4893 2200 50  0000 C CNN
 F 1 "165" V 4984 2200 50  0000 C CNN
 F 2 "Resistor_SMD:R_0805_2012Metric" V 5030 2200 50  0001 C CNN
@@
 $EndComp
 $Comp
-L Device:LED D2311
+L Device:LED D2411
 U 1 1 5B7830C7
 P 5500 2700
-F 0 "D2311" H 5492 2445 50  0000 C CNN
+F 0 "D2411" H 5492 2445 50  0000 C CNN
 F 1 "Red" H 5492 2536 50  0000 C CNN
 F 2 "LED_THT:LED_D5.0mm_Clear" H 5500 2700 50  0001 C CNN
@@
 	5650 2700 5850 2700
 $Comp
-L Device:R R2311
+L Device:R R2411
 U 1 1 5B7830D0
 P 5100 2700
-F 0 "R2311" V 4893 2700 50  0000 C CNN
+F 0 "R2411" V 4893 2700 50  0000 C CNN
 F 1 "165" V 4984 2700 50  0000 C CNN
 F 2 "Resistor_SMD:R_0805_2012Metric" V 5030 2700 50  0001 C CNN
@@
 $EndComp
 $Comp
-L Device:LED D2312
+L Device:LED D2412
 U 1 1 5B78347B
 P 5500 3150
-F 0 "D2312" H 5492 2895 50  0000 C CNN
+F 0 "D2412" H 5492 2895 50  0000 C CNN
 F 1 "Red" H 5492 2986 50  0000 C CNN
 F 2 "LED_THT:LED_D5.0mm_Clear" H 5500 3150 50  0001 C CNN
@@
 	5650 3150 5850 3150
 $Comp
-L Device:R R2312
+L Device:R R2412
 U 1 1 5B783484
 P 5100 3150
-F 0 "R2312" V 4893 3150 50  0000 C CNN
+F 0 "R2412" V 4893 3150 50  0000 C CNN
 F 1 "165" V 4984 3150 50  0000 C CNN
 F 2 "Resistor_SMD:R_0805_2012Metric" V 5030 3150 50  0001 C CNN
@@
 $EndComp
 $Comp
-L Device:LED D2313
+L Device:LED D2413
 U 1 1 5B7838C9
 P 5500 3600
-F 0 "D2313" H 5492 3345 50  0000 C CNN
+F 0 "D2413" H 5492 3345 50  0000 C CNN
 F 1 "Red" H 5492 3436 50  0000 C CNN
 F 2 "LED_THT:LED_D5.0mm_Clear" H 5500 3600 50  0001 C CNN
@@
 	5650 3600 5850 3600
 $Comp
-L Device:R R2313
+L Device:R R2413
 U 1 1 5B7838D2
 P 5100 3600
-F 0 "R2313" V 4893 3600 50  0000 C CNN
+F 0 "R2413" V 4893 3600 50  0000 C CNN
 F 1 "165" V 4984 3600 50  0000 C CNN
 F 2 "Resistor_SMD:R_0805_2012Metric" V 5030 3600 50  0001 C CNN
@@
 $EndComp
 $Comp
-L Device:LED D2314
+L Device:LED D2414
 U 1 1 5B783DB0
 P 5500 4050
-F 0 "D2314" H 5492 3795 50  0000 C CNN
+F 0 "D2414" H 5492 3795 50  0000 C CNN
 F 1 "Red" H 5492 3886 50  0000 C CNN
 F 2 "LED_THT:LED_D5.0mm_Clear" H 5500 4050 50  0001 C CNN
@@
 	5650 4050 5850 4050
 $Comp
-L Device:R R2314
+L Device:R R2414
 U 1 1 5B783DB9
 P 5100 4050
-F 0 "R2314" V 4893 4050 50  0000 C CNN
+F 0 "R2414" V 4893 4050 50  0000 C CNN
 F 1 "165" V 4984 4050 50  0000 C CNN
 F 2 "Resistor_SMD:R_0805_2012Metric" V 5030 4050 50  0001 C CNN
@@
 $EndComp
 $Comp
-L Device:LED D2315
+L Device:LED D2415
 U 1 1 5B784347
 P 5500 4500
-F 0 "D2315" H 5492 4245 50  0000 C CNN
+F 0 "D2415" H 5492 4245 50  0000 C CNN
 F 1 "Red" H 5492 4336 50  0000 C CNN
 F 2 "LED_THT:LED_D5.0mm_Clear" H 5500 4500 50  0001 C CNN
@@
 	5650 4500 5850 4500
 $Comp
-L Device:R R2315
+L Device:R R2415
 U 1 1 5B784350
 P 5100 4500
-F 0 "R2315" V 4893 4500 50  0000 C CNN
+F 0 "R2415" V 4893 4500 50  0000 C CNN
 F 1 "165" V 4984 4500 50  0000 C CNN
 F 2 "Resistor_SMD:R_0805_2012Metric" V 5030 4500 50  0001 C CNN
@@
 $EndComp
 $Comp
-L Device:LED D2316
+L Device:LED D2416
 U 1 1 5B7849A5
 P 5500 5000
-F 0 "D2316" H 5492 4745 50  0000 C CNN
+F 0 "D2416" H 5492 4745 50  0000 C CNN
 F 1 "Red" H 5492 4836 50  0000 C CNN
 F 2 "LED_THT:LED_D5.0mm_Clear" H 5500 5000 50  0001 C CNN
@@
 	5650 5000 5850 5000
 $Comp
-L Device:R R2316
+L Device:R R2416
 U 1 1 5B7849AE
 P 5100 5000
-F 0 "R2316" V 4893 5000 50  0000 C CNN
+F 0 "R2416" V 4893 5000 50  0000 C CNN
 F 1 "165" V 4984 5000 50  0000 C CNN
 F 2 "Resistor_SMD:R_0805_2012Metric" V 5030 5000 50  0001 C CNN
@@
 	2850 4500 2850 4950
 $Comp
-L power:+3V3 #PWR02302
+L power:+3V3 #PWR02402
 U 1 1 5B787261
 P 4950 1800
-F 0 "#PWR02302" H 4950 1650 50  0001 C CNN
+F 0 "#PWR02402" H 4950 1650 50  0001 C CNN
 F 1 "+3V3" V 4965 1928 50  0000 L CNN
 F 2 "" H 4950 1800 50  0001 C CNN

Commit message: Changes to input and outputs
Parts:
- removed D2401, D2402, D2403, D2404, D2405, D2406, D2407, D2408: Green, LED_THT:LED_D5.0mm_Clear, symbol Device:LED
- removed R2401, R2402, R2403, R2404, R2405, R2406, R2407, R2408: 165, Resistor_SMD:R_0805_2012Metric, symbol Device:R
Connections:
- net labels removed: Green1, Green2, Green3, Green4, Green5, Green6, Green7, Green8
- wire segments 46 -> 23
