File: G3/DigitalIO.sch (KiCad schematic (older format))
At the start: 11 parts, among them Q1301 ZXTN25050DFHTA, Q1302 ZXTN25050DFHTA, Q1303 ZXTN25050DFHTA, U1301 MCP23017

Commit message: Changed label on signal for digital input schema.
Changed lines of the file:
@@
 F2 "In1" B L 1500 1100 50
 F3 "In2" B L 1500 1200 50
-F4 "O1" O R 2250 1150 50
+F4 "~signal" O R 2250 1150 50
 $EndSheet
 Text GLabel 1400 1200 0    60   Input ~ 0
@@
 F2 "In1" B L 1500 1550 50
 F3 "In2" B L 1500 1650 50
-F4 "O1" O R 2250 1600 50
+F4 "~signal" O R 2250 1600 50
 $EndSheet
 Wire Wire Line
@@
 F2 "In1" B L 1500 2000 50
 F3 "In2" B L 1500 2100 50
-F4 "O1" O R 2250 2050 50
+F4 "~signal" O R 2250 2050 50
 $EndSheet
 $Sheet
@@
 F2 "In1" B L 1500 2450 50
 F3 "In2" B L 1500 2550 50
-F4 "O1" O R 2250 2500 50
+F4 "~signal" O R 2250 2500 50
 $EndSheet
 $Sheet
@@
 F2 "In1" B L 1500 2900 50
 F3 "In2" B L 1500 3000 50
-F4 "O1" O R 2250 2950 50
+F4 "~signal" O R 2250 2950 50
 $EndSheet
 $Sheet
@@
 F2 "In1" B L 1500 3350 50
 F3 "In2" B L 1500 3450 50
-F4 "O1" O R 2250 3400 50
+F4 "~signal" O R 2250 3400 50
 $EndSheet
 $Sheet
@@
 F2 "In1" B L 1500 3800 50
 F3 "In2" B L 1500 3900 50
-F4 "O1" O R 2250 3850 50
+F4 "~signal" O R 2250 3850 50
 $EndSheet
 $Sheet
@@
 F2 "In1" B L 1500 4250 50
 F3 "In2" B L 1500 4350 50
-F4 "O1" O R 2250 4300 50
+F4 "~signal" O R 2250 4300 50
 $EndSheet
 Wire Wire Line

Commit message: Touch up
Parts:
- removed Q1301, Q1302, Q1303: ZXTN25050DFHTA, Package_TO_SOT_SMD:SOT-23, symbol Device:Q_NPN_BCE
- removed R1304, R1305: 470, Resistor_SMD:R_0805_2012Metric, symbol Device:R
- added D1301: Red, LED_THT:LED_D5.0mm_Clear, symbol Device:LED
- R1303: value 470 -> 165
Connections:
- net labels added: StatusLED
- wire segments 67 -> 61
Changed lines of the file:
@@
 $Descr A3 16535 11693
 encoding utf-8
-Sheet 13 31
+Sheet 13 35
 Title ""
 Date ""
@@
 	1    0    0    -1
 $EndComp
-$Comp
-L Device:Q_NPN_BCE Q1303
-U 1 1 59CCBF12
-P 9050 5250
-F 0 "Q1303" V 9250 5200 50  0000 L CNN
-F 1 "ZXTN25050DFHTA" H 8450 5100 50  0000 L CNN
-F 2 "Package_TO_SOT_SMD:SOT-23" H 9250 5350 50  0001 C CNN
-F 3 "" H 9050 5250 50  0001 C CNN
-	1    9050 5250
-	1    0    0    -1
-$EndComp
-$Comp
-L power:GND #PWR01313
-U 1 1 59CCBF1E
-P 9150 5550
-F 0 "#PWR01313" H 9150 5300 50  0001 C CNN
-F 1 "GND" H 9155 5377 50  0000 C CNN
-F 2 "" H 9150 5550 50  0001 C CNN
-F 3 "" H 9150 5550 50  0001 C CNN
-	1    9150 5550
-	1    0    0    -1
-$EndComp
-$Comp
-L Device:R R1305
-U 1 1 59CCBF29
-P 8650 5250
-F 0 "R1305" V 8550 5250 50  0000 C CNN
-F 1 "470" V 8650 5250 50  0000 C CNN
-F 2 "Resistor_SMD:R_0805_2012Metric" V 8580 5250 50  0001 C CNN
-F 3 "" H 8650 5250 50  0001 C CNN
-	1    8650 5250
-	0    1    1    0
-$EndComp
-Text GLabel 9450 5050 2    60   Input ~ 0
+Text GLabel 6500 6450 2    60   Input ~ 0
 BELL_GND_BREAK
-Text GLabel 8500 5250 0    60   Input ~ 0
+Text GLabel 5700 6450 0    60   Input ~ 0
 BELL_CTRL
 Wire Wire Line
@@
 Wire Notes Line
 	3300 600  3300 1500
-Wire Wire Line
-	9150 5550 9150 5450
-Wire Wire Line
-	9450 5050 9150 5050
-Wire Wire Line
-	8800 5250 8850 5250
 $Comp
 L power:+3.3V #PWR01303
@@
 L Device:Buzzer BZ1301
 U 1 1 5B635F18
-P 6950 4950
-F 0 "BZ1301" H 7103 4979 50  0000 L CNN
-F 1 "SDC1610M5-01" H 7103 4888 50  0000 L CNN
-F 2 "PerMalmberg:SDC1610M5-01_Buzzer_16diam_5pitch" V 6925 5050 50  0001 C CNN
-F 3 "~" V 6925 5050 50  0001 C CNN
-	1    6950 4950
+P 6600 4900
+F 0 "BZ1301" H 6753 4929 50  0000 L CNN
+F 1 "SDC1610M5-01" H 6753 4838 50  0000 L CNN
+F 2 "PerMalmberg:SDC1610M5-01_Buzzer_16diam_5pitch" V 6575 5000 50  0001 C CNN
+F 3 "~" V 6575 5000 50  0001 C CNN
+	1    6600 4900
 	1    0    0    -1
 $EndComp
@@
 L power:+5V #PWR01310
 U 1 1 5B63AFA2
-P 6850 4850
-F 0 "#PWR01310" H 6850 4700 50  0001 C CNN
-F 1 "+5V" H 6865 5023 50  0000 C CNN
-F 2 "" H 6850 4850 50  0001 C CNN
-F 3 "" H 6850 4850 50  0001 C CNN
-	1    6850 4850
-	1    0    0    -1
-$EndComp
-$Comp
-L Device:Q_NPN_BCE Q1301
-U 1 1 5B640CA7
-P 6750 5250
-F 0 "Q1301" V 6950 5200 50  0000 L CNN
-F 1 "ZXTN25050DFHTA" H 6150 5100 50  0000 L CNN
-F 2 "Package_TO_SOT_SMD:SOT-23" H 6950 5350 50  0001 C CNN
-F 3 "" H 6750 5250 50  0001 C CNN
-	1    6750 5250
-	1    0    0    -1
-$EndComp
-$Comp
-L Device:R R1303
-U 1 1 5B640CAE
-P 6350 5250
-F 0 "R1303" V 6250 5250 50  0000 C CNN
-F 1 "470" V 6350 5250 50  0000 C CNN
-F 2 "Resistor_SMD:R_0805_2012Metric" V 6280 5250 50  0001 C CNN
-F 3 "" H 6350 5250 50  0001 C CNN
-	1    6350 5250
-	0    1    1    0
-$EndComp
-Text GLabel 6200 5250 0    60   Input ~ 0
+P 6500 4800
+F 0 "#PWR01310" H 6500 4650 50  0001 C CNN
+F 1 "+5V" H 6515 4973 50  0000 C CNN
+F 2 "" H 6500 4800 50  0001 C CNN
+F 3 "" H 6500 4800 50  0001 C CNN
+	1    6500 4800
+	1    0    0    -1
+$EndComp
+Text GLabel 5700 5000 0    60   Input ~ 0
 SIREN_CTRL
-Wire Wire Line
-	6500 5250 6550 5250
-$Comp
-L power:GND #PWR01311
-U 1 1 5B6493AF
-P 6850 5450
-F 0 "#PWR01311" H 6850 5200 50  0001 C CNN
-F 1 "GND" H 6855 5277 50  0000 C CNN
-F 2 "" H 6850 5450 50  0001 C CNN
-F 3 "" H 6850 5450 50  0001 C CNN
-	1    6850 5450
-	1    0    0    -1
-$EndComp
 Text GLabel 1400 4350 0    60   Input ~ 0
 DI8_2
@@
 Wire Wire Line
 	6900 4200 6650 4200
-$Comp
-L Device:Q_NPN_BCE Q1302
-U 1 1 5B72A32D
-P 6750 6000
-F 0 "Q1302" V 6950 5950 50  0000 L CNN
-F 1 "ZXTN25050DFHTA" H 6150 5850 50  0000 L CNN
-F 2 "Package_TO_SOT_SMD:SOT-23" H 6950 6100 50  0001 C CNN
-F 3 "" H 6750 6000 50  0001 C CNN
-	1    6750 6000
-	1    0    0    -1
-$EndComp
-$Comp
-L Device:R R1304
-U 1 1 5B72A333
-P 6350 6000
-F 0 "R1304" V 6250 6000 50  0000 C CNN
-F 1 "470" V 6350 6000 50  0000 C CNN
-F 2 "Resistor_SMD:R_0805_2012Metric" V 6280 6000 50  0001 C CNN
-F 3 "" H 6350 6000 50  0001 C CNN
-	1    6350 6000
-	0    1    1    0
-$EndComp
-Text GLabel 6200 6000 0    60   Input ~ 0
+Text GLabel 5700 5450 0    60   Input ~ 0
 SIREN_CTRL
-Wire Wire Line
-	6500 6000 6550 6000
-$Comp
-L power:GND #PWR01312
-U 1 1 5B72A33B
-P 6850 6200
-F 0 "#PWR01312" H 6850 5950 50  0001 C CNN
-F 1 "GND" H 6855 6027 50  0000 C CNN
-F 2 "" H 6850 6200 50  0001 C CNN
-F 3 "" H 6850 6200 50  0001 C CNN
-	1    6850 6200
-	1    0    0    -1
-$EndComp
-Text GLabel 7050 5750 2    50   Input ~ 0
+Text GLabel 6500 5450 2    50   Input ~ 0
 SIREN_GND_BREAK
-Wire Wire Line
-	7050 5750 6850 5750
-Wire Wire Line
-	6850 5750 6850 5800
 $Sheet
 S 9800 1900 800  900
@@
 Wire Wire Line
 	9650 2700 9800 2700
+$Comp
+L Device:LED D?
+U 1 1 5B8AAF3E
+P 6650 5950
+AR Path="/5B62EDB8/5B780EE8/5B8AAF3E" Ref="D?"  Part="1"
+AR Path="/5B62EDB8/5B8AAF3E" Ref="D1301"  Part="1"
+F 0 "D1301" H 6642 5695 50  0000 C CNN
+F 1 "Red" H 6642 5786 50  0000 C CNN
+F 2 "LED_THT:LED_D5.0mm_Clear" H 6650 5950 50  0001 C CNN
+F 3 "https://www.mouser.se/ProductDetail/Lumex/SSL-LX55103ID-FL?qs=sGAEpiMZZMtmwHDZQCdlqUPJk6OnVfwF%252bWo7zgs2%252bqE%3d" H 6650 5950 50  0001 C CNN
+	1    6650 5950
+	1    0    0    -1
+$EndComp
+Wire Wire Line
+	6900 5950 6800 5950
+$Comp
+L Device:R R?
+U 1 1 5B8AAF47
+P 7050 5950
+AR Path="/5B62EDB8/5B780EE8/5B8AAF47" Ref="R?"  Part="1"
+AR Path="/5B62EDB8/5B8AAF47" Ref="R1303"  Part="1"
+F 0 "R1303" V 6843 5950 50  0000 C CNN
+F 1 "165" V 6934 5950 50  0000 C CNN
+F 2 "Resistor_SMD:R_0805_2012Metric" V 6980 5950 50  0001 C CNN
+F 3 "https://www.mouser.se/ProductDetail/Bourns/CR0805-FX-1650ELF?qs=sGAEpiMZZMtlubZbdhIBIKn39ibjI6WbHbnDBzjqA1U%3d" H 7050 5950 50  0001 C CNN
+	1    7050 5950
+	0    -1   -1   0
+$EndComp
+$Comp
+L power:+3.3V #PWR01311
+U 1 1 5B8B47B5
+P 7200 5950
+F 0 "#PWR01311" H 7200 5800 50  0001 C CNN
+F 1 "+3.3V" V 7215 6078 50  0000 L CNN
+F 2 "" H 7200 5950 50  0001 C CNN
+F 3 "" H 7200 5950 50  0001 C CNN
+	1    7200 5950
+	0    1    1    0
+$EndComp
+Text GLabel 5700 5950 0    50   Input ~ 0
+StatusLED
+$Sheet
+S 5700 4900 800  200
+U 5B8B425B
+F0 "SimpleOutput" 50
+F1 "SimpleOutput.sch" 50
+F2 "CTRL" I L 5700 5000 50
+F3 "~Out" I R 6500 5000 50
+$EndSheet
+$Sheet
+S 5700 5350 800  200
+U 5B8BDF9E
+F0 "sheet5B8BDF9A" 50
+F1 "SimpleOutput.sch" 50
+F2 "CTRL" I L 5700 5450 50
+F3 "~Out" I R 6500 5450 50
+$EndSheet
+$Sheet
+S 5700 5850 800  200
+U 5B8CC011
+F0 "sheet5B8CC00D" 50
+F1 "SimpleOutput.sch" 50
+F2 "CTRL" I L 5700 5950 50
+F3 "~Out" I R 6500 5950 50
+$EndSheet
+$Sheet
+S 5700 6350 800  200
+U 5B8CD7E8
+F0 "sheet5B8CD7E4" 50
+F1 "SimpleOutput.sch" 50
+F2 "CTRL" I L 5700 6450 50
+F3 "~Out" I R 6500 6450 50
+$EndSheet
 $EndSCHEMATC

Commit message: Added SDCard slot.
Parts:
- renumbered BZ1301 to BZ1401, C1301 to C1401, D1301 to D1401, R1301 to R1401, R1302 to R1402, R1303 to R1403, U1301 to U1401
Changed lines of the file:
@@
 $Descr A3 16535 11693
 encoding utf-8
-Sheet 13 35
+Sheet 14 36
 Title ""
 Date ""
@@
 $EndDescr
 $Comp
-L PerMalmberg:MCP23017 U1301
+L PerMalmberg:MCP23017 U1401
 U 1 1 59C2CB37
 P 3600 4100
-F 0 "U1301" H 3400 5250 50  0000 C CNN
+F 0 "U1401" H 3400 5250 50  0000 C CNN
 F 1 "MCP23017" H 3650 5150 50  0000 C CNN
 F 2 "Package_SO:SOIC-28W_7.5x17.9mm_P1.27mm" H 3650 3150 50  0001 L CNN
@@
 DO1
 $Comp
-L Device:C C1301
+L Device:C C1401
 U 1 1 59C4102A
 P 3600 1050
-F 0 "C1301" H 3715 1096 50  0000 L CNN
+F 0 "C1401" H 3715 1096 50  0000 L CNN
 F 1 "100n" H 3715 1005 50  0000 L CNN
 F 2 "Capacitor_SMD:C_0805_2012Metric" H 3638 900 50  0001 C CNN
@@
 $EndComp
 $Comp
-L power:GND #PWR01302
+L power:GND #PWR01402
 U 1 1 59C42024
 P 3600 1200
-F 0 "#PWR01302" H 3600 950 50  0001 C CNN
+F 0 "#PWR01402" H 3600 950 50  0001 C CNN
 F 1 "GND" H 3605 1027 50  0000 C CNN
 F 2 "" H 3600 1200 50  0001 C CNN
@@
 $EndComp
 $Comp
-L power:GND #PWR01304
+L power:GND #PWR01404
 U 1 1 59C42579
 P 3600 4000
-F 0 "#PWR01304" H 3600 3750 50  0001 C CNN
+F 0 "#PWR01404" H 3600 3750 50  0001 C CNN
 F 1 "GND" H 3605 3827 50  0000 C CNN
 F 2 "" H 3600 4000 50  0001 C CNN
@@
 DO8
 $Comp
-L power:GND #PWR01307
+L power:GND #PWR01407
 U 1 1 59C5AF84
 P 4100 3800
-F 0 "#PWR01307" H 4100 3550 50  0001 C CNN
+F 0 "#PWR01407" H 4100 3550 50  0001 C CNN
 F 1 "GND" V 4105 3672 50  0000 R CNN
 F 2 "" H 4100 3800 50  0001 C CNN
@@
 $EndComp
 $Comp
-L power:GND #PWR01306
+L power:GND #PWR01406
 U 1 1 59C5B1A8
 P 4100 3700
-F 0 "#PWR01306" H 4100 3450 50  0001 C CNN
+F 0 "#PWR01406" H 4100 3450 50  0001 C CNN
 F 1 "GND" V 4105 3572 50  0000 R CNN
 F 2 "" H 4100 3700 50  0001 C CNN
@@
 $EndComp
 $Comp
-L power:GND #PWR01305
+L power:GND #PWR01405
 U 1 1 59C5B287
 P 4100 3600
-F 0 "#PWR01305" H 4100 3350 50  0001 C CNN
+F 0 "#PWR01405" H 4100 3350 50  0001 C CNN
 F 1 "GND" V 4105 3472 50  0000 R CNN
 F 2 "" H 4100 3600 50  0001 C CNN
@@
 Adress 0x20
 $Comp
-L Device:R R1302
+L Device:R R1402
 U 1 1 59C5F580
 P 4200 2550
-F 0 "R1302" H 4270 2596 50  0000 L CNN
+F 0 "R1402" H 4270 2596 50  0000 L CNN
 F 1 "10k" H 4270 2505 50  0000 L CNN
 F 2 "Resistor_SMD:R_0805_2012Metric" V 4130 2550 50  0001 C CNN
-F 3 "" H 4200 2550 50  0001 C CNN
+F 3 "https://www.mouser.se/ProductDetail/Panasonic-Industrial-Devices/ERJ-6ENF1002V?qs=sGAEpiMZZMu61qfTUdNhGzRxdwze5h8ZcGDx6geba20%3d" H 4200 2550 50  0001 C CNN
 	1    4200 2550
 	1    0    0    -1
 $EndComp
 $Comp
-L power:+3.3V #PWR01309
+L power:+3.3V #PWR01409
 U 1 1 59C5F699
 P 4200 2400
-F 0 "#PWR01309" H 4200 2250 50  0001 C CNN
+F 0 "#PWR01409" H 4200 2250 50  0001 C CNN
 F 1 "+3.3V" H 4350 2450 50  0000 C CNN
 F 2 "" H 4200 2400 50  0001 C CNN
@@
 Near MCP23017
 $Comp
-L power:+3.3V #PWR01308
+L power:+3.3V #PWR01408
 U 1 1 59CA4C36
 P 4200 1900
-F 0 "#PWR01308" H 4200 1750 50  0001 C CNN
+F 0 "#PWR01408" H 4200 1750 50  0001 C CNN
 F 1 "+3.3V" V 4150 2100 50  0000 C CNN
 F 2 "" H 4200 1900 50  0001 C CNN
@@
 	3300 600  3300 1500
 $Comp
-L power:+3.3V #PWR01303
+L power:+3.3V #PWR01403
 U 1 1 5A53CE41
 P 3600 2000
-F 0 "#PWR01303" H 3600 1850 50  0001 C CNN
+F 0 "#PWR01403" H 3600 1850 50  0001 C CNN
 F 1 "+3.3V" V 3600 2250 50  0000 C CNN
 F 2 "" H 3600 2000 50  0001 C CNN
@@
 $EndComp
 $Comp
-L power:+3.3V #PWR01301
+L power:+3.3V #PWR01401
 U 1 1 5A53D1F2
 P 3600 900
-F 0 "#PWR01301" H 3600 750 50  0001 C CNN
+F 0 "#PWR01401" H 3600 750 50  0001 C CNN
 F 1 "+3.3V" H 3600 1100 50  0000 C CNN
 F 2 "" H 3600 900 50  0001 C CNN
@@
 	4200 2700 4250 2700
 $Comp
-L Device:Buzzer BZ1301
+L Device:Buzzer BZ1401
 U 1 1 5B635F18
 P 6750 4700
-F 0 "BZ1301" H 6903 4729 50  0000 L CNN
+F 0 "BZ1401" H 6903 4729 50  0000 L CNN
 F 1 "SDC1610M5-01" H 6903 4638 50  0000 L CNN
 F 2 "PerMalmberg:SDC1610M5-01_Buzzer_16diam_5pitch" V 6725 4800 50  0001 C CNN
@@
 $EndComp
 $Comp
-L power:+5V #PWR01310
+L power:+5V #PWR01410
 U 1 1 5B63AFA2
 P 6650 4600
-F 0 "#PWR01310" H 6650 4450 50  0001 C CNN
+F 0 "#PWR01410" H 6650 4450 50  0001 C CNN
 F 1 "+5V" H 6665 4773 50  0000 C CNN
 F 2 "" H 6650 4600 50  0001 C CNN
@@
 	5400 4200 5550 4200
 $Comp
-L Device:R R1301
+L Device:R R1401
 U 1 1 5B6DFD32
 P 4200 2050
-F 0 "R1301" H 4270 2096 50  0000 L CNN
+F 0 "R1401" H 4270 2096 50  0000 L CNN
 F 1 "10k" H 4270 2005 50  0000 L CNN
 F 2 "Resistor_SMD:R_0805_2012Metric" V 4130 2050 50  0001 C CNN
-F 3 "" H 4200 2050 50  0001 C CNN
+F 3 "https://www.mouser.se/ProductDetail/Panasonic-Industrial-Devices/ERJ-6ENF1002V?qs=sGAEpiMZZMu61qfTUdNhGzRxdwze5h8ZcGDx6geba20%3d" H 4200 2050 50  0001 C CNN
 	1    4200 2050
 	1    0    0    -1
@@
 P 6800 5750
 AR Path="/5B62EDB8/5B780EE8/5B8AAF3E" Ref="D?"  Part="1"
-AR Path="/5B62EDB8/5B8AAF3E" Ref="D1301"  Part="1"
-F 0 "D1301" H 6792 5495 50  0000 C CNN
+AR Path="/5B62EDB8/5B8AAF3E" Ref="D1401"  Part="1"
+F 0 "D1401" H 6792 5495 50  0000 C CNN
 F 1 "Red" H 6792 5586 50  0000 C CNN
 F 2 "LED_THT:LED_D5.0mm_Clear" H 6800 5750 50  0001 C CNN
@@
 P 7200 5750
 AR Path="/5B62EDB8/5B780EE8/5B8AAF47" Ref="R?"  Part="1"
-AR Path="/5B62EDB8/5B8AAF47" Ref="R1303"  Part="1"
-F 0 "R1303" V 6993 5750 50  0000 C CNN
+AR Path="/5B62EDB8/5B8AAF47" Ref="R1403"  Part="1"
+F 0 "R1403" V 6993 5750 50  0000 C CNN
 F 1 "165" V 7084 5750 50  0000 C CNN
 F 2 "Resistor_SMD:R_0805_2012Metric" V 7130 5750 50  0001 C CNN
@@
 $EndComp
 $Comp
-L power:+3.3V #PWR01311
+L power:+3.3V #PWR01411
 U 1 1 5B8B47B5
 P 7350 5750
-F 0 "#PWR01311" H 7350 5600 50  0001 C CNN
+F 0 "#PWR01411" H 7350 5600 50  0001 C CNN
 F 1 "+3.3V" V 7365 5878 50  0000 L CNN
 F 2 "" H 7350 5750 50  0001 C CNN

Commit message: Using MAX4948 instead of DIPs
Parts:
- removed R1401, R1402: 10k, Resistor_SMD:R_0805_2012Metric, symbol Device:R
- added C1401: 100n, Capacitor_SMD:C_0805_2012Metric, symbol Device:C
- added U1401: MCP23017, Package_SO:SOIC-28W_7.5x17.9mm_P1.27mm, symbol PerMalmberg:MCP23017
- renumbered C1401 to C1402, R1403 to R1401, U1401 to U1402
Connections:
- net labels added: I2C_SCL, I2C_SDA, SD_ENABLE, SD_MODE
- net labels removed: DIGITAL_I2C_SCL, DIGITAL_I2C_SDA
- wire segments 61 -> 58
- no-connect marks 1 -> 15
Other:
- note added: "Adress 0x21"

Commit message: Pulldowns added to unused IO on MCP23017
Parts:
- added R1401, R1402: 10k, Resistor_SMD:R_0805_2012Metric, symbol Device:R
- renumbered R1401 to R1403
Connections:
- wire segments 58 -> 68
- no-connect marks 15 -> 3

Commit message: Changes to input and outputs
Parts:
- removed D1401: Red, LED_THT:LED_D5.0mm_Clear, symbol Device:LED
- removed R1403: 165, Resistor_SMD:R_0805_2012Metric, symbol Device:R
- renumbered U1402 to U1401, U1401 to U1402
Connections:
- net labels added: BELL_PWR, DI1_PWR, DI2_PWR, DI3_PWR, DI4_PWR, DI5_PWR, DI6_PWR, DI7_PWR, DI8_PWR, DO1_PWR, DO2_PWR, DO3_PWR, DO4_PWR, DO5_PWR, DO6_PWR, DO7_PWR, DO8_PWR, SIREN_PWR
- net labels removed: +5V, BELL_GND_BREAK, DO1_GND_BREAK, DO2_GND_BREAK, DO3_GND_BREAK, DO4_GND_BREAK, DO5_GND_BREAK, DO6_GND_BREAK, DO7_GND_BREAK, DO8_GND_BREAK, SIREN_GND_BREAK
- wire segments 68 -> 11

Commit message: WIP - PCB
Parts:
- added D1401: Armed, LED_THT:LED_D5.0mm_Clear, symbol Device:LED
- added D1402: Wifi, LED_THT:LED_D5.0mm_Clear, symbol Device:LED
- added D1403: MQTT, LED_THT:LED_D5.0mm_Clear, symbol Device:LED
- added D1404, D1405, D1406: Red, LED_THT:LED_D5.0mm_Clear, symbol Device:LED
- added R1403, R1404, R1405, R1406, R1407: 165, Resistor_SMD:R_0805_2012Metric, symbol Device:R
- R1401: value 10k -> 165
Connections:
- net labels removed: StatusLED
- wire segments 11 -> 25
