File: G3/G3.sch (KiCad schematic (older format))
At the start: 0 parts

Commit message: Texts and moutningholes.
Parts:
- added MH101, MH102, MH103, MH104: MountingHole, MountingHole:MountingHole_4.3mm_M4, symbol Mechanical:MountingHole
Changed lines of the file:
@@
 F1 "Connectors.sch" 50
 $EndSheet
+$Comp
+L Mechanical:MountingHole MH101
+U 1 1 5BA7C209
+P 4750 900
+F 0 "MH101" H 4850 946 50  0000 L CNN
+F 1 "MountingHole" H 4850 855 50  0000 L CNN
+F 2 "MountingHole:MountingHole_4.3mm_M4" H 4750 900 50  0001 C CNN
+F 3 "~" H 4750 900 50  0001 C CNN
+	1    4750 900
+	1    0    0    -1
+$EndComp
+$Comp
+L Mechanical:MountingHole MH102
+U 1 1 5BA7C4D2
+P 4750 1100
+F 0 "MH102" H 4850 1146 50  0000 L CNN
+F 1 "MountingHole" H 4850 1055 50  0000 L CNN
+F 2 "MountingHole:MountingHole_4.3mm_M4" H 4750 1100 50  0001 C CNN
+F 3 "~" H 4750 1100 50  0001 C CNN
+	1    4750 1100
+	1    0    0    -1
+$EndComp
+$Comp
+L Mechanical:MountingHole MH103
+U 1 1 5BA7C4E5
+P 4750 1300
+F 0 "MH103" H 4850 1346 50  0000 L CNN
+F 1 "MountingHole" H 4850 1255 50  0000 L CNN
+F 2 "MountingHole:MountingHole_4.3mm_M4" H 4750 1300 50  0001 C CNN
+F 3 "~" H 4750 1300 50  0001 C CNN
+	1    4750 1300
+	1    0    0    -1
+$EndComp
+$Comp
+L Mechanical:MountingHole MH104
+U 1 1 5BA7C4F9
+P 4750 1500
+F 0 "MH104" H 4850 1546 50  0000 L CNN
+F 1 "MountingHole" H 4850 1455 50  0000 L CNN
+F 2 "MountingHole:MountingHole_4.3mm_M4" H 4750 1500 50  0001 C CNN
+F 3 "~" H 4750 1500 50  0001 C CNN
+	1    4750 1500
+	1    0    0    -1
+$EndComp
 $EndSCHEMATC

Commit message: Text adjustements. Added OS H/W Logo. Added PCB manufacturing files.
Parts:
- added LOGO101: Logo_Open_Hardware_Small, Symbol:OSHW-Logo2_7.3x6mm_SilkScreen, symbol Graphic:Logo_Open_Hardware_Small
Changed lines of the file:
@@
+	1    0    0    -1
+$EndComp
+$Comp
+L Graphic:Logo_Open_Hardware_Small LOGO101
+U 1 1 5BAAC245
+P 5800 1150
+F 0 "LOGO101" H 5800 1425 50  0001 C CNN
+F 1 "Logo_Open_Hardware_Small" H 5800 925 50  0001 C CNN
+F 2 "Symbol:OSHW-Logo2_7.3x6mm_SilkScreen" H 5800 1150 50  0001 C CNN
+F 3 "~" H 5800 1150 50  0001 C CNN
+	1    5800 1150
 	1    0    0    -1
 $EndComp
