File: G3/G3.kicad_pcb (KiCad board)
At the start: 2 copper layers, 334 parts, among them J1501 Digital input supply, J1502 Digital input GND, J1601 Power_select, J1701 Power_select, J1801 Power_select, J1901 Power_select, J2001 Power_select, J201 Conn_02x02_Top_Bottom, J202 GS2, J203 GS2, J2101 Power_select, J2201 Power_select, J2301 Power_select, J2601 Power_select, J2801 Digital input supply, J2802 Digital input GND, J2901 Digital input supply, J2902 Digital input GND, J3001 Digital input supply, J3002 Digital input GND, J301 Debug, J302 BME280, J3101 Digital input supply, J3102 Digital input GND, J3201 Digital input supply, J3202 Digital input GND, J3301 Digital input supply, J3302 Digital input GND, J3401 Digital input supply, J3402 Digital input GND, J3501 Sense, J3502 Digital Input, J3503 Sense, J3504 Digital input, J3505 Power 12/5/3, J3506 Digital input, J3507 Digital Output, J3508 Digital output, J3509 Digital output, J401 Micro_SD_Card_Det, Q1601 ZXTN25050DFHTA, Q1602 ZXTN25050DFHTA, Q1701 ZXTN25050DFHTA, Q1702 ZXTN25050DFHTA, Q1801 ZXTN25050DFHTA, Q1802 ZXTN25050DFHTA, Q1901 ZXTN25050DFHTA, Q1902 ZXTN25050DFHTA, Q2001 ZXTN25050DFHTA, Q2002 ZXTN25050DFHTA, Q2101 ZXTN25050DFHTA, Q2102 ZXTN25050DFHTA, Q2201 ZXTN25050DFHTA, Q2202 ZXTN25050DFHTA, Q2301 ZXTN25050DFHTA, Q2302 ZXTN25050DFHTA, Q2401 ZXTN25050DFHTA, Q2402 ZXTN25050DFHTA, Q2601 ZXTN25050DFHTA, Q2602 ZXTN25050DFHTA, Q2701 ZXTN25050DFHTA, Q2702 ZXTN25050DFHTA, SW301 Boot option, SW302 Reset, SW303 Factory reset, SW401 SD SPI/MMC mode, U1401 MCP23017, U1402 MCP23017, U1501 LTV-354T, U201 LM1084-3.3, U202 LM1084-5.0, U2801 LTV-354T, U2901 LTV-354T, U3001 LTV-354T, U301 ESP32_WROVER, U302 TXB0102DCU, U3101 LTV-354T, U3201 LTV-354T, U3301 LTV-354T, U3401 LTV-354T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

Commit message: WIP - PCB
Parts:
- moved J3509 402.2 mm to (393.7, 247.7), turned to 270 degrees
- moved J3507 357.7 mm to (393.7, 154.3), turned to 270 degrees
- moved J2601 352.6 mm to (427.6, 280.6), turned to 180 degrees
- moved F2601 349.5 mm to (417.4, 277.4)
- moved J3508 344.2 mm to (393.7, 200.7), turned to 270 degrees
- moved R2603 336.8 mm to (406.0, 275.6)
- moved R2601 332.3 mm to (406.0, 271.8)
- moved Q2602 329.7 mm to (411.1, 275.6), turned to 180 degrees
- moved Q2601 328.4 mm to (411.1, 280.7), turned to 180 degrees
- moved D2601 326.9 mm to (404.7, 279.4), turned to 270 degrees
- moved J2301 324.1 mm to (427.6, 265.6), turned to 180 degrees
- moved R2602 323.9 mm to (402.2, 274.3), turned to 90 degrees
- moved F2301 321.1 mm to (417.4, 262.4)
- moved R2303 308.4 mm to (406.0, 260.6)
- moved Q2301 303.0 mm to (411.1, 265.7), turned to 180 degrees
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Routing:
- net 12V_PWR: track 151.6 -> 342.1 mm
- net +5V: track 155.9 -> 296.2 mm
- net DO7_PWR: track 0.00 -> 44.4 mm
- net BELL_PWR: track 0.00 -> 42.6 mm
- net DO8_PWR: track 0.00 -> 41.0 mm, vias 0 -> 1
- net DO6_PWR: track 0.00 -> 39.5 mm
- net DO4_PWR: track 0.00 -> 30.6 mm
- net DO3_PWR: track 0.00 -> 25.9 mm
- net DO2_PWR: track 0.00 -> 21.1 mm
- net DO1_PWR: track 0.00 -> 19.3 mm
- net Net-(Q2201-Pad1): track 0.00 -> 18.9 mm
- net Net-(Q2101-Pad1): track 0.00 -> 18.9 mm
- net Net-(Q2001-Pad1): track 0.00 -> 18.9 mm
- net Net-(Q1901-Pad1): track 0.00 -> 18.9 mm
- net Net-(Q1701-Pad1): track 0.00 -> 18.9 mm
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
Commit message: WIP - PCB
Parts:
- moved D2601 452.7 mm to (513.5, -160.0), turned to 90 degrees
- moved Q2601 452.3 mm to (507.1, -161.3), turned to 0 degrees
- moved J2601 446.3 mm to (490.6, -161.2), turned to 0 degrees
- moved R2603 444.7 mm to (512.2, -156.2), turned to 180 degrees
- moved R2602 444.1 mm to (516.0, -154.9), turned to 270 degrees
- moved F2601 443.4 mm to (500.8, -158.0), turned to 180 degrees
- moved Q2602 442.4 mm to (507.1, -156.2), turned to 0 degrees
- moved R2601 437.3 mm to (512.2, -152.4), turned to 180 degrees
- moved D1406 433.1 mm to (452.1, -96.5), turned to 180 degrees
- moved D2301 423.6 mm to (513.5, -145.0), turned to 90 degrees
- moved Q2301 423.0 mm to (507.1, -146.3), turned to 0 degrees
- moved D1405 420.3 mm to (452.1, -88.9), turned to 180 degrees
- moved D1403 418.8 mm to (452.1, -73.7), turned to 180 degrees
- moved J2301 416.7 mm to (490.6, -146.2), turned to 0 degrees
- moved R2303 415.6 mm to (512.2, -141.2), turned to 180 degrees
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Routing:
- net SIREN_PWR: track 0.00 -> 49.5 mm
- net Net-(Q2401-Pad1): track 0.00 -> 17.6 mm
- net /DigitalIO/Internal siren/Output: track 0.00 -> 17.3 mm
- net 12V_PWR: track 342.1 -> 359.2 mm
- net Net-(Q2701-Pad1): track 0.00 -> 13.0 mm, vias 0 -> 2
- net Net-(Q2402-Pad3): track 0.00 -> 9.27 mm, vias 0 -> 2
- net Net-(D2701-Pad2): track 0.00 -> 7.26 mm
- net Net-(D2401-Pad2): track 0.00 -> 7.26 mm
- net Net-(Q2702-Pad3): track 0.00 -> 3.14 mm

Commit message: WiP PCB
Parts:
- moved J201 472.5 mm to (618.5, 162.6), turned to 270 degrees
- moved J3502 438.1 mm to (363.5, 267.5), turned to 0 degrees
- moved F201 428.6 mm to (600.7, 165.1)
- moved D1501 427.7 mm to (363.5, 257.3), turned to 90 degrees
- moved U201 426.5 mm to (580.4, 179.1), turned to 270 degrees
- moved D202 424.0 mm to (589.3, 167.6)
- moved FL201 423.2 mm to (595.6, 167.6), turned to 180 degrees
- moved F1501 418.9 mm to (362.3, 247.2), turned to 0 degrees
- moved U202 416.6 mm to (581.7, 151.1), turned to 90 degrees
- moved R1501 416.5 mm to (373.7, 256.1), turned to 270 degrees
- moved R1503 411.6 mm to (361.0, 238.3), turned to 0 degrees
- moved R201 410.2 mm to (582.0, 165.1)
- moved D2801 408.4 mm to (383.5, 257.3), turned to 90 degrees
- moved J202 407.4 mm to (569.0, 179.1), turned to 180 degrees
- moved R1504 406.8 mm to (361.0, 233.2), turned to 180 degrees
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Routing:
- net I2C_SDA: track 0.00 -> 53.8 mm
- net I2C_SCL: track 0.00 -> 53.7 mm
- net +3V3: track 189.8 -> 225.9 mm, vias 8 -> 10
- net +5V: track 296.2 -> 325.7 mm
- net Net-(C901-Pad1): track 0.00 -> 24.5 mm
- net Net-(C801-Pad1): track 0.00 -> 24.5 mm
- net Net-(C701-Pad1): track 0.00 -> 24.5 mm
- net Net-(C1301-Pad1): track 0.00 -> 24.5 mm
- net Net-(C1201-Pad1): track 0.00 -> 24.5 mm
- net Net-(C1101-Pad1): track 0.00 -> 24.5 mm
- net Net-(C1001-Pad1): track 0.00 -> 24.5 mm
- net Net-(C601-Pad1): track 0.00 -> 24.5 mm
- net /AnalogInput/AnalogSensCircuit4/Adc: track 0.00 -> 21.7 mm
- net /AnalogInput/AnalogSensCircuit8/Adc: track 0.00 -> 21.6 mm
- net /AnalogInput/AnalogSensCircuit5/Adc: track 0.00 -> 20.9 mm
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
Commit message: WiP PCB
Parts:
- moved J401 110.7 mm to (156.2, 172.7), turned to 90 degrees
- moved R409 99.2 mm to (162.6, 185.4), turned to 90 degrees
- moved D407 98.2 mm to (157.5, 185.4), turned to 270 degrees
- moved D405 96.0 mm to (149.9, 185.4), turned to 270 degrees
- moved D404 90.5 mm to (146.1, 185.4), turned to 270 degrees
- moved C402 89.8 mm to (149.9, 156.2)
- moved D406 88.9 mm to (153.7, 185.4), turned to 270 degrees
- moved R304 87.2 mm to (-7.62, 141.0), turned to 270 degrees
- moved C306 86.4 mm to (-2.54, 141.0), turned to 90 degrees
- moved C403 82.1 mm to (149.9, 162.6), turned to 180 degrees
- moved D402 81.8 mm to (138.4, 185.4), turned to 270 degrees
- moved U401 81.2 mm to (137.2, 172.7), turned to 180 degrees
- moved D403 81.2 mm to (142.2, 185.4), turned to 270 degrees
- moved U302 79.2 mm to (5.08, 141.0), turned to 180 degrees
- moved C305 69.8 mm to (12.7, 141.0), turned to 90 degrees
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Connections:
- D403 pad 1: SD_SPI_CS -> /MCU/SDCard/SD_MMC_Data3
- D404 pad 1: SD_SPI_MOSI -> /MCU/SDCard/SD_MMC_CMD
- D405 pad 1: SD_SPI_CLK -> /MCU/SDCard/SD_MMC_CLK
- D406 pad 1: SD_SPI_MISO -> /MCU/SDCard/SD_MMC_DATA0
- J401 pad 2: SD_SPI_CS -> /MCU/SDCard/SD_MMC_Data3
- J401 pad 3: SD_SPI_MOSI -> /MCU/SDCard/SD_MMC_CMD
- J401 pad 5: SD_SPI_CLK -> /MCU/SDCard/SD_MMC_CLK
- J401 pad 7: SD_SPI_MISO -> /MCU/SDCard/SD_MMC_DATA0
- U401 pad 20: SD_DATA0 -> /MCU/SDCard/SD_MMC_DATA0
- U401 pad 23: SD_SPI_MOSI -> /MCU/SDCard/SD_MMC_CMD
- U401 pad 3: SD_SPI_CLK -> /MCU/SDCard/SD_MMC_CLK
- U401 pad 7: SD_SPI_CS -> /MCU/SDCard/SD_MMC_Data3

Commit message: WiP PCB
Parts:
- D2401: value Green -> Siren active
- moved D1301 453.3 mm to (15.0, 112.8), turned to 270 degrees
- moved RV1301 448.2 mm to (15.1, 106.4), turned to 180 degrees
- moved C1301 448.1 mm to (20.7, 114.4), turned to 270 degrees
- moved R1301 445.0 mm to (20.7, 110.5), turned to 90 degrees
- moved D1201 443.2 mm to (15.0, 99.8), turned to 270 degrees
- moved D1303 442.0 mm to (25.8, 114.0), turned to 180 degrees
- moved R1302 441.9 mm to (20.7, 106.7), turned to 270 degrees
- moved R1303 439.7 mm to (25.0, 110.2), turned to 0 degrees
- moved RV1201 438.3 mm to (15.1, 93.4), turned to 180 degrees
- moved C1201 437.7 mm to (20.7, 101.4), turned to 270 degrees
- moved D1302 435.7 mm to (25.8, 106.4), turned to 0 degrees
- moved R1201 434.8 mm to (20.7, 97.5), turned to 90 degrees
- moved D1101 433.6 mm to (15.0, 86.8), turned to 270 degrees
- moved R1202 431.9 mm to (20.7, 93.7), turned to 270 degrees
- moved D1203 431.5 mm to (25.8, 101.0), turned to 180 degrees
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Connections:
- U401 pad 10: Net-(U401-Pad10) -> SD_SPI_CS
- U401 pad 11: /MCU/SDCard/SD_MMC_Data2 -> /MCU/SDCard/SD_MMC_Data3
- U401 pad 12: SD_DATA2 -> SD_DATA3
- U401 pad 15: SD_DATA1 -> SD_CLK
- U401 pad 16: /MCU/SDCard/SD_MMC_DATA1 -> /MCU/SDCard/SD_MMC_CLK
- U401 pad 17: Net-(U401-Pad17) -> SD_SPI_CLK
- U401 pad 18: SD_DATA0 -> SD_DATA1
- U401 pad 19: SD_SPI_MISO -> Net-(U401-Pad19)
- U401 pad 2: SD_SPI_CLK -> SD_SPI_MISO
- U401 pad 20: /MCU/SDCard/SD_MMC_DATA0 -> /MCU/SDCard/SD_MMC_DATA1
- U401 pad 3: /MCU/SDCard/SD_MMC_CLK -> /MCU/SDCard/SD_MMC_DATA0
- U401 pad 4: SD_CLK -> SD_DATA0
- U401 pad 7: /MCU/SDCard/SD_MMC_Data3 -> /MCU/SDCard/SD_MMC_Data2
- U401 pad 8: SD_SPI_CS -> Net-(U401-Pad8)
- U401 pad 9: SD_DATA3 -> SD_DATA2
Routing:
- net +3V3: track 225.8 -> 366.5 mm, vias 10 -> 16
- net /MCU/CH_Enable: track 0.00 -> 86.0 mm, vias 0 -> 2
- net SD_DATA2: track 0.00 -> 69.5 mm, vias 0 -> 2
- net SD_DATA3: track 0.00 -> 55.7 mm, vias 0 -> 6
- net /MCU/Boot_option: track 0.00 -> 52.2 mm, vias 0 -> 8
- net SD_MODE: track 0.00 -> 50.8 mm
- net SD_CLK: track 0.00 -> 49.4 mm, vias 0 -> 3
- net /MCU/SDCard/SD_MMC_DATA1: track 0.00 -> 45.8 mm
- net /MCU/SDCard/SD_MMC_CLK: track 0.00 -> 34.6 mm, vias 0 -> 2
- net /MCU/SDCard/SD_MMC_CMD: track 0.00 -> 34.5 mm, vias 0 -> 2
- net SD_CMD: track 0.00 -> 33.1 mm, vias 0 -> 2
- net SD_SPI_MOSI: track 0.00 -> 33.1 mm, vias 0 -> 2
- net SD_SPI_CS: track 0.00 -> 32.2 mm, vias 0 -> 2
- net /MCU/SDCard/SD_MMC_DATA0: track 0.00 -> 32.1 mm
- net SD_SPI_MISO: track 0.00 -> 28.2 mm, vias 0 -> 2
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Other:
- board text added: "JTAG"
- board text added: "SD SPI Selected/ JTAG supported"

Commit message: WiP PCB
Parts:
- added REF**: MountingHole_4.3mm_M4, MountingHole:MountingHole_4.3mm_M4, F.Cu at (28.6, -9.27)
- added REF**: MountingHole_4.3mm_M4, MountingHole:MountingHole_4.3mm_M4, F.Cu at (208.4, 152.8)
- added REF**: MountingHole_4.3mm_M4, MountingHole:MountingHole_4.3mm_M4, F.Cu at (208.3, -9.27)
- added REF**: MountingHole_4.3mm_M4, MountingHole:MountingHole_4.3mm_M4, F.Cu at (28.6, 152.5)
- moved R3401 276.9 mm to (32.8, 4.72), turned to 90 degrees
- moved U3401 265.7 mm to (32.8, 14.9), turned to 270 degrees
- moved D3401 262.1 mm to (43.0, 3.45), turned to 270 degrees
- moved J3507 255.6 mm to (36.7, 148.1), turned to 0 degrees
- moved C3401 254.5 mm to (34.1, 23.8), turned to 180 degrees
- moved F3401 247.9 mm to (44.3, 13.6), turned to 180 degrees
- moved R3301 245.3 mm to (52.8, 4.72), turned to 90 degrees
- moved J3402 244.5 mm to (34.1, 35.2), turned to 270 degrees
- moved R1602 243.5 mm to (36.7, 139.6), turned to 180 degrees
- moved R1601 241.9 mm to (34.2, 135.8), turned to 90 degrees
- moved R2401 237.6 mm to (112.8, 63.6), turned to 180 degrees
- moved R1603 236.3 mm to (38.0, 135.8), turned to 90 degrees
- moved R3403 236.0 mm to (45.5, 22.5), turned to 180 degrees
- moved D1601 232.7 mm to (41.8, 137.0), turned to 0 degrees
- moved U3301 232.6 mm to (52.8, 14.9), turned to 270 degrees
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Routing:
- net +3V3: track 366.5 -> 1128.4 mm, vias 16 -> 32
- net +5V: track 344.9 -> 780.8 mm, vias 0 -> 17
- net BELL_CTRL: track 0.00 -> 263.7 mm, vias 0 -> 2
- net Wiegand_D0: track 0.00 -> 152.6 mm
- net Wiegand_D1: track 0.00 -> 145.9 mm
- net Sense8_DUT: track 10.7 -> 143.7 mm
- net SIREN_CTRL: track 0.00 -> 132.3 mm, vias 0 -> 6
- net 12V_PWR: track 369.6 -> 500.0 mm, vias 0 -> 2
- net DO5: track 0.00 -> 126.6 mm, vias 0 -> 2
- net DO8: track 0.00 -> 125.8 mm, vias 0 -> 2
- net DI1: track 47.7 -> 169.0 mm, vias 0 -> 2
- net DO7: track 0.00 -> 120.6 mm, vias 0 -> 2
- net DO4: track 0.00 -> 114.6 mm, vias 0 -> 2
- net DO1: track 0.00 -> 110.9 mm, vias 0 -> 2
- net DO6: track 0.00 -> 110.6 mm, vias 0 -> 2
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- added copper zone on B.Cu, net GND
- added copper zone on F.Cu, net GND
Other:
- board outline added: 191.3 x 175.3 mm
- board text added: "GND"
- board text added: "GND BELL"
- board text added: "GND SIREN"
- board text removed: "12V"

Commit message: Updated ESP32 Wrover footprint
Parts:
- removed REF** (x4): MountingHole_4.3mm_M4, MountingHole:MountingHole_4.3mm_M4
- moved D206 32.5 mm to (114.7, 137.3)
- moved F1601 32.5 mm to (35.1, 156.5)
- moved F1701 32.5 mm to (50.1, 156.5)
- moved F1801 32.5 mm to (65.1, 156.5)
- moved F1901 32.5 mm to (80.1, 156.5)
- moved F2001 32.5 mm to (95.1, 156.5)
- moved F2101 32.5 mm to (110.1, 156.5)
- moved J301 32.5 mm to (67.0, 137.8)
- moved J3505 32.5 mm to (191.9, 141.5)
- moved R2701 32.5 mm to (166.0, 158.6)
- moved R2702 32.5 mm to (171.1, 158.6)
- moved SW401 32.5 mm to (99.7, 134.8)
- moved C1402 32.5 mm to (61.7, 74.5)
- moved F2201 32.5 mm to (125.1, 156.5)
- moved F2301 32.5 mm to (140.1, 156.5)
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Routing:
- net +3V3: track 1128.4 -> 1122.2 mm
- net GND: track 32.1 -> 29.0 mm, vias 300 -> 301
- net SD_CMD: track 43.1 -> 41.0 mm
- net /MCU/CH_Enable: track 102.0 -> 101.2 mm
- net I2C_SCL: track 158.1 -> 158.0 mm, vias 4 -> 5
Other:
- board size 191.3 x 175.3 mm -> 191.3 x 176.8 mm
- board text added: "12V"
- board text added: "3.3V"
- board text added: "D inp 1 PWR 1 2"
- board text added: "D inp 2 PWR 1 2"
- board text added: "D inp 3 PWR 1 2"
- board text added: "D inp 4 PWR 1 2"
- board text added: "D inp 5 PWR 1 2"
- board text added: "D inp 6 PWR 1 2"
- board text added: "D inp 7 PWR 1 2"
- board text added: "D inp 8 PWR 1 2"
- board text added: "G3 I/O Card | PerMalmberg@GitHub 2018"
- board text added: "JLCJLCJLCJLC"
- board text added: "PWR SPLY"
- board text added: "Sense 1 GND 2"
- board text added: "Sense 3 GND 4"
- board text added: "Sense 5 GND 6"
- board text added: "Sense 7 GND 8"
- board text added: "Wiegand D0 D1"

Commit message: Updated ESP32 Wrover footprint
Routing:
- net SD_DATA2: track 74.3 -> 74.8 mm
- net GND: vias 301 -> 302
- net I2C_SCL: vias 5 -> 4
Changed lines of the file:
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@@
     (thickness 1.6)
     (drawings 79)
-    (tracks 2989)
+    (tracks 2990)
     (zones 0)
     (modules 334)
@@
   (segment (start 51.953914 113.14804) (end 51.200874 112.395) (width 0.25) (layer F.Cu) (net 32))
   (segment (start 52.178914 113.14804) (end 51.953914 113.14804) (width 0.25) (layer F.Cu) (net 32))
-  (via (at 61.214 103.632) (size 0.8) (drill 0.4) (layers F.Cu B.Cu) (net 32))
-  (via (at 65.278 103.759) (size 0.8) (drill 0.4) (layers F.Cu B.Cu) (net 32))
+  (via (at 61.214 103.886) (size 0.8) (drill 0.4) (layers F.Cu B.Cu) (net 32))
+  (via (at 65.278 103.886) (size 0.8) (drill 0.4) (layers F.Cu B.Cu) (net 32))
   (via (at 84.455 108.077) (size 0.8) (drill 0.4) (layers F.Cu B.Cu) (net 32))
   (via (at 75.565 101.854) (size 0.8) (drill 0.4) (layers F.Cu B.Cu) (net 32))
-  (via (at 81.153 110.236) (size 0.8) (drill 0.4) (layers F.Cu B.Cu) (net 115))
   (via (at 84.201 113.411) (size 0.8) (drill 0.4) (layers F.Cu B.Cu) (net 32))
   (via (at 79.629 117.094) (size 0.8) (drill 0.4) (layers F.Cu B.Cu) (net 32))
@@
   (via (at 23.622 178.308) (size 0.8) (drill 0.4) (layers F.Cu B.Cu) (net 32))
   (via (at 19.431 178.308) (size 0.8) (drill 0.4) (layers F.Cu B.Cu) (net 32))
+  (segment (start 65.864 103.759) (end 65.843685 103.759) (width 0.25) (layer F.Cu) (net 32))
+  (via (at 61.722 101.473) (size 0.8) (drill 0.4) (layers F.Cu B.Cu) (net 32))
   (segment (start 75.145914 94.51154) (end 72.732914 96.92454) (width 0.25) (layer F.Cu) (net 33))
   (segment (start 62.572914 100.232702) (end 64.139252 101.79904) (width 0.25) (layer F.Cu) (net 33))
@@
   (via (at 57.15 102.743) (size 0.8) (drill 0.4) (layers F.Cu B.Cu) (net 104))
   (segment (start 57.715685 102.743) (end 57.15 102.743) (width 0.25) (layer F.Cu) (net 104))
-  (segment (start 66.118 102.743) (end 57.715685 102.743) (width 0.25) (layer F.Cu) (net 104))
-  (segment (start 68.137 104.762) (end 66.118 102.743) (width 0.25) (layer F.Cu) (net 104))
-  (segment (start 68.137 106.012) (end 68.137 104.762) (width 0.25) (layer F.Cu) (net 104))
+  (segment (start 67.056 102.743) (end 57.715685 102.743) (width 0.25) (layer F.Cu) (net 104))
+  (segment (start 68.137 106.012) (end 68.137 103.824) (width 0.25) (layer F.Cu) (net 104))
+  (segment (start 68.137 103.824) (end 67.056 102.743) (width 0.25) (layer F.Cu) (net 104))
   (via (at 74.422 108.966) (size 0.8) (drill 0.4) (layers F.Cu B.Cu) (net 105))
   (segment (start 74.422 108.966) (end 76.410454 108.966) (width 0.25) (layer F.Cu) (net 105))
