File: G3/12VDigitalOutput.sch (KiCad schematic (older format))
At the start: 6 parts, among them Q2701 ZXTN25050DFHTA, Q2702 ZXTN25050DFHTA

Commit message: #Updated with Mouser-links for all components.
Parts:
- D2701: footprint LED_THT:LED_D5.0mm_Clear -> LED_THT:LED_D5.0mm
- R2703: value 165 -> 1.65k
Changed lines of the file:
@@
 F 1 "ZXTN25050DFHTA" H 3800 1750 50  0000 L CNN
 F 2 "Package_TO_SOT_SMD:SOT-23" H 3750 1950 50  0001 C CNN
-F 3 "" H 3550 1850 50  0001 C CNN
+F 3 "https://www.mouser.se/ProductDetail/Diodes-Incorporated/ZXTN25050DFHTA?qs=sGAEpiMZZMshyDBzk1%2fWi6gR%252bqBmAG1j52KxSCCDz6c%3d" H 3550 1850 50  0001 C CNN
 	1    3550 1850
 	1    0    0    -1
@@
 AR Path="/5B62EDB8/5BA35DC6/5BA13C13" Ref="R2703"  Part="1"
 F 0 "R2703" V 3443 3050 50  0000 C CNN
-F 1 "165" V 3534 3050 50  0000 C CNN
+F 1 "1.65k" V 3534 3050 50  0000 C CNN
 F 2 "Resistor_SMD:R_0805_2012Metric" V 3580 3050 50  0001 C CNN
-F 3 "https://www.mouser.se/ProductDetail/Bourns/CR0805-FX-1650ELF?qs=sGAEpiMZZMtlubZbdhIBIKn39ibjI6WbHbnDBzjqA1U%3d" H 3650 3050 50  0001 C CNN
+F 3 "https://www.mouser.se/ProductDetail/Vishay/CRCW08051K65FKEA?qs=sGAEpiMZZMtlubZbdhIBIFvv2%252blmU1cYk%2fKBbkOVYDU%3d" H 3650 3050 50  0001 C CNN
 	1    3650 3050
 	-1   0    0    1
@@
 F 0 "D2701" H 3642 3095 50  0000 C CNN
 F 1 "Green" H 3642 3186 50  0000 C CNN
-F 2 "LED_THT:LED_D5.0mm_Clear" H 3650 3350 50  0001 C CNN
-F 3 "https://www.mouser.se/ProductDetail/Lumex/SSL-LX55103GD-FL?qs=sGAEpiMZZMtmwHDZQCdlqVsz6Sp3LtaXcNplsbJfBSw%3d" H 3650 3350 50  0001 C CNN
+F 2 "LED_THT:LED_D5.0mm" H 3650 3350 50  0001 C CNN
+F 3 "https://www.mouser.se/ProductDetail/Lite-On/LTL2R3KGD-EM?qs=sGAEpiMZZMtmwHDZQCdlqY3QuPVQdrfivxVgVo2hFbg%3d" H 3650 3350 50  0001 C CNN
 	1    3650 3350
 	0    -1   -1   0
@@
 F 1 "ZXTN25050DFHTA" H 3800 2600 50  0000 L CNN
 F 2 "Package_TO_SOT_SMD:SOT-23" H 3750 2800 50  0001 C CNN
-F 3 "" H 3550 2700 50  0001 C CNN
+F 3 "https://www.mouser.se/ProductDetail/Diodes-Incorporated/ZXTN25050DFHTA?qs=sGAEpiMZZMshyDBzk1%2fWi6gR%252bqBmAG1j52KxSCCDz6c%3d" H 3550 2700 50  0001 C CNN
 	1    3550 2700
 	1    0    0    -1
