File: G3/AnalogInput.sch (KiCad schematic (older format))
At the start: 6 parts, among them U401 ADS1115IDGST, U402 ADS1115IDGST

Commit message: More touch ups
Changed lines of the file:
@@
 S 1300 900  550  200
 U 5B7620B9
-F0 "AnalogSensCircuit" 50
+F0 "AnalogSensCircuit1" 50
 F1 "AnalogSensCircuit.sch" 50
 F2 "DUT" I L 1300 1000 50
@@
 S 1300 1300 550  200
 U 5B774401
-F0 "sheet5B7743FD" 50
+F0 "AnalogSensCircuit2" 50
 F1 "AnalogSensCircuit.sch" 50
 F2 "DUT" I L 1300 1400 50
@@
 S 1300 1700 550  200
 U 5B7744D6
-F0 "sheet5B7744D2" 50
+F0 "AnalogSensCircuit3" 50
 F1 "AnalogSensCircuit.sch" 50
 F2 "DUT" I L 1300 1800 50
@@
 S 1300 2100 550  200
 U 5B77465F
-F0 "sheet5B77465B" 50
+F0 "AnalogSensCircuit4" 50
 F1 "AnalogSensCircuit.sch" 50
 F2 "DUT" I L 1300 2200 50
@@
 S 1300 2500 550  200
 U 5B7747EB
-F0 "sheet5B7747E7" 50
+F0 "AnalogSensCircuit5" 50
 F1 "AnalogSensCircuit.sch" 50
 F2 "DUT" I L 1300 2600 50
@@
 S 1300 2900 550  200
 U 5B774A61
-F0 "sheet5B774A5D" 50
+F0 "AnalogSensCircuit6" 50
 F1 "AnalogSensCircuit.sch" 50
 F2 "DUT" I L 1300 3000 50
@@
 S 1300 3300 550  200
 U 5B774D4C
-F0 "sheet5B774D48" 50
+F0 "AnalogSensCircuit7" 50
 F1 "AnalogSensCircuit.sch" 50
 F2 "DUT" I L 1300 3400 50
@@
 S 1300 3700 550  200
 U 5B77572B
-F0 "sheet5B775727" 50
+F0 "AnalogSensCircuit8" 50
 F1 "AnalogSensCircuit.sch" 50
 F2 "DUT" I L 1300 3800 50

Commit message: Added SDCard slot.
Parts:
- renumbered C401 to C501, C402 to C502, R401 to R501, R402 to R502, U401 to U501, U402 to U502
Changed lines of the file:
@@
 $Descr A4 11693 8268
 encoding utf-8
-Sheet 4 35
+Sheet 5 36
 Title ""
 Date ""
@@
 I2C address: 0x49
 $Comp
-L power:+3.3V #PWR0403
+L power:+3.3V #PWR0503
 U 1 1 59C73F9C
 P 3650 2850
-F 0 "#PWR0403" H 3650 2700 50  0001 C CNN
+F 0 "#PWR0503" H 3650 2700 50  0001 C CNN
 F 1 "+3.3V" V 3665 2978 50  0000 L CNN
 F 2 "" H 3650 2850 50  0001 C CNN
@@
 $EndComp
 $Comp
-L power:+3.3V #PWR0408
+L power:+3.3V #PWR0508
 U 1 1 59C73C46
 P 4200 1050
-F 0 "#PWR0408" H 4200 900 50  0001 C CNN
+F 0 "#PWR0508" H 4200 900 50  0001 C CNN
 F 1 "+3.3V" H 4215 1223 50  0000 C CNN
 F 2 "" H 4200 1050 50  0001 C CNN
@@
 ANALOG_RDY_1
 $Comp
-L Device:R R402
+L Device:R R502
 U 1 1 59C73C3C
 P 4200 1200
-F 0 "R402" H 4270 1246 50  0000 L CNN
+F 0 "R502" H 4270 1246 50  0000 L CNN
 F 1 "10k" H 4270 1155 50  0000 L CNN
 F 2 "Resistor_SMD:R_0805_2012Metric" V 4130 1200 50  0001 C CNN
-F 3 "" H 4200 1200 50  0001 C CNN
+F 3 "https://www.mouser.se/ProductDetail/Panasonic-Industrial-Devices/ERJ-6ENF1002V?qs=sGAEpiMZZMu61qfTUdNhGzRxdwze5h8ZcGDx6geba20%3d" H 4200 1200 50  0001 C CNN
 	1    4200 1200
 	1    0    0    -1
@@
 	5300 3750 6000 3750
 $Comp
-L power:GND #PWR0412
+L power:GND #PWR0512
 U 1 1 59C72B0C
 P 5500 3450
-F 0 "#PWR0412" H 5500 3200 50  0001 C CNN
+F 0 "#PWR0512" H 5500 3200 50  0001 C CNN
 F 1 "GND" H 5505 3277 50  0000 C CNN
 F 2 "" H 5500 3450 50  0001 C CNN
@@
 $EndComp
 $Comp
-L Device:C C402
+L Device:C C502
 U 1 1 59C72B05
 P 5500 3300
-F 0 "C402" H 5615 3346 50  0000 L CNN
+F 0 "C502" H 5615 3346 50  0000 L CNN
 F 1 "100n" H 5615 3255 50  0000 L CNN
 F 2 "Capacitor_SMD:C_0805_2012Metric" H 5538 3150 50  0001 C CNN
@@
 	5250 2000 5950 2000
 $Comp
-L power:GND #PWR0410
+L power:GND #PWR0510
 U 1 1 59C720F6
 P 5450 1700
-F 0 "#PWR0410" H 5450 1450 50  0001 C CNN
+F 0 "#PWR0510" H 5450 1450 50  0001 C CNN
 F 1 "GND" H 5455 1527 50  0000 C CNN
 F 2 "" H 5450 1700 50  0001 C CNN
@@
 $EndComp
 $Comp
-L Device:C C401
+L Device:C C501
 U 1 1 59C71FCA
 P 5450 1550
-F 0 "C401" H 5565 1596 50  0000 L CNN
+F 0 "C501" H 5565 1596 50  0000 L CNN
 F 1 "100n" H 5565 1505 50  0000 L CNN
 F 2 "Capacitor_SMD:C_0805_2012Metric" H 5488 1400 50  0001 C CNN
@@
 $EndComp
 $Comp
-L power:GND #PWR0404
+L power:GND #PWR0504
 U 1 1 59C70E9B
 P 3650 3750
-F 0 "#PWR0404" H 3650 3500 50  0001 C CNN
+F 0 "#PWR0504" H 3650 3500 50  0001 C CNN
 F 1 "GND" V 3655 3622 50  0000 R CNN
 F 2 "" H 3650 3750 50  0001 C CNN
@@
 I2C address: 0x48
 $Comp
-L power:GND #PWR0402
+L power:GND #PWR0502
 U 1 1 59C6F2E6
 P 3650 1950
-F 0 "#PWR0402" H 3650 1700 50  0001 C CNN
+F 0 "#PWR0502" H 3650 1700 50  0001 C CNN
 F 1 "GND" V 3655 1822 50  0000 R CNN
 F 2 "" H 3650 1950 50  0001 C CNN
@@
 $EndComp
 $Comp
-L power:+3.3V #PWR0407
+L power:+3.3V #PWR0507
 U 1 1 59C6D362
 P 4150 2850
-F 0 "#PWR0407" H 4150 2700 50  0001 C CNN
+F 0 "#PWR0507" H 4150 2700 50  0001 C CNN
 F 1 "+3.3V" H 4165 3023 50  0000 C CNN
 F 2 "" H 4150 2850 50  0001 C CNN
@@
 ANALOG_RDY_2
 $Comp
-L Device:R R401
+L Device:R R501
 U 1 1 59C6CAF7
 P 4150 3000
-F 0 "R401" H 4220 3046 50  0000 L CNN
+F 0 "R501" H 4220 3046 50  0000 L CNN
 F 1 "10k" H 4220 2955 50  0000 L CNN
 F 2 "Resistor_SMD:R_0805_2012Metric" V 4080 3000 50  0001 C CNN
-F 3 "" H 4150 3000 50  0001 C CNN
+F 3 "https://www.mouser.se/ProductDetail/Panasonic-Industrial-Devices/ERJ-6ENF1002V?qs=sGAEpiMZZMu61qfTUdNhGzRxdwze5h8ZcGDx6geba20%3d" H 4150 3000 50  0001 C CNN
 	1    4150 3000
 	1    0    0    -1
 $EndComp
 $Comp
-L Analog_ADC:ADS1115IDGS U401
+L Analog_ADC:ADS1115IDGS U501
 U 1 1 59C694AA
 P 3650 1550
-F 0 "U401" H 3850 2100 50  0000 C CNN
+F 0 "U501" H 3850 2100 50  0000 C CNN
 F 1 "ADS1115IDGST" H 3300 2050 50  0000 C CNN
 F 2 "Package_SO:TSSOP-10_3x3mm_P0.5mm" H 3650 1550 50  0001 L CNN
@@
 Sense1_DUT
 $Comp
-L power:+3.3V #PWR0409
+L power:+3.3V #PWR0509
 U 1 1 5A53E0D6
 P 5450 1400
-F 0 "#PWR0409" H 5450 1250 50  0001 C CNN
+F 0 "#PWR0509" H 5450 1250 50  0001 C CNN
 F 1 "+3.3V" H 5465 1573 50  0000 C CNN
 F 2 "" H 5450 1400 50  0001 C CNN
@@
 $EndComp
 $Comp
-L power:+3.3V #PWR0411
+L power:+3.3V #PWR0511
 U 1 1 5A53E39D
 P 5500 3150
-F 0 "#PWR0411" H 5500 3000 50  0001 C CNN
+F 0 "#PWR0511" H 5500 3000 50  0001 C CNN
 F 1 "+3.3V" H 5515 3323 50  0000 C CNN
 F 2 "" H 5500 3150 50  0001 C CNN
@@
 $EndComp
 $Comp
-L power:+3.3V #PWR0401
+L power:+3.3V #PWR0501
 U 1 1 5A53E8E5
 P 3650 1050
-F 0 "#PWR0401" H 3650 900 50  0001 C CNN
+F 0 "#PWR0501" H 3650 900 50  0001 C CNN
 F 1 "+3.3V" H 3665 1223 50  0000 C CNN
 F 2 "" H 3650 1050 50  0001 C CNN
@@
 Connection ~ 4200 1350
 $Comp
-L Analog_ADC:ADS1115IDGS U402
+L Analog_ADC:ADS1115IDGS U502
 U 1 1 5B62F45A
 P 3650 3350
-F 0 "U402" H 3850 3850 50  0000 C CNN
+F 0 "U502" H 3850 3850 50  0000 C CNN
 F 1 "ADS1115IDGST" H 3300 3850 50  0000 C CNN
 F 2 "Package_SO:TSSOP-10_3x3mm_P0.5mm" H 3650 3350 50  0001 L CNN
@@
 Connection ~ 4150 3150
 $Comp
-L power:GND #PWR0405
+L power:GND #PWR0505
 U 1 1 5B63FAD0
 P 4050 1750
-F 0 "#PWR0405" H 4050 1500 50  0001 C CNN
+F 0 "#PWR0505" H 4050 1500 50  0001 C CNN
 F 1 "GND" V 4055 1622 50  0000 R CNN
 F 2 "" H 4050 1750 50  0001 C CNN
@@
 $EndComp
 $Comp
-L power:+3.3V #PWR0406
+L power:+3.3V #PWR0506
 U 1 1 5B63FDDD
 P 4050 3550
-F 0 "#PWR0406" H 4050 3400 50  0001 C CNN
+F 0 "#PWR0506" H 4050 3400 50  0001 C CNN
 F 1 "+3.3V" V 4065 3678 50  0000 L CNN
 F 2 "" H 4050 3550 50  0001 C CNN

Commit message: Using MAX4948 instead of DIPs
Connections:
- net labels added: I2C_SCL, I2C_SDA
- net labels removed: ANALOG_I2C_SCL, ANALOG_I2C_SDA
Changed lines of the file:
@@
 	1    0    0    -1
 $EndComp
-Text GLabel 4050 1550 2    60   Input ~ 0
-ANALOG_I2C_SCL
-Text GLabel 4050 3350 2    60   Input ~ 0
-ANALOG_I2C_SCL
-Text GLabel 4050 3450 2    60   Input ~ 0
-ANALOG_I2C_SDA
-Text GLabel 4050 1650 2    60   Input ~ 0
-ANALOG_I2C_SDA
 Text Notes 4700 2000 2    60   ~ 0
 I2C address: 0x48
@@
 Wire Wire Line
 	2950 3800 1850 3800
+Text GLabel 4050 1550 2    60   Input ~ 0
+I2C_SCL
+Text GLabel 4050 1650 2    60   Input ~ 0
+I2C_SDA
+Text GLabel 4050 3350 2    60   Input ~ 0
+I2C_SCL
+Text GLabel 4050 3450 2    60   Input ~ 0
+I2C_SDA
 $EndSCHEMATC
