File: G3/AnalogSensCircuit.sch (KiCad schematic (older format))
At the start: 8 parts

Commit message: Added SDCard slot.
Parts:
- renumbered C501 to C601, D501 to D601, D502 to D602, D503 to D603, R501 to R601, R502 to R602, R503 to R603, RV501 to RV601

Commit message: Changes to input and outputs
Connections:
- wire segments 9 -> 10
Changed lines of the file:
@@
 $Descr A4 11693 8268
 encoding utf-8
-Sheet 6 36
+Sheet 6 35
 Title ""
 Date ""
@@
 Comment4 ""
 $EndDescr
-Wire Wire Line
-	2750 1700 2450 1700
 $Comp
 L Device:D_Schottky D602
@@
 Connection ~ 2600 1400
 $Comp
-L power:+5V #PWR0603
+L power:+5V #PWR0601
 U 1 1 5B762247
 P 2600 1400
-AR Path="/5B61F011/5B7620B9/5B762247" Ref="#PWR0603"  Part="1"
-AR Path="/5B61F011/5B774401/5B762247" Ref="#PWR0703"  Part="1"
-AR Path="/5B61F011/5B7744D6/5B762247" Ref="#PWR0803"  Part="1"
-AR Path="/5B61F011/5B77465F/5B762247" Ref="#PWR0903"  Part="1"
-AR Path="/5B61F011/5B7747EB/5B762247" Ref="#PWR01003"  Part="1"
-AR Path="/5B61F011/5B774A61/5B762247" Ref="#PWR01103"  Part="1"
-AR Path="/5B61F011/5B774D4C/5B762247" Ref="#PWR01203"  Part="1"
-AR Path="/5B61F011/5B77572B/5B762247" Ref="#PWR01303"  Part="1"
-F 0 "#PWR01303" H 2600 1250 50  0001 C CNN
+AR Path="/5B61F011/5B7620B9/5B762247" Ref="#PWR0601"  Part="1"
+AR Path="/5B61F011/5B774401/5B762247" Ref="#PWR0701"  Part="1"
+AR Path="/5B61F011/5B7744D6/5B762247" Ref="#PWR0801"  Part="1"
+AR Path="/5B61F011/5B77465F/5B762247" Ref="#PWR0901"  Part="1"
+AR Path="/5B61F011/5B7747EB/5B762247" Ref="#PWR01001"  Part="1"
+AR Path="/5B61F011/5B774A61/5B762247" Ref="#PWR01101"  Part="1"
+AR Path="/5B61F011/5B774D4C/5B762247" Ref="#PWR01201"  Part="1"
+AR Path="/5B61F011/5B77572B/5B762247" Ref="#PWR01301"  Part="1"
+F 0 "#PWR01301" H 2600 1250 50  0001 C CNN
 F 1 "+5V" H 2615 1573 50  0000 C CNN
 F 2 "" H 2600 1400 50  0001 C CNN
@@
 Wire Wire Line
 	2450 1400 2600 1400
-$Comp
-L power:GND #PWR0601
-U 1 1 5B76224E
-P 1750 1700
-AR Path="/5B61F011/5B7620B9/5B76224E" Ref="#PWR0601"  Part="1"
-AR Path="/5B61F011/5B774401/5B76224E" Ref="#PWR0701"  Part="1"
-AR Path="/5B61F011/5B7744D6/5B76224E" Ref="#PWR0801"  Part="1"
-AR Path="/5B61F011/5B77465F/5B76224E" Ref="#PWR0901"  Part="1"
-AR Path="/5B61F011/5B7747EB/5B76224E" Ref="#PWR01001"  Part="1"
-AR Path="/5B61F011/5B774A61/5B76224E" Ref="#PWR01101"  Part="1"
-AR Path="/5B61F011/5B774D4C/5B76224E" Ref="#PWR01201"  Part="1"
-AR Path="/5B61F011/5B77572B/5B76224E" Ref="#PWR01301"  Part="1"
-F 0 "#PWR01301" H 1750 1450 50  0001 C CNN
-F 1 "GND" V 1755 1572 50  0000 R CNN
-F 2 "" H 1750 1700 50  0001 C CNN
-F 3 "" H 1750 1700 50  0001 C CNN
-	1    1750 1700
-	0    1    -1   0
-$EndComp
 Connection ~ 2100 1700
-Wire Wire Line
-	2050 1700 2100 1700
 Connection ~ 2450 2000
 Wire Wire Line
@@
 L power:GND #PWR0602
 U 1 1 5B762258
-P 2450 2000
+P 2750 2000
 AR Path="/5B61F011/5B7620B9/5B762258" Ref="#PWR0602"  Part="1"
 AR Path="/5B61F011/5B774401/5B762258" Ref="#PWR0702"  Part="1"
@@
 AR Path="/5B61F011/5B774D4C/5B762258" Ref="#PWR01202"  Part="1"
 AR Path="/5B61F011/5B77572B/5B762258" Ref="#PWR01302"  Part="1"
-F 0 "#PWR01302" H 2450 1750 50  0001 C CNN
-F 1 "GND" H 2455 1827 50  0000 C CNN
-F 2 "" H 2450 2000 50  0001 C CNN
-F 3 "" H 2450 2000 50  0001 C CNN
-	1    2450 2000
+F 0 "#PWR01302" H 2750 1750 50  0001 C CNN
+F 1 "GND" H 2755 1827 50  0000 C CNN
+F 2 "" H 2750 2000 50  0001 C CNN
+F 3 "" H 2750 2000 50  0001 C CNN
+	1    2750 2000
 	-1   0    0    -1
 $EndComp
@@
 AR Path="/5B61F011/5B774D4C/5B76225E" Ref="D1201"  Part="1"
 AR Path="/5B61F011/5B77572B/5B76225E" Ref="D1301"  Part="1"
-F 0 "D1301" V 2100 1950 50  0000 L CNN
-F 1 "CDBA3100-HF" V 2200 1900 50  0000 L CNN
+F 0 "D1301" V 2300 1750 50  0000 L CNN
+F 1 "CDBA3100-HF" V 2400 1600 50  0000 L CNN
 F 2 "Diode_SMD:D_SMA" H 2100 1850 50  0001 C CNN
 F 3 "http://www.mouser.se/Search/ProductDetail.aspx?R=CDBA3100-HFvirtualkey59960000virtualkey750-CDBA3100-HF" H 2100 1850 50  0001 C CNN
@@
 L Device:Varistor RV601
 U 1 1 5B76226C
-P 1900 1700
+P 1800 1850
 AR Path="/5B61F011/5B7620B9/5B76226C" Ref="RV601"  Part="1"
 AR Path="/5B61F011/5B774401/5B76226C" Ref="RV701"  Part="1"
@@
 AR Path="/5B61F011/5B774D4C/5B76226C" Ref="RV1201"  Part="1"
 AR Path="/5B61F011/5B77572B/5B76226C" Ref="RV1301"  Part="1"
-F 0 "RV1301" V 1650 1750 50  0000 C CNN
-F 1 "B72510E250K062" V 1750 1900 50  0000 C CNN
-F 2 "Capacitor_SMD:C_0805_2012Metric" V 1830 1700 50  0001 C CNN
-F 3 "https://www.mouser.se/ProductDetail/EPCOS-TDK/B72510E0250K062/?qs=%2fha2pyFadugVCK9yiqateTD%252bWTZyWxpU55VnsqI3B1Kd%2fbUd9GEicg%3d%3d" H 1900 1700 50  0001 C CNN
-	1    1900 1700
-	0    -1   1    0
+F 0 "RV1301" V 1550 1900 50  0000 C CNN
+F 1 "B72510E250K062" V 1650 2050 50  0000 C CNN
+F 2 "Capacitor_SMD:C_0805_2012Metric" V 1730 1850 50  0001 C CNN
+F 3 "https://www.mouser.se/ProductDetail/EPCOS-TDK/B72510E0250K062/?qs=%2fha2pyFadugVCK9yiqateTD%252bWTZyWxpU55VnsqI3B1Kd%2fbUd9GEicg%3d%3d" H 1800 1850 50  0001 C CNN
+	1    1800 1850
+	1    0    0    1
 $EndComp
 $Comp
@@
 Wire Wire Line
 	3150 1700 3050 1700
+Wire Wire Line
+	2100 1700 1800 1700
+Wire Wire Line
+	1800 2000 2100 2000
+Connection ~ 2100 2000
+Wire Wire Line
+	2750 1700 2450 1700
+Connection ~ 2750 1700
+Connection ~ 2450 1700
+Connection ~ 2750 2000
 $EndSCHEMATC
