File: G3/Power.sch (KiCad schematic (older format))
At the start: 24 parts, among them J201 GS2, J202 GS2, U201 LM1084-3.3, U202 LM1084-5.0

Commit message: Use smaller TR5 fuse holders
Parts:
- F201, F202, F203: footprint Fuse:Fuseholder_Cylinder-5x20mm_Schurter_0031_8201_Horizontal_Open -> Fuse:Fuseholder_TR5_Littlefuse_No560_No460
Changed lines of the file:
@@
 	1    0    0    -1
 $EndComp
-Text Notes 6450 2200 0    60   ~ 0
+Text Notes 6450 2150 0    60   ~ 0
 Max 5A / 16.5 W
 $Comp
@@
 F 0 "F201" V 1403 2500 50  0000 C CNN
 F 1 "3.5A" V 1494 2500 50  0000 C CNN
-F 2 "Fuse:Fuseholder_Cylinder-5x20mm_Schurter_0031_8201_Horizontal_Open" V 1530 2500 50  0001 C CNN
+F 2 "Fuse:Fuseholder_TR5_Littlefuse_No560_No460" V 1530 2500 50  0001 C CNN
 F 3 "https://www.mouser.se/ProductDetail/Schurter/00318201?qs=sGAEpiMZZMtRmoYvq3OwzLrTj1%252b%252bxBWBiZ2DdJg9oKI%3d" H 1600 2500 50  0001 C CNN
 	1    1600 2500
@@
 F 0 "F202" V 4703 2500 50  0000 C CNN
 F 1 "5A" V 4794 2500 50  0000 C CNN
-F 2 "Fuse:Fuseholder_Cylinder-5x20mm_Schurter_0031_8201_Horizontal_Open" V 4830 2500 50  0001 C CNN
+F 2 "Fuse:Fuseholder_TR5_Littlefuse_No560_No460" V 4830 2500 50  0001 C CNN
 F 3 "https://www.mouser.se/ProductDetail/Schurter/00318201?qs=sGAEpiMZZMtRmoYvq3OwzLrTj1%252b%252bxBWBiZ2DdJg9oKI%3d" H 4900 2500 50  0001 C CNN
 	1    4900 2500
@@
 F 0 "F203" V 4703 3200 50  0000 C CNN
 F 1 "5A" V 4794 3200 50  0000 C CNN
-F 2 "Fuse:Fuseholder_Cylinder-5x20mm_Schurter_0031_8201_Horizontal_Open" V 4830 3200 50  0001 C CNN
+F 2 "Fuse:Fuseholder_TR5_Littlefuse_No560_No460" V 4830 3200 50  0001 C CNN
 F 3 "https://www.mouser.se/ProductDetail/Schurter/00318201?qs=sGAEpiMZZMtRmoYvq3OwzLrTj1%252b%252bxBWBiZ2DdJg9oKI%3d" H 4900 3200 50  0001 C CNN
 	1    4900 3200

Commit message: PCB started
Connections:
- net labels added: 3.3V_PWR_after_switch, 5V_PWR_after_switch
- net labels removed: 12V_filtered
Changed lines of the file:
@@
 	-1   0    0    1
 $EndComp
-Text Label 2850 3150 1    50   ~ 0
-12V_filtered
 $Comp
 L power:+12V #PWR?
@@
 Wire Wire Line
 	6200 2500 7300 2500
+Text Label 4650 3200 3    50   ~ 0
+5V_PWR_after_switch
+Text Label 4700 2500 1    50   ~ 0
+3.3V_PWR_after_switch
 $EndSCHEMATC

Commit message: Changes to input and outputs
Parts:
- added J201: Conn_02x02_Top_Bottom, Connector_Molex:Molex_Mega-Fit_76825-0004_2x02_P5.70mm_Horizontal, symbol Connector_Generic:Conn_02x02_Top_Bottom
- renumbered J201 to J202, J202 to J203
Connections:
- net labels removed: +12V_IN, GND_IN
- wire segments 36 -> 34
- no-connect marks 0 -> 2
Other:
- moved on the sheet: U202

Commit message: Changed special power supply connector to free contacts at regular connector. Moved power LEDs.
Parts:
- removed J201: Conn_02x02_Top_Bottom, Connector_Molex:Molex_Mega-Fit_76825-0004_2x02_P5.70mm_Horizontal, symbol Connector_Generic:Conn_02x02_Top_Bottom
Connections:
- net labels added: POWER_SUPPLY_12V
- no-connect marks 2 -> 0
Changed lines of the file:
@@
 	-1   0    0    1
-$EndComp
-$Comp
-L power:GND #PWR0202
-U 1 1 5B3933C3
-P 2000 2550
-F 0 "#PWR0202" H 2000 2300 50  0001 C CNN
-F 1 "GND" H 2005 2377 50  0000 C CNN
-F 2 "" H 2000 2550 50  0001 C CNN
-F 3 "" H 2000 2550 50  0001 C CNN
-	1    2000 2550
-	1    0    0    -1
 $EndComp
 Wire Wire Line
@@
 Text Label 5450 2450 1    50   ~ 0
 3.3V_PWR_after_switch
-$Comp
-L Connector_Generic:Conn_02x02_Top_Bottom J?
-U 1 1 5BA02922
-P 1800 2550
-AR Path="/5BA02922" Ref="J?"  Part="1"
-AR Path="/5B61ECB9/5BA02922" Ref="J201"  Part="1"
-F 0 "J201" H 1850 2225 50  0000 C CNN
-F 1 "Conn_02x02_Top_Bottom" H 1850 2316 50  0000 C CNN
-F 2 "Connector_Molex:Molex_Mega-Fit_76825-0004_2x02_P5.70mm_Horizontal" H 1800 2550 50  0001 C CNN
-F 3 "https://www.mouser.se/ProductDetail/Molex/76825-0002?qs=%2fha2pyFadug9gwVXW%252b6PjoTJPsbwjZb7D5oQ430PjGyxKDLr9emXmA%3d%3d" H 1800 2550 50  0001 C CNN
-	1    1800 2550
-	-1   0    0    1
-$EndComp
-NoConn ~ 1500 2450
-NoConn ~ 1500 2550
-Connection ~ 2000 2450
+Text GLabel 2000 2450 0    50   Input ~ 0
+POWER_SUPPLY_12V
 $EndSCHEMATC

Commit message: #Updated with Mouser-links for all components.
Parts:
- D201: value Power -> Red
- D206: value Power3V3 -> Red
- D207: value Power5V -> Red
- F201: value 3.5A -> xA
- F202, F203: value 5A -> xA
Changed lines of the file:
@@
 F 1 "100n" H 6565 2555 50  0000 L CNN
 F 2 "Capacitor_SMD:C_0805_2012Metric" H 6488 2450 50  0001 C CNN
-F 3 "https://www.mouser.se/ProductDetail/77-VJ0805Y104JXARBC" H 6450 2600 50  0001 C CNN
+F 3 "https://www.mouser.se/ProductDetail/KEMET/C0805C104J5RACTU?qs=sGAEpiMZZMs0AnBnWHyRQFCCI5cSbRT%2fIwsdZoDYv9I%3d" H 6450 2600 50  0001 C CNN
 	1    6450 2600
 	1    0    0    -1
@@
 F 1 "100n" H 6565 3255 50  0000 L CNN
 F 2 "Capacitor_SMD:C_0805_2012Metric" H 6488 3150 50  0001 C CNN
-F 3 "https://www.mouser.se/ProductDetail/77-VJ0805Y104JXARBC" H 6450 3300 50  0001 C CNN
+F 3 "https://www.mouser.se/ProductDetail/KEMET/C0805C104J5RACTU?qs=sGAEpiMZZMs0AnBnWHyRQFCCI5cSbRT%2fIwsdZoDYv9I%3d" H 6450 3300 50  0001 C CNN
 	1    6450 3300
 	1    0    0    -1
@@
 F 1 "100n" H 4315 3255 50  0000 L CNN
 F 2 "Capacitor_SMD:C_0805_2012Metric" H 4238 3150 50  0001 C CNN
-F 3 "https://www.mouser.se/ProductDetail/77-VJ0805Y104JXARBC" H 4200 3300 50  0001 C CNN
+F 3 "https://www.mouser.se/ProductDetail/KEMET/C0805C104J5RACTU?qs=sGAEpiMZZMs0AnBnWHyRQFCCI5cSbRT%2fIwsdZoDYv9I%3d" H 4200 3300 50  0001 C CNN
 	1    4200 3300
 	1    0    0    -1
@@
 F 1 "100n" H 4315 2555 50  0000 L CNN
 F 2 "Capacitor_SMD:C_0805_2012Metric" H 4238 2450 50  0001 C CNN
-F 3 "https://www.mouser.se/ProductDetail/77-VJ0805Y104JXARBC" H 4200 2600 50  0001 C CNN
+F 3 "https://www.mouser.se/ProductDetail/KEMET/C0805C104J5RACTU?qs=sGAEpiMZZMs0AnBnWHyRQFCCI5cSbRT%2fIwsdZoDYv9I%3d" H 4200 2600 50  0001 C CNN
 	1    4200 2600
 	1    0    0    -1
@@
 P 2350 2450
 F 0 "F201" V 2153 2450 50  0000 C CNN
-F 1 "3.5A" V 2244 2450 50  0000 C CNN
+F 1 "xA" V 2244 2450 50  0000 C CNN
 F 2 "Fuse:Fuseholder_TR5_Littlefuse_No560_No460" V 2280 2450 50  0001 C CNN
-F 3 "https://www.mouser.se/ProductDetail/Schurter/00318201?qs=sGAEpiMZZMtRmoYvq3OwzLrTj1%252b%252bxBWBiZ2DdJg9oKI%3d" H 2350 2450 50  0001 C CNN
+F 3 "https://www.mouser.se/ProductDetail/Littelfuse/56000001019?qs=sGAEpiMZZMtRmoYvq3OwzKEcK5xXAR8uiSqvDZfRA1w%3d" H 2350 2450 50  0001 C CNN
 	1    2350 2450
 	0    1    1    0
@@
 P 5650 2450
 F 0 "F202" V 5453 2450 50  0000 C CNN
-F 1 "5A" V 5544 2450 50  0000 C CNN
+F 1 "xA" V 5544 2450 50  0000 C CNN
 F 2 "Fuse:Fuseholder_TR5_Littlefuse_No560_No460" V 5580 2450 50  0001 C CNN
-F 3 "https://www.mouser.se/ProductDetail/Schurter/00318201?qs=sGAEpiMZZMtRmoYvq3OwzLrTj1%252b%252bxBWBiZ2DdJg9oKI%3d" H 5650 2450 50  0001 C CNN
+F 3 "https://www.mouser.se/ProductDetail/Littelfuse/56000001019?qs=sGAEpiMZZMtRmoYvq3OwzKEcK5xXAR8uiSqvDZfRA1w%3d" H 5650 2450 50  0001 C CNN
 	1    5650 2450
 	0    1    1    0
@@
 P 5650 3150
 F 0 "F203" V 5453 3150 50  0000 C CNN
-F 1 "5A" V 5544 3150 50  0000 C CNN
+F 1 "xA" V 5544 3150 50  0000 C CNN
 F 2 "Fuse:Fuseholder_TR5_Littlefuse_No560_No460" V 5580 3150 50  0001 C CNN
-F 3 "https://www.mouser.se/ProductDetail/Schurter/00318201?qs=sGAEpiMZZMtRmoYvq3OwzLrTj1%252b%252bxBWBiZ2DdJg9oKI%3d" H 5650 3150 50  0001 C CNN
+F 3 "https://www.mouser.se/ProductDetail/Littelfuse/56000001019?qs=sGAEpiMZZMtRmoYvq3OwzKEcK5xXAR8uiSqvDZfRA1w%3d" H 5650 3150 50  0001 C CNN
 	1    5650 3150
 	0    1    1    0
@@
 P 3750 1850
 F 0 "D201" H 3742 1595 50  0000 C CNN
-F 1 "Power" H 3742 1686 50  0000 C CNN
+F 1 "Red" H 3742 1686 50  0000 C CNN
 F 2 "LED_THT:LED_D5.0mm" H 3750 1850 50  0001 C CNN
 F 3 "https://www.mouser.se/ProductDetail/Lite-On/LTL2R3KGD-EM?qs=sGAEpiMZZMtmwHDZQCdlqY3QuPVQdrfivxVgVo2hFbg%3d" H 3750 1850 50  0001 C CNN
@@
 P 8500 2450
 F 0 "D206" H 8492 2195 50  0000 C CNN
-F 1 "Power3V3" H 8492 2286 50  0000 C CNN
+F 1 "Red" H 8492 2286 50  0000 C CNN
 F 2 "LED_THT:LED_D5.0mm" H 8500 2450 50  0001 C CNN
 F 3 "https://www.mouser.se/ProductDetail/Lite-On/LTL2R3KGD-EM?qs=sGAEpiMZZMtmwHDZQCdlqY3QuPVQdrfivxVgVo2hFbg%3d" H 8500 2450 50  0001 C CNN
@@
 P 8550 3150
 F 0 "D207" H 8542 2895 50  0000 C CNN
-F 1 "Power5V" H 8542 2986 50  0000 C CNN
+F 1 "Red" H 8542 2986 50  0000 C CNN
 F 2 "LED_THT:LED_D5.0mm" H 8550 3150 50  0001 C CNN
 F 3 "https://www.mouser.se/ProductDetail/Lite-On/LTL2R3KGD-EM?qs=sGAEpiMZZMtmwHDZQCdlqY3QuPVQdrfivxVgVo2hFbg%3d" H 8550 3150 50  0001 C CNN
