File: G3/Power.sch (KiCad schematic (older format))
At the start: 24 parts, among them J202 GS2, J203 GS2, U201 LM1084-3.3, U202 LM1084-5.0

Commit message: Changed footprint of J202 and J203. Regenerated manufacturing files.
Parts:
- J202, J203: footprint Connector_PinHeader_2.54mm:PinHeader_1x02_P2.54mm_Vertical_SMD_Pin1Left -> Connector_PinHeader_2.54mm:PinHeader_1x02_P2.54mm_Vertical
Changed lines of the file:
@@
 F 0 "J202" V 5400 2200 50  0000 C CNN
 F 1 "GS2" V 5300 2400 50  0000 C CNN
-F 2 "Connector_PinHeader_2.54mm:PinHeader_1x02_P2.54mm_Vertical_SMD_Pin1Left" V 5374 2250 50  0001 C CNN
+F 2 "Connector_PinHeader_2.54mm:PinHeader_1x02_P2.54mm_Vertical" V 5374 2250 50  0001 C CNN
 F 3 "" H 5300 2250 50  0001 C CNN
 	1    5300 2250
@@
 F 0 "J203" V 5400 2900 50  0000 C CNN
 F 1 "GS2" V 5250 3100 50  0000 C CNN
-F 2 "Connector_PinHeader_2.54mm:PinHeader_1x02_P2.54mm_Vertical_SMD_Pin1Left" V 5374 2950 50  0001 C CNN
+F 2 "Connector_PinHeader_2.54mm:PinHeader_1x02_P2.54mm_Vertical" V 5374 2950 50  0001 C CNN
 F 3 "" H 5300 2950 50  0001 C CNN
 	1    5300 2950
