File: G3/SDCard.sch (KiCad schematic (older format))
At the start: 16 parts, among them J401 Micro_SD_Card_Det

Commit message: MMC and SPI mode for SDCard
Parts:
- added J402: SDCard MMC mode, Connector_PinHeader_2.54mm:PinHeader_2x06_P2.54mm_Vertical, symbol Connector_Generic:Conn_02x06_Odd_Even
- added J403: SDCard SPI mode, Connector_PinHeader_2.54mm:PinHeader_2x04_P2.54mm_Vertical, symbol Connector_Generic:Conn_02x04_Odd_Even
Connections:
- net labels added: SD_SPI_CLK, SD_SPI_CS, SD_SPI_MISO, SD_SPI_MOSI
- wire segments 35 -> 53
Other:
- note added: "http://www.interfacebus.com/MicroSD_Card_Pinout.html"

Commit message: Using MAX4948 instead of DIPs
Parts:
- removed J402: SDCard MMC mode, Connector_PinHeader_2.54mm:PinHeader_2x06_P2.54mm_Vertical, symbol Connector_Generic:Conn_02x06_Odd_Even
- removed J403: SDCard SPI mode, Connector_PinHeader_2.54mm:PinHeader_2x04_P2.54mm_Vertical, symbol Connector_Generic:Conn_02x04_Odd_Even
- added C401: 100n, Capacitor_SMD:C_0805_2012Metric, symbol Device:C
- added D401: SD SPI Selected/JTAG supported, LED_THT:LED_D5.0mm_Clear, symbol Device:LED
- added R407: 10k, Resistor_SMD:R_0805_2012Metric, symbol Device:R
- added R408: 165, Resistor_SMD:R_0805_2012Metric, symbol Device:R
- added SW401: SD SPI/MMC mode, Button_Switch_SMD:SW_DIP_SPSTx01_Slide_Omron_A6S-110x_W8.9mm_P2.54mm, symbol Switch:SW_DIP_x01
- added U401: MAX4948, Package_DFN_QFN:QFN-24-1EP_4x4mm_P0.5mm_EP2.6x2.6mm_ThermalVias, symbol PerMalmberg:MAX4948
- renumbered C401 to C402, C402 to C403, D401 to D402, D402 to D403, D403 to D404, D404 to D405, D405 to D406, D406 to D407, R402 to R401, R401 to R402, R406 to R403, R405 to R404, R403 to R405, R404 to R406, R407 to R409
Connections:
- net labels added: SD_ENABLE, SD_MMC_CLK, SD_MMC_CMD, SD_MMC_DATA0, SD_MMC_DATA1, SD_MMC_Data2, SD_MMC_Data3, SD_MODE
- wire segments 53 -> 37
- no-connect marks 0 -> 2
Other:
- note added: "MMC Signals"
- note added: "On = SPI mode and\nJTAG support"
- note added: "Place near MAX4948"
- note added: "SPI signals"

Commit message: WiP PCB
Connections:
- net labels added: SD_SPI_CLK_CARD, SD_SPI_CS_CARD, SD_SPI_MISO_CARD, SD_SPI_MOSI_CARD
Other:
- note added: "https://www.acmesystems.it/pcb_microsd"
Changed lines of the file:
@@
 Wire Wire Line
 	6750 3000 6900 3000
-Text Label 7100 2400 2    50   ~ 0
-SD_SPI_MOSI
-Text Label 7100 2800 2    50   ~ 0
-SD_SPI_MISO
-Text Label 7100 2300 2    50   ~ 0
-SD_SPI_CS
-Text Label 7100 2600 2    50   ~ 0
-SD_SPI_CLK
+Text Label 7300 2400 2    50   ~ 0
+SD_SPI_MOSI_CARD
+Text Label 7300 2800 2    50   ~ 0
+SD_SPI_MISO_CARD
+Text Label 7300 2300 2    50   ~ 0
+SD_SPI_CS_CARD
+Text Label 7300 2600 2    50   ~ 0
+SD_SPI_CLK_CARD
 Text Notes 8050 3800 0    50   ~ 0
 http://www.interfacebus.com/MicroSD_Card_Pinout.html
@@
 SD_MMC_Data2
 Text Label 2050 3550 2    50   ~ 0
-SD_DATA0
+SD_MMC_DATA0
 Text Label 3200 3750 0    50   ~ 0
 SD_MMC_Data3
@@
 	6600 2000 6600 2850
 Wire Notes Line
-	6600 2850 7150 2850
-Wire Notes Line
-	7150 2850 7150 2000
-Wire Notes Line
-	7150 2000 6600 2000
+	6600 2850 7300 2850
+Wire Notes Line
+	7300 2850 7300 2000
+Wire Notes Line
+	7300 2000 6600 2000
 Text Notes 6650 2100 0    50   ~ 0
 SPI signals
@@
 Text Notes 1400 5600 1    50   ~ 0
 Place near MAX4948
+Text Notes 8050 3950 0    50   ~ 0
+https://www.acmesystems.it/pcb_microsd
 $EndSCHEMATC

Commit message: WiP PCB
Changed lines of the file:
@@
 Text Notes 8050 3800 0    50   ~ 0
 http://www.interfacebus.com/MicroSD_Card_Pinout.html
-Text GLabel 3200 3650 2    50   Input ~ 0
+Text GLabel 2050 4250 0    50   Input ~ 0
 SD_SPI_CS
 Text GLabel 3200 4250 2    50   Input ~ 0
 SD_SPI_MOSI
+Text GLabel 2050 3950 0    50   Input ~ 0
+SD_SPI_CLK
 Text GLabel 3200 3950 2    50   Input ~ 0
-SD_SPI_CLK
-Text GLabel 2050 3650 0    50   Input ~ 0
 SD_SPI_MISO
 Wire Wire Line
@@
 Wire Wire Line
 	5900 2600 7400 2600
+Text Label 3200 3750 0    50   ~ 0
+SD_MMC_Data2
+Text Label 3200 4050 0    50   ~ 0
+SD_MMC_DATA0
 Text Label 2050 4150 2    50   ~ 0
-SD_MMC_Data2
+SD_MMC_Data3
 Text Label 2050 3550 2    50   ~ 0
-SD_MMC_DATA0
-Text Label 3200 3750 0    50   ~ 0
-SD_MMC_Data3
+SD_MMC_DATA1
 Text Label 2050 3850 2    50   ~ 0
-SD_MMC_DATA1
-Text Label 3200 4050 0    50   ~ 0
 SD_MMC_CLK
 Text Label 3200 4350 0    50   ~ 0
 SD_MMC_CMD
+Text GLabel 2050 3750 0    50   Input ~ 0
+SD_DATA1
+Text GLabel 3200 3850 2    50   Input ~ 0
+SD_DATA0
 Text GLabel 2050 4050 0    50   Input ~ 0
-SD_DATA1
-Text GLabel 2050 3750 0    50   Input ~ 0
-SD_DATA0
-Text GLabel 3200 3850 2    50   Input ~ 0
 SD_CLK
 Text GLabel 3200 4150 2    50   Input ~ 0
 SD_CMD
+Text GLabel 2050 4350 0    50   Input ~ 0
+SD_DATA3
 Text GLabel 3200 3550 2    50   Input ~ 0
-SD_DATA3
-Text GLabel 2050 4350 0    50   Input ~ 0
 SD_DATA2
 $Comp
@@
 SD_MODE
 Connection ~ 3000 2600
-NoConn ~ 2050 3950
-NoConn ~ 2050 4250
 Wire Notes Line
 	6600 2000 6600 2850
@@
 Text Notes 8050 3950 0    50   ~ 0
 https://www.acmesystems.it/pcb_microsd
+NoConn ~ 3200 3650
+NoConn ~ 2050 3650
 $EndSCHEMATC

Commit message: Texts and moutningholes.
Parts:
- D401: value SD SPI Selected/JTAG supported -> SPI/JTAG Active
Changed lines of the file:
@@
 AR Path="/5B61FB63/5B98DF5D/5BA18619" Ref="D401"  Part="1"
 F 0 "D401" V 3350 2850 50  0000 C CNN
-F 1 "SD SPI Selected/JTAG supported" V 3450 2350 50  0000 C CNN
+F 1 "SPI/JTAG Active" H 3400 3200 50  0000 C CNN
 F 2 "LED_THT:LED_D5.0mm_Clear" H 3450 3050 50  0001 C CNN
 F 3 "https://www.mouser.se/ProductDetail/Lumex/SSL-LX55103ID-FL?qs=sGAEpiMZZMtmwHDZQCdlqUPJk6OnVfwF%252bWo7zgs2%252bqE%3d" H 3450 3050 50  0001 C CNN

Commit message: #Updated with Mouser-links for all components.
Parts:
- D401: value SPI/JTAG Active -> Red; footprint LED_THT:LED_D5.0mm_Clear -> LED_THT:LED_D5.0mm
- R408: value 165 -> 1.65k
Changed lines of the file:
@@
 F 1 "100n" H 10185 2445 50  0000 R CNN
 F 2 "Capacitor_SMD:C_0805_2012Metric" H 10338 2250 50  0001 C CNN
-F 3 "https://www.mouser.se/ProductDetail/AVX/08055C104JAZ2A?qs=%2fha2pyFaduhAZO93RAy6IIlm7PKA7PN%2fjITVSPkVEftSFjliFvU6%2fw%3d%3d" H 10300 2400 50  0001 C CNN
+F 3 "https://www.mouser.se/ProductDetail/KEMET/C0805C104J5RACTU?qs=sGAEpiMZZMs0AnBnWHyRQFCCI5cSbRT%2fIwsdZoDYv9I%3d" H 10300 2400 50  0001 C CNN
 	1    10300 2400
 	-1   0    0    1
@@
 F 1 "10u" H 9950 2500 50  0000 C CNN
 F 2 "Capacitor_SMD:CP_Elec_5x4.5" H 9888 2250 50  0001 C CNN
-F 3 "" H 9850 2400 50  0001 C CNN
+F 3 "https://www.mouser.se/ProductDetail/710-865080440002" H 9850 2400 50  0001 C CNN
 	1    9850 2400
 	1    0    0    -1
@@
 F 1 "MAX4948" H 2600 5000 50  0000 C CNN
 F 2 "Package_DFN_QFN:QFN-24-1EP_4x4mm_P0.5mm_EP2.6x2.6mm_ThermalVias" H 2100 4500 50  0001 C CNN
-F 3 "" H 2100 4500 50  0001 C CNN
+F 3 "https://www.mouser.se/ProductDetail/Maxim-Integrated/MAX4948ETG%2b?qs=sGAEpiMZZMuuBt6TL7D%2f6HEUAj%252bJt3CD" H 2100 4500 50  0001 C CNN
 	1    2150 4500
 	1    0    0    -1
@@
 AR Path="/5B61FB63/5B98DF5D/5BA18619" Ref="D401"  Part="1"
 F 0 "D401" V 3350 2850 50  0000 C CNN
-F 1 "SPI/JTAG Active" H 3400 3200 50  0000 C CNN
-F 2 "LED_THT:LED_D5.0mm_Clear" H 3450 3050 50  0001 C CNN
-F 3 "https://www.mouser.se/ProductDetail/Lumex/SSL-LX55103ID-FL?qs=sGAEpiMZZMtmwHDZQCdlqUPJk6OnVfwF%252bWo7zgs2%252bqE%3d" H 3450 3050 50  0001 C CNN
+F 1 "Red" H 3400 3200 50  0000 C CNN
+F 2 "LED_THT:LED_D5.0mm" H 3450 3050 50  0001 C CNN
+F 3 "https://www.mouser.se/ProductDetail/Lite-On/LTL2R3KGD-EM?qs=sGAEpiMZZMtmwHDZQCdlqY3QuPVQdrfivxVgVo2hFbg%3d" H 3450 3050 50  0001 C CNN
 	1    3450 3050
 	0    -1   -1   0
@@
 AR Path="/5B61FB63/5B98DF5D/5BA18621" Ref="R408"  Part="1"
 F 0 "R408" V 3243 2750 50  0000 C CNN
-F 1 "165" V 3334 2750 50  0000 C CNN
+F 1 "1.65k" V 3334 2750 50  0000 C CNN
 F 2 "Resistor_SMD:R_0805_2012Metric" V 3380 2750 50  0001 C CNN
-F 3 "https://www.mouser.se/ProductDetail/Bourns/CR0805-FX-1650ELF?qs=sGAEpiMZZMtlubZbdhIBIKn39ibjI6WbHbnDBzjqA1U%3d" H 3450 2750 50  0001 C CNN
+F 3 "https://www.mouser.se/ProductDetail/Vishay/CRCW08051K65FKEA?qs=sGAEpiMZZMtlubZbdhIBIFvv2%252blmU1cYk%2fKBbkOVYDU%3d" H 3450 2750 50  0001 C CNN
 	1    3450 2750
 	-1   0    0    1
@@
 F 1 "100n" H 1435 5295 50  0000 R CNN
 F 2 "Capacitor_SMD:C_0805_2012Metric" H 1588 5100 50  0001 C CNN
-F 3 "https://www.mouser.se/ProductDetail/AVX/08055C104JAZ2A?qs=%2fha2pyFaduhAZO93RAy6IIlm7PKA7PN%2fjITVSPkVEftSFjliFvU6%2fw%3d%3d" H 1550 5250 50  0001 C CNN
+F 3 "https://www.mouser.se/ProductDetail/KEMET/C0805C104J5RACTU?qs=sGAEpiMZZMs0AnBnWHyRQFCCI5cSbRT%2fIwsdZoDYv9I%3d" H 1550 5250 50  0001 C CNN
 	1    1550 5250
 	-1   0    0    1
