File: G3/SelectableVoltageOutput.sch (KiCad schematic (older format))
At the start: 8 parts, among them J1601 Power_select, Q1601 ZXTN25050DFHTA, Q1602 ZXTN25050DFHTA

Commit message: #Updated with Mouser-links for all components.
Parts:
- D1601: footprint LED_THT:LED_D5.0mm_Clear -> LED_THT:LED_D5.0mm
- R1603: value 165 -> 1.65k
Changed lines of the file:
@@
 AR Path="/5B62EDB8/5BA2E71A/5B8D6899" Ref="Q2301"  Part="1"
 AR Path="/5B62EDB8/5BA3564E/5B8D6899" Ref="Q2601"  Part="1"
-F 0 "Q2601" V 3750 1800 50  0000 L CNN
+F 0 "Q2301" V 3750 1800 50  0000 L CNN
 F 1 "ZXTN25050DFHTA" H 3800 1750 50  0000 L CNN
 F 2 "Package_TO_SOT_SMD:SOT-23" H 3750 1950 50  0001 C CNN
-F 3 "" H 3550 1850 50  0001 C CNN
+F 3 "https://www.mouser.se/ProductDetail/Diodes-Incorporated/ZXTN25050DFHTA?qs=sGAEpiMZZMshyDBzk1%2fWi6gR%252bqBmAG1j52KxSCCDz6c%3d" H 3550 1850 50  0001 C CNN
 	1    3550 1850
 	1    0    0    -1
@@
 AR Path="/5B62EDB8/5BA2E71A/5BA36D5C" Ref="R2301"  Part="1"
 AR Path="/5B62EDB8/5BA3564E/5BA36D5C" Ref="R2601"  Part="1"
-F 0 "R2601" V 2450 2300 50  0000 C CNN
+F 0 "R2301" V 2450 2300 50  0000 C CNN
 F 1 "470" V 2550 2300 50  0000 C CNN
 F 2 "Resistor_SMD:R_0805_2012Metric" V 2480 2300 50  0001 C CNN
@@
 AR Path="/5B62EDB8/5BA2E71A/5BA36D5F" Ref="R2302"  Part="1"
 AR Path="/5B62EDB8/5BA3564E/5BA36D5F" Ref="R2602"  Part="1"
-F 0 "R2602" H 3070 2496 50  0000 L CNN
+F 0 "R2302" H 3070 2496 50  0000 L CNN
 F 1 "10k" H 3070 2405 50  0000 L CNN
 F 2 "Resistor_SMD:R_0805_2012Metric" V 2930 2450 50  0001 C CNN
@@
 AR Path="/5B62EDB8/5BA2E71A/5BA13007" Ref="J2301"  Part="1"
 AR Path="/5B62EDB8/5BA3564E/5BA13007" Ref="J2601"  Part="1"
-F 0 "J2601" H 1600 1175 50  0000 C CNN
+F 0 "J2301" H 1600 1175 50  0000 C CNN
 F 1 "Power_select" H 1600 1266 50  0000 C CNN
 F 2 "Connector_PinHeader_2.54mm:PinHeader_1x03_P2.54mm_Vertical" V 1688 1426 50  0001 C CNN
-F 3 "" H 1600 1500 50  0001 C CNN
+F 3 "https://www.mouser.se/ProductDetail/Molex/22-28-0030?qs=sGAEpiMZZMs%252bGHln7q6pmxD%2f5kNJnZVeZCYy0rFr0qA%3d" H 1600 1500 50  0001 C CNN
 	1    1600 1500
 	-1   0    0    1
@@
 AR Path="/5B62EDB8/5BA2E71A/5BA36D69" Ref="F2301"  Part="1"
 AR Path="/5B62EDB8/5BA3564E/5BA36D69" Ref="F2601"  Part="1"
-F 0 "F2601" V 2553 1500 50  0000 C CNN
+F 0 "F2301" V 2553 1500 50  0000 C CNN
 F 1 "xA" V 2644 1500 50  0000 C CNN
 F 2 "Fuse:Fuseholder_TR5_Littlefuse_No560_No460" V 2680 1500 50  0001 C CNN
-F 3 "https://www.mouser.se/ProductDetail/Schurter/00318201?qs=sGAEpiMZZMtRmoYvq3OwzLrTj1%252b%252bxBWBiZ2DdJg9oKI%3d" H 2750 1500 50  0001 C CNN
+F 3 "https://www.mouser.se/ProductDetail/Littelfuse/56000001019?qs=sGAEpiMZZMtRmoYvq3OwzKEcK5xXAR8uiSqvDZfRA1w%3d" H 2750 1500 50  0001 C CNN
 	1    2750 1500
 	0    1    1    0
@@
 AR Path="/5B62EDB8/5BA2E71A/5BA36D6B" Ref="R2303"  Part="1"
 AR Path="/5B62EDB8/5BA3564E/5BA36D6B" Ref="R2603"  Part="1"
-F 0 "R2603" V 3443 3050 50  0000 C CNN
-F 1 "165" V 3534 3050 50  0000 C CNN
+F 0 "R2303" V 3443 3050 50  0000 C CNN
+F 1 "1.65k" V 3534 3050 50  0000 C CNN
 F 2 "Resistor_SMD:R_0805_2012Metric" V 3580 3050 50  0001 C CNN
-F 3 "https://www.mouser.se/ProductDetail/Bourns/CR0805-FX-1650ELF?qs=sGAEpiMZZMtlubZbdhIBIKn39ibjI6WbHbnDBzjqA1U%3d" H 3650 3050 50  0001 C CNN
+F 3 "https://www.mouser.se/ProductDetail/Vishay/CRCW08051K65FKEA?qs=sGAEpiMZZMtlubZbdhIBIFvv2%252blmU1cYk%2fKBbkOVYDU%3d" H 3650 3050 50  0001 C CNN
 	1    3650 3050
 	-1   0    0    1
@@
 AR Path="/5B62EDB8/5BA2E71A/5BA36D6E" Ref="D2301"  Part="1"
 AR Path="/5B62EDB8/5BA3564E/5BA36D6E" Ref="D2601"  Part="1"
-F 0 "D2601" H 3642 3095 50  0000 C CNN
+F 0 "D2301" H 3642 3095 50  0000 C CNN
 F 1 "Green" H 3642 3186 50  0000 C CNN
-F 2 "LED_THT:LED_D5.0mm_Clear" H 3650 3350 50  0001 C CNN
-F 3 "https://www.mouser.se/ProductDetail/Lumex/SSL-LX55103GD-FL?qs=sGAEpiMZZMtmwHDZQCdlqVsz6Sp3LtaXcNplsbJfBSw%3d" H 3650 3350 50  0001 C CNN
+F 2 "LED_THT:LED_D5.0mm" H 3650 3350 50  0001 C CNN
+F 3 "https://www.mouser.se/ProductDetail/Lite-On/LTL2R3KGD-EM?qs=sGAEpiMZZMtmwHDZQCdlqY3QuPVQdrfivxVgVo2hFbg%3d" H 3650 3350 50  0001 C CNN
 	1    3650 3350
 	0    -1   -1   0
@@
 AR Path="/5B62EDB8/5BA2E71A/5BA36D74" Ref="Q2302"  Part="1"
 AR Path="/5B62EDB8/5BA3564E/5BA36D74" Ref="Q2602"  Part="1"
-F 0 "Q2602" V 3750 2650 50  0000 L CNN
+F 0 "Q2302" V 3750 2650 50  0000 L CNN
 F 1 "ZXTN25050DFHTA" H 3800 2600 50  0000 L CNN
 F 2 "Package_TO_SOT_SMD:SOT-23" H 3750 2800 50  0001 C CNN
-F 3 "" H 3550 2700 50  0001 C CNN
+F 3 "https://www.mouser.se/ProductDetail/Diodes-Incorporated/ZXTN25050DFHTA?qs=sGAEpiMZZMshyDBzk1%2fWi6gR%252bqBmAG1j52KxSCCDz6c%3d" H 3550 2700 50  0001 C CNN
 	1    3550 2700
 	1    0    0    -1
