File: hardware/G3.kicad_pcb (KiCad board)
At the start: 2 copper layers, 191.3 x 181.7 mm, 338 parts, among them J1501 Digital input supply, J1502 Digital input GND, J1601 Power_select, J1701 Power_select, J1801 Power_select, J1901 Power_select, J2001 Power_select, J202 GS2, J203 GS2, J2101 Power_select, J2201 Power_select, J2301 Power_select, J2601 Power_select, J2801 Digital input supply, J2802 Digital input GND, J2901 Digital input supply, J2902 Digital input GND, J3001 Digital input supply, J3002 Digital input GND, J301 Debug, J302 BME280, J3101 Digital input supply, J3102 Digital input GND, J3201 Digital input supply, J3202 Digital input GND, J3301 Digital input supply, J3302 Digital input GND, J3401 Digital input supply, J3402 Digital input GND, J3501 Sense, J3502 Digital Input, J3503 Sense, J3504 Digital input, J3505 Power 12/5/3, J3506 Digital input, J3507 Digital Output, J3508 Digital output, J3509 Digital output, J401 Micro_SD_Card_Det, Q1601 ZXTN25050DFHTA, Q1602 ZXTN25050DFHTA, Q1701 ZXTN25050DFHTA, Q1702 ZXTN25050DFHTA, Q1801 ZXTN25050DFHTA, Q1802 ZXTN25050DFHTA, Q1901 ZXTN25050DFHTA, Q1902 ZXTN25050DFHTA, Q2001 ZXTN25050DFHTA, Q2002 ZXTN25050DFHTA, Q2101 ZXTN25050DFHTA, Q2102 ZXTN25050DFHTA, Q2201 ZXTN25050DFHTA, Q2202 ZXTN25050DFHTA, Q2301 ZXTN25050DFHTA, Q2302 ZXTN25050DFHTA, Q2401 ZXTN25050DFHTA, Q2402 ZXTN25050DFHTA, Q2601 ZXTN25050DFHTA, Q2602 ZXTN25050DFHTA, Q2701 ZXTN25050DFHTA, Q2702 ZXTN25050DFHTA, SW301 Boot option, SW302 Reset, SW303 Factory reset, SW401 SD SPI/MMC mode, U1401 MCP23017, U1402 MCP23017, U1501 LTV-354T, U201 LM1084-3.3, U202 LM1084-5.0, U2801 LTV-354T, U2901 LTV-354T, U3001 LTV-354T, U301 ESP32_WROVER, U302 TXB0102DCU, U3101 LTV-354T, U3201 LTV-354T, U3301 LTV-354T, U3401 LTV-354T, U401 MAX4948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

Commit message: #5 - Moved All SD pullup resistors except R406 (SD_DATA2/MTDI/GPIO12) to SD-side of MAX4948. #3 - Added jumper for GPIO2 <-> GPOI0 for flash download. Removed affected items from PCB.
Parts:
- removed SW401: SD SPI/MMC mode, Button_Switch_SMD:SW_DIP_SPSTx01_Slide_Omron_A6S-110x_W8.9mm_P2.54mm
- added SW1: SD SPI/MMC mode, Button_Switch_SMD:SW_DIP_SPSTx02_Slide_Omron_A6S-210x_W8.9mm_P2.54mm, F.Cu at (99.7, 136.8)
- R401, R402, R403, R404, R405, R406: value 10k -> 50k
- moved R405 73.4 mm to (5.39, 122.9), turned to 0 degrees
- moved R402 67.9 mm to (5.39, 120.9), turned to 0 degrees
- moved R406 54.2 mm to (8.80, 120.9), turned to 0 degrees
- moved R401 53.4 mm to (8.80, 119.0)
- moved R403 51.2 mm to (5.39, 119.0), turned to 0 degrees
- moved R404 46.8 mm to (12.2, 119.0), turned to 0 degrees
- moved D402 30.5 mm to (12.8, 128.9)
- moved D404 30.5 mm to (7.20, 128.9)
- moved D407 30.5 mm to (-2.45, 128.9)
- moved D403 30.5 mm to (9.99, 128.9)
- moved D405 30.5 mm to (4.03, 128.9)
- moved D406 30.5 mm to (0.60, 128.9)
Connections:
- net /MCU/Boot_option renamed BootOption
- D402 pad 1: /MCU/SDCard/SD_MMC_Data2 -> /MCU/SDCard/SD_MMC_DATA1
- D403 pad 1: /MCU/SDCard/SD_MMC_Data3 -> /MCU/SDCard/SD_MMC_DATA0
- D404 pad 1: /MCU/SDCard/SD_MMC_CMD -> /MCU/SDCard/SD_MMC_CLK
- D405 pad 1: /MCU/SDCard/SD_MMC_CLK -> /MCU/SDCard/SD_MMC_CMD
- D406 pad 1: /MCU/SDCard/SD_MMC_DATA0 -> /MCU/SDCard/SD_MMC_Data3
- D407 pad 1: /MCU/SDCard/SD_MMC_DATA1 -> /MCU/SDCard/SD_MMC_Data2
- R401 pad 2: SD_DATA0 -> /MCU/SDCard/SD_MMC_DATA1
- R402 pad 2: SD_DATA1 -> /MCU/SDCard/SD_MMC_DATA0
- R403 pad 2: SD_DATA2 -> /MCU/SDCard/SD_MMC_CLK
- R404 pad 2: SD_DATA3 -> /MCU/SDCard/SD_MMC_CMD
- R405 pad 2: SD_CLK -> /MCU/SDCard/SD_MMC_Data3
- R406 pad 2: SD_CMD -> SD_DATA2
Routing:
- net DO7_PWR: track 44.4 -> 0.00 mm
- net BELL_PWR: track 56.7 -> 14.1 mm
- net DO6_PWR: track 39.5 -> 0.00 mm
- net +3V3: track 1127.2 -> 1101.0 mm, vias 32 -> 28
- net /MCU/SDCard/SD_MMC_DATA1: track 45.8 -> 21.6 mm
- net /MCU/SDCard/SD_MMC_DATA0: track 32.4 -> 10.8 mm
- net DO2_PWR: track 21.1 -> 0.00 mm
- net /MCU/SDCard/SD_MMC_CLK: track 37.0 -> 18.1 mm
- net /MCU/SDCard/SD_MMC_CMD: track 34.7 -> 18.7 mm
- net SD_DATA0: track 40.5 -> 25.3 mm
- net GND: track 29.0 -> 14.1 mm, vias 302 -> 2
- net /MCU/SDCard/SD_MMC_Data3: track 20.7 -> 7.31 mm
- net /MCU/SDCard/SD_MMC_Data2: track 19.9 -> 10.7 mm
- net SD_CMD: track 41.0 -> 33.8 mm
- net SD_DATA1: track 25.7 -> 19.9 mm
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
Commit message: #1 SD_ENABLE removed; pin grounded. #7 All pins on seconds MCP2317 used. Updated I2CTask to match new H/W layout. Closes #1. Closes #7.
Parts:
- removed R1402: 10k, Resistor_SMD:R_0805_2012Metric
- added C1: 100n, Capacitor_SMD:C_0805_2012Metric, F.Cu at (-9.38, 66.8)
- added D1: Red, LED_THT:LED_D5.0mm, F.Cu at (-23.2, 75.6)
- added D2: Red, LED_THT:LED_D5.0mm, F.Cu at (-29.7, 75.6)
- added D3: Red, LED_THT:LED_D5.0mm, F.Cu at (-23.2, 69.1)
- added D4: Red, LED_THT:LED_D5.0mm, F.Cu at (-36.2, 82.2)
- added D5: Red, LED_THT:LED_D5.0mm, F.Cu at (-36.2, 75.6)
- added D6: Red, LED_THT:LED_D5.0mm, F.Cu at (-42.7, 82.2)
- added D7: Red, LED_THT:LED_D5.0mm, F.Cu at (-49.2, 75.6)
- added R1: 1.65k, Resistor_SMD:R_0805_2012Metric, F.Cu at (-17.0, 68.7)
- added R2: 1.65k, Resistor_SMD:R_0805_2012Metric, F.Cu at (-17.0, 74.6)
- added R3: 1.65k, Resistor_SMD:R_0805_2012Metric, F.Cu at (-30.0, 79.9)
- added R4: 1.65k, Resistor_SMD:R_0805_2012Metric, F.Cu at (-17.0, 66.8)
- added R5: 1.65k, Resistor_SMD:R_0805_2012Metric, F.Cu at (-26.6, 79.9)
- added R6: 1.65k, Resistor_SMD:R_0805_2012Metric, F.Cu at (-17.0, 70.7)
- added R7: 1.65k, Resistor_SMD:R_0805_2012Metric, F.Cu at (-30.0, 81.8)
- added R9: 10k, Resistor_SMD:R_0805_2012Metric, F.Cu at (-9.38, 68.7)
- moved D1406 81.5 mm to (-42.7, 69.1), turned to 0 degrees
- moved D1402 78.4 mm to (-49.2, 69.1), turned to 0 degrees
- moved D1405 77.7 mm to (-49.2, 82.2), turned to 0 degrees
- moved D1403 73.3 mm to (-42.7, 75.6), turned to 0 degrees
- moved R1406 72.1 mm to (-30.0, 83.8)
- moved D1404 72.1 mm to (-36.2, 69.1), turned to 0 degrees
- moved R1407 69.7 mm to (-26.6, 81.8)
- moved R1403 69.4 mm to (-26.6, 83.8)
- moved D1401 67.1 mm to (-29.7, 69.1), turned to 0 degrees
- moved R1401 65.4 mm to (-23.2, 81.8)
- moved R1405 65.3 mm to (-23.2, 79.9)
- moved R1404 61.5 mm to (-17.0, 72.6)
Connections:
- net BootOption renamed Boot_option
- R2401 pad 2: SIREN_CTRL -> INTERNAL_SIREN_CTRL
- R2701 pad 2: SIREN_CTRL -> EXTERNAL_SIREN_CTRL
- U1402 pad 1: SD_ENABLE -> BELL_CTRL
- U1402 pad 2: BELL_CTRL -> INTERNAL_SIREN_CTRL
- U1402 pad 21: SD_MODE -> Net-(R1-Pad2)
- U1402 pad 22: Net-(R1402-Pad2) -> Net-(R2-Pad2)
- U1402 pad 23: Net-(R1402-Pad2) -> Net-(R3-Pad2)
- U1402 pad 24: Net-(R1402-Pad2) -> Net-(R4-Pad2)
- U1402 pad 25: Net-(R1402-Pad2) -> Net-(R5-Pad2)
- U1402 pad 26: Net-(R1402-Pad2) -> Net-(R6-Pad2)
- U1402 pad 27: Net-(R1402-Pad2) -> Net-(R7-Pad2)
- U1402 pad 28: Net-(R1402-Pad2) -> SD_MODE
- U301 pad 36: SIREN_CTRL -> EXTERNAL_SIREN_CTRL
- U401 pad 5: SD_ENABLE -> GND
Routing:
- net BELL_CTRL: track 263.7 -> 0.00 mm, vias 2 -> 0
- net SIREN_CTRL: track 132.4 -> 0.00 mm, vias 6 -> 0
- net SD_ENABLE: track 64.0 -> 0.00 mm, vias 2 -> 0
- net Net-(R1401-Pad2): track 16.2 -> 0.00 mm, vias 2 -> 0
- net Net-(R1404-Pad2): track 15.4 -> 0.14 mm, vias 2 -> 0
- net Net-(D1402-Pad2): track 14.5 -> 0.00 mm
- net Net-(D1405-Pad2): track 14.0 -> 0.00 mm
- net Net-(R1407-Pad2): track 14.5 -> 0.70 mm
- net Net-(D1403-Pad2): track 13.5 -> 0.00 mm
- net Net-(R1402-Pad2): track 11.2 -> 0.00 mm
- net SD_MODE: track 117.8 -> 109.9 mm
- net Net-(R1403-Pad2): track 7.73 -> 0.00 mm
- net Net-(D1406-Pad2): track 7.26 -> 0.00 mm
- net Net-(D1401-Pad2): track 6.76 -> 0.00 mm
- net Net-(D1404-Pad2): track 6.35 -> 0.00 mm
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
Commit message: #8 - Added SD Card power circuit controlled via I2C.
Parts:
- removed D1401: Red, LED_THT:LED_D5.0mm
- removed R1401: 1.65k, Resistor_SMD:R_0805_2012Metric
- added Q1: ZXTN25050DFHTA, Package_TO_SOT_SMD:SOT-23, F.Cu at (-20.4, 107.3)
- added R10: 10k, Resistor_SMD:R_0805_2012Metric, F.Cu at (-16.9, 108.5)
- added R8: 470, Resistor_SMD:R_0805_2012Metric, F.Cu at (-16.9, 106.5)
Connections:
- J401 pad 4: +3V3 -> SD_CARD_PWR
- U1402 pad 3: Net-(R1401-Pad2) -> SD_CARD_PWR_CTRL

Commit message: #6 Switched SIREN_CTRL and SD_SPI_MOSI.
Connections:
- U301 pad 36: EXTERNAL_SIREN_CTRL -> SD_SPI_MOSI
- U301 pad 37: SD_SPI_MOSI -> EXTERNAL_SIREN_CTRL
Routing:
- net SD_SPI_MOSI: track 33.2 -> 32.6 mm
Changed lines of the file:
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@@
   )
   (setup
-    (last_trace_width 2.1)
+    (last_trace_width 0.25)
     (user_trace_width 0.25)
     (user_trace_width 1.7)
@@
       (net 87 /MCU/RDX))
     (pad 36 smd rect (at 8.96 -21.02 270) (size 2 0.9) (layers F.Cu F.Paste F.Mask)
-      (net 258 EXTERNAL_SIREN_CTRL))
-    (pad 37 smd rect (at 8.96 -22.29 270) (size 2 0.9) (layers F.Cu F.Paste F.Mask)
       (net 104 SD_SPI_MOSI))
+    (pad 37 smd rect (at 8.96 -22.29 270) (size 2 0.9) (layers F.Cu F.Paste F.Mask)
+      (net 258 EXTERNAL_SIREN_CTRL))
     (pad 38 smd rect (at 8.96 -23.56 270) (size 2 0.9) (layers F.Cu F.Paste F.Mask)
       (net 32 GND))
@@
   (segment (start 62.955259 117.86077) (end 62.767178 117.672689) (width 0.25) (layer F.Cu) (net 104))
   (segment (start 78.46577 117.86077) (end 62.955259 117.86077) (width 0.25) (layer F.Cu) (net 104))
-  (segment (start 83.377 122.772) (end 78.46577 117.86077) (width 0.25) (layer F.Cu) (net 104))
-  (segment (start 83.377 124.022) (end 83.377 122.772) (width 0.25) (layer F.Cu) (net 104) (status 10))
+  (segment (start 82.107 121.502) (end 82.107 124.022) (width 0.25) (layer F.Cu) (net 104))
+  (segment (start 78.46577 117.86077) (end 82.107 121.502) (width 0.25) (layer F.Cu) (net 104))
   (segment (start 56.635933 119.569518) (end 64.76011 119.569518) (width 0.25) (layer F.Cu) (net 105))
   (segment (start 64.981084 119.348544) (end 66.45869 119.348544) (width 0.25) (layer F.Cu) (net 105))

Commit message: #2 - Wiegand OE pulled high at all times. Closes #2.
Parts:
- removed R304: 10k, Resistor_SMD:R_0805_2012Metric
- moved C306 1.48 mm to (39.1, 136.1), turned to 0 degrees
Connections:
- U302 pad 6: Net-(R304-Pad1) -> +3V3
Routing:
- net Net-(R304-Pad1): track 12.6 -> 0.00 mm
- net +3V3: track 1101.0 -> 1111.6 mm
- net +5V: track 789.3 -> 791.0 mm
- net Wiegand_D0: track 152.6 -> 154.1 mm
- net Wiegand_D1: track 145.9 -> 146.7 mm

Commit message: #4 Added test points to MAX4948. Closes #4.
Parts:
- added TP1: COM1, TestPoint:TestPoint_Pad_D1.5mm, F.Cu at (-14.6, 145.2)
- added TP10: COM4, TestPoint:TestPoint_Pad_D1.5mm, F.Cu at (-4.39, 150.3)
- added TP12: NC4, TestPoint:TestPoint_Pad_D1.5mm, F.Cu at (-6.94, 150.3)
- added TP13: COM5, TestPoint:TestPoint_Pad_D1.5mm, F.Cu at (-4.39, 145.2)
- added TP14: NO5, TestPoint:TestPoint_Pad_D1.5mm, F.Cu at (-6.94, 147.7)
- added TP15: NC5, TestPoint:TestPoint_Pad_D1.5mm, F.Cu at (-9.49, 150.3)
- added TP16: COM6, TestPoint:TestPoint_Pad_D1.5mm, F.Cu at (-6.94, 145.2)
- added TP17: NO6, TestPoint:TestPoint_Pad_D1.5mm, F.Cu at (-9.49, 147.7)
- added TP18: NC6, TestPoint:TestPoint_Pad_D1.5mm, F.Cu at (-12.0, 150.3)
- added TP3: NC1, TestPoint:TestPoint_Pad_D1.5mm, F.Cu at (-14.6, 147.7)
- added TP4: COM2, TestPoint:TestPoint_Pad_D1.5mm, F.Cu at (-12.0, 145.2)
- added TP5: NO2, TestPoint:TestPoint_Pad_D1.5mm, F.Cu at (-17.1, 147.7)
- added TP6: NC2, TestPoint:TestPoint_Pad_D1.5mm, F.Cu at (-14.6, 150.3)
- added TP7: COM3, TestPoint:TestPoint_Pad_D1.5mm, F.Cu at (-12.0, 147.7)
- added TP8: NO3, TestPoint:TestPoint_Pad_D1.5mm, F.Cu at (-9.49, 145.2)
- added TP9: NC3, TestPoint:TestPoint_Pad_D1.5mm, F.Cu at (-17.1, 145.2)
Routing:
- net +3V3: track 1111.6 -> 1088.4 mm, vias 28 -> 26

Commit message: Removed track near pad.
Routing:
- net +3V3: track 1088.4 -> 1078.5 mm
Changed lines of the file:
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@@
     (thickness 1.6)
     (drawings 105)
-    (tracks 2350)
+    (tracks 2347)
     (zones 0)
     (modules 369)
@@
   (segment (start 64.789599 98.06754) (end 66.255914 99.533855) (width 0.25) (layer F.Cu) (net 12))
   (segment (start 64.139252 99.92404) (end 66.255914 99.92404) (width 1.7) (layer F.Cu) (net 12) (status 10))
-  (segment (start 45.485914 114.57754) (end 45.532914 114.53054) (width 0.25) (layer F.Cu) (net 12) (status 30))
   (segment (start 55.366414 114.83554) (end 56.677912 114.83554) (width 0.25) (layer F.Cu) (net 12) (status 10))
   (segment (start 37.680914 103.69654) (end 42.768414 103.69654) (width 1.7) (layer F.Cu) (net 12) (status 10))
@@
   (segment (start 37.680914 109.75154) (end 37.680914 103.69654) (width 1.7) (layer F.Cu) (net 12) (status 20))
   (segment (start 24.853914 122.57854) (end 37.680914 109.75154) (width 1.7) (layer F.Cu) (net 12))
-  (segment (start 42.459914 114.53054) (end 37.680914 109.75154) (width 0.25) (layer F.Cu) (net 12))
-  (segment (start 45.532914 114.53054) (end 42.459914 114.53054) (width 0.25) (layer F.Cu) (net 12) (status 10))
   (segment (start 48.45749 131.33999) (end 53.086 135.9685) (width 2.1) (layer F.Cu) (net 12) (status 20))
   (segment (start 27.45399 131.33999) (end 48.45749 131.33999) (width 2.1) (layer F.Cu) (net 12))

Commit message: Started to re-route PCB for schematics changes.
Parts:
- removed C1: 100n, Capacitor_SMD:C_0805_2012Metric
- removed D1, D2, D3, D4, D5, D6, D7: Red, LED_THT:LED_D5.0mm
- removed Q1: ZXTN25050DFHTA, Package_TO_SOT_SMD:SOT-23
- removed R1, R2, R3, R4, R5, R6, R7: 1.65k, Resistor_SMD:R_0805_2012Metric
- removed R10, R9: 10k, Resistor_SMD:R_0805_2012Metric
- removed R8: 470, Resistor_SMD:R_0805_2012Metric
- added C307: 100n, Capacitor_SMD:C_0805_2012Metric, F.Cu at (56.6, 95.4)
- added D1401: Red, LED_THT:LED_D5.0mm, F.Cu at (22.6, 75.2)
- added D1407: Red, LED_THT:LED_D5.0mm, F.Cu at (35.6, 75.2)
- added D1408: Red, LED_THT:LED_D5.0mm, F.Cu at (35.6, 81.7)
- added D1409: Red, LED_THT:LED_D5.0mm, F.Cu at (35.6, 88.1)
- added D1410: Red, LED_THT:LED_D5.0mm, F.Cu at (42.0, 75.2)
- added D1411: Red, LED_THT:LED_D5.0mm, F.Cu at (42.0, 81.7)
- added D1412: Red, LED_THT:LED_D5.0mm, F.Cu at (42.0, 88.1)
- added Q401: ZXTN25050DFHTA, Package_TO_SOT_SMD:SOT-23, F.Cu at (29.7, 106.5)
- added R1401: 1.65k, Resistor_SMD:R_0805_2012Metric, F.Cu at (22.5, 102.1)
- added R1402: 1.65k, Resistor_SMD:R_0805_2012Metric, F.Cu at (22.6, 97.5)
- added R1408: 1.65k, Resistor_SMD:R_0805_2012Metric, F.Cu at (32.0, 97.5)
- added R1409: 1.65k, Resistor_SMD:R_0805_2012Metric, F.Cu at (31.9, 93.8)
- added R1410: 1.65k, Resistor_SMD:R_0805_2012Metric, F.Cu at (36.5, 102.1)
- added R1411: 1.65k, Resistor_SMD:R_0805_2012Metric, F.Cu at (36.6, 97.5)
- added R1412: 1.65k, Resistor_SMD:R_0805_2012Metric, F.Cu at (36.5, 93.8)
- added R304: 10k, Resistor_SMD:R_0805_2012Metric, F.Cu at (66.1, 95.4)
- added R410: 470, Resistor_SMD:R_0805_2012Metric, F.Cu at (34.1, 105.7)
- added R411: 10k, Resistor_SMD:R_0805_2012Metric, F.Cu at (25.2, 105.7)
- moved D1405 78.3 mm to (29.1, 81.7)
- moved D1406 74.3 mm to (29.1, 88.1)
- moved D1402 72.9 mm to (22.6, 81.7)
- moved D1403 66.5 mm to (22.6, 88.1)
- moved D1404 65.6 mm to (29.1, 75.2)
- moved R1407 61.9 mm to (31.9, 102.1)
- moved R1406 57.9 mm to (27.1, 93.8)
- moved R1405 53.3 mm to (27.2, 97.5)
- moved R1404 53.0 mm to (27.1, 102.1)
- moved R1403 50.1 mm to (22.5, 93.8)
- moved TP1 20.0 mm to (3.14, 135.9)
- moved TP10 20.0 mm to (13.3, 141.0)
- moved TP12 20.0 mm to (10.8, 141.0)
- moved TP13 20.0 mm to (13.3, 135.9)
- moved TP14 20.0 mm to (10.8, 138.5)
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Connections:
- R1403 pad 1: Net-(D1402-Pad2) -> Net-(D1403-Pad2)
- R1404 pad 1: Net-(D1403-Pad2) -> Net-(D1404-Pad2)
- R1405 pad 1: Net-(D1404-Pad2) -> Net-(D1405-Pad2)
- R1406 pad 1: Net-(D1405-Pad2) -> Net-(D1406-Pad2)
- R1407 pad 1: Net-(D1406-Pad2) -> Net-(D1407-Pad2)
- U1402 pad 21: Net-(R1-Pad2) -> Net-(R1406-Pad2)
- U1402 pad 22: Net-(R2-Pad2) -> Net-(R1407-Pad2)
- U1402 pad 4: Net-(R1403-Pad2) -> Net-(R1401-Pad2)
- U1402 pad 5: Net-(R1404-Pad2) -> Net-(R1402-Pad2)
- U1402 pad 6: Net-(R1405-Pad2) -> Net-(R1403-Pad2)
- U1402 pad 7: Net-(R1406-Pad2) -> Net-(R1404-Pad2)
- U1402 pad 8: Net-(R1407-Pad2) -> Net-(R1405-Pad2)
Routing:
- net +3V3: track 1078.5 -> 970.0 mm, vias 26 -> 22
- net SD_CD: track 96.5 -> 5.40 mm, vias 4 -> 0
- net SD_DATA2: track 71.2 -> 0.00 mm, vias 3 -> 0
- net SD_DATA3: track 55.6 -> 1.84 mm, vias 6 -> 0
- net Net-(R1406-Pad2): track 0.00 -> 52.0 mm, vias 0 -> 2
- net SD_CARD_PWR_CTRL: track 0.00 -> 50.8 mm
- net SD_CLK: track 50.5 -> 0.00 mm, vias 3 -> 0
- net Net-(R1403-Pad2): track 0.00 -> 44.9 mm, vias 0 -> 2
- net Net-(R1401-Pad2): track 0.00 -> 43.5 mm, vias 0 -> 2
- net Net-(R1407-Pad2): track 0.70 -> 41.2 mm, vias 0 -> 2
- net Net-(R1410-Pad2): track 0.00 -> 35.9 mm, vias 0 -> 2
- net Net-(R1402-Pad2): track 0.00 -> 35.5 mm, vias 0 -> 2
- net Net-(R1409-Pad2): track 0.00 -> 35.2 mm, vias 0 -> 4
- net Net-(R1408-Pad2): track 0.00 -> 35.1 mm, vias 0 -> 4
- net Net-(R1404-Pad2): track 0.14 -> 33.8 mm, vias 0 -> 4
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