File: hardware/G3.kicad_pcb (KiCad board)
At the start: 2 copper layers, 191.3 x 181.7 mm, 369 parts, among them J1501 Digital input supply, J1502 Digital input GND, J1601 Power_select, J1701 Power_select, J1801 Power_select, J1901 Power_select, J2001 Power_select, J202 GS2, J203 GS2, J2101 Power_select, J2201 Power_select, J2301 Power_select, J2601 Power_select, J2801 Digital input supply, J2802 Digital input GND, J2901 Digital input supply, J2902 Digital input GND, J3001 Digital input supply, J3002 Digital input GND, J301 Debug, J302 BME280, J3101 Digital input supply, J3102 Digital input GND, J3201 Digital input supply, J3202 Digital input GND, J3301 Digital input supply, J3302 Digital input GND, J3401 Digital input supply, J3402 Digital input GND, J3501 Sense, J3502 Digital Input, J3503 Sense, J3504 Digital input, J3505 Power 12/5/3, J3506 Digital input, J3507 Digital Output, J3508 Digital output, J3509 Digital output, J401 Micro_SD_Card_Det, Q1601 ZXTN25050DFHTA, Q1602 ZXTN25050DFHTA, Q1701 ZXTN25050DFHTA, Q1702 ZXTN25050DFHTA, Q1801 ZXTN25050DFHTA, Q1802 ZXTN25050DFHTA, Q1901 ZXTN25050DFHTA, Q1902 ZXTN25050DFHTA, Q2001 ZXTN25050DFHTA, Q2002 ZXTN25050DFHTA, Q2101 ZXTN25050DFHTA, Q2102 ZXTN25050DFHTA, Q2201 ZXTN25050DFHTA, Q2202 ZXTN25050DFHTA, Q2301 ZXTN25050DFHTA, Q2302 ZXTN25050DFHTA, Q2401 ZXTN25050DFHTA, Q2402 ZXTN25050DFHTA, Q2601 ZXTN25050DFHTA, Q2602 ZXTN25050DFHTA, Q2701 ZXTN25050DFHTA, Q2702 ZXTN25050DFHTA, Q401 ZXTN25050DFHTA, SW1 SD SPI/MMC mode, SW301 Boot option, SW302 Reset, SW303 Factory reset, U1401 MCP23017, U1402 MCP23017, U1501 LTV-354T, U201 LM1084-3.3, U202 LM1084-5.0, U2801 LTV-354T, U2901 LTV-354T, U3001 LTV-354T, U301 ESP32_WROVER, U302 TXB0102DCU, U3101 LTV-354T, U3201 LTV-354T, U3301 LTV-354T, U3401 LTV-354T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

Commit message: Continued routing
Parts:
- moved D407 40.0 mm to (37.5, 126.9)
- moved R406 39.6 mm to (46.5, 108.7), turned to 270 degrees
- moved D406 33.9 mm to (34.4, 126.9)
- moved R405 32.1 mm to (36.4, 131.2), turned to 90 degrees
- moved R403 27.3 mm to (29.8, 131.2), turned to 90 degrees
- moved D405 27.1 mm to (31.0, 126.9)
- moved R404 24.2 mm to (33.1, 131.2), turned to 90 degrees
- moved R402 23.5 mm to (26.5, 131.2), turned to 90 degrees
- moved R409 21.6 mm to (21.8, 106.9), turned to 90 degrees
- moved D404 20.7 mm to (27.8, 126.9)
- moved R401 18.9 mm to (23.2, 131.2), turned to 90 degrees
- moved D403 15.2 mm to (25.0, 126.9)
- moved TP3 12.1 mm to (13.4, 144.8), turned to 270 degrees
- moved TP9 11.9 mm to (8.36, 144.9), turned to 270 degrees
- moved TP5 11.0 mm to (10.9, 142.2), turned to 270 degrees
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Routing:
- net BELL_CTRL: track 0.00 -> 162.4 mm, vias 0 -> 2
- net EXTERNAL_SIREN_CTRL: track 0.00 -> 100.7 mm, vias 0 -> 4
- net SD_CD: track 5.40 -> 97.6 mm, vias 0 -> 2
- net +3V3: track 970.0 -> 1051.1 mm, vias 22 -> 26
- net SD_DATA0: track 0.00 -> 80.5 mm, vias 0 -> 10
- net SD_DATA2: track 0.00 -> 79.8 mm, vias 0 -> 3
- net INTERNAL_SIREN_CTRL: track 0.00 -> 77.2 mm, vias 0 -> 2
- net SD_CLK: track 0.00 -> 63.4 mm, vias 0 -> 2
- net SD_DATA3: track 1.84 -> 64.2 mm, vias 0 -> 3
- net /MCU/SDCard/SD_MMC_DATA1: track 0.00 -> 59.8 mm
- net /MCU/SDCard/SD_MMC_DATA0: track 0.00 -> 58.2 mm
- net /MCU/SDCard/SD_MMC_CLK: track 0.00 -> 55.8 mm
- net /MCU/SDCard/SD_MMC_CMD: track 0.00 -> 50.3 mm, vias 0 -> 2
- net /MCU/SDCard/SD_MMC_Data3: track 0.00 -> 49.1 mm, vias 0 -> 2
- net DO7_PWR: track 0.00 -> 44.5 mm
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
Commit message: Continued routing
Parts:
- moved R407 8.98 mm to (105.7, 124.4), turned to 90 degrees
Routing:
- net GND: track 24.9 -> 29.0 mm, vias 1 -> 2
- net SD_MODE: track 154.5 -> 157.8 mm
- net Wiegand_D0: track 160.5 -> 160.0 mm

Commit message: PCB DRC Ok. Removed test points for MAX4948, takes up too much space.
Parts:
- removed TP1: COM1, TestPoint:TestPoint_Pad_D1.5mm
- removed TP10: COM4, TestPoint:TestPoint_Pad_D1.5mm
- removed TP12: NC4, TestPoint:TestPoint_Pad_D1.5mm
- removed TP13: COM5, TestPoint:TestPoint_Pad_D1.5mm
- removed TP14: NO5, TestPoint:TestPoint_Pad_D1.5mm
- removed TP15: NC5, TestPoint:TestPoint_Pad_D1.5mm
- removed TP16: COM6, TestPoint:TestPoint_Pad_D1.5mm
- removed TP17: NO6, TestPoint:TestPoint_Pad_D1.5mm
- removed TP18: NC6, TestPoint:TestPoint_Pad_D1.5mm
- removed TP3: NC1, TestPoint:TestPoint_Pad_D1.5mm
- removed TP4: COM2, TestPoint:TestPoint_Pad_D1.5mm
- removed TP5: NO2, TestPoint:TestPoint_Pad_D1.5mm
- removed TP6: NC2, TestPoint:TestPoint_Pad_D1.5mm
- removed TP7: COM3, TestPoint:TestPoint_Pad_D1.5mm
- removed TP8: NO3, TestPoint:TestPoint_Pad_D1.5mm
- removed TP9: NC3, TestPoint:TestPoint_Pad_D1.5mm
- moved D1404 0.18 mm to (29.1, 75.0)
- moved D1401 0.18 mm to (22.6, 75.0)
- moved D1407 0.18 mm to (35.6, 75.0)
- moved D1410 0.18 mm to (42.0, 75.0)
- moved D1402 0.11 mm to (22.6, 81.6)
- moved D1405 0.11 mm to (29.1, 81.6)
- moved D1408 0.11 mm to (35.6, 81.6)
- moved D1411 0.11 mm to (42.0, 81.6)
Routing:
- net GND: track 29.0 -> 46.1 mm, vias 2 -> 348
- net SD_DATA0: track 80.5 -> 73.8 mm
- net Net-(R1404-Pad2): track 33.8 -> 38.3 mm
- net /MCU/SDCard/SD_MMC_CMD: track 50.3 -> 53.6 mm
- net Net-(R1402-Pad2): track 35.5 -> 37.7 mm
- net SD_CD: track 97.6 -> 98.9 mm
- net DI1_2: track 46.5 -> 47.5 mm
- net /MCU/SDCard/SD_MMC_DATA1: track 59.8 -> 60.8 mm
- net SD_CARD_PWR_CTRL: track 50.8 -> 51.4 mm
- net SD_SPI_MOSI: track 37.0 -> 37.5 mm
Other:
- board text added: "G3 I/O Card | 2018 | GitHub: PerMalmberg | IRC/freenode: Yoari / permal"
- board text removed: "G3 I/O Card | 2018 | GitHub: PerMalmberg | IRC/freenode: Yoari"

Commit message: Hardware: Added a few ground areas. Software: Updated smooth submodule.
Routing:
- net GND: vias 348 -> 370
Changed lines of the file:
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@@
     (thickness 1.6)
     (drawings 105)
-    (tracks 4892)
+    (tracks 4914)
     (zones 0)
     (modules 353)
@@
   (via (at 81.92516 110.93704) (size 0.8) (drill 0.4) (layers F.Cu B.Cu) (net 32))
   (via (at 84.31784 113.42624) (size 0.8) (drill 0.4) (layers F.Cu B.Cu) (net 32))
-  (via (at 76.08316 117.44452) (size 0.8) (drill 0.4) (layers F.Cu B.Cu) (net 32))
   (via (at 90.35796 72.17664) (size 0.8) (drill 0.4) (layers F.Cu B.Cu) (net 32))
   (via (at 83.8708 72.15124) (size 0.8) (drill 0.4) (layers F.Cu B.Cu) (net 32))
@@
   (via (at 122.05208 107.95) (size 0.8) (drill 0.4) (layers F.Cu B.Cu) (net 32))
   (via (at 109.60608 107.99572) (size 0.8) (drill 0.4) (layers F.Cu B.Cu) (net 32))
-  (via (at 102.3112 108.34624) (size 0.8) (drill 0.4) (layers F.Cu B.Cu) (net 32))
+  (via (at 102.41788 108.01096) (size 0.8) (drill 0.4) (layers F.Cu B.Cu) (net 32))
   (via (at 102.08768 114.27968) (size 0.8) (drill 0.4) (layers F.Cu B.Cu) (net 32))
   (via (at 111.32312 123.4694) (size 0.8) (drill 0.4) (layers F.Cu B.Cu) (net 32))
@@
   (via (at 163.61156 59.49188) (size 0.8) (drill 0.4) (layers F.Cu B.Cu) (net 32))
   (via (at 166.64432 75.7936) (size 0.8) (drill 0.4) (layers F.Cu B.Cu) (net 32))
+  (via (at 58.71464 124.45492) (size 0.8) (drill 0.4) (layers F.Cu B.Cu) (net 32))
+  (via (at 65.5574 127.49276) (size 0.8) (drill 0.4) (layers F.Cu B.Cu) (net 32))
+  (via (at 54.73192 124.5108) (size 0.8) (drill 0.4) (layers F.Cu B.Cu) (net 32))
+  (via (at 58.96864 128.69672) (size 0.8) (drill 0.4) (layers F.Cu B.Cu) (net 32))
+  (via (at 69.37756 110.10392) (size 0.8) (drill 0.4) (layers F.Cu B.Cu) (net 32))
+  (via (at 67.2592 112.82172) (size 0.8) (drill 0.4) (layers F.Cu B.Cu) (net 32))
+  (via (at 67.96532 116.06276) (size 0.8) (drill 0.4) (layers F.Cu B.Cu) (net 32))
+  (via (at 70.47484 117.76456) (size 0.8) (drill 0.4) (layers F.Cu B.Cu) (net 32))
+  (via (at 75.22972 117.55628) (size 0.8) (drill 0.4) (layers F.Cu B.Cu) (net 32))
+  (via (at 80.38084 118.10492) (size 0.8) (drill 0.4) (layers F.Cu B.Cu) (net 32))
+  (via (at 79.15148 121.34596) (size 0.8) (drill 0.4) (layers F.Cu B.Cu) (net 32))
+  (via (at 84.91728 134.05612) (size 0.8) (drill 0.4) (layers F.Cu B.Cu) (net 32))
+  (via (at 79.883 141.25448) (size 0.8) (drill 0.4) (layers F.Cu B.Cu) (net 32))
+  (via (at 91.90228 141.27988) (size 0.8) (drill 0.4) (layers F.Cu B.Cu) (net 32))
+  (via (at 88.265 137.53592) (size 0.8) (drill 0.4) (layers F.Cu B.Cu) (net 32))
+  (via (at 85.90788 141.25448) (size 0.8) (drill 0.4) (layers F.Cu B.Cu) (net 32))
+  (via (at 81.407 137.39876) (size 0.8) (drill 0.4) (layers F.Cu B.Cu) (net 32))
+  (via (at 117.45976 136.10336) (size 0.8) (drill 0.4) (layers F.Cu B.Cu) (net 32))
+  (via (at 110.91164 137.7188) (size 0.8) (drill 0.4) (layers F.Cu B.Cu) (net 32))
+  (via (at 111.65332 141.29512) (size 0.8) (drill 0.4) (layers F.Cu B.Cu) (net 32))
+  (via (at 122.51944 141.16812) (size 0.8) (drill 0.4) (layers F.Cu B.Cu) (net 32))
+  (via (at 116.93144 141.47292) (size 0.8) (drill 0.4) (layers F.Cu B.Cu) (net 32))
+  (via (at 120.77192 137.7188) (size 0.8) (drill 0.4) (layers F.Cu B.Cu) (net 32))
   (segment (start 54.543698 99.92404) (end 59.341475 99.92404) (width 0.25) (layer F.Cu) (net 33) (status 30))
   (via (at 70.231 104.267) (size 0.8) (drill 0.4) (layers F.Cu B.Cu) (net 33))

Commit message: More ground vias. Moved text label
Parts:
- moved LOGO101 6.95 mm to (205.0, 84.3)
Routing:
- net GND: vias 370 -> 440
Changed lines of the file:
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@@
     (thickness 1.6)
     (drawings 105)
-    (tracks 4914)
+    (tracks 4984)
     (zones 0)
     (modules 353)
@@
   )
   (module Symbol:OSHW-Logo2_7.3x6mm_SilkScreen (layer F.Cu)
-    (at 205.171 91.201 90)
+    (at 205.01352 84.25664 90)
     (descr "Open Source Hardware Symbol")
     (tags "Logo Symbol OSHW")
@@
     (effects (font (size 1.5 1.5) (thickness 0.3)))
   )
-  (gr_text "G3 I/O Card | 2018 | GitHub: PerMalmberg | IRC/freenode: Yoari / permal" (at 205.261 141.251 90) (layer F.SilkS)
+  (gr_text "G3 I/O Card | 2018 | GitHub: PerMalmberg | IRC/freenode: Yoari / permal" (at 205.10352 134.30664 90) (layer F.SilkS)
     (effects (font (size 1.5 1.5) (thickness 0.3)))
   )
@@
   (via (at 116.93144 141.47292) (size 0.8) (drill 0.4) (layers F.Cu B.Cu) (net 32))
   (via (at 120.77192 137.7188) (size 0.8) (drill 0.4) (layers F.Cu B.Cu) (net 32))
+  (via (at 95.34652 107.90428) (size 0.8) (drill 0.4) (layers F.Cu B.Cu) (net 32))
+  (via (at 95.34652 112.90428) (size 0.8) (drill 0.4) (layers F.Cu B.Cu) (net 32))
+  (via (at 95.34652 117.90428) (size 0.8) (drill 0.4) (layers F.Cu B.Cu) (net 32))
+  (via (at 92.45092 127.00508) (size 0.8) (drill 0.4) (layers F.Cu B.Cu) (net 32))
+  (via (at 90.26144 127.06096) (size 0.8) (drill 0.4) (layers F.Cu B.Cu) (net 32))
+  (via (at 88.83396 132.7912) (size 0.8) (drill 0.4) (layers F.Cu B.Cu) (net 32))
+  (via (at 92.80144 137.0076) (size 0.8) (drill 0.4) (layers F.Cu B.Cu) (net 32))
+  (via (at 82.18424 132.85216) (size 0.8) (drill 0.4) (layers F.Cu B.Cu) (net 32))
+  (via (at 82.2198 130.95732) (size 0.8) (drill 0.4) (layers F.Cu B.Cu) (net 32))
+  (via (at 82.10296 126.52756) (size 0.8) (drill 0.4) (layers F.Cu B.Cu) (net 32))
+  (via (at 82.12328 127.97536) (size 0.8) (drill 0.4) (layers F.Cu B.Cu) (net 32))
+  (via (at 101.81844 100.02012) (size 0.8) (drill 0.4) (layers F.Cu B.Cu) (net 32))
+  (via (at 101.81844 96.02216) (size 0.8) (drill 0.4) (layers F.Cu B.Cu) (net 32))
+  (via (at 103.37292 104.79532) (size 0.8) (drill 0.4) (layers F.Cu B.Cu) (net 32))
+  (via (at 109.601 104.79532) (size 0.8) (drill 0.4) (layers F.Cu B.Cu) (net 32))
+  (via (at 116.02212 104.89692) (size 0.8) (drill 0.4) (layers F.Cu B.Cu) (net 32))
+  (via (at 126.56312 104.89692) (size 0.8) (drill 0.4) (layers F.Cu B.Cu) (net 32))
+  (via (at 105.9688 97.93224) (size 0.8) (drill 0.4) (layers F.Cu B.Cu) (net 32))
+  (via (at 106.0196 101.46284) (size 0.8) (drill 0.4) (layers F.Cu B.Cu) (net 32))
+  (via (at 111.6076 98.02876) (size 0.8) (drill 0.4) (layers F.Cu B.Cu) (net 32))
+  (via (at 102.11816 52.15636) (size 0.8) (drill 0.4) (layers F.Cu B.Cu) (net 32))
+  (via (at 104.40924 45.20692) (size 0.8) (drill 0.4) (layers F.Cu B.Cu) (net 32))
+  (via (at 103.33736 34.86912) (size 0.8) (drill 0.4) (layers F.Cu B.Cu) (net 32))
+  (via (at 101.03612 36.3728) (size 0.8) (drill 0.4) (layers F.Cu B.Cu) (net 32))
+  (via (at 99.31908 42.26052) (size 0.8) (drill 0.4) (layers F.Cu B.Cu) (net 32))
+  (via (at 120.04548 57.25668) (size 0.8) (drill 0.4) (layers F.Cu B.Cu) (net 32))
+  (via (at 122.8852 51.52644) (size 0.8) (drill 0.4) (layers F.Cu B.Cu) (net 32))
+  (via (at 124.3838 45.04436) (size 0.8) (drill 0.4) (layers F.Cu B.Cu) (net 32))
+  (via (at 122.82932 35.72764) (size 0.8) (drill 0.4) (layers F.Cu B.Cu) (net 32))
+  (via (at 121.5898 47.7774) (size 0.8) (drill 0.4) (layers F.Cu B.Cu) (net 32))
+  (via (at 118.29796 58.40476) (size 0.8) (drill 0.4) (layers F.Cu B.Cu) (net 32))
+  (via (at 119.2022 48.93056) (size 0.8) (drill 0.4) (layers F.Cu B.Cu) (net 32))
+  (via (at 144.98828 45.09516) (size 0.8) (drill 0.4) (layers F.Cu B.Cu) (net 32))
+  (via (at 143.11884 33.19272) (size 0.8) (drill 0.4) (layers F.Cu B.Cu) (net 32))
+  (via (at 141.53388 47.82312) (size 0.8) (drill 0.4) (layers F.Cu B.Cu) (net 32))
+  (via (at 139.192 49.29124) (size 0.8) (drill 0.4) (layers F.Cu B.Cu) (net 32))
+  (via (at 142.37208 51.87696) (size 0.8) (drill 0.4) (layers F.Cu B.Cu) (net 32))
+  (via (at 140.716 57.16524) (size 0.8) (drill 0.4) (layers F.Cu B.Cu) (net 32))
+  (via (at 138.6332 58.17616) (size 0.8) (drill 0.4) (layers F.Cu B.Cu) (net 32))
+  (via (at 163.03244 29.8704) (size 0.8) (drill 0.4) (layers F.Cu B.Cu) (net 32))
+  (via (at 164.11956 44.86148) (size 0.8) (drill 0.4) (layers F.Cu B.Cu) (net 32))
+  (via (at 162.0774 48.17872) (size 0.8) (drill 0.4) (layers F.Cu B.Cu) (net 32))
+  (via (at 159.90824 49.8348) (size 0.8) (drill 0.4) (layers F.Cu B.Cu) (net 32))
+  (via (at 181.27472 47.73168) (size 0.8) (drill 0.4) (layers F.Cu B.Cu) (net 32))
+  (via (at 179.35956 50.15484) (size 0.8) (drill 0.4) (layers F.Cu B.Cu) (net 32))
+  (via (at 180.44668 56.97728) (size 0.8) (drill 0.4) (layers F.Cu B.Cu) (net 32))
+  (via (at 178.65852 58.25236) (size 0.8) (drill 0.4) (layers F.Cu B.Cu) (net 32))
+  (via (at 160.74644 56.76392) (size 0.8) (drill 0.4) (layers F.Cu B.Cu) (net 32))
+  (via (at 158.71952 58.1152) (size 0.8) (drill 0.4) (layers F.Cu B.Cu) (net 32))
+  (via (at 162.49904 89.76868) (size 0.8) (drill 0.4) (layers F.Cu B.Cu) (net 32))
+  (via (at 162.44316 93.01988) (size 0.8) (drill 0.4) (layers F.Cu B.Cu) (net 32))
+  (via (at 168.33088 93.07576) (size 0.8) (drill 0.4) (layers F.Cu B.Cu) (net 32))
+  (via (at 168.19372 89.60104) (size 0.8) (drill 0.4) (layers F.Cu B.Cu) (net 32))
+  (via (at 177.9524 88.05672) (size 0.8) (drill 0.4) (layers F.Cu B.Cu) (net 32))
+  (via (at 175.37176 90.74912) (size 0.8) (drill 0.4) (layers F.Cu B.Cu) (net 32))
+  (via (at 174.36084 94.53372) (size 0.8) (drill 0.4) (layers F.Cu B.Cu) (net 32))
+  (via (at 178.28768 90.35796) (size 0.8) (drill 0.4) (layers F.Cu B.Cu) (net 32))
+  (via (at 169.19956 96.55556) (size 0.8) (drill 0.4) (layers F.Cu B.Cu) (net 32))
+  (via (at 167.93972 97.8154) (size 0.8) (drill 0.4) (layers F.Cu B.Cu) (net 32))
+  (via (at 154.55392 102.8192) (size 0.8) (drill 0.4) (layers F.Cu B.Cu) (net 32))
+  (via (at 163.68268 103.06304) (size 0.8) (drill 0.4) (layers F.Cu B.Cu) (net 32))
+  (via (at 163.4998 113.88344) (size 0.8) (drill 0.4) (layers F.Cu B.Cu) (net 32))
+  (via (at 141.67612 111.28248) (size 0.8) (drill 0.4) (layers F.Cu B.Cu) (net 32))
+  (via (at 138.10996 115.15344) (size 0.8) (drill 0.4) (layers F.Cu B.Cu) (net 32))
+  (via (at 22.73808 136.59612) (size 0.8) (drill 0.4) (layers F.Cu B.Cu) (net 32))
+  (via (at 27.73808 136.59612) (size 0.8) (drill 0.4) (layers F.Cu B.Cu) (net 32))
+  (via (at 32.73808 136.59612) (size 0.8) (drill 0.4) (layers F.Cu B.Cu) (net 32))
+  (via (at 118.60276 117.23116) (size 0.8) (drill 0.4) (layers F.Cu B.Cu) (net 32))
+  (via (at 132.09524 113.36528) (size 0.8) (drill 0.4) (layers F.Cu B.Cu) (net 32))
+  (via (at 128.73736 117.3988) (size 0.8) (drill 0.4) (layers F.Cu B.Cu) (net 32))
   (segment (start 54.543698 99.92404) (end 59.341475 99.92404) (width 0.25) (layer F.Cu) (net 33) (status 30))
   (via (at 70.231 104.267) (size 0.8) (drill 0.4) (layers F.Cu B.Cu) (net 33))

Commit message: Text update. New manufacturing files.
Parts:
- moved LOGO101 35.9 mm to (199.7, 119.8)
Other:
- board text added: "G3 I/O Card | 2018 | GitHub: PerMalmberg"
- board text removed: "G3 I/O Card | 2018 | GitHub: PerMalmberg | IRC/freenode: Yoari / permal"
Changed lines of the file:
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@@
   )
   (module Symbol:OSHW-Logo2_7.3x6mm_SilkScreen (layer F.Cu)
-    (at 205.01352 84.25664 90)
+    (at 199.72528 119.75592 90)
     (descr "Open Source Hardware Symbol")
     (tags "Logo Symbol OSHW")
@@
     (effects (font (size 1.5 1.5) (thickness 0.3)))
   )
-  (gr_text "G3 I/O Card | 2018 | GitHub: PerMalmberg | IRC/freenode: Yoari / permal" (at 205.10352 134.30664 90) (layer F.SilkS)
+  (gr_text "G3 I/O Card | 2018 | GitHub: PerMalmberg" (at 205.0542 118.4402 90) (layer F.SilkS)
     (effects (font (size 1.5 1.5) (thickness 0.3)))
   )

Commit message: Replaced TXB0102DCU with SN74LV4T125. Closes #13
Parts:
- removed C306: 100n, Capacitor_SMD:C_0805_2012Metric
- D1401: value Red -> SDCard Init OK
- D1404: value Red -> Wifi Connected
- D1407: value Red -> SNTP Time set
- D1410: value Red -> MQTT Connected
- U302: value TXB0102DCU -> SN74LV4T125; footprint Package_SO:VSSOP-8_2.4x2.1mm_P0.5mm -> Package_SO:TSSOP-14_4.4x5mm_P0.65mm
- moved U302 17.4 mm to (28.1, 137.6), turned to 0 degrees
- moved C305 11.6 mm to (27.9, 142.8)
Connections:
- U302 pad 1: Wiegand_D1 -> GND
- U302 pad 2: GND -> Wiegand_D0
- U302 pad 3: +3V3 -> Net-(U301-Pad12)
- U302 pad 4: Net-(U301-Pad11) -> GND
- U302 pad 5: Net-(U301-Pad12) -> Wiegand_D1
- U302 pad 6: +3V3 -> Net-(U301-Pad11)
- U302 pad 7: +5V -> GND
- U302 pad 8: Wiegand_D0 -> Net-(U302-Pad8)
Routing:
- net +3V3: track 1050.8 -> 1237.5 mm, vias 26 -> 27
- net Net-(U301-Pad11): track 72.0 -> 101.4 mm
- net Wiegand_D0: track 159.7 -> 138.1 mm
- net +5V: track 791.0 -> 770.1 mm, vias 17 -> 16
- net Wiegand_D1: track 152.8 -> 132.2 mm, vias 0 -> 2
- net GND: track 46.1 -> 63.3 mm, vias 440 -> 496
- net Net-(U301-Pad12): track 81.1 -> 94.7 mm, vias 4 -> 2
