File: hardware/SDCard.sch (KiCad schematic (older format))
At the start: 22 parts, among them J401 Micro_SD_Card_Det, SW401 SD SPI/MMC mode, U401 MAX4948

Commit message: #5 - Moved All SD pullup resistors except R406 (SD_DATA2/MTDI/GPIO12) to SD-side of MAX4948. #3 - Added jumper for GPIO2 <-> GPOI0 for flash download. Removed affected items from PCB.
Parts:
- removed SW401: SD SPI/MMC mode, Button_Switch_SMD:SW_DIP_SPSTx01_Slide_Omron_A6S-110x_W8.9mm_P2.54mm, symbol Switch:SW_DIP_x01
- added SW1: SD SPI/MMC mode, Button_Switch_SMD:SW_DIP_SPSTx02_Slide_Omron_A6S-210x_W8.9mm_P2.54mm, symbol Switch:SW_DIP_x02
- R401, R402, R403, R404, R405, R406: value 10k -> 50k
Connections:
- net labels added: BootOption
- wire segments 37 -> 34
Other:
- note added: "Both On = SPI mode and JTAG support.\nGPIO2 needs to be LOW during boot to enter download mode;\nshorting it to GPIO0 (SD_DATA0) will allow this to happen."
- note added: "SD Pullups. R406 is placed on other side of MAX4948 to comply with ESP32\nWrover GPIO12 strapping pin for flash voltage (1.8V) selection regardless\nof SPI or MMC mode."
- note removed: "NC"
- note removed: "On = SPI mode and\nJTAG support"
- moved on the sheet: C401, C402, C403, D401, D402, D403, D404, D405, D406, D407, J401, R401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

Commit message: #1 SD_ENABLE removed; pin grounded. #7 All pins on seconds MCP2317 used. Updated I2CTask to match new H/W layout. Closes #1. Closes #7.
Connections:
- net SD_ENABLE is gone; now on net GND: U401.5 (~EN)
- net BootOption renamed Boot_option
Changed lines of the file:
@@
 	1    0    0    -1
 $EndComp
-Text GLabel 2100 1800 1    50   Input ~ 0
-SD_ENABLE
 Text GLabel 2350 1000 1    50   Input ~ 0
 SD_MODE
@@
 $EndComp
 Text GLabel 4300 1100 0    50   Input ~ 0
-BootOption
+Boot_option
 Text GLabel 4900 1100 2    50   Input ~ 0
 SD_DATA0
+$Comp
+L power:GND #PWR01
+U 1 1 5BF07627
+P 2100 1800
+F 0 "#PWR01" H 2100 1550 50  0001 C CNN
+F 1 "GND" H 2105 1627 50  0000 C CNN
+F 2 "" H 2100 1800 50  0001 C CNN
+F 3 "" H 2100 1800 50  0001 C CNN
+	1    2100 1800
+	-1   0    0    1
+$EndComp
 $EndSCHEMATC

Commit message: #8 - Added SD Card power circuit controlled via I2C.
Parts:
- added Q1: ZXTN25050DFHTA, Package_TO_SOT_SMD:SOT-23, symbol Device:Q_NPN_BCE
- added R10: 10k, Resistor_SMD:R_0805_2012Metric, symbol Device:R
- added R8: 470, Resistor_SMD:R_0805_2012Metric, symbol Device:R
Connections:
- net +3V3: no longer J401.4 (VDD)
- net GND: now also R10.1
- new net: Q1.1 (B), R10.2, R8.1
- new net +5V: Q1.2 (C)
- new net SD_CARD_PWR: J401.4 (VDD), Q1.3 (E)
- new net SD_CARD_PWR_CTRL: R8.2
Changed lines of the file:
@@
 Text Notes 8850 5650 0    50   ~ 0
 Card present = SD_CD low
-$Comp
-L power:+3.3V #PWR0416
-U 1 1 5B9DC236
-P 9250 4800
-F 0 "#PWR0416" H 9250 4650 50  0001 C CNN
-F 1 "+3.3V" V 9265 4928 50  0000 L CNN
-F 2 "" H 9250 4800 50  0001 C CNN
-F 3 "" H 9250 4800 50  0001 C CNN
-	1    9250 4800
-	0    -1   -1   0
-$EndComp
 Wire Notes Line
 	8950 3950 8950 3100
@@
 	-1   0    0    1
 $EndComp
+Text GLabel 9250 4800 0    50   Input ~ 0
+SD_CARD_PWR
+Text GLabel 9600 1450 3    50   Input ~ 0
+SD_CARD_PWR
+$Comp
+L Device:Q_NPN_BCE Q?
+U 1 1 5BF764A8
+P 9500 1250
+AR Path="/5B62EDB8/5BF764A8" Ref="Q?"  Part="1"
+AR Path="/5B62EDB8/5B8B425B/5BF764A8" Ref="Q?"  Part="1"
+AR Path="/5B62EDB8/5B8BDF9E/5BF764A8" Ref="Q?"  Part="1"
+AR Path="/5B62EDB8/5B8CC011/5BF764A8" Ref="Q?"  Part="1"
+AR Path="/5B62EDB8/5B8CD7E8/5BF764A8" Ref="Q?"  Part="1"
+AR Path="/5B62EDB8/5B6C04D0/5BF764A8" Ref="Q?"  Part="1"
+AR Path="/5B62EDB8/5B8DFA1F/5BF764A8" Ref="Q?"  Part="1"
+AR Path="/5B62EDB8/5B8D6A51/5BF764A8" Ref="Q?"  Part="1"
+AR Path="/5B62EDB8/5B8D8275/5BF764A8" Ref="Q?"  Part="1"
+AR Path="/5B62EDB8/5B8D9A4C/5BF764A8" Ref="Q?"  Part="1"
+AR Path="/5B62EDB8/5B8DB29A/5BF764A8" Ref="Q?"  Part="1"
+AR Path="/5B62EDB8/5B8DCA71/5BF764A8" Ref="Q?"  Part="1"
+AR Path="/5B62EDB8/5B8DE248/5BF764A8" Ref="Q?"  Part="1"
+AR Path="/5B62EDB8/5B8EE9B3/5BF764A8" Ref="Q?"  Part="1"
+AR Path="/5B62EDB8/5B8F19D7/5BF764A8" Ref="Q?"  Part="1"
+AR Path="/5B62EDB8/5B8F31AE/5BF764A8" Ref="Q?"  Part="1"
+AR Path="/5B62EDB8/5B8F4985/5BF764A8" Ref="Q?"  Part="1"
+AR Path="/5B62EDB8/5BA037E0/5BF764A8" Ref="Q?"  Part="1"
+AR Path="/5B62EDB8/5B9EF457/5BF764A8" Ref="Q?"  Part="1"
+AR Path="/5B62EDB8/5B9F3247/5BF764A8" Ref="Q?"  Part="1"
+AR Path="/5B62EDB8/5BA1CD69/5BF764A8" Ref="Q?"  Part="1"
+AR Path="/5B62EDB8/5BA1DF84/5BF764A8" Ref="Q?"  Part="1"
+AR Path="/5B62EDB8/5BA1E7D8/5BF764A8" Ref="Q?"  Part="1"
+AR Path="/5B62EDB8/5BA1F02C/5BF764A8" Ref="Q?"  Part="1"
+AR Path="/5B62EDB8/5BA1F880/5BF764A8" Ref="Q?"  Part="1"
+AR Path="/5B62EDB8/5BA200D4/5BF764A8" Ref="Q?"  Part="1"
+AR Path="/5B62EDB8/5BA20928/5BF764A8" Ref="Q?"  Part="1"
+AR Path="/5B62EDB8/5BA2F275/5BF764A8" Ref="Q?"  Part="1"
+AR Path="/5B61FB63/5B98DF5D/5BF764A8" Ref="Q1"  Part="1"
+F 0 "Q1" V 9700 1200 50  0000 L CNN
+F 1 "ZXTN25050DFHTA" H 9750 1150 50  0000 L CNN
+F 2 "Package_TO_SOT_SMD:SOT-23" H 9700 1350 50  0001 C CNN
+F 3 "https://www.mouser.se/ProductDetail/Diodes-Incorporated/ZXTN25050DFHTA?qs=sGAEpiMZZMshyDBzk1%2fWi6gR%252bqBmAG1j52KxSCCDz6c%3d" H 9500 1250 50  0001 C CNN
+	1    9500 1250
+	1    0    0    -1
+$EndComp
+$Comp
+L Device:R R?
+U 1 1 5BF764AF
+P 8750 1250
+AR Path="/5B62EDB8/5BF764AF" Ref="R?"  Part="1"
+AR Path="/5B62EDB8/5B8B425B/5BF764AF" Ref="R?"  Part="1"
+AR Path="/5B62EDB8/5B8BDF9E/5BF764AF" Ref="R?"  Part="1"
+AR Path="/5B62EDB8/5B8CC011/5BF764AF" Ref="R?"  Part="1"
+AR Path="/5B62EDB8/5B8CD7E8/5BF764AF" Ref="R?"  Part="1"
+AR Path="/5B62EDB8/5B6C04D0/5BF764AF" Ref="R?"  Part="1"
+AR Path="/5B62EDB8/5B8DFA1F/5BF764AF" Ref="R?"  Part="1"
+AR Path="/5B62EDB8/5B8D6A51/5BF764AF" Ref="R?"  Part="1"
+AR Path="/5B62EDB8/5B8D8275/5BF764AF" Ref="R?"  Part="1"
+AR Path="/5B62EDB8/5B8D9A4C/5BF764AF" Ref="R?"  Part="1"
+AR Path="/5B62EDB8/5B8DB29A/5BF764AF" Ref="R?"  Part="1"
+AR Path="/5B62EDB8/5B8DCA71/5BF764AF" Ref="R?"  Part="1"
+AR Path="/5B62EDB8/5B8DE248/5BF764AF" Ref="R?"  Part="1"
+AR Path="/5B62EDB8/5B8EE9B3/5BF764AF" Ref="R?"  Part="1"
+AR Path="/5B62EDB8/5B8F19D7/5BF764AF" Ref="R?"  Part="1"
+AR Path="/5B62EDB8/5B8F31AE/5BF764AF" Ref="R?"  Part="1"
+AR Path="/5B62EDB8/5B8F4985/5BF764AF" Ref="R?"  Part="1"
+AR Path="/5B62EDB8/5BA037E0/5BF764AF" Ref="R?"  Part="1"
+AR Path="/5B62EDB8/5B9EF457/5BF764AF" Ref="R?"  Part="1"
+AR Path="/5B62EDB8/5B9F3247/5BF764AF" Ref="R?"  Part="1"
+AR Path="/5B62EDB8/5BA1CD69/5BF764AF" Ref="R?"  Part="1"
+AR Path="/5B62EDB8/5BA1DF84/5BF764AF" Ref="R?"  Part="1"
+AR Path="/5B62EDB8/5BA1E7D8/5BF764AF" Ref="R?"  Part="1"
+AR Path="/5B62EDB8/5BA1F02C/5BF764AF" Ref="R?"  Part="1"
+AR Path="/5B62EDB8/5BA1F880/5BF764AF" Ref="R?"  Part="1"
+AR Path="/5B62EDB8/5BA200D4/5BF764AF" Ref="R?"  Part="1"
+AR Path="/5B62EDB8/5BA20928/5BF764AF" Ref="R?"  Part="1"
+AR Path="/5B62EDB8/5BA2F275/5BF764AF" Ref="R?"  Part="1"
+AR Path="/5B61FB63/5B98DF5D/5BF764AF" Ref="R8"  Part="1"
+F 0 "R8" V 8650 1250 50  0000 C CNN
+F 1 "470" V 8750 1250 50  0000 C CNN
+F 2 "Resistor_SMD:R_0805_2012Metric" V 8680 1250 50  0001 C CNN
+F 3 "https://www.mouser.se/ProductDetail/Bourns/CR0805-FX-4700ELF?qs=sGAEpiMZZMu61qfTUdNhG6LqqFhkr6pUJHKuKfp2v90%3d" H 8750 1250 50  0001 C CNN
+	1    8750 1250
+	0    1    1    0
+$EndComp
+$Comp
+L Device:R R?
+U 1 1 5BF764B6
+P 9150 1400
+AR Path="/5B62EDB8/5BF764B6" Ref="R?"  Part="1"
+AR Path="/5B62EDB8/5B8B425B/5BF764B6" Ref="R?"  Part="1"
+AR Path="/5B62EDB8/5B8BDF9E/5BF764B6" Ref="R?"  Part="1"
+AR Path="/5B62EDB8/5B8CC011/5BF764B6" Ref="R?"  Part="1"
+AR Path="/5B62EDB8/5B8CD7E8/5BF764B6" Ref="R?"  Part="1"
+AR Path="/5B62EDB8/5B6C04D0/5BF764B6" Ref="R?"  Part="1"
+AR Path="/5B62EDB8/5B8DFA1F/5BF764B6" Ref="R?"  Part="1"
+AR Path="/5B62EDB8/5B8D6A51/5BF764B6" Ref="R?"  Part="1"
+AR Path="/5B62EDB8/5B8D8275/5BF764B6" Ref="R?"  Part="1"
+AR Path="/5B62EDB8/5B8D9A4C/5BF764B6" Ref="R?"  Part="1"
+AR Path="/5B62EDB8/5B8DB29A/5BF764B6" Ref="R?"  Part="1"
+AR Path="/5B62EDB8/5B8DCA71/5BF764B6" Ref="R?"  Part="1"
+AR Path="/5B62EDB8/5B8DE248/5BF764B6" Ref="R?"  Part="1"
+AR Path="/5B62EDB8/5B8EE9B3/5BF764B6" Ref="R?"  Part="1"
+AR Path="/5B62EDB8/5B8F19D7/5BF764B6" Ref="R?"  Part="1"
+AR Path="/5B62EDB8/5B8F31AE/5BF764B6" Ref="R?"  Part="1"
+AR Path="/5B62EDB8/5B8F4985/5BF764B6" Ref="R?"  Part="1"
+AR Path="/5B62EDB8/5BA037E0/5BF764B6" Ref="R?"  Part="1"
+AR Path="/5B62EDB8/5B9EF457/5BF764B6" Ref="R?"  Part="1"
+AR Path="/5B62EDB8/5B9F3247/5BF764B6" Ref="R?"  Part="1"
+AR Path="/5B62EDB8/5BA1CD69/5BF764B6" Ref="R?"  Part="1"
+AR Path="/5B62EDB8/5BA1DF84/5BF764B6" Ref="R?"  Part="1"
+AR Path="/5B62EDB8/5BA1E7D8/5BF764B6" Ref="R?"  Part="1"
+AR Path="/5B62EDB8/5BA1F02C/5BF764B6" Ref="R?"  Part="1"
+AR Path="/5B62EDB8/5BA1F880/5BF764B6" Ref="R?"  Part="1"
+AR Path="/5B62EDB8/5BA200D4/5BF764B6" Ref="R?"  Part="1"
+AR Path="/5B62EDB8/5BA20928/5BF764B6" Ref="R?"  Part="1"
+AR Path="/5B62EDB8/5BA2F275/5BF764B6" Ref="R?"  Part="1"
+AR Path="/5B61FB63/5B98DF5D/5BF764B6" Ref="R10"  Part="1"
+F 0 "R10" H 9220 1446 50  0000 L CNN
+F 1 "10k" H 9220 1355 50  0000 L CNN
+F 2 "Resistor_SMD:R_0805_2012Metric" V 9080 1400 50  0001 C CNN
+F 3 "https://www.mouser.se/ProductDetail/Panasonic-Industrial-Devices/ERJ-6ENF1002V?qs=sGAEpiMZZMu61qfTUdNhGzRxdwze5h8ZcGDx6geba20%3d" H 9150 1400 50  0001 C CNN
+	1    9150 1400
+	-1   0    0    1
+$EndComp
+$Comp
+L power:GND #PWR?
+U 1 1 5BF764BD
+P 9150 1550
+AR Path="/5B62EDB8/5BF764BD" Ref="#PWR?"  Part="1"
+AR Path="/5B62EDB8/5B8B425B/5BF764BD" Ref="#PWR?"  Part="1"
+AR Path="/5B62EDB8/5B8BDF9E/5BF764BD" Ref="#PWR?"  Part="1"
+AR Path="/5B62EDB8/5B8CC011/5BF764BD" Ref="#PWR?"  Part="1"
+AR Path="/5B62EDB8/5B8CD7E8/5BF764BD" Ref="#PWR?"  Part="1"
+AR Path="/5B62EDB8/5B6C04D0/5BF764BD" Ref="#PWR?"  Part="1"
+AR Path="/5B62EDB8/5B8DFA1F/5BF764BD" Ref="#PWR?"  Part="1"
+AR Path="/5B62EDB8/5B8D6A51/5BF764BD" Ref="#PWR?"  Part="1"
+AR Path="/5B62EDB8/5B8D8275/5BF764BD" Ref="#PWR?"  Part="1"
+AR Path="/5B62EDB8/5B8D9A4C/5BF764BD" Ref="#PWR?"  Part="1"
+AR Path="/5B62EDB8/5B8DB29A/5BF764BD" Ref="#PWR?"  Part="1"
+AR Path="/5B62EDB8/5B8DCA71/5BF764BD" Ref="#PWR?"  Part="1"
+AR Path="/5B62EDB8/5B8DE248/5BF764BD" Ref="#PWR?"  Part="1"
+AR Path="/5B62EDB8/5B8EE9B3/5BF764BD" Ref="#PWR?"  Part="1"
+AR Path="/5B62EDB8/5B8F19D7/5BF764BD" Ref="#PWR?"  Part="1"
+AR Path="/5B62EDB8/5B8F31AE/5BF764BD" Ref="#PWR?"  Part="1"
+AR Path="/5B62EDB8/5B8F4985/5BF764BD" Ref="#PWR?"  Part="1"
+AR Path="/5B62EDB8/5BA037E0/5BF764BD" Ref="#PWR?"  Part="1"
+AR Path="/5B62EDB8/5B9EF457/5BF764BD" Ref="#PWR?"  Part="1"
+AR Path="/5B62EDB8/5B9F3247/5BF764BD" Ref="#PWR?"  Part="1"
+AR Path="/5B62EDB8/5BA1CD69/5BF764BD" Ref="#PWR?"  Part="1"
+AR Path="/5B62EDB8/5BA1DF84/5BF764BD" Ref="#PWR?"  Part="1"
+AR Path="/5B62EDB8/5BA1E7D8/5BF764BD" Ref="#PWR?"  Part="1"
+AR Path="/5B62EDB8/5BA1F02C/5BF764BD" Ref="#PWR?"  Part="1"
+AR Path="/5B62EDB8/5BA1F880/5BF764BD" Ref="#PWR?"  Part="1"
+AR Path="/5B62EDB8/5BA200D4/5BF764BD" Ref="#PWR?"  Part="1"
+AR Path="/5B62EDB8/5BA20928/5BF764BD" Ref="#PWR?"  Part="1"
+AR Path="/5B62EDB8/5BA2F275/5BF764BD" Ref="#PWR?"  Part="1"
+AR Path="/5B61FB63/5B98DF5D/5BF764BD" Ref="#PWR09"  Part="1"
+F 0 "#PWR09" H 9150 1300 50  0001 C CNN
+F 1 "GND" H 9155 1377 50  0000 C CNN
+F 2 "" H 9150 1550 50  0001 C CNN
+F 3 "" H 9150 1550 50  0001 C CNN
+	1    9150 1550
+	1    0    0    -1
+$EndComp
+$Comp
+L power:+5V #PWR?
+U 1 1 5BF764C3
+P 9600 1050
+AR Path="/5B62EDB8/5BF764C3" Ref="#PWR?"  Part="1"
+AR Path="/5B72552B/5BF764C3" Ref="#PWR?"  Part="1"
+AR Path="/5B62EDB8/5B6C04D0/5BF764C3" Ref="#PWR?"  Part="1"
+AR Path="/5B62EDB8/5B8EE9B3/5BF764C3" Ref="#PWR?"  Part="1"
+AR Path="/5B62EDB8/5BA1CD69/5BF764C3" Ref="#PWR?"  Part="1"
+AR Path="/5B62EDB8/5BA1DF84/5BF764C3" Ref="#PWR?"  Part="1"
+AR Path="/5B62EDB8/5BA1E7D8/5BF764C3" Ref="#PWR?"  Part="1"
+AR Path="/5B62EDB8/5BA1F02C/5BF764C3" Ref="#PWR?"  Part="1"
+AR Path="/5B62EDB8/5BA1F880/5BF764C3" Ref="#PWR?"  Part="1"
+AR Path="/5B62EDB8/5BA200D4/5BF764C3" Ref="#PWR?"  Part="1"
+AR Path="/5B62EDB8/5BA20928/5BF764C3" Ref="#PWR?"  Part="1"
+AR Path="/5B62EDB8/5BA2F275/5BF764C3" Ref="#PWR?"  Part="1"
+AR Path="/5B61FB63/5B98DF5D/5BF764C3" Ref="#PWR010"  Part="1"
+F 0 "#PWR010" H 9600 900 50  0001 C CNN
+F 1 "+5V" V 9615 1178 50  0000 L CNN
+F 2 "" H 9600 1050 50  0001 C CNN
+F 3 "" H 9600 1050 50  0001 C CNN
+	1    9600 1050
+	1    0    0    -1
+$EndComp
+Wire Wire Line
+	8900 1250 9150 1250
+Connection ~ 9150 1250
+Wire Wire Line
+	9150 1250 9300 1250
+Text GLabel 8600 1250 0    50   Input ~ 0
+SD_CARD_PWR_CTRL
 $EndSCHEMATC

Commit message: #4 Added test points to MAX4948. Closes #4.
Parts:
- added TP1: COM1, TestPoint:TestPoint_Pad_D1.5mm, symbol Connector:TestPoint
- added TP10: COM4, TestPoint:TestPoint_Pad_D1.5mm, symbol Connector:TestPoint
- added TP12: NC4, TestPoint:TestPoint_Pad_D1.5mm, symbol Connector:TestPoint
- added TP13: COM5, TestPoint:TestPoint_Pad_D1.5mm, symbol Connector:TestPoint
- added TP14: NO5, TestPoint:TestPoint_Pad_D1.5mm, symbol Connector:TestPoint
- added TP15: NC5, TestPoint:TestPoint_Pad_D1.5mm, symbol Connector:TestPoint
- added TP16: COM6, TestPoint:TestPoint_Pad_D1.5mm, symbol Connector:TestPoint
- added TP17: NO6, TestPoint:TestPoint_Pad_D1.5mm, symbol Connector:TestPoint
- added TP18: NC6, TestPoint:TestPoint_Pad_D1.5mm, symbol Connector:TestPoint
- added TP3: NC1, TestPoint:TestPoint_Pad_D1.5mm, symbol Connector:TestPoint
- added TP4: COM2, TestPoint:TestPoint_Pad_D1.5mm, symbol Connector:TestPoint
- added TP5: NO2, TestPoint:TestPoint_Pad_D1.5mm, symbol Connector:TestPoint
- added TP6: NC2, TestPoint:TestPoint_Pad_D1.5mm, symbol Connector:TestPoint
- added TP7: COM3, TestPoint:TestPoint_Pad_D1.5mm, symbol Connector:TestPoint
- added TP8: NO3, TestPoint:TestPoint_Pad_D1.5mm, symbol Connector:TestPoint
- added TP9: NC3, TestPoint:TestPoint_Pad_D1.5mm, symbol Connector:TestPoint
Connections:
- net SD_CLK: now also TP6.1
- net SD_CMD: now also TP18.1
- net SD_DATA0: now also TP15.1
- net SD_DATA1: now also TP3.1
- net SD_DATA2: now also TP12.1
- net SD_DATA3: now also TP9.1
- net SD_MMC_CLK: now also TP4.1
- net SD_MMC_CMD: now also TP16.1
- net SD_MMC_DATA0: now also TP13.1
- net SD_MMC_DATA1: now also TP1.1
- net SD_MMC_Data2: now also TP10.1
- net SD_MMC_Data3: now also TP7.1
- net SD_SPI_CLK: now also TP5.1
- net SD_SPI_CS: now also TP8.1
- net SD_SPI_MISO: now also TP14.1
- net SD_SPI_MOSI: now also TP17.1
Changed lines of the file:
@@
 Text GLabel 8600 1250 0    50   Input ~ 0
 SD_CARD_PWR_CTRL
+$Comp
+L Connector:TestPoint TP1
+U 1 1 5BF8579D
+P 850 5350
+F 0 "TP1" V 800 5750 50  0000 R CNN
+F 1 "COM1" V 900 5900 50  0000 R CNN
+F 2 "TestPoint:TestPoint_Pad_D1.5mm" H 1050 5350 50  0001 C CNN
+F 3 "~" H 1050 5350 50  0001 C CNN
+	1    850  5350
+	-1   0    0    1
+$EndComp
+Text Label 850  5350 1    50   ~ 0
+SD_MMC_DATA1
+Text GLabel 1050 5350 1    50   Input ~ 0
+SD_DATA1
+Text GLabel 1450 5350 1    50   Input ~ 0
+SD_SPI_CLK
+Text Label 1250 5350 1    50   ~ 0
+SD_MMC_CLK
+Text GLabel 1650 5350 1    50   Input ~ 0
+SD_CLK
+$Comp
+L Connector:TestPoint TP3
+U 1 1 5BF93E2D
+P 1050 5350
+F 0 "TP3" V 1000 5750 50  0000 R CNN
+F 1 "NC1" V 1100 5900 50  0000 R CNN
+F 2 "TestPoint:TestPoint_Pad_D1.5mm" H 1250 5350 50  0001 C CNN
+F 3 "~" H 1250 5350 50  0001 C CNN
+	1    1050 5350
+	-1   0    0    1
+$EndComp
+$Comp
+L Connector:TestPoint TP4
+U 1 1 5BF94693
+P 1250 5350
+F 0 "TP4" V 1200 5750 50  0000 R CNN
+F 1 "COM2" V 1300 5900 50  0000 R CNN
+F 2 "TestPoint:TestPoint_Pad_D1.5mm" H 1450 5350 50  0001 C CNN
+F 3 "~" H 1450 5350 50  0001 C CNN
+	1    1250 5350
+	-1   0    0    1
+$EndComp
+$Comp
+L Connector:TestPoint TP5
+U 1 1 5BF94EFB
+P 1450 5350
+F 0 "TP5" V 1400 5750 50  0000 R CNN
+F 1 "NO2" V 1500 5900 50  0000 R CNN
+F 2 "TestPoint:TestPoint_Pad_D1.5mm" H 1650 5350 50  0001 C CNN
+F 3 "~" H 1650 5350 50  0001 C CNN
+	1    1450 5350
+	-1   0    0    1
+$EndComp
+$Comp
+L Connector:TestPoint TP6
+U 1 1 5BF95765
+P 1650 5350
+F 0 "TP6" V 1600 5750 50  0000 R CNN
+F 1 "NC2" V 1700 5900 50  0000 R CNN
+F 2 "TestPoint:TestPoint_Pad_D1.5mm" H 1850 5350 50  0001 C CNN
+F 3 "~" H 1850 5350 50  0001 C CNN
+	1    1650 5350
+	-1   0    0    1
+$EndComp
+$Comp
+L Connector:TestPoint TP7
+U 1 1 5BF960E6
+P 1800 5350
+F 0 "TP7" V 1750 5750 50  0000 R CNN
+F 1 "COM3" V 1850 5900 50  0000 R CNN
+F 2 "TestPoint:TestPoint_Pad_D1.5mm" H 2000 5350 50  0001 C CNN
+F 3 "~" H 2000 5350 50  0001 C CNN
+	1    1800 5350
+	-1   0    0    1
+$EndComp
+$Comp
+L Connector:TestPoint TP8
+U 1 1 5BF960ED
+P 2000 5350
+F 0 "TP8" V 1950 5750 50  0000 R CNN
+F 1 "NO3" V 2050 5900 50  0000 R CNN
+F 2 "TestPoint:TestPoint_Pad_D1.5mm" H 2200 5350 50  0001 C CNN
+F 3 "~" H 2200 5350 50  0001 C CNN
+	1    2000 5350
+	-1   0    0    1
+$EndComp
+$Comp
+L Connector:TestPoint TP9
+U 1 1 5BF960F4
+P 2200 5350
+F 0 "TP9" V 2150 5750 50  0000 R CNN
+F 1 "NC3" V 2250 5900 50  0000 R CNN
+F 2 "TestPoint:TestPoint_Pad_D1.5mm" H 2400 5350 50  0001 C CNN
+F 3 "~" H 2400 5350 50  0001 C CNN
+	1    2200 5350
+	-1   0    0    1
+$EndComp
+$Comp
+L Connector:TestPoint TP10
+U 1 1 5BF960FB
+P 2400 5350
+F 0 "TP10" V 2350 5750 50  0000 R CNN
+F 1 "COM4" V 2450 5900 50  0000 R CNN
+F 2 "TestPoint:TestPoint_Pad_D1.5mm" H 2600 5350 50  0001 C CNN
+F 3 "~" H 2600 5350 50  0001 C CNN
+	1    2400 5350
+	-1   0    0    1
+$EndComp
+$Comp
+L Connector:TestPoint TP12
+U 1 1 5BF96102
+P 2550 5350
+F 0 "TP12" V 2500 5750 50  0000 R CNN
+F 1 "NC4" V 2600 5900 50  0000 R CNN
+F 2 "TestPoint:TestPoint_Pad_D1.5mm" H 2750 5350 50  0001 C CNN
+F 3 "~" H 2750 5350 50  0001 C CNN
+	1    2550 5350
+	-1   0    0    1
+$EndComp
+$Comp
+L Connector:TestPoint TP13
+U 1 1 5BF96A3D
+P 2750 5350
+F 0 "TP13" V 2700 5750 50  0000 R CNN
+F 1 "COM5" V 2800 5900 50  0000 R CNN
+F 2 "TestPoint:TestPoint_Pad_D1.5mm" H 2950 5350 50  0001 C CNN
+F 3 "~" H 2950 5350 50  0001 C CNN
+	1    2750 5350
+	-1   0    0    1
+$EndComp
+$Comp
+L Connector:TestPoint TP14
+U 1 1 5BF96A44
+P 2950 5350
+F 0 "TP14" V 2900 5750 50  0000 R CNN
+F 1 "NO5" V 3000 5900 50  0000 R CNN
+F 2 "TestPoint:TestPoint_Pad_D1.5mm" H 3150 5350 50  0001 C CNN
+F 3 "~" H 3150 5350 50  0001 C CNN
+	1    2950 5350
+	-1   0    0    1
+$EndComp
+$Comp
+L Connector:TestPoint TP15
+U 1 1 5BF96A4B
+P 3150 5350
+F 0 "TP15" V 3100 5750 50  0000 R CNN
+F 1 "NC5" V 3200 5900 50  0000 R CNN
+F 2 "TestPoint:TestPoint_Pad_D1.5mm" H 3350 5350 50  0001 C CNN
+F 3 "~" H 3350 5350 50  0001 C CNN
+	1    3150 5350
+	-1   0    0    1
+$EndComp
+$Comp
+L Connector:TestPoint TP16
+U 1 1 5BF96A52
+P 3350 5350
+F 0 "TP16" V 3300 5750 50  0000 R CNN
+F 1 "COM6" V 3400 5900 50  0000 R CNN
+F 2 "TestPoint:TestPoint_Pad_D1.5mm" H 3550 5350 50  0001 C CNN
+F 3 "~" H 3550 5350 50  0001 C CNN
+	1    3350 5350
+	-1   0    0    1
+$EndComp
+$Comp
+L Connector:TestPoint TP17
+U 1 1 5BF972C8
+P 3550 5350
+F 0 "TP17" V 3500 5750 50  0000 R CNN
+F 1 "NO6" V 3600 5900 50  0000 R CNN
+F 2 "TestPoint:TestPoint_Pad_D1.5mm" H 3750 5350 50  0001 C CNN
+F 3 "~" H 3750 5350 50  0001 C CNN
+	1    3550 5350
+	-1   0    0    1
+$EndComp
+$Comp
+L Connector:TestPoint TP18
+U 1 1 5BF97336
+P 3750 5350
+F 0 "TP18" V 3700 5750 50  0000 R CNN
+F 1 "NC6" V 3800 5900 50  0000 R CNN
+F 2 "TestPoint:TestPoint_Pad_D1.5mm" H 3950 5350 50  0001 C CNN
+F 3 "~" H 3950 5350 50  0001 C CNN
+	1    3750 5350
+	-1   0    0    1
+$EndComp
+Text GLabel 2000 5350 1    50   Input ~ 0
+SD_SPI_CS
+Text Label 1800 5350 1    50   ~ 0
+SD_MMC_Data3
+Text GLabel 2200 5350 1    50   Input ~ 0
+SD_DATA3
+Text GLabel 2550 5350 1    50   Input ~ 0
+SD_DATA2
+Text Label 2400 5350 1    50   ~ 0
+SD_MMC_Data2
+Text GLabel 2950 5350 1    50   Input ~ 0
+SD_SPI_MISO
+Text Label 2750 5350 1    50   ~ 0
+SD_MMC_DATA0
+Text GLabel 3150 5350 1    50   Input ~ 0
+SD_DATA0
+Text GLabel 3550 5350 1    50   Input ~ 0
+SD_SPI_MOSI
+Text Label 3350 5350 1    50   ~ 0
+SD_MMC_CMD
+Text GLabel 3750 5350 1    50   Input ~ 0
+SD_CMD
 $EndSCHEMATC

Commit message: Started to re-route PCB for schematics changes.
Parts:
- renumbered Q1 to Q401, R8 to R410, R10 to R411
Connections:
- net +5V is gone; now on net +3V3: Q401.2 (C)
Changed lines of the file:
@@
 AR Path="/5B62EDB8/5BA20928/5BF764A8" Ref="Q?"  Part="1"
 AR Path="/5B62EDB8/5BA2F275/5BF764A8" Ref="Q?"  Part="1"
-AR Path="/5B61FB63/5B98DF5D/5BF764A8" Ref="Q1"  Part="1"
-F 0 "Q1" V 9700 1200 50  0000 L CNN
+AR Path="/5B61FB63/5B98DF5D/5BF764A8" Ref="Q401"  Part="1"
+F 0 "Q401" V 9700 1200 50  0000 L CNN
 F 1 "ZXTN25050DFHTA" H 9750 1150 50  0000 L CNN
 F 2 "Package_TO_SOT_SMD:SOT-23" H 9700 1350 50  0001 C CNN
@@
 AR Path="/5B62EDB8/5BA20928/5BF764AF" Ref="R?"  Part="1"
 AR Path="/5B62EDB8/5BA2F275/5BF764AF" Ref="R?"  Part="1"
-AR Path="/5B61FB63/5B98DF5D/5BF764AF" Ref="R8"  Part="1"
-F 0 "R8" V 8650 1250 50  0000 C CNN
+AR Path="/5B61FB63/5B98DF5D/5BF764AF" Ref="R410"  Part="1"
+F 0 "R410" V 8650 1250 50  0000 C CNN
 F 1 "470" V 8750 1250 50  0000 C CNN
 F 2 "Resistor_SMD:R_0805_2012Metric" V 8680 1250 50  0001 C CNN
@@
 AR Path="/5B62EDB8/5BA20928/5BF764B6" Ref="R?"  Part="1"
 AR Path="/5B62EDB8/5BA2F275/5BF764B6" Ref="R?"  Part="1"
-AR Path="/5B61FB63/5B98DF5D/5BF764B6" Ref="R10"  Part="1"
-F 0 "R10" H 9220 1446 50  0000 L CNN
+AR Path="/5B61FB63/5B98DF5D/5BF764B6" Ref="R411"  Part="1"
+F 0 "R411" H 9220 1446 50  0000 L CNN
 F 1 "10k" H 9220 1355 50  0000 L CNN
 F 2 "Resistor_SMD:R_0805_2012Metric" V 9080 1400 50  0001 C CNN
@@
 	1    0    0    -1
 $EndComp
-$Comp
-L power:+5V #PWR?
-U 1 1 5BF764C3
-P 9600 1050
-AR Path="/5B62EDB8/5BF764C3" Ref="#PWR?"  Part="1"
-AR Path="/5B72552B/5BF764C3" Ref="#PWR?"  Part="1"
-AR Path="/5B62EDB8/5B6C04D0/5BF764C3" Ref="#PWR?"  Part="1"
-AR Path="/5B62EDB8/5B8EE9B3/5BF764C3" Ref="#PWR?"  Part="1"
-AR Path="/5B62EDB8/5BA1CD69/5BF764C3" Ref="#PWR?"  Part="1"
-AR Path="/5B62EDB8/5BA1DF84/5BF764C3" Ref="#PWR?"  Part="1"
-AR Path="/5B62EDB8/5BA1E7D8/5BF764C3" Ref="#PWR?"  Part="1"
-AR Path="/5B62EDB8/5BA1F02C/5BF764C3" Ref="#PWR?"  Part="1"
-AR Path="/5B62EDB8/5BA1F880/5BF764C3" Ref="#PWR?"  Part="1"
-AR Path="/5B62EDB8/5BA200D4/5BF764C3" Ref="#PWR?"  Part="1"
-AR Path="/5B62EDB8/5BA20928/5BF764C3" Ref="#PWR?"  Part="1"
-AR Path="/5B62EDB8/5BA2F275/5BF764C3" Ref="#PWR?"  Part="1"
-AR Path="/5B61FB63/5B98DF5D/5BF764C3" Ref="#PWR010"  Part="1"
-F 0 "#PWR010" H 9600 900 50  0001 C CNN
-F 1 "+5V" V 9615 1178 50  0000 L CNN
-F 2 "" H 9600 1050 50  0001 C CNN
-F 3 "" H 9600 1050 50  0001 C CNN
-	1    9600 1050
-	1    0    0    -1
-$EndComp
 Wire Wire Line
 	8900 1250 9150 1250
@@
 Text GLabel 3750 5350 1    50   Input ~ 0
 SD_CMD
+$Comp
+L power:+3.3V #PWR0118
+U 1 1 5BEA97EE
+P 9600 1050
+F 0 "#PWR0118" H 9600 900 50  0001 C CNN
+F 1 "+3.3V" H 9615 1223 50  0000 C CNN
+F 2 "" H 9600 1050 50  0001 C CNN
+F 3 "" H 9600 1050 50  0001 C CNN
+	1    9600 1050
+	1    0    0    -1
+$EndComp
 $EndSCHEMATC
