File: hardware/MCU.sch (KiCad schematic (older format))
At the start: 20 parts, among them J301 Debug, J302 BME280, SW301 Boot option, SW302 Reset, SW303 Factory reset, U301 ESP32_WROVER, U302 SN74LV4T125

Commit message: Updated PCB with additional vias. Added decoupler caps for Wiegand.
Parts:
- added C306, C308, C309, C310: 100n, Capacitor_SMD:C_0805_2012Metric, symbol Device:C
Connections:
- net GND: now also C306.1, C308.2, C309.1, C310.1
- net Wiegand_D0: now also C309.2
- net Wiegand_D1: now also C310.2
- net at U301.11 (GPIO26), U302.6 (2Y): now also C306.2
- net at U301.12 (GPIO27), U302.3 (1Y): now also C308.1
Changed lines of the file:
@@
 	5450 3300 7100 3300
 Wire Wire Line
-	7100 3300 7100 4850
+	7100 3300 7100 4000
 Wire Wire Line
 	5450 2800 6750 2800
@@
 $EndComp
 Wire Wire Line
-	7200 3200 7200 4700
+	7200 3200 7200 4000
 Wire Wire Line
 	7200 4700 8000 4700
@@
 	8650 5000 8700 5000
 Wire Wire Line
-	9150 4750 8500 4750
-Wire Wire Line
-	9150 4900 8500 4900
+	9150 4750 9100 4750
+Wire Wire Line
+	9150 4900 9100 4900
 $Comp
 L power:GND #PWR0319
@@
 NoConn ~ 8000 5000
 NoConn ~ 8000 5150
+$Comp
+L Device:C C306
+U 1 1 5C4671A8
+P 6950 4000
+F 0 "C306" V 7202 4000 50  0000 C CNN
+F 1 "100n" V 7111 4000 50  0000 C CNN
+F 2 "Capacitor_SMD:C_0805_2012Metric" H 6988 3850 50  0001 C CNN
+F 3 "https://www.mouser.se/ProductDetail/KEMET/C0805C104J5RACTU?qs=sGAEpiMZZMs0AnBnWHyRQFCCI5cSbRT%2fIwsdZoDYv9I%3d" H 6950 4000 50  0001 C CNN
+	1    6950 4000
+	0    -1   -1   0
+$EndComp
+Connection ~ 7100 4000
+Wire Wire Line
+	7100 4000 7100 4850
+$Comp
+L Device:C C308
+U 1 1 5C46724B
+P 7350 4000
+F 0 "C308" V 7602 4000 50  0000 C CNN
+F 1 "100n" V 7511 4000 50  0000 C CNN
+F 2 "Capacitor_SMD:C_0805_2012Metric" H 7388 3850 50  0001 C CNN
+F 3 "https://www.mouser.se/ProductDetail/KEMET/C0805C104J5RACTU?qs=sGAEpiMZZMs0AnBnWHyRQFCCI5cSbRT%2fIwsdZoDYv9I%3d" H 7350 4000 50  0001 C CNN
+	1    7350 4000
+	0    -1   -1   0
+$EndComp
+Connection ~ 7200 4000
+Wire Wire Line
+	7200 4000 7200 4700
+$Comp
+L power:GND #PWR0323
+U 1 1 5C4672B9
+P 7500 4000
+F 0 "#PWR0323" H 7500 3750 50  0001 C CNN
+F 1 "GND" V 7505 3872 50  0000 R CNN
+F 2 "" H 7500 4000 50  0001 C CNN
+F 3 "" H 7500 4000 50  0001 C CNN
+	1    7500 4000
+	0    -1   -1   0
+$EndComp
+$Comp
+L power:GND #PWR0322
+U 1 1 5C467348
+P 6800 4000
+F 0 "#PWR0322" H 6800 3750 50  0001 C CNN
+F 1 "GND" V 6805 3872 50  0000 R CNN
+F 2 "" H 6800 4000 50  0001 C CNN
+F 3 "" H 6800 4000 50  0001 C CNN
+	1    6800 4000
+	0    1    1    0
+$EndComp
+$Comp
+L Device:C C309
+U 1 1 5C4693F4
+P 9100 4600
+F 0 "C309" V 9352 4600 50  0000 C CNN
+F 1 "100n" V 9261 4600 50  0000 C CNN
+F 2 "Capacitor_SMD:C_0805_2012Metric" H 9138 4450 50  0001 C CNN
+F 3 "https://www.mouser.se/ProductDetail/KEMET/C0805C104J5RACTU?qs=sGAEpiMZZMs0AnBnWHyRQFCCI5cSbRT%2fIwsdZoDYv9I%3d" H 9100 4600 50  0001 C CNN
+	1    9100 4600
+	1    0    0    -1
+$EndComp
+$Comp
+L power:GND #PWR0324
+U 1 1 5C4693FB
+P 9100 4450
+F 0 "#PWR0324" H 9100 4200 50  0001 C CNN
+F 1 "GND" V 9105 4322 50  0000 R CNN
+F 2 "" H 9100 4450 50  0001 C CNN
+F 3 "" H 9100 4450 50  0001 C CNN
+	1    9100 4450
+	-1   0    0    1
+$EndComp
+Connection ~ 9100 4750
+Wire Wire Line
+	9100 4750 8500 4750
+$Comp
+L Device:C C310
+U 1 1 5C4701F0
+P 9100 5050
+F 0 "C310" V 8850 5050 50  0000 C CNN
+F 1 "100n" V 8950 5050 50  0000 C CNN
+F 2 "Capacitor_SMD:C_0805_2012Metric" H 9138 4900 50  0001 C CNN
+F 3 "https://www.mouser.se/ProductDetail/KEMET/C0805C104J5RACTU?qs=sGAEpiMZZMs0AnBnWHyRQFCCI5cSbRT%2fIwsdZoDYv9I%3d" H 9100 5050 50  0001 C CNN
+	1    9100 5050
+	-1   0    0    1
+$EndComp
+$Comp
+L power:GND #PWR0325
+U 1 1 5C4701F7
+P 9100 5200
+F 0 "#PWR0325" H 9100 4950 50  0001 C CNN
+F 1 "GND" V 9105 5072 50  0000 R CNN
+F 2 "" H 9100 5200 50  0001 C CNN
+F 3 "" H 9100 5200 50  0001 C CNN
+	1    9100 5200
+	1    0    0    -1
+$EndComp
+Connection ~ 9100 4900
+Wire Wire Line
+	9100 4900 8500 4900
 $EndSCHEMATC
