File: hardware/5VDigitalOutput.sch (KiCad schematic (older format))
At the start: 6 parts, among them Q2401 ZXTN25050DFHTA, Q2402 ZXTN25050DFHTA

Commit message: Outputs now uses MOSFETs
Parts:
- removed Q2401, Q2402: ZXTN25050DFHTA, Package_TO_SOT_SMD:SOT-23, symbol Device:Q_NPN_BCE
- added Q2401: Si2312CD, Package_TO_SOT_SMD:SOT-23, symbol PerMalmberg:Si2312CD
- added Q2402: Si2323CDS, Package_TO_SOT_SMD:SOT-23, symbol PerMalmberg:Si2323CDS
- added R2404: 4.7k, symbol Device:R
- added R2405: 120, Resistor_SMD:R_0805_2012Metric, symbol Device:R
- D2401: value Red -> Green
- R2401: value 470 -> 10k
- R2402: value 10k -> 1.65k
- R2403: value 1.65k -> 120
Connections:
- net +5V: now also Q2402.2 (S), R2404.1
- net CTRL: now also R2402.2, R2403.2
- net GND: now also R2401.1, Q2401.2 (S); no longer R2402.1
- net Output: now also Q2402.3 (D)
- net at D2401.2 (A): now also R2402.1; no longer R2403.1
- new net: Q2401.1 (G), R2403.1
- new net: Q2401.3 (D), R2404.2, R2405.2
- new net: Q2402.1 (G), R2405.1
Other:
- note added: "Zener diodes and stop resisitors must be placed as close\nto mosfets as possible with shortest possible traces to reduce\noscillation and reduce capacitance."

Commit message: Preparing to replicate layout for outputs.
Parts:
- R2404: footprint (none) -> Resistor_SMD:R_0805_2012Metric
Other:
- note added: "Stop resisitors must be placed as close\nto mosfets as possible with shortest possible traces to reduce\noscillation and reduce capacitance."
- note removed: "Zener diodes and stop resisitors must be placed as close\nto mosfets as possible with shortest possible traces to reduce\noscillation and reduce capacitance."
Changed lines of the file:
@@
 F 1 "120" V 4600 5750 50  0000 C CNN
 F 2 "Resistor_SMD:R_0805_2012Metric" V 4530 5750 50  0001 C CNN
-F 3 "~" H 4600 5750 50  0001 C CNN
+F 3 "https://www.mouser.se/ProductDetail/Yageo/RT0805FRE07120RL?qs=sGAEpiMZZMu61qfTUdNhGxEjuuBLd0B4GJARAMhcGkM%3d" H 4600 5750 50  0001 C CNN
 	1    4600 5750
 	0    1    1    0
@@
 F 0 "R2404" V 4350 5350 50  0000 L CNN
 F 1 "4.7k" V 4450 5350 50  0000 L CNN
-F 2 "" V 4380 5450 50  0001 C CNN
-F 3 "~" H 4450 5450 50  0001 C CNN
+F 2 "Resistor_SMD:R_0805_2012Metric" V 4380 5450 50  0001 C CNN
+F 3 "https://www.mouser.se/ProductDetail/Yageo/RT0805FRE134K7L?qs=sGAEpiMZZMu61qfTUdNhG7aYZMPoYcGCBsSWytAGlDAzZPdys9pEHA%3d%3d" H 4450 5450 50  0001 C CNN
 	1    4450 5450
 	1    0    0    -1
@@
 Connection ~ 4450 5750
 Text Notes 3100 4800 0    50   ~ 0
-Zener diodes and stop resisitors must be placed as close\nto mosfets as possible with shortest possible traces to reduce\noscillation and reduce capacitance.
+Stop resisitors must be placed as close\nto mosfets as possible with shortest possible traces to reduce\noscillation and reduce capacitance.
 Wire Wire Line
 	5200 5650 5200 5200
