File: hardware/AnalogSensCircuit.sch (KiCad schematic (older format))
At the start: 8 parts

Commit message: #5 - Moved All SD pullup resistors except R406 (SD_DATA2/MTDI/GPIO12) to SD-side of MAX4948. #3 - Added jumper for GPIO2 <-> GPOI0 for flash download. Removed affected items from PCB.
Changed lines of the file:
@@
 AR Path="/5B61F011/5B774D4C/5B76223E" Ref="D1202"  Part="1"
 AR Path="/5B61F011/5B77572B/5B76223E" Ref="D1302"  Part="1"
-F 0 "D602" H 2700 1650 50  0000 L CNN
+F 0 "D1302" H 2700 1650 50  0000 L CNN
 F 1 "STPS0560Z" V 2600 1100 50  0000 L CNN
 F 2 "Diode_SMD:D_SOD-123" H 2750 1550 50  0001 C CNN
@@
 AR Path="/5B61F011/5B774D4C/5B76225E" Ref="D1201"  Part="1"
 AR Path="/5B61F011/5B77572B/5B76225E" Ref="D1301"  Part="1"
-F 0 "D601" V 2300 1750 50  0000 L CNN
+F 0 "D1301" V 2300 1750 50  0000 L CNN
 F 1 "CDBA3100-HF" V 2400 1600 50  0000 L CNN
 F 2 "Diode_SMD:D_SMA" H 2100 1850 50  0001 C CNN
@@
 AR Path="/5B61F011/5B774D4C/5B762265" Ref="C1201"  Part="1"
 AR Path="/5B61F011/5B77572B/5B762265" Ref="C1301"  Part="1"
-F 0 "C601" H 2565 1896 50  0000 L CNN
+F 0 "C1301" H 2565 1896 50  0000 L CNN
 F 1 "100n" H 2550 1800 50  0000 L CNN
 F 2 "Capacitor_SMD:C_0805_2012Metric" H 2488 1700 50  0001 C CNN
@@
 AR Path="/5B61F011/5B774D4C/5B76226C" Ref="RV1201"  Part="1"
 AR Path="/5B61F011/5B77572B/5B76226C" Ref="RV1301"  Part="1"
-F 0 "RV601" V 1550 1900 50  0000 C CNN
+F 0 "RV1301" V 1550 1900 50  0000 C CNN
 F 1 "B72510E250K062" V 1650 2050 50  0000 C CNN
 F 2 "Capacitor_SMD:C_0805_2012Metric" V 1730 1850 50  0001 C CNN
@@
 AR Path="/5B61F011/5B774D4C/5B762273" Ref="R1202"  Part="1"
 AR Path="/5B61F011/5B77572B/5B762273" Ref="R1302"  Part="1"
-F 0 "R602" H 2520 1596 50  0000 L CNN
+F 0 "R1302" H 2520 1596 50  0000 L CNN
 F 1 "2k" V 2450 1500 50  0000 L CNN
 F 2 "Resistor_SMD:R_0805_2012Metric" V 2380 1550 50  0001 C CNN
@@
 AR Path="/5B61F011/5B774D4C/5B76227A" Ref="R1201"  Part="1"
 AR Path="/5B61F011/5B77572B/5B76227A" Ref="R1301"  Part="1"
-F 0 "R601" V 2200 1700 50  0000 C CNN
+F 0 "R1301" V 2200 1700 50  0000 C CNN
 F 1 "1k" V 2300 1700 50  0000 C CNN
 F 2 "Resistor_SMD:R_0805_2012Metric" V 2230 1700 50  0001 C CNN
@@
 AR Path="/5B61F011/5B774D4C/5B762281" Ref="D1203"  Part="1"
 AR Path="/5B61F011/5B77572B/5B762281" Ref="D1303"  Part="1"
-F 0 "D603" H 2700 1950 50  0000 L CNN
+F 0 "D1303" H 2700 1950 50  0000 L CNN
 F 1 "STPS0560Z" H 2700 1750 50  0000 L CNN
 F 2 "Diode_SMD:D_SOD-123" H 2750 1850 50  0001 C CNN
@@
 AR Path="/5B61F011/5B774D4C/5B762288" Ref="R1203"  Part="1"
 AR Path="/5B61F011/5B77572B/5B762288" Ref="R1303"  Part="1"
-F 0 "R603" V 2800 1650 50  0000 C CNN
+F 0 "R1303" V 2800 1650 50  0000 C CNN
 F 1 "100" V 2900 1700 50  0000 C CNN
 F 2 "Resistor_SMD:R_0805_2012Metric" V 2830 1700 50  0001 C CNN

Commit message: #11 Put transistor on the low side for SD Card power.
Changed lines of the file:
@@
 $Descr A4 11693 8268
 encoding utf-8
-Sheet 6 34
+Sheet 11 34
 Title ""
 Date ""
@@
 AR Path="/5B61F011/5B774D4C/5B76223E" Ref="D1202"  Part="1"
 AR Path="/5B61F011/5B77572B/5B76223E" Ref="D1302"  Part="1"
-F 0 "D1302" H 2700 1650 50  0000 L CNN
+F 0 "D1102" H 2700 1650 50  0000 L CNN
 F 1 "STPS0560Z" V 2600 1100 50  0000 L CNN
 F 2 "Diode_SMD:D_SOD-123" H 2750 1550 50  0001 C CNN
@@
 AR Path="/5B61F011/5B774D4C/5B762247" Ref="#PWR01201"  Part="1"
 AR Path="/5B61F011/5B77572B/5B762247" Ref="#PWR01301"  Part="1"
-F 0 "#PWR01301" H 2600 1250 50  0001 C CNN
+F 0 "#PWR01101" H 2600 1250 50  0001 C CNN
 F 1 "+5V" H 2615 1573 50  0000 C CNN
 F 2 "" H 2600 1400 50  0001 C CNN
@@
 AR Path="/5B61F011/5B774D4C/5B762258" Ref="#PWR01202"  Part="1"
 AR Path="/5B61F011/5B77572B/5B762258" Ref="#PWR01302"  Part="1"
-F 0 "#PWR01302" H 2750 1750 50  0001 C CNN
+F 0 "#PWR01102" H 2750 1750 50  0001 C CNN
 F 1 "GND" H 2755 1827 50  0000 C CNN
 F 2 "" H 2750 2000 50  0001 C CNN
@@
 AR Path="/5B61F011/5B774D4C/5B76225E" Ref="D1201"  Part="1"
 AR Path="/5B61F011/5B77572B/5B76225E" Ref="D1301"  Part="1"
-F 0 "D1301" V 2300 1750 50  0000 L CNN
+F 0 "D1101" V 2300 1750 50  0000 L CNN
 F 1 "CDBA3100-HF" V 2400 1600 50  0000 L CNN
 F 2 "Diode_SMD:D_SMA" H 2100 1850 50  0001 C CNN
@@
 AR Path="/5B61F011/5B774D4C/5B762265" Ref="C1201"  Part="1"
 AR Path="/5B61F011/5B77572B/5B762265" Ref="C1301"  Part="1"
-F 0 "C1301" H 2565 1896 50  0000 L CNN
+F 0 "C1101" H 2565 1896 50  0000 L CNN
 F 1 "100n" H 2550 1800 50  0000 L CNN
 F 2 "Capacitor_SMD:C_0805_2012Metric" H 2488 1700 50  0001 C CNN
@@
 AR Path="/5B61F011/5B774D4C/5B76226C" Ref="RV1201"  Part="1"
 AR Path="/5B61F011/5B77572B/5B76226C" Ref="RV1301"  Part="1"
-F 0 "RV1301" V 1550 1900 50  0000 C CNN
+F 0 "RV1101" V 1550 1900 50  0000 C CNN
 F 1 "B72510E250K062" V 1650 2050 50  0000 C CNN
 F 2 "Capacitor_SMD:C_0805_2012Metric" V 1730 1850 50  0001 C CNN
@@
 AR Path="/5B61F011/5B774D4C/5B762273" Ref="R1202"  Part="1"
 AR Path="/5B61F011/5B77572B/5B762273" Ref="R1302"  Part="1"
-F 0 "R1302" H 2520 1596 50  0000 L CNN
+F 0 "R1102" H 2520 1596 50  0000 L CNN
 F 1 "2k" V 2450 1500 50  0000 L CNN
 F 2 "Resistor_SMD:R_0805_2012Metric" V 2380 1550 50  0001 C CNN
@@
 AR Path="/5B61F011/5B774D4C/5B76227A" Ref="R1201"  Part="1"
 AR Path="/5B61F011/5B77572B/5B76227A" Ref="R1301"  Part="1"
-F 0 "R1301" V 2200 1700 50  0000 C CNN
+F 0 "R1101" V 2200 1700 50  0000 C CNN
 F 1 "1k" V 2300 1700 50  0000 C CNN
 F 2 "Resistor_SMD:R_0805_2012Metric" V 2230 1700 50  0001 C CNN
@@
 AR Path="/5B61F011/5B774D4C/5B762281" Ref="D1203"  Part="1"
 AR Path="/5B61F011/5B77572B/5B762281" Ref="D1303"  Part="1"
-F 0 "D1303" H 2700 1950 50  0000 L CNN
+F 0 "D1103" H 2700 1950 50  0000 L CNN
 F 1 "STPS0560Z" H 2700 1750 50  0000 L CNN
 F 2 "Diode_SMD:D_SOD-123" H 2750 1850 50  0001 C CNN
@@
 AR Path="/5B61F011/5B774D4C/5B762288" Ref="R1203"  Part="1"
 AR Path="/5B61F011/5B77572B/5B762288" Ref="R1303"  Part="1"
-F 0 "R1303" V 2800 1650 50  0000 C CNN
+F 0 "R1103" V 2800 1650 50  0000 C CNN
 F 1 "100" V 2900 1700 50  0000 C CNN
 F 2 "Resistor_SMD:R_0805_2012Metric" V 2830 1700 50  0001 C CNN

Commit message: Outputs now uses MOSFETs
Changed lines of the file:
@@
 AR Path="/5B61F011/5B774D4C/5B76223E" Ref="D1202"  Part="1"
 AR Path="/5B61F011/5B77572B/5B76223E" Ref="D1302"  Part="1"
-F 0 "D1102" H 2700 1650 50  0000 L CNN
+F 0 "D1302" H 2700 1650 50  0000 L CNN
 F 1 "STPS0560Z" V 2600 1100 50  0000 L CNN
 F 2 "Diode_SMD:D_SOD-123" H 2750 1550 50  0001 C CNN
@@
 AR Path="/5B61F011/5B774D4C/5B762247" Ref="#PWR01201"  Part="1"
 AR Path="/5B61F011/5B77572B/5B762247" Ref="#PWR01301"  Part="1"
-F 0 "#PWR01101" H 2600 1250 50  0001 C CNN
+F 0 "#PWR01301" H 2600 1250 50  0001 C CNN
 F 1 "+5V" H 2615 1573 50  0000 C CNN
 F 2 "" H 2600 1400 50  0001 C CNN
@@
 AR Path="/5B61F011/5B774D4C/5B762258" Ref="#PWR01202"  Part="1"
 AR Path="/5B61F011/5B77572B/5B762258" Ref="#PWR01302"  Part="1"
-F 0 "#PWR01102" H 2750 1750 50  0001 C CNN
+F 0 "#PWR01302" H 2750 1750 50  0001 C CNN
 F 1 "GND" H 2755 1827 50  0000 C CNN
 F 2 "" H 2750 2000 50  0001 C CNN
@@
 AR Path="/5B61F011/5B774D4C/5B76225E" Ref="D1201"  Part="1"
 AR Path="/5B61F011/5B77572B/5B76225E" Ref="D1301"  Part="1"
-F 0 "D1101" V 2300 1750 50  0000 L CNN
+F 0 "D1301" V 2300 1750 50  0000 L CNN
 F 1 "CDBA3100-HF" V 2400 1600 50  0000 L CNN
 F 2 "Diode_SMD:D_SMA" H 2100 1850 50  0001 C CNN
@@
 AR Path="/5B61F011/5B774D4C/5B762265" Ref="C1201"  Part="1"
 AR Path="/5B61F011/5B77572B/5B762265" Ref="C1301"  Part="1"
-F 0 "C1101" H 2565 1896 50  0000 L CNN
+F 0 "C1301" H 2565 1896 50  0000 L CNN
 F 1 "100n" H 2550 1800 50  0000 L CNN
 F 2 "Capacitor_SMD:C_0805_2012Metric" H 2488 1700 50  0001 C CNN
@@
 AR Path="/5B61F011/5B774D4C/5B76226C" Ref="RV1201"  Part="1"
 AR Path="/5B61F011/5B77572B/5B76226C" Ref="RV1301"  Part="1"
-F 0 "RV1101" V 1550 1900 50  0000 C CNN
+F 0 "RV1301" V 1550 1900 50  0000 C CNN
 F 1 "B72510E250K062" V 1650 2050 50  0000 C CNN
 F 2 "Capacitor_SMD:C_0805_2012Metric" V 1730 1850 50  0001 C CNN
@@
 AR Path="/5B61F011/5B774D4C/5B762273" Ref="R1202"  Part="1"
 AR Path="/5B61F011/5B77572B/5B762273" Ref="R1302"  Part="1"
-F 0 "R1102" H 2520 1596 50  0000 L CNN
+F 0 "R1302" H 2520 1596 50  0000 L CNN
 F 1 "2k" V 2450 1500 50  0000 L CNN
 F 2 "Resistor_SMD:R_0805_2012Metric" V 2380 1550 50  0001 C CNN
@@
 AR Path="/5B61F011/5B774D4C/5B76227A" Ref="R1201"  Part="1"
 AR Path="/5B61F011/5B77572B/5B76227A" Ref="R1301"  Part="1"
-F 0 "R1101" V 2200 1700 50  0000 C CNN
+F 0 "R1301" V 2200 1700 50  0000 C CNN
 F 1 "1k" V 2300 1700 50  0000 C CNN
 F 2 "Resistor_SMD:R_0805_2012Metric" V 2230 1700 50  0001 C CNN
@@
 AR Path="/5B61F011/5B774D4C/5B762281" Ref="D1203"  Part="1"
 AR Path="/5B61F011/5B77572B/5B762281" Ref="D1303"  Part="1"
-F 0 "D1103" H 2700 1950 50  0000 L CNN
+F 0 "D1303" H 2700 1950 50  0000 L CNN
 F 1 "STPS0560Z" H 2700 1750 50  0000 L CNN
 F 2 "Diode_SMD:D_SOD-123" H 2750 1850 50  0001 C CNN
@@
 AR Path="/5B61F011/5B774D4C/5B762288" Ref="R1203"  Part="1"
 AR Path="/5B61F011/5B77572B/5B762288" Ref="R1303"  Part="1"
-F 0 "R1103" V 2800 1650 50  0000 C CNN
+F 0 "R1303" V 2800 1650 50  0000 C CNN
 F 1 "100" V 2900 1700 50  0000 C CNN
 F 2 "Resistor_SMD:R_0805_2012Metric" V 2830 1700 50  0001 C CNN
