File: hardware/DigitalIO.sch (KiCad schematic (older format))
At the start: 18 parts, among them U1401 MCP23017, U1402 MCP23017

Commit message: #1 SD_ENABLE removed; pin grounded. #7 All pins on seconds MCP2317 used. Updated I2CTask to match new H/W layout. Closes #1. Closes #7.
Parts:
- removed R1402: 10k, Resistor_SMD:R_0805_2012Metric, symbol Device:R
- added D1, D2, D3, D4, D5, D6, D7: Red, LED_THT:LED_D5.0mm, symbol Device:LED
- added R1, R2, R3, R4, R5, R6, R7: 1.65k, Resistor_SMD:R_0805_2012Metric, symbol Device:R
Connections:
- net SD_ENABLE is gone; now on net BELL_CTRL: U1402.1 (GPB0)
- net BELL_CTRL: no longer U1402.2 (GPB1)
- net GND: now also D1.1 (K), D2.1 (K), D3.1 (K), D4.1 (K), D5.1 (K), D6.1 (K), D7.1 (K)
- net SD_MODE: now also U1402.28 (GPA7); no longer U1402.21 (GPA0)
- new net: R1.2, U1402.21 (GPA0)
- new net: R2.2, U1402.22 (GPA1)
- new net: R3.2, U1402.23 (GPA2)
- new net: R4.2, U1402.24 (GPA3)
- new net: R5.2, U1402.25 (GPA4)
- new net: R6.2, U1402.26 (GPA5)
- new net: R7.2, U1402.27 (GPA6)
- new net: D1.2 (A), R1.1
- new net: D2.2 (A), R2.1
- new net: D3.2 (A), R3.1
- new net: D4.2 (A), R4.1
- new net: D5.2 (A), R5.1
- new net: D6.2 (A), R6.1
- new net: D7.2 (A), R7.1
- new net INTERNAL_SIREN_CTRL: U1402.2 (GPB1)
Other:
- moved on the sheet: U1402

Commit message: #8 - Added SD Card power circuit controlled via I2C.
Parts:
- removed D1401: Red, LED_THT:LED_D5.0mm, symbol Device:LED
- removed R1401: 1.65k, Resistor_SMD:R_0805_2012Metric, symbol Device:R
Connections:
- net SD_CARD_PWR_CTRL: now reaches U1402.3 (GPB2)
Changed lines of the file:
@@
-$Comp
-L Device:LED D?
-U 1 1 5BA5B3F8
-P 1450 5150
-AR Path="/5B62EDB8/5B780EE8/5BA5B3F8" Ref="D?"  Part="1"
-AR Path="/5B62EDB8/5B66E27E/5BA5B3F8" Ref="D?"  Part="1"
-AR Path="/5B62EDB8/5B66FC5D/5BA5B3F8" Ref="D?"  Part="1"
-AR Path="/5B62EDB8/5B685B64/5BA5B3F8" Ref="D?"  Part="1"
-AR Path="/5B62EDB8/5B687263/5BA5B3F8" Ref="D?"  Part="1"
-AR Path="/5B62EDB8/5B688B1A/5BA5B3F8" Ref="D?"  Part="1"
-AR Path="/5B62EDB8/5B68A219/5BA5B3F8" Ref="D?"  Part="1"
-AR Path="/5B62EDB8/5B68BAA8/5BA5B3F8" Ref="D?"  Part="1"
-AR Path="/5B62EDB8/5B68D1A7/5BA5B3F8" Ref="D?"  Part="1"
-AR Path="/5B62EDB8/5BA53A47/5BA5B3F8" Ref="D?"  Part="1"
-AR Path="/5B62EDB8/5BA53BAF/5BA5B3F8" Ref="D?"  Part="1"
-AR Path="/5B62EDB8/5BA53CC3/5BA5B3F8" Ref="D?"  Part="1"
-AR Path="/5B62EDB8/5BA53E16/5BA5B3F8" Ref="D?"  Part="1"
-AR Path="/5B62EDB8/5BA53F23/5BA5B3F8" Ref="D?"  Part="1"
-AR Path="/5B62EDB8/5BA54030/5BA5B3F8" Ref="D?"  Part="1"
-AR Path="/5B62EDB8/5BA5413D/5BA5B3F8" Ref="D?"  Part="1"
-AR Path="/5B62EDB8/5BA5B3F8" Ref="D1401"  Part="1"
-F 0 "D1401" H 1442 4895 50  0000 C CNN
-F 1 "Red" H 1442 4986 50  0000 C CNN
-F 2 "LED_THT:LED_D5.0mm" H 1450 5150 50  0001 C CNN
-F 3 "https://www.mouser.se/ProductDetail/Lite-On/LTL2R3KGD-EM?qs=sGAEpiMZZMtmwHDZQCdlqY3QuPVQdrfivxVgVo2hFbg%3d" H 1450 5150 50  0001 C CNN
-	1    1450 5150
-	1    0    0    -1
-$EndComp
-$Comp
-L Device:R R?
-U 1 1 5BA5B3FF
-P 1750 5150
-AR Path="/5B62EDB8/5B780EE8/5BA5B3FF" Ref="R?"  Part="1"
-AR Path="/5B62EDB8/5B66E27E/5BA5B3FF" Ref="R?"  Part="1"
-AR Path="/5B62EDB8/5B66FC5D/5BA5B3FF" Ref="R?"  Part="1"
-AR Path="/5B62EDB8/5B685B64/5BA5B3FF" Ref="R?"  Part="1"
-AR Path="/5B62EDB8/5B687263/5BA5B3FF" Ref="R?"  Part="1"
-AR Path="/5B62EDB8/5B688B1A/5BA5B3FF" Ref="R?"  Part="1"
-AR Path="/5B62EDB8/5B68A219/5BA5B3FF" Ref="R?"  Part="1"
-AR Path="/5B62EDB8/5B68BAA8/5BA5B3FF" Ref="R?"  Part="1"
-AR Path="/5B62EDB8/5B68D1A7/5BA5B3FF" Ref="R?"  Part="1"
-AR Path="/5B62EDB8/5BA53A47/5BA5B3FF" Ref="R?"  Part="1"
-AR Path="/5B62EDB8/5BA53BAF/5BA5B3FF" Ref="R?"  Part="1"
-AR Path="/5B62EDB8/5BA53CC3/5BA5B3FF" Ref="R?"  Part="1"
-AR Path="/5B62EDB8/5BA53E16/5BA5B3FF" Ref="R?"  Part="1"
-AR Path="/5B62EDB8/5BA53F23/5BA5B3FF" Ref="R?"  Part="1"
-AR Path="/5B62EDB8/5BA54030/5BA5B3FF" Ref="R?"  Part="1"
-AR Path="/5B62EDB8/5BA5413D/5BA5B3FF" Ref="R?"  Part="1"
-AR Path="/5B62EDB8/5BA5B3FF" Ref="R1401"  Part="1"
-F 0 "R1401" V 1543 5150 50  0000 C CNN
-F 1 "1.65k" V 1634 5150 50  0000 C CNN
-F 2 "Resistor_SMD:R_0805_2012Metric" V 1680 5150 50  0001 C CNN
-F 3 "https://www.mouser.se/ProductDetail/Vishay/CRCW08051K65FKEA?qs=sGAEpiMZZMtlubZbdhIBIFvv2%252blmU1cYk%2fKBbkOVYDU%3d" H 1750 5150 50  0001 C CNN
-	1    1750 5150
-	0    -1   -1   0
-$EndComp
-$Comp
-L power:GND #PWR0101
-U 1 1 5BA5B6E6
-P 1300 5150
-F 0 "#PWR0101" H 1300 4900 50  0001 C CNN
-F 1 "GND" V 1305 5022 50  0000 R CNN
-F 2 "" H 1300 5150 50  0001 C CNN
-F 3 "" H 1300 5150 50  0001 C CNN
-	1    1300 5150
-	0    1    1    0
-$EndComp
 $Comp
 L Device:LED D?
@@
 INTERNAL_SIREN_CTRL
 Wire Wire Line
-	3800 5300 1900 5300
-Wire Wire Line
-	1900 5300 1900 5150
-Wire Wire Line
 	1900 5400 1900 5500
 Wire Wire Line
@@
 Wire Wire Line
 	2600 6600 3800 6600
+Text GLabel 3800 5300 0    50   Input ~ 0
+SD_CARD_PWR_CTRL
 $EndSCHEMATC

Commit message: Started to re-route PCB for schematics changes.
Parts:
- renumbered D1402 to D1401, D1403 to D1402, D1404 to D1403, D1405 to D1404, D1406 to D1405, D1 to D1406, D2 to D1407, D3 to D1408, D4 to D1409, D5 to D1410, D6 to D1411, D7 to D1412, R1403 to R1401, R1404 to R1402, R1405 to R1403, R1406 to R1404, R1407 to R1405, R1 to R1406, R2 to R1407, R3 to R1408, R4 to R1409, R5 to R1410, R6 to R1411, R7 to R1412
Changed lines of the file:
@@
 AR Path="/5B62EDB8/5BA54030/5BA5B774" Ref="D?"  Part="1"
 AR Path="/5B62EDB8/5BA5413D/5BA5B774" Ref="D?"  Part="1"
-AR Path="/5B62EDB8/5BA5B774" Ref="D1402"  Part="1"
-F 0 "D1402" H 1442 5245 50  0000 C CNN
+AR Path="/5B62EDB8/5BA5B774" Ref="D1401"  Part="1"
+F 0 "D1401" H 1442 5245 50  0000 C CNN
 F 1 "Red" H 1442 5336 50  0000 C CNN
 F 2 "LED_THT:LED_D5.0mm" H 1450 5500 50  0001 C CNN
@@
 AR Path="/5B62EDB8/5BA54030/5BA5B77B" Ref="R?"  Part="1"
 AR Path="/5B62EDB8/5BA5413D/5BA5B77B" Ref="R?"  Part="1"
-AR Path="/5B62EDB8/5BA5B77B" Ref="R1403"  Part="1"
-F 0 "R1403" V 1543 5500 50  0000 C CNN
+AR Path="/5B62EDB8/5BA5B77B" Ref="R1401"  Part="1"
+F 0 "R1401" V 1543 5500 50  0000 C CNN
 F 1 "1.65k" V 1634 5500 50  0000 C CNN
 F 2 "Resistor_SMD:R_0805_2012Metric" V 1680 5500 50  0001 C CNN
@@
 AR Path="/5B62EDB8/5BA54030/5BA5B879" Ref="D?"  Part="1"
 AR Path="/5B62EDB8/5BA5413D/5BA5B879" Ref="D?"  Part="1"
-AR Path="/5B62EDB8/5BA5B879" Ref="D1403"  Part="1"
-F 0 "D1403" H 1442 5595 50  0000 C CNN
+AR Path="/5B62EDB8/5BA5B879" Ref="D1402"  Part="1"
+F 0 "D1402" H 1442 5595 50  0000 C CNN
 F 1 "Red" H 1442 5686 50  0000 C CNN
 F 2 "LED_THT:LED_D5.0mm" H 1450 5850 50  0001 C CNN
@@
 AR Path="/5B62EDB8/5BA54030/5BA5B880" Ref="R?"  Part="1"
 AR Path="/5B62EDB8/5BA5413D/5BA5B880" Ref="R?"  Part="1"
-AR Path="/5B62EDB8/5BA5B880" Ref="R1404"  Part="1"
-F 0 "R1404" V 1543 5850 50  0000 C CNN
+AR Path="/5B62EDB8/5BA5B880" Ref="R1402"  Part="1"
+F 0 "R1402" V 1543 5850 50  0000 C CNN
 F 1 "1.65k" V 1634 5850 50  0000 C CNN
 F 2 "Resistor_SMD:R_0805_2012Metric" V 1680 5850 50  0001 C CNN
@@
 AR Path="/5B62EDB8/5BA54030/5BA5BA0A" Ref="D?"  Part="1"
 AR Path="/5B62EDB8/5BA5413D/5BA5BA0A" Ref="D?"  Part="1"
-AR Path="/5B62EDB8/5BA5BA0A" Ref="D1404"  Part="1"
-F 0 "D1404" H 1442 5995 50  0000 C CNN
+AR Path="/5B62EDB8/5BA5BA0A" Ref="D1403"  Part="1"
+F 0 "D1403" H 1442 5995 50  0000 C CNN
 F 1 "Red" H 1442 6086 50  0000 C CNN
 F 2 "LED_THT:LED_D5.0mm" H 1450 6250 50  0001 C CNN
@@
 AR Path="/5B62EDB8/5BA54030/5BA5BA11" Ref="R?"  Part="1"
 AR Path="/5B62EDB8/5BA5413D/5BA5BA11" Ref="R?"  Part="1"
-AR Path="/5B62EDB8/5BA5BA11" Ref="R1405"  Part="1"
-F 0 "R1405" V 1543 6250 50  0000 C CNN
+AR Path="/5B62EDB8/5BA5BA11" Ref="R1403"  Part="1"
+F 0 "R1403" V 1543 6250 50  0000 C CNN
 F 1 "1.65k" V 1634 6250 50  0000 C CNN
 F 2 "Resistor_SMD:R_0805_2012Metric" V 1680 6250 50  0001 C CNN
@@
 AR Path="/5B62EDB8/5BA54030/5BA5BDA3" Ref="D?"  Part="1"
 AR Path="/5B62EDB8/5BA5413D/5BA5BDA3" Ref="D?"  Part="1"
-AR Path="/5B62EDB8/5BA5BDA3" Ref="D1405"  Part="1"
-F 0 "D1405" H 1442 6395 50  0000 C CNN
+AR Path="/5B62EDB8/5BA5BDA3" Ref="D1404"  Part="1"
+F 0 "D1404" H 1442 6395 50  0000 C CNN
 F 1 "Red" H 1442 6486 50  0000 C CNN
 F 2 "LED_THT:LED_D5.0mm" H 1450 6650 50  0001 C CNN
@@
 AR Path="/5B62EDB8/5BA54030/5BA5BDAA" Ref="R?"  Part="1"
 AR Path="/5B62EDB8/5BA5413D/5BA5BDAA" Ref="R?"  Part="1"
-AR Path="/5B62EDB8/5BA5BDAA" Ref="R1406"  Part="1"
-F 0 "R1406" V 1543 6650 50  0000 C CNN
+AR Path="/5B62EDB8/5BA5BDAA" Ref="R1404"  Part="1"
+F 0 "R1404" V 1543 6650 50  0000 C CNN
 F 1 "1.65k" V 1634 6650 50  0000 C CNN
 F 2 "Resistor_SMD:R_0805_2012Metric" V 1680 6650 50  0001 C CNN
@@
 AR Path="/5B62EDB8/5BA54030/5BA5D5BE" Ref="D?"  Part="1"
 AR Path="/5B62EDB8/5BA5413D/5BA5D5BE" Ref="D?"  Part="1"
-AR Path="/5B62EDB8/5BA5D5BE" Ref="D1406"  Part="1"
-F 0 "D1406" H 1442 6795 50  0000 C CNN
+AR Path="/5B62EDB8/5BA5D5BE" Ref="D1405"  Part="1"
+F 0 "D1405" H 1442 6795 50  0000 C CNN
 F 1 "Red" H 1442 6886 50  0000 C CNN
 F 2 "LED_THT:LED_D5.0mm" H 1450 7050 50  0001 C CNN
@@
 AR Path="/5B62EDB8/5BA54030/5BA5D5C5" Ref="R?"  Part="1"
 AR Path="/5B62EDB8/5BA5413D/5BA5D5C5" Ref="R?"  Part="1"
-AR Path="/5B62EDB8/5BA5D5C5" Ref="R1407"  Part="1"
-F 0 "R1407" V 1543 7050 50  0000 C CNN
+AR Path="/5B62EDB8/5BA5D5C5" Ref="R1405"  Part="1"
+F 0 "R1405" V 1543 7050 50  0000 C CNN
 F 1 "1.65k" V 1634 7050 50  0000 C CNN
 F 2 "Resistor_SMD:R_0805_2012Metric" V 1680 7050 50  0001 C CNN
@@
 AR Path="/5B62EDB8/5BA54030/5BF0FC57" Ref="D?"  Part="1"
 AR Path="/5B62EDB8/5BA5413D/5BF0FC57" Ref="D?"  Part="1"
-AR Path="/5B62EDB8/5BF0FC57" Ref="D1"  Part="1"
-F 0 "D1" H 1442 7195 50  0000 C CNN
+AR Path="/5B62EDB8/5BF0FC57" Ref="D1406"  Part="1"
+F 0 "D1406" H 1442 7195 50  0000 C CNN
 F 1 "Red" H 1442 7286 50  0000 C CNN
 F 2 "LED_THT:LED_D5.0mm" H 1450 7450 50  0001 C CNN
@@
 AR Path="/5B62EDB8/5BA54030/5BF0FC5E" Ref="R?"  Part="1"
 AR Path="/5B62EDB8/5BA5413D/5BF0FC5E" Ref="R?"  Part="1"
-AR Path="/5B62EDB8/5BF0FC5E" Ref="R1"  Part="1"
-F 0 "R1" V 1543 7450 50  0000 C CNN
+AR Path="/5B62EDB8/5BF0FC5E" Ref="R1406"  Part="1"
+F 0 "R1406" V 1543 7450 50  0000 C CNN
 F 1 "1.65k" V 1634 7450 50  0000 C CNN
 F 2 "Resistor_SMD:R_0805_2012Metric" V 1680 7450 50  0001 C CNN
@@
 AR Path="/5B62EDB8/5BA54030/5BF0FE5D" Ref="D?"  Part="1"
 AR Path="/5B62EDB8/5BA5413D/5BF0FE5D" Ref="D?"  Part="1"
-AR Path="/5B62EDB8/5BF0FE5D" Ref="D2"  Part="1"
-F 0 "D2" H 1442 7595 50  0000 C CNN
+AR Path="/5B62EDB8/5BF0FE5D" Ref="D1407"  Part="1"
+F 0 "D1407" H 1442 7595 50  0000 C CNN
 F 1 "Red" H 1442 7686 50  0000 C CNN
 F 2 "LED_THT:LED_D5.0mm" H 1450 7850 50  0001 C CNN
@@
 AR Path="/5B62EDB8/5BA54030/5BF0FE64" Ref="R?"  Part="1"
 AR Path="/5B62EDB8/5BA5413D/5BF0FE64" Ref="R?"  Part="1"
-AR Path="/5B62EDB8/5BF0FE64" Ref="R2"  Part="1"
-F 0 "R2" V 1543 7850 50  0000 C CNN
+AR Path="/5B62EDB8/5BF0FE64" Ref="R1407"  Part="1"
+F 0 "R1407" V 1543 7850 50  0000 C CNN
 F 1 "1.65k" V 1634 7850 50  0000 C CNN
 F 2 "Resistor_SMD:R_0805_2012Metric" V 1680 7850 50  0001 C CNN
@@
 AR Path="/5B62EDB8/5BA54030/5BF1006B" Ref="D?"  Part="1"
 AR Path="/5B62EDB8/5BA5413D/5BF1006B" Ref="D?"  Part="1"
-AR Path="/5B62EDB8/5BF1006B" Ref="D3"  Part="1"
-F 0 "D3" H 1442 7995 50  0000 C CNN
+AR Path="/5B62EDB8/5BF1006B" Ref="D1408"  Part="1"
+F 0 "D1408" H 1442 7995 50  0000 C CNN
 F 1 "Red" H 1442 8086 50  0000 C CNN
 F 2 "LED_THT:LED_D5.0mm" H 1450 8250 50  0001 C CNN
@@
 AR Path="/5B62EDB8/5BA54030/5BF10072" Ref="R?"  Part="1"
 AR Path="/5B62EDB8/5BA5413D/5BF10072" Ref="R?"  Part="1"
-AR Path="/5B62EDB8/5BF10072" Ref="R3"  Part="1"
-F 0 "R3" V 1543 8250 50  0000 C CNN
+AR Path="/5B62EDB8/5BF10072" Ref="R1408"  Part="1"
+F 0 "R1408" V 1543 8250 50  0000 C CNN
 F 1 "1.65k" V 1634 8250 50  0000 C CNN
 F 2 "Resistor_SMD:R_0805_2012Metric" V 1680 8250 50  0001 C CNN
@@
 AR Path="/5B62EDB8/5BA54030/5BF102D1" Ref="D?"  Part="1"
 AR Path="/5B62EDB8/5BA5413D/5BF102D1" Ref="D?"  Part="1"
-AR Path="/5B62EDB8/5BF102D1" Ref="D4"  Part="1"
-F 0 "D4" H 1442 8395 50  0000 C CNN
+AR Path="/5B62EDB8/5BF102D1" Ref="D1409"  Part="1"
+F 0 "D1409" H 1442 8395 50  0000 C CNN
 F 1 "Red" H 1442 8486 50  0000 C CNN
 F 2 "LED_THT:LED_D5.0mm" H 1450 8650 50  0001 C CNN
@@
 AR Path="/5B62EDB8/5BA54030/5BF102D8" Ref="R?"  Part="1"
 AR Path="/5B62EDB8/5BA5413D/5BF102D8" Ref="R?"  Part="1"
-AR Path="/5B62EDB8/5BF102D8" Ref="R4"  Part="1"
-F 0 "R4" V 1543 8650 50  0000 C CNN
+AR Path="/5B62EDB8/5BF102D8" Ref="R1409"  Part="1"
+F 0 "R1409" V 1543 8650 50  0000 C CNN
 F 1 "1.65k" V 1634 8650 50  0000 C CNN
 F 2 "Resistor_SMD:R_0805_2012Metric" V 1680 8650 50  0001 C CNN
@@
 AR Path="/5B62EDB8/5BA54030/5BF106D4" Ref="D?"  Part="1"
 AR Path="/5B62EDB8/5BA5413D/5BF106D4" Ref="D?"  Part="1"
-AR Path="/5B62EDB8/5BF106D4" Ref="D5"  Part="1"
-F 0 "D5" H 1442 8795 50  0000 C CNN
+AR Path="/5B62EDB8/5BF106D4" Ref="D1410"  Part="1"
+F 0 "D1410" H 1442 8795 50  0000 C CNN
 F 1 "Red" H 1442 8886 50  0000 C CNN
 F 2 "LED_THT:LED_D5.0mm" H 1450 9050 50  0001 C CNN
@@
 AR Path="/5B62EDB8/5BA54030/5BF106DB" Ref="R?"  Part="1"
 AR Path="/5B62EDB8/5BA5413D/5BF106DB" Ref="R?"  Part="1"
-AR Path="/5B62EDB8/5BF106DB" Ref="R5"  Part="1"
-F 0 "R5" V 1543 9050 50  0000 C CNN
+AR Path="/5B62EDB8/5BF106DB" Ref="R1410"  Part="1"
+F 0 "R1410" V 1543 9050 50  0000 C CNN
 F 1 "1.65k" V 1634 9050 50  0000 C CNN
 F 2 "Resistor_SMD:R_0805_2012Metric" V 1680 9050 50  0001 C CNN
@@
 AR Path="/5B62EDB8/5BA54030/5BF10C65" Ref="D?"  Part="1"
 AR Path="/5B62EDB8/5BA5413D/5BF10C65" Ref="D?"  Part="1"
-AR Path="/5B62EDB8/5BF10C65" Ref="D6"  Part="1"
-F 0 "D6" H 1442 9195 50  0000 C CNN
+AR Path="/5B62EDB8/5BF10C65" Ref="D1411"  Part="1"
+F 0 "D1411" H 1442 9195 50  0000 C CNN
 F 1 "Red" H 1442 9286 50  0000 C CNN
 F 2 "LED_THT:LED_D5.0mm" H 1450 9450 50  0001 C CNN
@@
 AR Path="/5B62EDB8/5BA54030/5BF10C6C" Ref="R?"  Part="1"
 AR Path="/5B62EDB8/5BA5413D/5BF10C6C" Ref="R?"  Part="1"
-AR Path="/5B62EDB8/5BF10C6C" Ref="R6"  Part="1"
-F 0 "R6" V 1543 9450 50  0000 C CNN
+AR Path="/5B62EDB8/5BF10C6C" Ref="R1411"  Part="1"
+F 0 "R1411" V 1543 9450 50  0000 C CNN
 F 1 "1.65k" V 1634 9450 50  0000 C CNN
 F 2 "Resistor_SMD:R_0805_2012Metric" V 1680 9450 50  0001 C CNN
@@
 AR Path="/5B62EDB8/5BA54030/5BF65E41" Ref="D?"  Part="1"
 AR Path="/5B62EDB8/5BA5413D/5BF65E41" Ref="D?"  Part="1"
-AR Path="/5B62EDB8/5BF65E41" Ref="D7"  Part="1"
-F 0 "D7" H 1442 9595 50  0000 C CNN
+AR Path="/5B62EDB8/5BF65E41" Ref="D1412"  Part="1"
+F 0 "D1412" H 1442 9595 50  0000 C CNN
 F 1 "Red" H 1442 9686 50  0000 C CNN
 F 2 "LED_THT:LED_D5.0mm" H 1450 9850 50  0001 C CNN
@@
 AR Path="/5B62EDB8/5BA54030/5BF65E48" Ref="R?"  Part="1"
 AR Path="/5B62EDB8/5BA5413D/5BF65E48" Ref="R?"  Part="1"
-AR Path="/5B62EDB8/5BF65E48" Ref="R7"  Part="1"
-F 0 "R7" V 1543 9850 50  0000 C CNN
+AR Path="/5B62EDB8/5BF65E48" Ref="R1412"  Part="1"
+F 0 "R1412" V 1543 9850 50  0000 C CNN
 F 1 "1.65k" V 1634 9850 50  0000 C CNN
 F 2 "Resistor_SMD:R_0805_2012Metric" V 1680 9850 50  0001 C CNN

Commit message: - Initialization of SD Card. - Wifi - SNTP - Status LEDs
Parts:
- D1401: value Red -> SDCard Init OK
- D1402: value Red -> SNTP Time set
- D1403: value Red -> Wifi connected
- D1404: value Red -> MQTT connected
Other:
- note added: ""Input output" device"
- note added: ""Status" device"
Changed lines of the file:
@@
 AR Path="/5B62EDB8/5BA5B774" Ref="D1401"  Part="1"
 F 0 "D1401" H 1442 5245 50  0000 C CNN
-F 1 "Red" H 1442 5336 50  0000 C CNN
+F 1 "SDCard Init OK" H 1250 5350 50  0000 C CNN
 F 2 "LED_THT:LED_D5.0mm" H 1450 5500 50  0001 C CNN
 F 3 "https://www.mouser.se/ProductDetail/Lite-On/LTL2R3KGD-EM?qs=sGAEpiMZZMtmwHDZQCdlqY3QuPVQdrfivxVgVo2hFbg%3d" H 1450 5500 50  0001 C CNN
@@
 AR Path="/5B62EDB8/5BA5B879" Ref="D1402"  Part="1"
 F 0 "D1402" H 1442 5595 50  0000 C CNN
-F 1 "Red" H 1442 5686 50  0000 C CNN
+F 1 "SNTP Time set" H 1300 5700 50  0000 C CNN
 F 2 "LED_THT:LED_D5.0mm" H 1450 5850 50  0001 C CNN
 F 3 "https://www.mouser.se/ProductDetail/Lite-On/LTL2R3KGD-EM?qs=sGAEpiMZZMtmwHDZQCdlqY3QuPVQdrfivxVgVo2hFbg%3d" H 1450 5850 50  0001 C CNN
@@
 AR Path="/5B62EDB8/5BA5BA0A" Ref="D1403"  Part="1"
 F 0 "D1403" H 1442 5995 50  0000 C CNN
-F 1 "Red" H 1442 6086 50  0000 C CNN
+F 1 "Wifi connected" H 1300 6100 50  0000 C CNN
 F 2 "LED_THT:LED_D5.0mm" H 1450 6250 50  0001 C CNN
 F 3 "https://www.mouser.se/ProductDetail/Lite-On/LTL2R3KGD-EM?qs=sGAEpiMZZMtmwHDZQCdlqY3QuPVQdrfivxVgVo2hFbg%3d" H 1450 6250 50  0001 C CNN
@@
 AR Path="/5B62EDB8/5BA5BDA3" Ref="D1404"  Part="1"
 F 0 "D1404" H 1442 6395 50  0000 C CNN
-F 1 "Red" H 1442 6486 50  0000 C CNN
+F 1 "MQTT connected" H 1250 6500 50  0000 C CNN
 F 2 "LED_THT:LED_D5.0mm" H 1450 6650 50  0001 C CNN
 F 3 "https://www.mouser.se/ProductDetail/Lite-On/LTL2R3KGD-EM?qs=sGAEpiMZZMtmwHDZQCdlqY3QuPVQdrfivxVgVo2hFbg%3d" H 1450 6650 50  0001 C CNN
@@
 Text GLabel 3800 5300 0    50   Input ~ 0
 SD_CARD_PWR_CTRL
+Text Notes 4800 5900 0    50   ~ 0
+"Status" device
+Text Notes 4250 3050 0    50   ~ 0
+"Input output" device
 $EndSCHEMATC

Commit message: LED indicators for SDCard Wifi, SNTP & MQTT functional.
Parts:
- D1402: value SNTP Time set -> Red
- D1403: value Wifi connected -> Red
- D1404: value MQTT connected -> Wifi Connected
- D1407: value Red -> SNTP Time set
- D1410: value Red -> MQTT Connected
Changed lines of the file:
@@
 AR Path="/5B62EDB8/5BA5B879" Ref="D1402"  Part="1"
 F 0 "D1402" H 1442 5595 50  0000 C CNN
-F 1 "SNTP Time set" H 1300 5700 50  0000 C CNN
+F 1 "Red" H 1300 5700 50  0000 C CNN
 F 2 "LED_THT:LED_D5.0mm" H 1450 5850 50  0001 C CNN
 F 3 "https://www.mouser.se/ProductDetail/Lite-On/LTL2R3KGD-EM?qs=sGAEpiMZZMtmwHDZQCdlqY3QuPVQdrfivxVgVo2hFbg%3d" H 1450 5850 50  0001 C CNN
@@
 AR Path="/5B62EDB8/5BA5BA0A" Ref="D1403"  Part="1"
 F 0 "D1403" H 1442 5995 50  0000 C CNN
-F 1 "Wifi connected" H 1300 6100 50  0000 C CNN
+F 1 "Red" H 1300 6100 50  0000 C CNN
 F 2 "LED_THT:LED_D5.0mm" H 1450 6250 50  0001 C CNN
 F 3 "https://www.mouser.se/ProductDetail/Lite-On/LTL2R3KGD-EM?qs=sGAEpiMZZMtmwHDZQCdlqY3QuPVQdrfivxVgVo2hFbg%3d" H 1450 6250 50  0001 C CNN
@@
 AR Path="/5B62EDB8/5BA5BDA3" Ref="D1404"  Part="1"
 F 0 "D1404" H 1442 6395 50  0000 C CNN
-F 1 "MQTT connected" H 1250 6500 50  0000 C CNN
+F 1 "Wifi Connected" H 1250 6500 50  0000 C CNN
 F 2 "LED_THT:LED_D5.0mm" H 1450 6650 50  0001 C CNN
 F 3 "https://www.mouser.se/ProductDetail/Lite-On/LTL2R3KGD-EM?qs=sGAEpiMZZMtmwHDZQCdlqY3QuPVQdrfivxVgVo2hFbg%3d" H 1450 6650 50  0001 C CNN
@@
 AR Path="/5B62EDB8/5BF0FE5D" Ref="D1407"  Part="1"
 F 0 "D1407" H 1442 7595 50  0000 C CNN
-F 1 "Red" H 1442 7686 50  0000 C CNN
+F 1 "SNTP Time set" H 1350 7700 50  0000 C CNN
 F 2 "LED_THT:LED_D5.0mm" H 1450 7850 50  0001 C CNN
 F 3 "https://www.mouser.se/ProductDetail/Lite-On/LTL2R3KGD-EM?qs=sGAEpiMZZMtmwHDZQCdlqY3QuPVQdrfivxVgVo2hFbg%3d" H 1450 7850 50  0001 C CNN
@@
 AR Path="/5B62EDB8/5BF106D4" Ref="D1410"  Part="1"
 F 0 "D1410" H 1442 8795 50  0000 C CNN
-F 1 "Red" H 1442 8886 50  0000 C CNN
+F 1 "MQTT Connected" H 1442 8886 50  0000 C CNN
 F 2 "LED_THT:LED_D5.0mm" H 1450 9050 50  0001 C CNN
 F 3 "https://www.mouser.se/ProductDetail/Lite-On/LTL2R3KGD-EM?qs=sGAEpiMZZMtmwHDZQCdlqY3QuPVQdrfivxVgVo2hFbg%3d" H 1450 9050 50  0001 C CNN

Commit message: Updated PCB to match new schematics with MOSFETs.
Changed lines of the file:
@@
 Text Notes 4100 1400 1    60   ~ 0
 Near MCP23017
-Text GLabel 8750 4000 0    60   Input ~ 0
+Text GLabel 8700 3900 0    60   Input ~ 0
 BELL_CTRL
 Wire Notes Line
@@
 Text GLabel 6650 2900 2    50   Input ~ 0
 DO5_PWR
-Text GLabel 8750 3600 0    60   Input ~ 0
+Text GLabel 8700 4350 0    60   Input ~ 0
 EXTERNAL_SIREN_CTRL
 Text GLabel 3800 5100 0    60   Input ~ 0
@@
 F3 "Output" I R 9700 3150 50
 $EndSheet
-$Sheet
-S 8750 3900 1100 200
-U 5BA3564E
-F0 "Bell control" 50
-F1 "SelectableVoltageOutput.sch" 50
-F2 "CTRL" I L 8750 4000 50
-F3 "Output" I R 9850 4000 50
-$EndSheet
-Text GLabel 9850 4000 2    50   Input ~ 0
+Text GLabel 9800 3900 2    50   Input ~ 0
 BELL_PWR
-Text GLabel 9700 3600 2    50   Input ~ 0
+Text GLabel 9800 4350 2    50   Input ~ 0
 SIREN_PWR
-$Sheet
-S 8750 3500 950  200
-U 5BA35DC6
-F0 "External siren" 50
-F1 "12VDigitalOutput.sch" 50
-F2 "CTRL" I L 8750 3600 50
-F3 "Output" I R 9700 3600 50
-$EndSheet
 Text GLabel 1500 1300 0    50   Input ~ 0
 DI1_PWR
@@
 Text Notes 4250 3050 0    50   ~ 0
 "Input output" device
+$Sheet
+S 8700 4250 1100 200
+U 5C44CE71
+F0 "ExternalSiren" 50
+F1 "SelectableVoltageOutput.sch" 50
+F2 "CTRL" I L 8700 4350 50
+F3 "Output" I R 9800 4350 50
+$EndSheet
+$Sheet
+S 8700 3800 1100 200
+U 5C44D366
+F0 "Bell" 50
+F1 "SelectableVoltageOutput.sch" 50
+F2 "CTRL" I L 8700 3900 50
+F3 "Output" I R 9800 3900 50
+$EndSheet
 $EndSCHEMATC
