File: hardware/DigitalInput.sch (KiCad schematic (older format))
At the start: 10 parts, among them J1501 Digital input supply, J1502 Digital input GND, U1501 LTV-354T

Commit message: #5 - Moved All SD pullup resistors except R406 (SD_DATA2/MTDI/GPIO12) to SD-side of MAX4948. #3 - Added jumper for GPIO2 <-> GPOI0 for flash download. Removed affected items from PCB.
Changed lines of the file:
@@
 AR Path="/5B62EDB8/5BA54030/5B66E449" Ref="U3301"  Part="1"
 AR Path="/5B62EDB8/5BA5413D/5B66E449" Ref="U3401"  Part="1"
-F 0 "U1501" H 3650 2875 50  0000 C CNN
+F 0 "U3401" H 3650 2875 50  0000 C CNN
 F 1 "LTV-354T" H 3650 2784 50  0000 C CNN
 F 2 "Package_SO:SO-4_4.4x3.6mm_P2.54mm" H 3450 2350 50  0001 L CIN
@@
 AR Path="/5B62EDB8/5BA54030/5B66E450" Ref="R3301"  Part="1"
 AR Path="/5B62EDB8/5BA5413D/5B66E450" Ref="R3401"  Part="1"
-F 0 "R1501" V 1750 2450 50  0000 C CNN
+F 0 "R3401" V 1750 2450 50  0000 C CNN
 F 1 "1k" V 1850 2450 50  0000 C CNN
 F 2 "Resistor_SMD:R_2512_6332Metric" V 1780 2450 50  0001 C CNN
@@
 AR Path="/5B62EDB8/5BA54030/5B66E457" Ref="R3303"  Part="1"
 AR Path="/5B62EDB8/5BA5413D/5B66E457" Ref="R3403"  Part="1"
-F 0 "R1503" V 4500 2650 50  0000 C CNN
+F 0 "R3403" V 4500 2650 50  0000 C CNN
 F 1 "100" V 4600 2650 50  0000 C CNN
 F 2 "Resistor_SMD:R_0805_2012Metric" V 4530 2650 50  0001 C CNN
@@
 AR Path="/5B62EDB8/5BA54030/5B66E45E" Ref="C3301"  Part="1"
 AR Path="/5B62EDB8/5BA5413D/5B66E45E" Ref="C3401"  Part="1"
-F 0 "C1501" V 4050 2650 50  0000 C CNN
+F 0 "C3401" V 4050 2650 50  0000 C CNN
 F 1 "10u" H 4300 2750 50  0000 C CNN
 F 2 "Capacitor_SMD:CP_Elec_5x4.5" H 4238 2500 50  0001 C CNN
@@
 AR Path="/5B62EDB8/5BA54030/5B66E465" Ref="R3304"  Part="1"
 AR Path="/5B62EDB8/5BA5413D/5B66E465" Ref="R3404"  Part="1"
-F 0 "R1504" H 4900 2250 50  0000 C CNN
+F 0 "R3404" H 4900 2250 50  0000 C CNN
 F 1 "10k" H 4900 2350 50  0000 C CNN
 F 2 "Resistor_SMD:R_0805_2012Metric" V 4680 2300 50  0001 C CNN
@@
 AR Path="/5B62EDB8/5BA54030/5B66E46C" Ref="#PWR03303"  Part="1"
 AR Path="/5B62EDB8/5BA5413D/5B66E46C" Ref="#PWR03403"  Part="1"
-F 0 "#PWR01503" H 4000 2400 50  0001 C CNN
+F 0 "#PWR03403" H 4000 2400 50  0001 C CNN
 F 1 "GND" H 4005 2477 50  0000 C CNN
 F 2 "" H 4000 2650 50  0001 C CNN
@@
 AR Path="/5B62EDB8/5BA54030/5BA245A9" Ref="D3301"  Part="1"
 AR Path="/5B62EDB8/5BA5413D/5BA245A9" Ref="D3401"  Part="1"
-F 0 "D1501" H 4342 2045 50  0000 C CNN
+F 0 "D3401" H 4342 2045 50  0000 C CNN
 F 1 "Red" H 4342 2136 50  0000 C CNN
 F 2 "LED_THT:LED_D5.0mm" H 4350 2300 50  0001 C CNN
@@
 AR Path="/5B62EDB8/5BA54030/5BA245B2" Ref="R3302"  Part="1"
 AR Path="/5B62EDB8/5BA5413D/5BA245B2" Ref="R3402"  Part="1"
-F 0 "R1502" V 4143 2000 50  0000 C CNN
+F 0 "R3402" V 4143 2000 50  0000 C CNN
 F 1 "1.65k" V 4234 2000 50  0000 C CNN
 F 2 "Resistor_SMD:R_0805_2012Metric" V 4280 2000 50  0001 C CNN
@@
 AR Path="/5B62EDB8/5BA54030/5BA245BA" Ref="#PWR03304"  Part="1"
 AR Path="/5B62EDB8/5BA5413D/5BA245BA" Ref="#PWR03404"  Part="1"
-F 0 "#PWR01504" H 4350 1700 50  0001 C CNN
+F 0 "#PWR03404" H 4350 1700 50  0001 C CNN
 F 1 "+3V3" V 4365 1978 50  0000 L CNN
 F 2 "" H 4350 1850 50  0001 C CNN
@@
 AR Path="/5B62EDB8/5BA54030/5BA49A14" Ref="J3302"  Part="1"
 AR Path="/5B62EDB8/5BA5413D/5BA49A14" Ref="J3402"  Part="1"
-F 0 "J1502" V 1900 2900 50  0000 C CNN
+F 0 "J3402" V 1900 2900 50  0000 C CNN
 F 1 "Digital input GND" V 2000 2850 50  0000 C CNN
 F 2 "Connector_PinHeader_2.54mm:PinHeader_1x02_P2.54mm_Vertical" V 1874 2950 50  0001 C CNN
@@
 AR Path="/5B62EDB8/5BA54030/5BA49FBA" Ref="#PWR03301"  Part="1"
 AR Path="/5B62EDB8/5BA5413D/5BA49FBA" Ref="#PWR03401"  Part="1"
-F 0 "#PWR01501" H 1600 2800 50  0001 C CNN
+F 0 "#PWR03401" H 1600 2800 50  0001 C CNN
 F 1 "GND" H 1605 2877 50  0000 C CNN
 F 2 "" H 1600 3050 50  0001 C CNN
@@
 AR Path="/5B62EDB8/5BA54030/5BA4A7BB" Ref="#PWR03302"  Part="1"
 AR Path="/5B62EDB8/5BA5413D/5BA4A7BB" Ref="#PWR03402"  Part="1"
-F 0 "#PWR01502" H 1700 1350 50  0001 C CNN
+F 0 "#PWR03402" H 1700 1350 50  0001 C CNN
 F 1 "+5V" V 1715 1628 50  0000 L CNN
 F 2 "" H 1700 1500 50  0001 C CNN
@@
 AR Path="/5B62EDB8/5BA54030/5BA4B9C4" Ref="J3301"  Part="1"
 AR Path="/5B62EDB8/5BA5413D/5BA4B9C4" Ref="J3401"  Part="1"
-F 0 "J1501" V 1566 1112 50  0000 R CNN
+F 0 "J3401" V 1566 1112 50  0000 R CNN
 F 1 "Digital input supply" V 1475 1112 50  0000 R CNN
 F 2 "Connector_PinHeader_2.54mm:PinHeader_1x03_P2.54mm_Vertical" H 1600 1300 50  0001 C CNN
@@
 AR Path="/5B62EDB8/5BA54030/5BA4C782" Ref="F3301"  Part="1"
 AR Path="/5B62EDB8/5BA5413D/5BA4C782" Ref="F3401"  Part="1"
-F 0 "F1501" V 1403 2100 50  0000 C CNN
+F 0 "F3401" V 1403 2100 50  0000 C CNN
 F 1 "xA" V 1494 2100 50  0000 C CNN
 F 2 "Fuse:Fuseholder_TR5_Littlefuse_No560_No460" V 1530 2100 50  0001 C CNN
