File: hardware/SelectableVoltageOutput.sch (KiCad schematic (older format))
At the start: 8 parts, among them J1601 Power_select, Q1601 ZXTN25050DFHTA, Q1602 ZXTN25050DFHTA

Commit message: Outputs now uses MOSFETs
Parts:
- removed Q1601, Q1602: ZXTN25050DFHTA, Package_TO_SOT_SMD:SOT-23, symbol Device:Q_NPN_BCE
- added D1602, D1603: CZRQR52C6V8-HF, Diode_SMD:D_0402_1005Metric, symbol Device:D_Zener
- added Q1601: Si2312CD, Package_TO_SOT_SMD:SOT-23, symbol PerMalmberg:Si2312CD
- added Q1602: Si2323CDS, Package_TO_SOT_SMD:SOT-23, symbol PerMalmberg:Si2323CDS
- added R1604: 470, Resistor_SMD:R_0805_2012Metric, symbol Device:R
- added R1605: 10k, Resistor_SMD:R_0805_2012Metric, symbol Device:R
- R1602: value 10k -> 2.2k; footprint Resistor_SMD:R_0805_2012Metric -> (none)
Connections:
- net CTRL: now also R1603.2, R1605.2
- net GND: now also D1602.2 (A), Q1601.2 (S), R1605.1; no longer R1602.1
- net Output: now also Q1602.3 (D)
- net at R1601.1: now also D1602.1 (K), Q1601.1 (G); no longer R1602.2
- net Fused_power: no longer names the net of F1601.1
- net Fused_power: now also R1602.1, D1603.1 (K), Q1602.2 (S)
- net Unfused_power: no longer names the net of F1601.2, J1601.2 (Pin_2)
- new net: Q1601.3 (D), R1602.2, R1604.2
- new net: D1603.2 (A), Q1602.1 (G), R1604.1
Other:
- note added: "Zener diodes and stop resisitors must be placed as close\nto mosfets as possible with shortest possible traces to reduce\noscillation and reduce capacitance."
- moved on the sheet: D1601, F1601, J1601, R1603

Commit message: Preparing to replicate layout for outputs.
Parts:
- F1601: footprint Fuse:Fuseholder_TR5_Littlefuse_No560_No460 -> Fuse:Fuseholder_TR5_Littelfuse_No560_No460
- R1602: footprint (none) -> Resistor_SMD:R_0805_2012Metric
Changed lines of the file:
@@
 F 0 "F1601" V 2153 1800 50  0000 C CNN
 F 1 "xA" V 2244 1800 50  0000 C CNN
-F 2 "Fuse:Fuseholder_TR5_Littlefuse_No560_No460" V 2280 1800 50  0001 C CNN
+F 2 "Fuse:Fuseholder_TR5_Littelfuse_No560_No460" V 2280 1800 50  0001 C CNN
 F 3 "https://www.mouser.se/ProductDetail/Littelfuse/56000001019?qs=sGAEpiMZZMtRmoYvq3OwzKEcK5xXAR8uiSqvDZfRA1w%3d" H 2350 1800 50  0001 C CNN
 	1    2350 1800
@@
 F 0 "R1602" V 3350 1950 50  0000 L CNN
 F 1 "2.2k" V 3450 1950 50  0000 L CNN
-F 2 "" V 3380 2050 50  0001 C CNN
-F 3 "~" H 3450 2050 50  0001 C CNN
+F 2 "Resistor_SMD:R_0805_2012Metric" V 3380 2050 50  0001 C CNN
+F 3 "https://www.mouser.se/ProductDetail/667-ERA-6AED222V" H 3450 2050 50  0001 C CNN
 	1    3450 2050
 	1    0    0    -1

Commit message: Updated PCB to match new schematics with MOSFETs.
Changed lines of the file:
@@
 $Descr A4 11693 8268
 encoding utf-8
-Sheet 16 34
+Sheet 32 34
 Title ""
 Date ""
@@
 AR Path="/5B62EDB8/5BA2E71A/5BA13007" Ref="J2301"  Part="1"
 AR Path="/5B62EDB8/5BA3564E/5BA13007" Ref="J2601"  Part="1"
-F 0 "J1601" H 1200 1475 50  0000 C CNN
+AR Path="/5B62EDB8/5C44CE71/5BA13007" Ref="J3203"  Part="1"
+AR Path="/5B62EDB8/5C44D366/5BA13007" Ref="J3303"  Part="1"
+F 0 "J3203" H 1200 1475 50  0000 C CNN
 F 1 "Power_select" H 1200 1566 50  0000 C CNN
 F 2 "Connector_PinHeader_2.54mm:PinHeader_1x03_P2.54mm_Vertical" V 1288 1726 50  0001 C CNN
@@
 AR Path="/5B62EDB8/5BA2E71A/5BA36D68" Ref="#PWR02301"  Part="1"
 AR Path="/5B62EDB8/5BA3564E/5BA36D68" Ref="#PWR02601"  Part="1"
-F 0 "#PWR02601" H 1400 1550 50  0001 C CNN
+AR Path="/5B62EDB8/5C44CE71/5BA36D68" Ref="#PWR03205"  Part="1"
+AR Path="/5B62EDB8/5C44D366/5BA36D68" Ref="#PWR03305"  Part="1"
+F 0 "#PWR03205" H 1400 1550 50  0001 C CNN
 F 1 "+5V" V 1415 1828 50  0000 L CNN
 F 2 "" H 1400 1700 50  0001 C CNN
@@
 AR Path="/5B62EDB8/5BA2E71A/5BA36D69" Ref="F2301"  Part="1"
 AR Path="/5B62EDB8/5BA3564E/5BA36D69" Ref="F2601"  Part="1"
-F 0 "F1601" V 2153 1800 50  0000 C CNN
+AR Path="/5B62EDB8/5C44CE71/5BA36D69" Ref="F3202"  Part="1"
+AR Path="/5B62EDB8/5C44D366/5BA36D69" Ref="F3302"  Part="1"
+F 0 "F3202" V 2153 1800 50  0000 C CNN
 F 1 "xA" V 2244 1800 50  0000 C CNN
 F 2 "Fuse:Fuseholder_TR5_Littelfuse_No560_No460" V 2280 1800 50  0001 C CNN
@@
 AR Path="/5B62EDB8/5BA2E71A/5BA36D6B" Ref="R2303"  Part="1"
 AR Path="/5B62EDB8/5BA3564E/5BA36D6B" Ref="R2603"  Part="1"
-F 0 "R1603" V 2500 2950 50  0000 C CNN
+AR Path="/5B62EDB8/5C44CE71/5BA36D6B" Ref="R3206"  Part="1"
+AR Path="/5B62EDB8/5C44D366/5BA36D6B" Ref="R3306"  Part="1"
+F 0 "R3206" V 2500 2950 50  0000 C CNN
 F 1 "1.65k" V 2600 2950 50  0000 C CNN
 F 2 "Resistor_SMD:R_0805_2012Metric" V 2530 2950 50  0001 C CNN
@@
 AR Path="/5B62EDB8/5BA2E71A/5BA36D6E" Ref="D2301"  Part="1"
 AR Path="/5B62EDB8/5BA3564E/5BA36D6E" Ref="D2601"  Part="1"
-F 0 "D1601" H 2650 3350 50  0000 C CNN
+AR Path="/5B62EDB8/5C44CE71/5BA36D6E" Ref="D3202"  Part="1"
+AR Path="/5B62EDB8/5C44D366/5BA36D6E" Ref="D3302"  Part="1"
+F 0 "D3202" H 2650 3350 50  0000 C CNN
 F 1 "Green" H 2400 3350 50  0000 C CNN
 F 2 "LED_THT:LED_D5.0mm" H 2600 3250 50  0001 C CNN
@@
 AR Path="/5B62EDB8/5BA2E71A/5BA36D70" Ref="#PWR02304"  Part="1"
 AR Path="/5B62EDB8/5BA3564E/5BA36D70" Ref="#PWR02604"  Part="1"
-F 0 "#PWR02604" H 2600 3150 50  0001 C CNN
+AR Path="/5B62EDB8/5C44CE71/5BA36D70" Ref="#PWR03207"  Part="1"
+AR Path="/5B62EDB8/5C44D366/5BA36D70" Ref="#PWR03307"  Part="1"
+F 0 "#PWR03207" H 2600 3150 50  0001 C CNN
 F 1 "GND" H 2605 3227 50  0000 C CNN
 F 2 "" H 2600 3400 50  0001 C CNN
@@
 AR Path="/5B62EDB8/5BA2E71A/5C3FF0E5" Ref="Q2301"  Part="1"
 AR Path="/5B62EDB8/5BA3564E/5C3FF0E5" Ref="Q2501"  Part="1"
-F 0 "Q1601" H 3250 2500 50  0000 C CNN
+AR Path="/5B62EDB8/5C44CE71/5C3FF0E5" Ref="Q3201"  Part="1"
+AR Path="/5B62EDB8/5C44D366/5C3FF0E5" Ref="Q3301"  Part="1"
+F 0 "Q3201" H 3250 2500 50  0000 C CNN
 F 1 "Si2312CD" H 3600 2700 50  0000 C CNN
 F 2 "Package_TO_SOT_SMD:SOT-23" H 3210 2705 50  0001 C CNN
@@
 AR Path="/5B62EDB8/5BA2E71A/5C3FF139" Ref="Q2302"  Part="1"
 AR Path="/5B62EDB8/5BA3564E/5C3FF139" Ref="Q2502"  Part="1"
-F 0 "Q1602" H 4000 2550 50  0000 C CNN
+AR Path="/5B62EDB8/5C44CE71/5C3FF139" Ref="Q3202"  Part="1"
+AR Path="/5B62EDB8/5C44D366/5C3FF139" Ref="Q3302"  Part="1"
+F 0 "Q3202" H 4000 2550 50  0000 C CNN
 F 1 "Si2323CDS" H 4000 2150 50  0000 C CNN
 F 2 "Package_TO_SOT_SMD:SOT-23" H 4000 2350 50  0001 C CNN
@@
 AR Path="/5B62EDB8/5BA2E71A/5C3FFFEC" Ref="R2304"  Part="1"
 AR Path="/5B62EDB8/5BA3564E/5C3FFFEC" Ref="R2503"  Part="1"
-F 0 "R1604" H 3400 2400 50  0000 C CNN
+AR Path="/5B62EDB8/5C44CE71/5C3FFFEC" Ref="R3209"  Part="1"
+AR Path="/5B62EDB8/5C44D366/5C3FFFEC" Ref="R3309"  Part="1"
+F 0 "R3209" H 3400 2400 50  0000 C CNN
 F 1 "470" V 3600 2350 50  0000 C CNN
 F 2 "Resistor_SMD:R_0805_2012Metric" V 3530 2350 50  0001 C CNN
@@
 AR Path="/5B62EDB8/5BA2E71A/5C40010C" Ref="R2302"  Part="1"
 AR Path="/5B62EDB8/5BA3564E/5C40010C" Ref="R2502"  Part="1"
-F 0 "R1602" V 3350 1950 50  0000 L CNN
+AR Path="/5B62EDB8/5C44CE71/5C40010C" Ref="R3208"  Part="1"
+AR Path="/5B62EDB8/5C44D366/5C40010C" Ref="R3308"  Part="1"
+F 0 "R3208" V 3350 1950 50  0000 L CNN
 F 1 "2.2k" V 3450 1950 50  0000 L CNN
 F 2 "Resistor_SMD:R_0805_2012Metric" V 3380 2050 50  0001 C CNN
@@
 AR Path="/5B62EDB8/5BA2E71A/5C4028BB" Ref="#PWR02302"  Part="1"
 AR Path="/5B62EDB8/5BA3564E/5C4028BB" Ref="#PWR02501"  Part="1"
-F 0 "#PWR02501" H 3000 2950 50  0001 C CNN
+AR Path="/5B62EDB8/5C44CE71/5C4028BB" Ref="#PWR03208"  Part="1"
+AR Path="/5B62EDB8/5C44D366/5C4028BB" Ref="#PWR03308"  Part="1"
+F 0 "#PWR03208" H 3000 2950 50  0001 C CNN
 F 1 "GND" H 3005 3027 50  0000 C CNN
 F 2 "" H 3000 3200 50  0001 C CNN
@@
 AR Path="/5B62EDB8/5BA2E71A/5C40A4E1" Ref="R2305"  Part="1"
 AR Path="/5B62EDB8/5BA3564E/5C40A4E1" Ref="R2504"  Part="1"
-F 0 "R1605" H 2320 2896 50  0000 L CNN
+AR Path="/5B62EDB8/5C44CE71/5C40A4E1" Ref="R3205"  Part="1"
+AR Path="/5B62EDB8/5C44D366/5C40A4E1" Ref="R3305"  Part="1"
+F 0 "R3205" H 2320 2896 50  0000 L CNN
 F 1 "10k" H 2320 2805 50  0000 L CNN
 F 2 "Resistor_SMD:R_0805_2012Metric" V 2180 2850 50  0001 C CNN
@@
 AR Path="/5B62EDB8/5BA2E71A/5C40A7A7" Ref="#PWR02303"  Part="1"
 AR Path="/5B62EDB8/5BA3564E/5C40A7A7" Ref="#PWR02502"  Part="1"
-F 0 "#PWR02502" H 2250 2750 50  0001 C CNN
+AR Path="/5B62EDB8/5C44CE71/5C40A7A7" Ref="#PWR03206"  Part="1"
+AR Path="/5B62EDB8/5C44D366/5C40A7A7" Ref="#PWR03306"  Part="1"
+F 0 "#PWR03206" H 2250 2750 50  0001 C CNN
 F 1 "GND" H 2255 2827 50  0000 C CNN
 F 2 "" H 2250 3000 50  0001 C CNN
@@
 AR Path="/5B62EDB8/5BA2E71A/5C40FA87" Ref="D2302"  Part="1"
 AR Path="/5B62EDB8/5BA3564E/5C40FA87" Ref="D2501"  Part="1"
-F 0 "D1602" V 2954 3129 50  0000 L CNN
+AR Path="/5B62EDB8/5C44CE71/5C40FA87" Ref="D3203"  Part="1"
+AR Path="/5B62EDB8/5C44D366/5C40FA87" Ref="D3303"  Part="1"
+F 0 "D3203" V 2954 3129 50  0000 L CNN
 F 1 "CZRQR52C6V8-HF" V 3045 3129 50  0000 L CNN
 F 2 "Diode_SMD:D_0402_1005Metric" H 3000 3050 50  0001 C CNN
@@
 AR Path="/5B62EDB8/5BA2E71A/5C40FC74" Ref="R2301"  Part="1"
 AR Path="/5B62EDB8/5BA3564E/5C40FC74" Ref="R2501"  Part="1"
-F 0 "R1601" V 2750 2700 50  0000 C CNN
+AR Path="/5B62EDB8/5C44CE71/5C40FC74" Ref="R3207"  Part="1"
+AR Path="/5B62EDB8/5C44D366/5C40FC74" Ref="R3307"  Part="1"
+F 0 "R3207" V 2750 2700 50  0000 C CNN
 F 1 "470" V 2850 2700 50  0000 C CNN
 F 2 "Resistor_SMD:R_0805_2012Metric" V 2780 2700 50  0001 C CNN
@@
 AR Path="/5B62EDB8/5BA2E71A/5C410A9C" Ref="D2303"  Part="1"
 AR Path="/5B62EDB8/5BA3564E/5C410A9C" Ref="D2502"  Part="1"
-F 0 "D1603" V 3704 2029 50  0000 L CNN
+AR Path="/5B62EDB8/5C44CE71/5C410A9C" Ref="D3204"  Part="1"
+AR Path="/5B62EDB8/5C44D366/5C410A9C" Ref="D3304"  Part="1"
+F 0 "D3204" V 3704 2029 50  0000 L CNN
 F 1 "CZRQR52C6V8-HF" V 3795 2029 50  0000 L CNN
 F 2 "Diode_SMD:D_0402_1005Metric" H 3750 1950 50  0001 C CNN
@@
 AR Path="/5B62EDB8/5BA2E71A/5C438377" Ref="#FLG0108"  Part="1"
 AR Path="/5B62EDB8/5BA3564E/5C438377" Ref="#FLG0109"  Part="1"
-F 0 "#FLG0109" H 4550 1875 50  0001 C CNN
+AR Path="/5B62EDB8/5C44CE71/5C438377" Ref="#FLG03201"  Part="1"
+AR Path="/5B62EDB8/5C44D366/5C438377" Ref="#FLG03301"  Part="1"
+F 0 "#FLG03201" H 4550 1875 50  0001 C CNN
 F 1 "PWR_FLAG" H 4550 1974 50  0000 C CNN
 F 2 "" H 4550 1800 50  0001 C CNN

Commit message: Updated PCB with additional vias. Added decoupler caps for Wiegand.
Changed lines of the file:
@@
 AR Path="/5B62EDB8/5C44CE71/5BA13007" Ref="J3203"  Part="1"
 AR Path="/5B62EDB8/5C44D366/5BA13007" Ref="J3303"  Part="1"
-F 0 "J3203" H 1200 1475 50  0000 C CNN
+F 0 "J3303" H 1200 1475 50  0000 C CNN
 F 1 "Power_select" H 1200 1566 50  0000 C CNN
 F 2 "Connector_PinHeader_2.54mm:PinHeader_1x03_P2.54mm_Vertical" V 1288 1726 50  0001 C CNN
@@
 AR Path="/5B62EDB8/5C44CE71/5BA36D68" Ref="#PWR03205"  Part="1"
 AR Path="/5B62EDB8/5C44D366/5BA36D68" Ref="#PWR03305"  Part="1"
-F 0 "#PWR03205" H 1400 1550 50  0001 C CNN
+F 0 "#PWR03305" H 1400 1550 50  0001 C CNN
 F 1 "+5V" V 1415 1828 50  0000 L CNN
 F 2 "" H 1400 1700 50  0001 C CNN
@@
 AR Path="/5B62EDB8/5C44CE71/5BA36D69" Ref="F3202"  Part="1"
 AR Path="/5B62EDB8/5C44D366/5BA36D69" Ref="F3302"  Part="1"
-F 0 "F3202" V 2153 1800 50  0000 C CNN
+F 0 "F3302" V 2153 1800 50  0000 C CNN
 F 1 "xA" V 2244 1800 50  0000 C CNN
 F 2 "Fuse:Fuseholder_TR5_Littelfuse_No560_No460" V 2280 1800 50  0001 C CNN
@@
 AR Path="/5B62EDB8/5C44CE71/5BA36D6B" Ref="R3206"  Part="1"
 AR Path="/5B62EDB8/5C44D366/5BA36D6B" Ref="R3306"  Part="1"
-F 0 "R3206" V 2500 2950 50  0000 C CNN
+F 0 "R3306" V 2500 2950 50  0000 C CNN
 F 1 "1.65k" V 2600 2950 50  0000 C CNN
 F 2 "Resistor_SMD:R_0805_2012Metric" V 2530 2950 50  0001 C CNN
@@
 AR Path="/5B62EDB8/5C44CE71/5BA36D6E" Ref="D3202"  Part="1"
 AR Path="/5B62EDB8/5C44D366/5BA36D6E" Ref="D3302"  Part="1"
-F 0 "D3202" H 2650 3350 50  0000 C CNN
+F 0 "D3302" H 2650 3350 50  0000 C CNN
 F 1 "Green" H 2400 3350 50  0000 C CNN
 F 2 "LED_THT:LED_D5.0mm" H 2600 3250 50  0001 C CNN
@@
 AR Path="/5B62EDB8/5C44CE71/5BA36D70" Ref="#PWR03207"  Part="1"
 AR Path="/5B62EDB8/5C44D366/5BA36D70" Ref="#PWR03307"  Part="1"
-F 0 "#PWR03207" H 2600 3150 50  0001 C CNN
+F 0 "#PWR03307" H 2600 3150 50  0001 C CNN
 F 1 "GND" H 2605 3227 50  0000 C CNN
 F 2 "" H 2600 3400 50  0001 C CNN
@@
 AR Path="/5B62EDB8/5C44CE71/5C3FF0E5" Ref="Q3201"  Part="1"
 AR Path="/5B62EDB8/5C44D366/5C3FF0E5" Ref="Q3301"  Part="1"
-F 0 "Q3201" H 3250 2500 50  0000 C CNN
+F 0 "Q3301" H 3250 2500 50  0000 C CNN
 F 1 "Si2312CD" H 3600 2700 50  0000 C CNN
 F 2 "Package_TO_SOT_SMD:SOT-23" H 3210 2705 50  0001 C CNN
@@
 AR Path="/5B62EDB8/5C44CE71/5C3FF139" Ref="Q3202"  Part="1"
 AR Path="/5B62EDB8/5C44D366/5C3FF139" Ref="Q3302"  Part="1"
-F 0 "Q3202" H 4000 2550 50  0000 C CNN
+F 0 "Q3302" H 4000 2550 50  0000 C CNN
 F 1 "Si2323CDS" H 4000 2150 50  0000 C CNN
 F 2 "Package_TO_SOT_SMD:SOT-23" H 4000 2350 50  0001 C CNN
@@
 AR Path="/5B62EDB8/5C44CE71/5C3FFFEC" Ref="R3209"  Part="1"
 AR Path="/5B62EDB8/5C44D366/5C3FFFEC" Ref="R3309"  Part="1"
-F 0 "R3209" H 3400 2400 50  0000 C CNN
+F 0 "R3309" H 3400 2400 50  0000 C CNN
 F 1 "470" V 3600 2350 50  0000 C CNN
 F 2 "Resistor_SMD:R_0805_2012Metric" V 3530 2350 50  0001 C CNN
@@
 AR Path="/5B62EDB8/5C44CE71/5C40010C" Ref="R3208"  Part="1"
 AR Path="/5B62EDB8/5C44D366/5C40010C" Ref="R3308"  Part="1"
-F 0 "R3208" V 3350 1950 50  0000 L CNN
+F 0 "R3308" V 3350 1950 50  0000 L CNN
 F 1 "2.2k" V 3450 1950 50  0000 L CNN
 F 2 "Resistor_SMD:R_0805_2012Metric" V 3380 2050 50  0001 C CNN
@@
 AR Path="/5B62EDB8/5C44CE71/5C4028BB" Ref="#PWR03208"  Part="1"
 AR Path="/5B62EDB8/5C44D366/5C4028BB" Ref="#PWR03308"  Part="1"
-F 0 "#PWR03208" H 3000 2950 50  0001 C CNN
+F 0 "#PWR03308" H 3000 2950 50  0001 C CNN
 F 1 "GND" H 3005 3027 50  0000 C CNN
 F 2 "" H 3000 3200 50  0001 C CNN
@@
 AR Path="/5B62EDB8/5C44CE71/5C40A4E1" Ref="R3205"  Part="1"
 AR Path="/5B62EDB8/5C44D366/5C40A4E1" Ref="R3305"  Part="1"
-F 0 "R3205" H 2320 2896 50  0000 L CNN
+F 0 "R3305" H 2320 2896 50  0000 L CNN
 F 1 "10k" H 2320 2805 50  0000 L CNN
 F 2 "Resistor_SMD:R_0805_2012Metric" V 2180 2850 50  0001 C CNN
@@
 AR Path="/5B62EDB8/5C44CE71/5C40A7A7" Ref="#PWR03206"  Part="1"
 AR Path="/5B62EDB8/5C44D366/5C40A7A7" Ref="#PWR03306"  Part="1"
-F 0 "#PWR03206" H 2250 2750 50  0001 C CNN
+F 0 "#PWR03306" H 2250 2750 50  0001 C CNN
 F 1 "GND" H 2255 2827 50  0000 C CNN
 F 2 "" H 2250 3000 50  0001 C CNN
@@
 AR Path="/5B62EDB8/5C44CE71/5C40FA87" Ref="D3203"  Part="1"
 AR Path="/5B62EDB8/5C44D366/5C40FA87" Ref="D3303"  Part="1"
-F 0 "D3203" V 2954 3129 50  0000 L CNN
+F 0 "D3303" V 2954 3129 50  0000 L CNN
 F 1 "CZRQR52C6V8-HF" V 3045 3129 50  0000 L CNN
 F 2 "Diode_SMD:D_0402_1005Metric" H 3000 3050 50  0001 C CNN
@@
 AR Path="/5B62EDB8/5C44CE71/5C40FC74" Ref="R3207"  Part="1"
 AR Path="/5B62EDB8/5C44D366/5C40FC74" Ref="R3307"  Part="1"
-F 0 "R3207" V 2750 2700 50  0000 C CNN
+F 0 "R3307" V 2750 2700 50  0000 C CNN
 F 1 "470" V 2850 2700 50  0000 C CNN
 F 2 "Resistor_SMD:R_0805_2012Metric" V 2780 2700 50  0001 C CNN
@@
 AR Path="/5B62EDB8/5C44CE71/5C410A9C" Ref="D3204"  Part="1"
 AR Path="/5B62EDB8/5C44D366/5C410A9C" Ref="D3304"  Part="1"
-F 0 "D3204" V 3704 2029 50  0000 L CNN
+F 0 "D3304" V 3704 2029 50  0000 L CNN
 F 1 "CZRQR52C6V8-HF" V 3795 2029 50  0000 L CNN
 F 2 "Diode_SMD:D_0402_1005Metric" H 3750 1950 50  0001 C CNN
@@
 AR Path="/5B62EDB8/5C44CE71/5C438377" Ref="#FLG03201"  Part="1"
 AR Path="/5B62EDB8/5C44D366/5C438377" Ref="#FLG03301"  Part="1"
-F 0 "#FLG03201" H 4550 1875 50  0001 C CNN
+F 0 "#FLG03301" H 4550 1875 50  0001 C CNN
 F 1 "PWR_FLAG" H 4550 1974 50  0000 C CNN
 F 2 "" H 4550 1800 50  0001 C CNN
